File: hw/kicad/appliance.kicad_pcb (KiCad board)
At the start: 12 copper layers, 312 x 111.2 mm, 52 parts

Commit message: hw: derive the ASIC package and ball map from the power model
hw/pinout.py turns the interface list, the power model and the
package_selection rules in board.yaml into the ball count the core rail
needs, the smallest candidate package that carries it, and a rule-based
ball map (links on the west and east edges as two columns of 18 rows,
both LPDDR channels on the north rows in byte lanes with ground returns,
management on the south row, ground and core in a checkerboard), written
as CSV, JSON and a report for the packaging house.  At the design point
the 400-ball draft package cannot carry 54 A of core current; a 784-ball
28x28 array at 0.8 mm in the same 23 mm body is selected.  The KiCad
generator now builds the ASIC footprint from this map: escape geometry
and lane pitch follow the ball pitch, ribbon paths run through each
port's lane centre, and hops between packages of different pitch rescale
their lanes.  DRC stays clean apart from the unrouted nets.

Co-Authored-By: Claude Fable 5.1 <noreply@anthropic.com>
Claude-Session: https://claude.ai/code/session_01VmmvkZe8Ctg3RAykNGsQBn
Parts:
- U_A0, U_A1, U_A2, U_A3, U_A4, U_A5, U_A6, U_A7, U_H0, U_H1: footprint appliance:FCBGA400_20x20_P1.0 -> appliance:FCBGA784_28x28_P0.8
Connections:
- U_A0 pad A10: A0_CH0_DQ9 -> A0_CH0_DQS0_N
- U_A0 pad A11: A0_CH0_DQ10 -> A0_CH0_DMI0
- U_A0 pad A12: A0_CH0_DQ11 -> GND
- U_A0 pad A13: A0_CH0_DQ12 -> A0_CH0_DQ8
- U_A0 pad A14: A0_CH0_DQ13 -> A0_CH0_DQ9
- U_A0 pad A15: A0_CH0_DQ14 -> A0_CH0_DQ10
- U_A0 pad A16: A0_CH0_DQ15 -> A0_CH0_DQ11
- U_A0 pad A17: A0_CH0_DQ16 -> A0_CH0_DQ12
- U_A0 pad A18: A0_CH0_DQ17 -> A0_CH0_DQ13
- U_A0 pad A19: A0_CH0_DQ18 -> A0_CH0_DQ14
- U_A0 pad A20: A0_CH0_DQ19 -> A0_CH0_DQ15
- U_A0 pad A9: A0_CH0_DQ8 -> A0_CH0_DQS0_P
- U_A0 pad B10: A0_CH0_DQ29 -> A0_CH0_DQ25
- U_A0 pad B11: A0_CH0_DQ30 -> A0_CH0_DQ26
- U_A0 pad B12: A0_CH0_DQ31 -> A0_CH0_DQ27
- U_A0 pad B13: A0_CH0_DQS0_P -> A0_CH0_DQ28
- U_A0 pad B14: A0_CH0_DQS0_N -> A0_CH0_DQ29
- U_A0 pad B15: A0_CH0_DQS1_P -> A0_CH0_DQ30
- U_A0 pad B16: A0_CH0_DQS1_N -> A0_CH0_DQ31
- U_A0 pad B17: A0_CH0_DQS2_P -> A0_CH0_DQS3_P
- U_A0 pad B18: A0_CH0_DQS2_N -> A0_CH0_DQS3_N
- U_A0 pad B19: A0_CH0_DQS3_P -> A0_CH0_DMI3
- U_A0 pad B20: A0_CH0_DQS3_N -> GND
- U_A0 pad B5: A0_CH0_DQ24 -> A0_CH0_DQS2_P
- U_A0 pad B6: A0_CH0_DQ25 -> A0_CH0_DQS2_N
- U_A0 pad B7: A0_CH0_DQ26 -> A0_CH0_DMI2
- U_A0 pad B8: A0_CH0_DQ27 -> GND
- U_A0 pad B9: A0_CH0_DQ28 -> A0_CH0_DQ24
- U_A0 pad C1: LINK0_DATA0 -> A0_CH0_CA8
- U_A0 pad C10: A0_CH0_CA3 -> A0_CH0_CK0_N
- U_A0 pad C11: A0_CH0_CA4 -> A0_CH0_CK1_P
- U_A0 pad C12: A0_CH0_CA5 -> A0_CH0_CK1_N
- U_A0 pad C13: A0_CH0_CA6 -> A0_CH0_RESET
- U_A0 pad C14: A0_CH0_CA7 -> GND
- U_A0 pad C15: A0_CH0_CA8 -> A0_CH1_DQ0
- U_A0 pad C16: A0_CH0_CA9 -> A0_CH1_DQ1
- U_A0 pad C17: A0_CH0_CA10 -> A0_CH1_DQ2
- U_A0 pad C18: A0_CH0_CA11 -> A0_CH1_DQ3
- U_A0 pad C19: LINK1_DATA1 -> A0_CH1_DQ4
- U_A0 pad C2: LINK0_DATA1 -> A0_CH0_CA9
- U_A0 pad C20: LINK1_DATA0 -> A0_CH1_DQ5
- U_A0 pad C3: A0_CH0_DMI0 -> A0_CH0_CA10
- U_A0 pad C4: A0_CH0_DMI1 -> A0_CH0_CA11
- U_A0 pad C5: A0_CH0_DMI2 -> A0_CH0_CA12
- U_A0 pad C6: A0_CH0_DMI3 -> A0_CH0_CA13
- U_A0 pad C7: A0_CH0_CA0 -> A0_CH0_CS0
- U_A0 pad C8: A0_CH0_CA1 -> A0_CH0_CS1
- U_A0 pad C9: A0_CH0_CA2 -> A0_CH0_CK0_P
- U_A0 pad D1: LINK0_DATA2 -> A0_CH1_DQ10
- U_A0 pad D10: A0_CH0_CK1_N -> GND
- U_A0 pad D11: A0_CH0_RESET -> A0_CH1_DQ16
- U_A0 pad D12: A0_CH1_DQ0 -> A0_CH1_DQ17
- U_A0 pad D13: A0_CH1_DQ1 -> A0_CH1_DQ18
- U_A0 pad D14: A0_CH1_DQ2 -> A0_CH1_DQ19
- U_A0 pad D15: A0_CH1_DQ3 -> A0_CH1_DQ20
- U_A0 pad D16: A0_CH1_DQ4 -> A0_CH1_DQ21
- U_A0 pad D17: A0_CH1_DQ5 -> A0_CH1_DQ22
- U_A0 pad D18: A0_CH1_DQ6 -> A0_CH1_DQ23
- U_A0 pad D19: LINK1_DATA3 -> A0_CH1_DQS2_P
- U_A0 pad D2: LINK0_DATA3 -> A0_CH1_DQ11
- U_A0 pad D20: LINK1_DATA2 -> A0_CH1_DQS2_N
- U_A0 pad D3: A0_CH0_CA12 -> A0_CH1_DQ12
- U_A0 pad D4: A0_CH0_CA13 -> A0_CH1_DQ13
- U_A0 pad D5: A0_CH0_CS0 -> A0_CH1_DQ14
- U_A0 pad D6: A0_CH0_CS1 -> A0_CH1_DQ15
- U_A0 pad D7: A0_CH0_CK0_P -> A0_CH1_DQS1_P
- U_A0 pad D8: A0_CH0_CK0_N -> A0_CH1_DQS1_N
- U_A0 pad D9: A0_CH0_CK1_P -> A0_CH1_DMI1
- U_A0 pad E1: LINK0_DATA4 -> A0_CH1_DQ30
- U_A0 pad E10: A0_CH1_DQ14 -> A0_CH1_CA3
- U_A0 pad E11: A0_CH1_DQ15 -> A0_CH1_CA4
- U_A0 pad E12: A0_CH1_DQ16 -> A0_CH1_CA5
- U_A0 pad E13: A0_CH1_DQ17 -> A0_CH1_CA6
- U_A0 pad E14: A0_CH1_DQ18 -> A0_CH1_CA7
- U_A0 pad E15: A0_CH1_DQ19 -> A0_CH1_CA8
- U_A0 pad E16: A0_CH1_DQ20 -> A0_CH1_CA9
- U_A0 pad E17: A0_CH1_DQ21 -> A0_CH1_CA10
- U_A0 pad E18: A0_CH1_DQ22 -> A0_CH1_CA11
- U_A0 pad E19: LINK1_DATA5 -> A0_CH1_CA12
- U_A0 pad E2: LINK0_DATA5 -> A0_CH1_DQ31
- U_A0 pad E20: LINK1_DATA4 -> A0_CH1_CA13
- U_A0 pad E3: A0_CH1_DQ7 -> A0_CH1_DQS3_P
- U_A0 pad E4: A0_CH1_DQ8 -> A0_CH1_DQS3_N
- U_A0 pad E5: A0_CH1_DQ9 -> A0_CH1_DMI3
- U_A0 pad E6: A0_CH1_DQ10 -> GND
- U_A0 pad E7: A0_CH1_DQ11 -> A0_CH1_CA0
- U_A0 pad E8: A0_CH1_DQ12 -> A0_CH1_CA1
- U_A0 pad E9: A0_CH1_DQ13 -> A0_CH1_CA2
- U_A0 pad F1: LINK0_DATA6 -> LINK0_DATA0
- U_A0 pad F10: A0_CH1_DQ30 -> GND
- U_A0 pad F11: A0_CH1_DQ31 -> VDD_IO_1V8
- U_A0 pad F12: A0_CH1_DQS0_P -> GND
- U_A0 pad F13: A0_CH1_DQS0_N -> VDD_CORE_A0
- U_A0 pad F14: A0_CH1_DQS1_P -> GND
- U_A0 pad F15: A0_CH1_DQS1_N -> VDD_CORE_A0
- U_A0 pad F16: A0_CH1_DQS2_P -> GND
- U_A0 pad F17: A0_CH1_DQS2_N -> VDD_CORE_A0
- U_A0 pad F18: A0_CH1_DQS3_P -> GND
- U_A0 pad F19: LINK1_DATA7 -> VDD_CORE_A0
- U_A0 pad F2: LINK0_DATA7 -> LINK0_DATA1
- U_A0 pad F20: LINK1_DATA6 -> GND
- U_A0 pad F3: A0_CH1_DQ23 -> VDD_CORE_A0
- U_A0 pad F4: A0_CH1_DQ24 -> GND
- U_A0 pad F5: A0_CH1_DQ25 -> VDD_CORE_A0
- U_A0 pad F6: A0_CH1_DQ26 -> GND
- U_A0 pad F7: A0_CH1_DQ27 -> VDD_CORE_A0
- U_A0 pad F8: A0_CH1_DQ28 -> GND
- U_A0 pad F9: A0_CH1_DQ29 -> VDD_CORE_A0
- U_A0 pad G1: LINK0_DATA8 -> LINK0_DATA2
- U_A0 pad G10: A0_CH1_CA2 -> VDD_CORE_A0
- U_A0 pad G11: A0_CH1_CA3 -> GND
- U_A0 pad G12: A0_CH1_CA4 -> VDD_IO_1V8
- U_A0 pad G13: A0_CH1_CA5 -> GND
- U_A0 pad G14: A0_CH1_CA6 -> VDD_CORE_A0
- U_A0 pad G15: A0_CH1_CA7 -> GND
- U_A0 pad G16: A0_CH1_CA8 -> VDD_CORE_A0
- U_A0 pad G17: A0_CH1_CA9 -> GND
- U_A0 pad G18: A0_CH1_CA10 -> VDD_CORE_A0
- U_A0 pad G19: LINK1_DATA9 -> GND
- U_A0 pad G2: LINK0_DATA9 -> LINK0_DATA3
- U_A0 pad G20: LINK1_DATA8 -> VDD_CORE_A0
- U_A0 pad G3: A0_CH1_DQS3_N -> GND
- U_A0 pad G4: A0_CH1_DMI0 -> VDD_CORE_A0
- U_A0 pad G5: A0_CH1_DMI1 -> GND
- U_A0 pad G6: A0_CH1_DMI2 -> VDD_CORE_A0
- U_A0 pad G7: A0_CH1_DMI3 -> GND
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Routing:
- net LINK0_SOF: track 56.0 -> 52.2 mm
- net LINK0_READY_BACK: track 54.1 -> 50.3 mm
- net LINK0_VALID: track 55.2 -> 51.6 mm
- net LINK0_CLOCK: track 53.2 -> 49.7 mm
- net LINK0_DATA31: track 54.5 -> 51.0 mm
- net LINK0_DATA30: track 52.4 -> 49.1 mm
- net LINK0_DATA29: track 53.8 -> 50.6 mm
- net LINK0_DATA28: track 51.8 -> 48.6 mm
- net LINK0_DATA27: track 53.3 -> 50.2 mm
- net LINK9_VALID: track 13.4 -> 10.3 mm
- net LINK9_DATA31: track 13.4 -> 10.3 mm
- net LINK9_DATA3: track 13.4 -> 10.3 mm
- net LINK9_DATA23: track 13.4 -> 10.3 mm
- net LINK9_DATA21: track 13.4 -> 10.3 mm
- net LINK9_DATA13: track 13.4 -> 10.3 mm
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
Commit message: Retarget the board to a host-attached 1U chassis
The energy model put the board at 0.5 to 1.6 kW of input across the
throughput range, which is a rack supply, not a PCIe slot.  The board is
now one 420 x 360 mm board in a 1U: two CRPS modules in a 1+1 pair, a
BMC with its own Ethernet, six front fans, and a SlimSAS 8i cable to the
host's PCIe.  With the room to carry it, the ASIC package is rated at the
50K tokens/s target (177 A core), which selects the 1225-ball 29 mm
package.

hw/board.yaml: 1U form factor, host cable, CRPS input, BMC, PSU, fan and
RJ45 parts and classes, 50K package rating.

hw/kicad_gen.py: form factors (1U default, card kept) that map the ring
frame onto the physical board with keep-outs (PSU bay, rear I/O, fans),
physical parts for the chassis connectors and BMC, a fit check, layout
derived from the package body, the FPGA beside H1 taking the ring on its
west edge (closing hop 74 mm instead of 95 mm with the 29 mm package),
PCIe pins on the FPGA's south edge, regulators spaced for the larger
package.  Every hop is within the 80 mm limit and pcbnew DRC reports only
the unrouted nets.

Tests cover both form factors, the keep-outs and the package rating;
docs describe the 1U, the rating decision and the floorplan findings.

Co-Authored-By: Claude Fable 5.1 <noreply@anthropic.com>
Claude-Session: https://claude.ai/code/session_01VmmvkZe8Ctg3RAykNGsQBn
Parts:
- removed J_AUX: 12V-2x6 aux, appliance:12V-2x6
- removed J_PCIE: PCIe x8 edge, appliance:PCIE_X8_EDGE
- added J_BMC_NET: BMC Ethernet, appliance:RJ45_MAGJACK, F.Cu at (50.0, 367.0)
- added J_FAN0: fan header, appliance:FAN_4PIN, F.Cu at (55.0, 32.0)
- added J_FAN1: fan header, appliance:FAN_4PIN, F.Cu at (125.0, 32.0)
- added J_FAN2: fan header, appliance:FAN_4PIN, F.Cu at (195.0, 32.0)
- added J_FAN3: fan header, appliance:FAN_4PIN, F.Cu at (265.0, 32.0)
- added J_FAN4: fan header, appliance:FAN_4PIN, F.Cu at (335.0, 32.0)
- added J_FAN5: fan header, appliance:FAN_4PIN, F.Cu at (405.0, 32.0)
- added J_HOST: SlimSAS 8i host cable, appliance:SLIMSAS_8I, F.Cu at (175.5, 374.0)
- added J_PSU0: CRPS 12 V output, appliance:CRPS_BLADES, F.Cu at (320.0, 200.0)
- added J_PSU1: CRPS 12 V output, appliance:CRPS_BLADES, F.Cu at (395.0, 200.0)
- added U_BMC: BMC SoC, appliance:BGA_BMC_21x21, F.Cu at (120.0, 320.0)
- U_A0, U_A1, U_A2, U_A3, U_A4, U_A5, U_A6, U_A7, U_H0, U_H1: footprint appliance:FCBGA784_28x28_P0.8 -> appliance:FCBGA1225_35x35_P0.8
- moved U_D0 343.5 mm to (185.0, 342.0)
- moved U_CLK 339.0 mm to (258.0, 362.0)
- moved U_D1 332.4 mm to (185.0, 333.5)
- moved U_FPGA 327.9 mm to (205.5, 341.5)
- moved U_D2 321.3 mm to (185.0, 325.0)
- moved J_SFP 310.6 mm to (80.0, 353.0)
- moved U_D3 310.3 mm to (185.0, 316.5)
- moved U_H1 308.9 mm to (236.0, 344.0)
- moved VRM_H1 299.4 mm to (255.8, 342.0)
- moved REG_3V3 290.8 mm to (183.0, 301.0)
- moved REG_DDR 283.2 mm to (191.0, 300.0)
- moved REG_FPGA 278.6 mm to (216.5, 315.0)
- moved U_H0 262.2 mm to (236.0, 308.0)
- moved VRM_H0 253.9 mm to (255.8, 306.0)
- moved U_M0a 250.7 mm to (176.5, 281.5)
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Connections:
- U_A0 pad AA1: LINK0_DATA30 -> LINK0_DATA24
- U_A0 pad AA2: LINK0_DATA31 -> LINK0_DATA25
- U_A0 pad AA27: LINK1_DATA31 -> GND
- U_A0 pad AA28: LINK1_DATA30 -> VDD_CORE_A0
- U_A0 pad AB1: LINK0_CLOCK -> LINK0_DATA26
- U_A0 pad AB2: LINK0_VALID -> LINK0_DATA27
- U_A0 pad AB27: LINK1_VALID -> VDD_CORE_A0
- U_A0 pad AB28: LINK1_CLOCK -> GND
- U_A0 pad AC1: LINK0_READY_BACK -> LINK0_DATA28
- U_A0 pad AC2: LINK0_SOF -> LINK0_DATA29
- U_A0 pad AC27: LINK1_SOF -> GND
- U_A0 pad AC28: LINK1_READY_BACK -> VDD_CORE_A0
- U_A0 pad AD1: VDD_CORE_A0 -> LINK0_DATA30
- U_A0 pad AD2: GND -> LINK0_DATA31
- U_A0 pad AE1: GND -> LINK0_CLOCK
- U_A0 pad AE2: VDD_CORE_A0 -> LINK0_VALID
- U_A0 pad AF1: VDD_CORE_A0 -> LINK0_READY_BACK
- U_A0 pad AF2: GND -> LINK0_SOF
- U_A0 pad AH10: JTAG_TMS -> GND
- U_A0 pad AH11: JTAG_TDO_FPGA -> VDD_CORE_A0
- U_A0 pad AH13: JTAG_TDO_A0 -> VDD_CORE_A0
- U_A0 pad AH14: JTAG_TRST -> GND
- U_A0 pad AH15: REFCLK_A0_P -> VDD_CORE_A0
- U_A0 pad AH16: REFCLK_A0_N -> GND
- U_A0 pad AH17: GND -> VDD_CORE_A0
- U_A0 pad AH18: MODE0_A0 -> GND
- U_A0 pad AH19: MODE1_A0 -> VDD_CORE_A0
- U_A0 pad AH3: MGMT_SCLK -> VDD_CORE_A0
- U_A0 pad AH4: MGMT_MOSI -> GND
- U_A0 pad AH5: MGMT_MISO -> VDD_CORE_A0
- U_A0 pad AH6: MGMT_CS_A0 -> GND
- U_A0 pad AH7: GND -> VDD_CORE_A0
- U_A0 pad AH8: MGMT_IRQ_A0 -> GND
- U_A0 pad AH9: JTAG_TCK -> VDD_CORE_A0
- U_A0 pad B1: A0_CH0_DQ20 -> GND
- U_A0 pad B10: A0_CH0_DQ25 -> A0_CH0_DQS3_P
- U_A0 pad B11: A0_CH0_DQ26 -> A0_CH0_DQS3_N
- U_A0 pad B12: A0_CH0_DQ27 -> A0_CH0_DMI3
- U_A0 pad B13: A0_CH0_DQ28 -> GND
- U_A0 pad B14: A0_CH0_DQ29 -> A0_CH0_CA0
- U_A0 pad B15: A0_CH0_DQ30 -> A0_CH0_CA1
- U_A0 pad B16: A0_CH0_DQ31 -> A0_CH0_CA2
- U_A0 pad B17: A0_CH0_DQS3_P -> A0_CH0_CA3
- U_A0 pad B18: A0_CH0_DQS3_N -> A0_CH0_CA4
- U_A0 pad B19: A0_CH0_DMI3 -> A0_CH0_CA5
- U_A0 pad B2: A0_CH0_DQ21 -> A0_CH0_DQ24
- U_A0 pad B20: GND -> A0_CH0_CA6
- U_A0 pad B21: A0_CH0_CA0 -> A0_CH0_CA7
- U_A0 pad B22: A0_CH0_CA1 -> A0_CH0_CA8
- U_A0 pad B23: A0_CH0_CA2 -> A0_CH0_CA9
- U_A0 pad B24: A0_CH0_CA3 -> A0_CH0_CA10
- U_A0 pad B25: A0_CH0_CA4 -> A0_CH0_CA11
- U_A0 pad B26: A0_CH0_CA5 -> A0_CH0_CA12
- U_A0 pad B27: A0_CH0_CA6 -> A0_CH0_CA13
- U_A0 pad B28: A0_CH0_CA7 -> A0_CH0_CS0
- U_A0 pad B3: A0_CH0_DQ22 -> A0_CH0_DQ25
- U_A0 pad B4: A0_CH0_DQ23 -> A0_CH0_DQ26
- U_A0 pad B5: A0_CH0_DQS2_P -> A0_CH0_DQ27
- U_A0 pad B6: A0_CH0_DQS2_N -> A0_CH0_DQ28
- U_A0 pad B7: A0_CH0_DMI2 -> A0_CH0_DQ29
- U_A0 pad B8: GND -> A0_CH0_DQ30
- U_A0 pad B9: A0_CH0_DQ24 -> A0_CH0_DQ31
- U_A0 pad C1: A0_CH0_CA8 -> A0_CH1_DQ0
- U_A0 pad C10: A0_CH0_CK0_N -> A0_CH1_DQS0_N
- U_A0 pad C11: A0_CH0_CK1_P -> A0_CH1_DMI0
- U_A0 pad C12: A0_CH0_CK1_N -> GND
- U_A0 pad C13: A0_CH0_RESET -> A0_CH1_DQ8
- U_A0 pad C14: GND -> A0_CH1_DQ9
- U_A0 pad C15: A0_CH1_DQ0 -> A0_CH1_DQ10
- U_A0 pad C16: A0_CH1_DQ1 -> A0_CH1_DQ11
- U_A0 pad C17: A0_CH1_DQ2 -> A0_CH1_DQ12
- U_A0 pad C18: A0_CH1_DQ3 -> A0_CH1_DQ13
- U_A0 pad C19: A0_CH1_DQ4 -> A0_CH1_DQ14
- U_A0 pad C2: A0_CH0_CA9 -> A0_CH1_DQ1
- U_A0 pad C20: A0_CH1_DQ5 -> A0_CH1_DQ15
- U_A0 pad C21: A0_CH1_DQ6 -> A0_CH1_DQS1_P
- U_A0 pad C22: A0_CH1_DQ7 -> A0_CH1_DQS1_N
- U_A0 pad C23: A0_CH1_DQS0_P -> A0_CH1_DMI1
- U_A0 pad C24: A0_CH1_DQS0_N -> GND
- U_A0 pad C25: A0_CH1_DMI0 -> A0_CH1_DQ16
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Routing:
- net LINK10_READY_BACK: track 70.0 -> 55.4 mm
- net LINK10_SOF: track 72.1 -> 57.7 mm
- net LINK10_CLOCK: track 69.9 -> 55.7 mm
- net LINK10_VALID: track 72.0 -> 58.1 mm
- net LINK10_DATA30: track 69.9 -> 56.1 mm
- net LINK10_DATA31: track 72.0 -> 58.5 mm
- net LINK10_DATA28: track 69.9 -> 56.5 mm
- net LINK10_DATA29: track 72.1 -> 58.9 mm
- net LINK10_DATA26: track 69.9 -> 57.0 mm
- net LINK10_DATA27: track 72.2 -> 59.5 mm
- net LINK10_DATA24: track 70.1 -> 57.6 mm
- net LINK10_DATA25: track 72.3 -> 60.1 mm
- net LINK10_DATA22: track 70.3 -> 58.3 mm
- net LINK10_DATA23: track 72.6 -> 60.8 mm
- net LINK10_DATA20: track 70.6 -> 59.1 mm
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Other:
- board size 312 x 111.2 mm -> 420 x 360 mm
- board text added: "PSU bay (two CRPS)"
- board text added: "appliance: 1U rack chassis, single board, host-attached, floorplan generated from hw/board.yaml"
- board text added: "front fans"
- board text added: "rear I/O"
- board text removed: "appliance: floorplan generated from hw/board.yaml"
