File: hw/kicad/appliance.kicad_pcb (KiCad board)
At the start: 12 copper layers, 420 x 360 mm, 61 parts

Commit message: Lay the activation ring out as a regular polygon
The two-row snake had two hops at the edge of the 80 mm link limit (row
change 76 mm, closing hop 74 mm) that only fit with compressed lanes split
over two layers, and each row of four sat in series in the airflow.  The
ring is now a regular 11-gon: one ring node per vertex (FPGA, eight layer
ASICs, two heads), each chip rotated tangentially with its two LPDDR5X
devices on its outer edge and its core regulator on its inner edge, the
shared regulators and the clock generator in the middle.  Every hop is
one 36-lane ribbon on one layer with two bends of 16 to 20 degrees; the
longest lane anywhere is 39 mm.  All eleven nodes are on the polygon
because a chip takes the ring in on one edge and out on the opposite one,
so a loop cannot dip into the middle without a hairpin.

hw/kicad_gen.py: arbitrary part rotation (rotated footprint outlines,
courtyards and pads), a polygon layout derived from the ring order and
the package body, a general bent-ribbon router (offset-line corners at
any angle, paths that start past the outer escape vias), oriented fit
and overlap checks, rotated rail islands; the ring frame and the card
form factor are gone.  hw/board.py draws the block diagram as the same
polygon; board.yaml names the vertices.  pcbnew DRC reports only the
unrouted nets; tests check the polygon geometry, orientation of memories
and regulators, bend angles and hop lengths.

Co-Authored-By: Claude Fable 5.1 <noreply@anthropic.com>
Claude-Session: https://claude.ai/code/session_01VmmvkZe8Ctg3RAykNGsQBn
Parts:
- moved U_CLK 198.0 mm to (160.0, 190.0)
- moved U_M2a 144.0 mm to (34.5, 181.6)
- moved U_A2 143.5 mm to (58.1, 175.4)
- moved U_M4a 143.0 mm to (115.5, 72.3)
- moved U_M2b 141.4 mm to (37.2, 162.7)
- moved VRM_A2 140.4 mm to (77.7, 178.2)
- moved U_M1b 138.5 mm to (42.0, 233.5)
- moved U_A1 134.6 mm to (66.4, 232.8)
- moved VRM_A1 133.2 mm to (84.3, 224.6)
- moved U_M1a 130.5 mm to (49.8, 250.7)
- moved U_M4b 127.9 mm to (133.8, 67.0)
- moved VRM_A3 124.6 mm to (97.1, 135.5)
- moved U_A3 122.4 mm to (82.2, 122.6)
- moved U_M3a 119.1 mm to (59.0, 115.0)
- moved REG_0V9 116.6 mm to (148.0, 208.0)
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Routing:
- net LINK4_DATA1: track 77.6 -> 39.1 mm
- net LINK4_DATA0: track 74.9 -> 37.0 mm
- net LINK4_DATA3: track 76.0 -> 38.7 mm
- net LINK4_DATA2: track 73.3 -> 36.5 mm
- net LINK4_DATA5: track 74.5 -> 38.2 mm
- net LINK4_DATA4: track 71.8 -> 36.0 mm
- net LINK4_DATA7: track 73.0 -> 37.7 mm
- net LINK4_DATA6: track 70.3 -> 35.6 mm
- net LINK10_DATA1: track 75.1 -> 40.5 mm
- net LINK4_DATA9: track 71.6 -> 37.3 mm
- net LINK10_DATA0: track 72.1 -> 38.1 mm
- net LINK4_DATA8: track 68.9 -> 35.1 mm
- net LINK4_DATA11: track 70.2 -> 36.8 mm
- net LINK10_DATA3: track 73.4 -> 40.0 mm
- net LINK4_DATA10: track 67.6 -> 34.7 mm
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
Commit message: Tighten the ring polygon to a 46 mm side
The neighbour spacing beyond the package body drops from 29 mm to 17 mm
(circumradius 103 mm to 82 mm, ring envelope about 230 mm), with the
straight run at each port shortened to 5 mm.  Every hop is now 27 mm at
most with bends of up to 23 degrees; pcbnew DRC still reports only the
unrouted nets.  A 15 mm gap also passes; below that the ports are too
close for a ribbon to bend.

Co-Authored-By: Claude Fable 5.1 <noreply@anthropic.com>
Claude-Session: https://claude.ai/code/session_01VmmvkZe8Ctg3RAykNGsQBn
Parts:
- moved VRM_A6 21.3 mm to (206.8, 149.5)
- moved VRM_A3 21.3 mm to (113.2, 149.5)
- moved U_M2b 21.3 mm to (58.3, 165.8)
- moved U_M7a 21.3 mm to (261.7, 165.8)
- moved U_M4a 21.3 mm to (121.5, 92.8)
- moved U_M5b 21.3 mm to (198.5, 92.8)
- moved VRM_H0 21.3 mm to (216.3, 215.7)
- moved U_M1b 21.3 mm to (61.3, 224.6)
- moved U_M1a 21.3 mm to (69.2, 241.9)
- moved VRM_A1 21.3 mm to (103.7, 215.7)
- moved U_A3 21.3 mm to (98.3, 136.5)
- moved U_A6 21.3 mm to (221.7, 136.5)
- moved REG_FPGA 21.3 mm to (160.0, 252.4)
- moved U_D0 21.3 mm to (172.8, 292.4)
- moved U_D1 21.3 mm to (164.2, 292.4)
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Routing:
- net LINK5_DATA9: track 37.3 -> 25.0 mm
- net LINK3_DATA16: track 33.3 -> 21.0 mm
- net LINK7_DATA16: track 33.3 -> 21.0 mm
- net LINK1_DATA21: track 34.5 -> 22.3 mm
- net LINK9_DATA21: track 34.5 -> 22.3 mm
- net LINK8_DATA19: track 35.0 -> 22.7 mm
- net LINK2_DATA19: track 35.0 -> 22.7 mm
- net LINK3_DATA0: track 37.0 -> 24.7 mm
- net LINK7_DATA0: track 37.0 -> 24.7 mm
- net LINK3_DATA27: track 33.1 -> 20.9 mm
- net LINK7_DATA27: track 33.1 -> 20.9 mm
- net LINK3_DATA11: track 36.8 -> 24.6 mm
- net LINK7_DATA11: track 36.8 -> 24.6 mm
- net LINK7_DATA31: track 32.2 -> 20.0 mm
- net LINK3_DATA31: track 32.2 -> 20.0 mm
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