File: hw/kicad/appliance.kicad_pcb (KiCad board)
At the start: 12 copper layers, 420 x 360 mm, 61 parts

Commit message: Add the four-plus-one high-end board variant with HBM in the package
hw/board_27b.yaml describes the 27B-class appliance on a 2 nm-class die:
four layer ASICs of sixteen layers, one head ASIC holding the whole LM
head, an HBM4 stack on each layer ASIC's interposer (no memory on the
board), direct-to-chip liquid cooling, a 1+1 pair of 3000 W CRPS modules,
rated at the 234K tokens/s fabric ceiling (525 W and 656 A per layer die,
a 55 x 55 package of 3025 balls, a hexagon ring of 85 mm side with 10 mm
between packages for the cold plates).  The simulator's 27B configs
become 4 + 1 too; throughput and board power are unchanged, per-die power
doubles.

To carry a second description the tools now take the memory channels
from the class's interfaces (none for in-package HBM), the rail ball
counts from the package rules, the regulators from the power tree (one
block per shared rail in the middle of the polygon, the FPGA's rails on
one block, DDR4 and 3.3 V beside the DDR4 row), a per-board ring gap, and
ball names past 40 rows; outputs are named after the source.  The
overlap test's margin had the wrong sign and let bodies touch by half a
millimetre; fixed, and both boards pass pcbnew DRC with only the unrouted
nets.  Tests cover the variant's hexagon, package, rails and fit.

Co-Authored-By: Claude Fable 5.1 <noreply@anthropic.com>
Claude-Session: https://claude.ai/code/session_01VmmvkZe8Ctg3RAykNGsQBn
Parts:
- added REG_IO_1V8: VDD_IO_1V8 regulator, appliance:REG_MODULE_20x6, F.Cu at (148.0, 180.0)
- REG_1V8: value VDD_IO_1V8 regulator -> VDD1_1V8 regulator
- REG_DDR: value VDD_1V2 regulator -> VDD_1V2, VPP_2V5 regulator
- REG_FPGA: value VCCINT_0V85 regulator -> VCCINT_0V85, VCCAUX_1V8, VCCO_1V8, VCCO_1V2, MGTAVCC, MGTAVTT regulator
- moved REG_0V3 8.00 mm to (172.0, 200.0)
- moved REG_0V9 8.00 mm to (148.0, 200.0)
- moved REG_1V05 8.00 mm to (172.0, 180.0)
Connections:
- REG_0V3 pad 7: VDDQ_0V3 -> GND
- REG_0V9 pad 5: VDD_PLL_0V9 -> VDD2L_0V9
- REG_0V9 pad 7: VDD2L_0V9 -> GND
- REG_1V05 pad 5: VCCO_1V2 -> VDD2H_1V05
- REG_1V05 pad 7: VDD2H_1V05 -> GND
- REG_1V8 pad 5: VCCO_1V8 -> VDD1_1V8
- REG_1V8 pad 6: VDD_IO_1V8 -> VDD1_1V8
- REG_1V8 pad 7: VDD_IO_1V8 -> GND
- REG_3V3 pad 7: VDD_3V3 -> GND
- REG_DDR pad 6: VPP_2V5 -> VDD_1V2
- REG_DDR pad 7: VDD_1V2 -> VPP_2V5
- REG_FPGA pad 10: GND -> MGTAVCC
- REG_FPGA pad 5: VCCAUX_1V8 -> VCCINT_0V85
- REG_FPGA pad 6: MGTAVCC -> VCCINT_0V85
- REG_FPGA pad 7: MGTAVTT -> VCCAUX_1V8
- REG_FPGA pad 8: GND -> VCCO_1V8
- REG_FPGA pad 9: GND -> VCCO_1V2
Routing:
- net VDD_IO_1V8: vias 83 -> 84
- net VCCINT_0V85: vias 175 -> 177
- net GND: vias 7513 -> 7516
- net +12V: vias 79 -> 82
