File: hw/kicad/asics.kicad_sch (KiCad schematic)
At the start: 10 parts

Commit message: hw: derive the ASIC package and ball map from the power model
hw/pinout.py turns the interface list, the power model and the
package_selection rules in board.yaml into the ball count the core rail
needs, the smallest candidate package that carries it, and a rule-based
ball map (links on the west and east edges as two columns of 18 rows,
both LPDDR channels on the north rows in byte lanes with ground returns,
management on the south row, ground and core in a checkerboard), written
as CSV, JSON and a report for the packaging house.  At the design point
the 400-ball draft package cannot carry 54 A of core current; a 784-ball
28x28 array at 0.8 mm in the same 23 mm body is selected.  The KiCad
generator now builds the ASIC footprint from this map: escape geometry
and lane pitch follow the ball pitch, ribbon paths run through each
port's lane centre, and hops between packages of different pitch rescale
their lanes.  DRC stays clean apart from the unrouted nets.

Co-Authored-By: Claude Fable 5.1 <noreply@anthropic.com>
Claude-Session: https://claude.ai/code/session_01VmmvkZe8Ctg3RAykNGsQBn
Parts:
- U_A0, U_A1, U_A2, U_A3, U_A4, U_A5, U_A6, U_A7, U_H0, U_H1: footprint appliance:FCBGA400_20x20_P1.0 -> appliance:FCBGA784_28x28_P0.8
Connections:
- net A0_CH0_CA0: now also U_A0.B21; no longer U_A0.C7
- net A0_CH0_CA1: now also U_A0.B22; no longer U_A0.C8
- net A0_CH0_CA10: now also U_A0.C3; no longer U_A0.C17
- net A0_CH0_CA11: now also U_A0.C4; no longer U_A0.C18
- net A0_CH0_CA12: now also U_A0.C5; no longer U_A0.D3
- net A0_CH0_CA13: now also U_A0.C6; no longer U_A0.D4
- net A0_CH0_CA2: now also U_A0.B23; no longer U_A0.C9
- net A0_CH0_CA3: now also U_A0.B24; no longer U_A0.C10
- net A0_CH0_CA4: now also U_A0.B25; no longer U_A0.C11
- net A0_CH0_CA5: now also U_A0.B26; no longer U_A0.C12
- net A0_CH0_CA6: now also U_A0.B27; no longer U_A0.C13
- net A0_CH0_CA7: now also U_A0.B28; no longer U_A0.C14
- net A0_CH0_CA8: now also U_A0.C1; no longer U_A0.C15
- net A0_CH0_CA9: now also U_A0.C2; no longer U_A0.C16
- net A0_CH0_CK0_N: now also U_A0.C10; no longer U_A0.D8
- net A0_CH0_CK0_P: now also U_A0.C9; no longer U_A0.D7
- net A0_CH0_CK1_N: now also U_A0.C12; no longer U_A0.D10
- net A0_CH0_CK1_P: now also U_A0.C11; no longer U_A0.D9
- net A0_CH0_CS0: now also U_A0.C7; no longer U_A0.D5
- net A0_CH0_CS1: now also U_A0.C8; no longer U_A0.D6
- net A0_CH0_DMI0: now also U_A0.A11; no longer U_A0.C3
- net A0_CH0_DMI1: now also U_A0.A23; no longer U_A0.C4
- net A0_CH0_DMI2: now also U_A0.B7; no longer U_A0.C5
- net A0_CH0_DMI3: now also U_A0.B19; no longer U_A0.C6
- net A0_CH0_DQ10: now also U_A0.A15; no longer U_A0.A11
- net A0_CH0_DQ11: now also U_A0.A16; no longer U_A0.A12
- net A0_CH0_DQ12: now also U_A0.A17; no longer U_A0.A13
- net A0_CH0_DQ13: now also U_A0.A18; no longer U_A0.A14
- net A0_CH0_DQ14: now also U_A0.A19; no longer U_A0.A15
- net A0_CH0_DQ15: now also U_A0.A20; no longer U_A0.A16
- net A0_CH0_DQ16: now also U_A0.A25; no longer U_A0.A17
- net A0_CH0_DQ17: now also U_A0.A26; no longer U_A0.A18
- net A0_CH0_DQ18: now also U_A0.A27; no longer U_A0.A19
- net A0_CH0_DQ19: now also U_A0.A28; no longer U_A0.A20
- net A0_CH0_DQ24: now also U_A0.B9; no longer U_A0.B5
- net A0_CH0_DQ25: now also U_A0.B10; no longer U_A0.B6
- net A0_CH0_DQ26: now also U_A0.B11; no longer U_A0.B7
- net A0_CH0_DQ27: now also U_A0.B12; no longer U_A0.B8
- net A0_CH0_DQ28: now also U_A0.B13; no longer U_A0.B9
- net A0_CH0_DQ29: now also U_A0.B14; no longer U_A0.B10
- net A0_CH0_DQ30: now also U_A0.B15; no longer U_A0.B11
- net A0_CH0_DQ31: now also U_A0.B16; no longer U_A0.B12
- net A0_CH0_DQ8: now also U_A0.A13; no longer U_A0.A9
- net A0_CH0_DQ9: now also U_A0.A14; no longer U_A0.A10
- net A0_CH0_DQS0_N: now also U_A0.A10; no longer U_A0.B14
- net A0_CH0_DQS0_P: now also U_A0.A9; no longer U_A0.B13
- net A0_CH0_DQS1_N: now also U_A0.A22; no longer U_A0.B16
- net A0_CH0_DQS1_P: now also U_A0.A21; no longer U_A0.B15
- net A0_CH0_DQS2_N: now also U_A0.B6; no longer U_A0.B18
- net A0_CH0_DQS2_P: now also U_A0.B5; no longer U_A0.B17
- net A0_CH0_DQS3_N: now also U_A0.B18; no longer U_A0.B20
- net A0_CH0_DQS3_P: now also U_A0.B17; no longer U_A0.B19
- net A0_CH0_RESET: now also U_A0.C13; no longer U_A0.D11
- net A0_CH1_CA0: now also U_A0.E7; no longer U_A0.G8
- net A0_CH1_CA1: now also U_A0.E8; no longer U_A0.G9
- net A0_CH1_CA10: now also U_A0.E17; no longer U_A0.G18
- net A0_CH1_CA11: now also U_A0.E18; no longer U_A0.H3
- net A0_CH1_CA12: now also U_A0.E19; no longer U_A0.H4
- net A0_CH1_CA13: now also U_A0.E20; no longer U_A0.H5
- net A0_CH1_CA2: now also U_A0.E9; no longer U_A0.G10
- net A0_CH1_CA3: now also U_A0.E10; no longer U_A0.G11
- net A0_CH1_CA4: now also U_A0.E11; no longer U_A0.G12
- net A0_CH1_CA5: now also U_A0.E12; no longer U_A0.G13
- net A0_CH1_CA6: now also U_A0.E13; no longer U_A0.G14
- net A0_CH1_CA7: now also U_A0.E14; no longer U_A0.G15
- net A0_CH1_CA8: now also U_A0.E15; no longer U_A0.G16
- net A0_CH1_CA9: now also U_A0.E16; no longer U_A0.G17
- net A0_CH1_CK0_N: now also U_A0.E24; no longer U_A0.H9
- net A0_CH1_CK0_P: now also U_A0.E23; no longer U_A0.H8
- net A0_CH1_CK1_N: now also U_A0.E26; no longer U_A0.H11
- net A0_CH1_CK1_P: now also U_A0.E25; no longer U_A0.H10
- net A0_CH1_CS0: now also U_A0.E21; no longer U_A0.H6
- net A0_CH1_CS1: now also U_A0.E22; no longer U_A0.H7
- net A0_CH1_DMI0: now also U_A0.C25; no longer U_A0.G4
- net A0_CH1_DMI1: now also U_A0.D9; no longer U_A0.G5
- net A0_CH1_DMI2: now also U_A0.D21; no longer U_A0.G6
- net A0_CH1_DMI3: now also U_A0.E5; no longer U_A0.G7
- net A0_CH1_DQ0: now also U_A0.C15; no longer U_A0.D12
- net A0_CH1_DQ1: now also U_A0.C16; no longer U_A0.D13
- net A0_CH1_DQ10: now also U_A0.D1; no longer U_A0.E6
- net A0_CH1_DQ11: now also U_A0.D2; no longer U_A0.E7
- net A0_CH1_DQ12: now also U_A0.D3; no longer U_A0.E8
- net A0_CH1_DQ13: now also U_A0.D4; no longer U_A0.E9
- net A0_CH1_DQ14: now also U_A0.D5; no longer U_A0.E10
- net A0_CH1_DQ15: now also U_A0.D6; no longer U_A0.E11
- net A0_CH1_DQ16: now also U_A0.D11; no longer U_A0.E12
- net A0_CH1_DQ17: now also U_A0.D12; no longer U_A0.E13
- net A0_CH1_DQ18: now also U_A0.D13; no longer U_A0.E14
- net A0_CH1_DQ19: now also U_A0.D14; no longer U_A0.E15
- net A0_CH1_DQ2: now also U_A0.C17; no longer U_A0.D14
- net A0_CH1_DQ20: now also U_A0.D15; no longer U_A0.E16
- net A0_CH1_DQ21: now also U_A0.D16; no longer U_A0.E17
- net A0_CH1_DQ22: now also U_A0.D17; no longer U_A0.E18
- net A0_CH1_DQ23: now also U_A0.D18; no longer U_A0.F3
- net A0_CH1_DQ24: now also U_A0.D23; no longer U_A0.F4
- net A0_CH1_DQ25: now also U_A0.D24; no longer U_A0.F5
- net A0_CH1_DQ26: now also U_A0.D25; no longer U_A0.F6
- net A0_CH1_DQ27: now also U_A0.D26; no longer U_A0.F7
- net A0_CH1_DQ28: now also U_A0.D27; no longer U_A0.F8
- net A0_CH1_DQ29: now also U_A0.D28; no longer U_A0.F9
- net A0_CH1_DQ3: now also U_A0.C18; no longer U_A0.D15
- net A0_CH1_DQ30: now also U_A0.E1; no longer U_A0.F10
- net A0_CH1_DQ31: now also U_A0.E2; no longer U_A0.F11
- net A0_CH1_DQ4: now also U_A0.C19; no longer U_A0.D16
- net A0_CH1_DQ5: now also U_A0.C20; no longer U_A0.D17
- net A0_CH1_DQ6: now also U_A0.C21; no longer U_A0.D18
- net A0_CH1_DQ7: now also U_A0.C22; no longer U_A0.E3
- net A0_CH1_DQ8: now also U_A0.C27; no longer U_A0.E4
- net A0_CH1_DQ9: now also U_A0.C28; no longer U_A0.E5
- net A0_CH1_DQS0_N: now also U_A0.C24; no longer U_A0.F13
- net A0_CH1_DQS0_P: now also U_A0.C23; no longer U_A0.F12
- net A0_CH1_DQS1_N: now also U_A0.D8; no longer U_A0.F15
- net A0_CH1_DQS1_P: now also U_A0.D7; no longer U_A0.F14
- net A0_CH1_DQS2_N: now also U_A0.D20; no longer U_A0.F17
- net A0_CH1_DQS2_P: now also U_A0.D19; no longer U_A0.F16
- net A0_CH1_DQS3_N: now also U_A0.E4; no longer U_A0.G3
- net A0_CH1_DQS3_P: now also U_A0.E3; no longer U_A0.F18
- net A0_CH1_RESET: now also U_A0.E27; no longer U_A0.H12
- net A1_CH0_CA0: now also U_A1.B21; no longer U_A1.C7
- net A1_CH0_CA1: now also U_A1.B22; no longer U_A1.C8
- net A1_CH0_CA10: now also U_A1.C3; no longer U_A1.C17
- net A1_CH0_CA11: now also U_A1.C4; no longer U_A1.C18
- net A1_CH0_CA12: now also U_A1.C5; no longer U_A1.D3
- net A1_CH0_CA13: now also U_A1.C6; no longer U_A1.D4
- net A1_CH0_CA2: now also U_A1.B23; no longer U_A1.C9
- net A1_CH0_CA3: now also U_A1.B24; no longer U_A1.C10
- net A1_CH0_CA4: now also U_A1.B25; no longer U_A1.C11
- net A1_CH0_CA5: now also U_A1.B26; no longer U_A1.C12
- net A1_CH0_CA6: now also U_A1.B27; no longer U_A1.C13
- net A1_CH0_CA7: now also U_A1.B28; no longer U_A1.C14
- net A1_CH0_CA8: now also U_A1.C1; no longer U_A1.C15
- net A1_CH0_CA9: now also U_A1.C2; no longer U_A1.C16
- net A1_CH0_CK0_N: now also U_A1.C10; no longer U_A1.D8
- net A1_CH0_CK0_P: now also U_A1.C9; no longer U_A1.D7
- net A1_CH0_CK1_N: now also U_A1.C12; no longer U_A1.D10
- net A1_CH0_CK1_P: now also U_A1.C11; no longer U_A1.D9
- net A1_CH0_CS0: now also U_A1.C7; no longer U_A1.D5
- net A1_CH0_CS1: now also U_A1.C8; no longer U_A1.D6
- net A1_CH0_DMI0: now also U_A1.A11; no longer U_A1.C3
- net A1_CH0_DMI1: now also U_A1.A23; no longer U_A1.C4
- net A1_CH0_DMI2: now also U_A1.B7; no longer U_A1.C5
- net A1_CH0_DMI3: now also U_A1.B19; no longer U_A1.C6
- net A1_CH0_DQ10: now also U_A1.A15; no longer U_A1.A11
- net A1_CH0_DQ11: now also U_A1.A16; no longer U_A1.A12
- net A1_CH0_DQ12: now also U_A1.A17; no longer U_A1.A13
- net A1_CH0_DQ13: now also U_A1.A18; no longer U_A1.A14
- net A1_CH0_DQ14: now also U_A1.A19; no longer U_A1.A15
- net A1_CH0_DQ15: now also U_A1.A20; no longer U_A1.A16
- net A1_CH0_DQ16: now also U_A1.A25; no longer U_A1.A17
- net A1_CH0_DQ17: now also U_A1.A26; no longer U_A1.A18
- net A1_CH0_DQ18: now also U_A1.A27; no longer U_A1.A19
- net A1_CH0_DQ19: now also U_A1.A28; no longer U_A1.A20
- net A1_CH0_DQ24: now also U_A1.B9; no longer U_A1.B5
- net A1_CH0_DQ25: now also U_A1.B10; no longer U_A1.B6
- net A1_CH0_DQ26: now also U_A1.B11; no longer U_A1.B7
- net A1_CH0_DQ27: now also U_A1.B12; no longer U_A1.B8
- net A1_CH0_DQ28: now also U_A1.B13; no longer U_A1.B9
- net A1_CH0_DQ29: now also U_A1.B14; no longer U_A1.B10
- net A1_CH0_DQ30: now also U_A1.B15; no longer U_A1.B11
- net A1_CH0_DQ31: now also U_A1.B16; no longer U_A1.B12
- net A1_CH0_DQ8: now also U_A1.A13; no longer U_A1.A9
- net A1_CH0_DQ9: now also U_A1.A14; no longer U_A1.A10
- net A1_CH0_DQS0_N: now also U_A1.A10; no longer U_A1.B14
- net A1_CH0_DQS0_P: now also U_A1.A9; no longer U_A1.B13
- net A1_CH0_DQS1_N: now also U_A1.A22; no longer U_A1.B16
- net A1_CH0_DQS1_P: now also U_A1.A21; no longer U_A1.B15
- net A1_CH0_DQS2_N: now also U_A1.B6; no longer U_A1.B18
- net A1_CH0_DQS2_P: now also U_A1.B5; no longer U_A1.B17
- net A1_CH0_DQS3_N: now also U_A1.B18; no longer U_A1.B20
- net A1_CH0_DQS3_P: now also U_A1.B17; no longer U_A1.B19
- net A1_CH0_RESET: now also U_A1.C13; no longer U_A1.D11
- net A1_CH1_CA0: now also U_A1.E7; no longer U_A1.G8
- net A1_CH1_CA1: now also U_A1.E8; no longer U_A1.G9
- net A1_CH1_CA10: now also U_A1.E17; no longer U_A1.G18
- net A1_CH1_CA11: now also U_A1.E18; no longer U_A1.H3
- net A1_CH1_CA12: now also U_A1.E19; no longer U_A1.H4
- net A1_CH1_CA13: now also U_A1.E20; no longer U_A1.H5
- net A1_CH1_CA2: now also U_A1.E9; no longer U_A1.G10
- net A1_CH1_CA3: now also U_A1.E10; no longer U_A1.G11
- net A1_CH1_CA4: now also U_A1.E11; no longer U_A1.G12
- net A1_CH1_CA5: now also U_A1.E12; no longer U_A1.G13
- net A1_CH1_CA6: now also U_A1.E13; no longer U_A1.G14
- net A1_CH1_CA7: now also U_A1.E14; no longer U_A1.G15
- net A1_CH1_CA8: now also U_A1.E15; no longer U_A1.G16
- net A1_CH1_CA9: now also U_A1.E16; no longer U_A1.G17
- net A1_CH1_CK0_N: now also U_A1.E24; no longer U_A1.H9
- net A1_CH1_CK0_P: now also U_A1.E23; no longer U_A1.H8
- net A1_CH1_CK1_N: now also U_A1.E26; no longer U_A1.H11
- net A1_CH1_CK1_P: now also U_A1.E25; no longer U_A1.H10
- net A1_CH1_CS0: now also U_A1.E21; no longer U_A1.H6
- net A1_CH1_CS1: now also U_A1.E22; no longer U_A1.H7
- net A1_CH1_DMI0: now also U_A1.C25; no longer U_A1.G4
- net A1_CH1_DMI1: now also U_A1.D9; no longer U_A1.G5
- net A1_CH1_DMI2: now also U_A1.D21; no longer U_A1.G6
- net A1_CH1_DMI3: now also U_A1.E5; no longer U_A1.G7
- net A1_CH1_DQ0: now also U_A1.C15; no longer U_A1.D12
- net A1_CH1_DQ1: now also U_A1.C16; no longer U_A1.D13
- net A1_CH1_DQ10: now also U_A1.D1; no longer U_A1.E6
- net A1_CH1_DQ11: now also U_A1.D2; no longer U_A1.E7
- net A1_CH1_DQ12: now also U_A1.D3; no longer U_A1.E8
- net A1_CH1_DQ13: now also U_A1.D4; no longer U_A1.E9
- net A1_CH1_DQ14: now also U_A1.D5; no longer U_A1.E10
- net A1_CH1_DQ15: now also U_A1.D6; no longer U_A1.E11
- net A1_CH1_DQ16: now also U_A1.D11; no longer U_A1.E12
- net A1_CH1_DQ17: now also U_A1.D12; no longer U_A1.E13
- net A1_CH1_DQ18: now also U_A1.D13; no longer U_A1.E14
- net A1_CH1_DQ19: now also U_A1.D14; no longer U_A1.E15
- net A1_CH1_DQ2: now also U_A1.C17; no longer U_A1.D14
- net A1_CH1_DQ20: now also U_A1.D15; no longer U_A1.E16
- net A1_CH1_DQ21: now also U_A1.D16; no longer U_A1.E17
- net A1_CH1_DQ22: now also U_A1.D17; no longer U_A1.E18
- net A1_CH1_DQ23: now also U_A1.D18; no longer U_A1.F3
- net A1_CH1_DQ24: now also U_A1.D23; no longer U_A1.F4
- net A1_CH1_DQ25: now also U_A1.D24; no longer U_A1.F5
- net A1_CH1_DQ26: now also U_A1.D25; no longer U_A1.F6
- net A1_CH1_DQ27: now also U_A1.D26; no longer U_A1.F7
- net A1_CH1_DQ28: now also U_A1.D27; no longer U_A1.F8
- net A1_CH1_DQ29: now also U_A1.D28; no longer U_A1.F9
- net A1_CH1_DQ3: now also U_A1.C18; no longer U_A1.D15
- net A1_CH1_DQ30: now also U_A1.E1; no longer U_A1.F10
- net A1_CH1_DQ31: now also U_A1.E2; no longer U_A1.F11
- net A1_CH1_DQ4: now also U_A1.C19; no longer U_A1.D16
- net A1_CH1_DQ5: now also U_A1.C20; no longer U_A1.D17
- net A1_CH1_DQ6: now also U_A1.C21; no longer U_A1.D18
- net A1_CH1_DQ7: now also U_A1.C22; no longer U_A1.E3
- net A1_CH1_DQ8: now also U_A1.C27; no longer U_A1.E4
- net A1_CH1_DQ9: now also U_A1.C28; no longer U_A1.E5
- net A1_CH1_DQS0_N: now also U_A1.C24; no longer U_A1.F13
- net A1_CH1_DQS0_P: now also U_A1.C23; no longer U_A1.F12
- net A1_CH1_DQS1_N: now also U_A1.D8; no longer U_A1.F15
- net A1_CH1_DQS1_P: now also U_A1.D7; no longer U_A1.F14
- net A1_CH1_DQS2_N: now also U_A1.D20; no longer U_A1.F17
- net A1_CH1_DQS2_P: now also U_A1.D19; no longer U_A1.F16
- net A1_CH1_DQS3_N: now also U_A1.E4; no longer U_A1.G3
- net A1_CH1_DQS3_P: now also U_A1.E3; no longer U_A1.F18
- net A1_CH1_RESET: now also U_A1.E27; no longer U_A1.H12
- net A2_CH0_CA0: now also U_A2.B21; no longer U_A2.C7
- net A2_CH0_CA1: now also U_A2.B22; no longer U_A2.C8
- net A2_CH0_CA10: now also U_A2.C3; no longer U_A2.C17
- net A2_CH0_CA11: now also U_A2.C4; no longer U_A2.C18
- net A2_CH0_CA12: now also U_A2.C5; no longer U_A2.D3
- net A2_CH0_CA13: now also U_A2.C6; no longer U_A2.D4
- net A2_CH0_CA2: now also U_A2.B23; no longer U_A2.C9
- net A2_CH0_CA3: now also U_A2.B24; no longer U_A2.C10
- net A2_CH0_CA4: now also U_A2.B25; no longer U_A2.C11
- net A2_CH0_CA5: now also U_A2.B26; no longer U_A2.C12
- net A2_CH0_CA6: now also U_A2.B27; no longer U_A2.C13
- net A2_CH0_CA7: now also U_A2.B28; no longer U_A2.C14
- net A2_CH0_CA8: now also U_A2.C1; no longer U_A2.C15
- net A2_CH0_CA9: now also U_A2.C2; no longer U_A2.C16
- net A2_CH0_CK0_N: now also U_A2.C10; no longer U_A2.D8
- net A2_CH0_CK0_P: now also U_A2.C9; no longer U_A2.D7
- net A2_CH0_CK1_N: now also U_A2.C12; no longer U_A2.D10
- net A2_CH0_CK1_P: now also U_A2.C11; no longer U_A2.D9
- net A2_CH0_CS0: now also U_A2.C7; no longer U_A2.D5
- net A2_CH0_CS1: now also U_A2.C8; no longer U_A2.D6
- net A2_CH0_DMI0: now also U_A2.A11; no longer U_A2.C3
- net A2_CH0_DMI1: now also U_A2.A23; no longer U_A2.C4
- net A2_CH0_DMI2: now also U_A2.B7; no longer U_A2.C5
- net A2_CH0_DMI3: now also U_A2.B19; no longer U_A2.C6
- net A2_CH0_DQ10: now also U_A2.A15; no longer U_A2.A11
- net A2_CH0_DQ11: now also U_A2.A16; no longer U_A2.A12
- net A2_CH0_DQ12: now also U_A2.A17; no longer U_A2.A13
- net A2_CH0_DQ13: now also U_A2.A18; no longer U_A2.A14
- net A2_CH0_DQ14: now also U_A2.A19; no longer U_A2.A15
- net A2_CH0_DQ15: now also U_A2.A20; no longer U_A2.A16
- net A2_CH0_DQ16: now also U_A2.A25; no longer U_A2.A17
- net A2_CH0_DQ17: now also U_A2.A26; no longer U_A2.A18
- net A2_CH0_DQ18: now also U_A2.A27; no longer U_A2.A19
- net A2_CH0_DQ19: now also U_A2.A28; no longer U_A2.A20
- net A2_CH0_DQ24: now also U_A2.B9; no longer U_A2.B5
- net A2_CH0_DQ25: now also U_A2.B10; no longer U_A2.B6
- net A2_CH0_DQ26: now also U_A2.B11; no longer U_A2.B7
- net A2_CH0_DQ27: now also U_A2.B12; no longer U_A2.B8
- net A2_CH0_DQ28: now also U_A2.B13; no longer U_A2.B9
- net A2_CH0_DQ29: now also U_A2.B14; no longer U_A2.B10
- net A2_CH0_DQ30: now also U_A2.B15; no longer U_A2.B11
- net A2_CH0_DQ31: now also U_A2.B16; no longer U_A2.B12
- net A2_CH0_DQ8: now also U_A2.A13; no longer U_A2.A9
- net A2_CH0_DQ9: now also U_A2.A14; no longer U_A2.A10
- net A2_CH0_DQS0_N: now also U_A2.A10; no longer U_A2.B14
- net A2_CH0_DQS0_P: now also U_A2.A9; no longer U_A2.B13
- net A2_CH0_DQS1_N: now also U_A2.A22; no longer U_A2.B16
- net A2_CH0_DQS1_P: now also U_A2.A21; no longer U_A2.B15
- net A2_CH0_DQS2_N: now also U_A2.B6; no longer U_A2.B18
- net A2_CH0_DQS2_P: now also U_A2.B5; no longer U_A2.B17
- net A2_CH0_DQS3_N: now also U_A2.B18; no longer U_A2.B20
- net A2_CH0_DQS3_P: now also U_A2.B17; no longer U_A2.B19
- net A2_CH0_RESET: now also U_A2.C13; no longer U_A2.D11
- net A2_CH1_CA0: now also U_A2.E7; no longer U_A2.G8
- net A2_CH1_CA1: now also U_A2.E8; no longer U_A2.G9
- net A2_CH1_CA10: now also U_A2.E17; no longer U_A2.G18
- net A2_CH1_CA11: now also U_A2.E18; no longer U_A2.H3
- net A2_CH1_CA12: now also U_A2.E19; no longer U_A2.H4
- net A2_CH1_CA13: now also U_A2.E20; no longer U_A2.H5
- net A2_CH1_CA2: now also U_A2.E9; no longer U_A2.G10
- net A2_CH1_CA3: now also U_A2.E10; no longer U_A2.G11
- net A2_CH1_CA4: now also U_A2.E11; no longer U_A2.G12
- net A2_CH1_CA5: now also U_A2.E12; no longer U_A2.G13
- net A2_CH1_CA6: now also U_A2.E13; no longer U_A2.G14
- net A2_CH1_CA7: now also U_A2.E14; no longer U_A2.G15
- net A2_CH1_CA8: now also U_A2.E15; no longer U_A2.G16
- net A2_CH1_CA9: now also U_A2.E16; no longer U_A2.G17
- net A2_CH1_CK0_N: now also U_A2.E24; no longer U_A2.H9
- net A2_CH1_CK0_P: now also U_A2.E23; no longer U_A2.H8
- net A2_CH1_CK1_N: now also U_A2.E26; no longer U_A2.H11
- net A2_CH1_CK1_P: now also U_A2.E25; no longer U_A2.H10
- net A2_CH1_CS0: now also U_A2.E21; no longer U_A2.H6
- net A2_CH1_CS1: now also U_A2.E22; no longer U_A2.H7
- net A2_CH1_DMI0: now also U_A2.C25; no longer U_A2.G4
- net A2_CH1_DMI1: now also U_A2.D9; no longer U_A2.G5
- net A2_CH1_DMI2: now also U_A2.D21; no longer U_A2.G6
- net A2_CH1_DMI3: now also U_A2.E5; no longer U_A2.G7
- net A2_CH1_DQ0: now also U_A2.C15; no longer U_A2.D12
- net A2_CH1_DQ1: now also U_A2.C16; no longer U_A2.D13
- net A2_CH1_DQ10: now also U_A2.D1; no longer U_A2.E6
- net A2_CH1_DQ11: now also U_A2.D2; no longer U_A2.E7
- net A2_CH1_DQ12: now also U_A2.D3; no longer U_A2.E8
- net A2_CH1_DQ13: now also U_A2.D4; no longer U_A2.E9
- net A2_CH1_DQ14: now also U_A2.D5; no longer U_A2.E10
- net A2_CH1_DQ15: now also U_A2.D6; no longer U_A2.E11
- net A2_CH1_DQ16: now also U_A2.D11; no longer U_A2.E12
- net A2_CH1_DQ17: now also U_A2.D12; no longer U_A2.E13
- net A2_CH1_DQ18: now also U_A2.D13; no longer U_A2.E14
- net A2_CH1_DQ19: now also U_A2.D14; no longer U_A2.E15
- net A2_CH1_DQ2: now also U_A2.C17; no longer U_A2.D14
- net A2_CH1_DQ20: now also U_A2.D15; no longer U_A2.E16
- net A2_CH1_DQ21: now also U_A2.D16; no longer U_A2.E17
- net A2_CH1_DQ22: now also U_A2.D17; no longer U_A2.E18
- net A2_CH1_DQ23: now also U_A2.D18; no longer U_A2.F3
- net A2_CH1_DQ24: now also U_A2.D23; no longer U_A2.F4
- net A2_CH1_DQ25: now also U_A2.D24; no longer U_A2.F5
- net A2_CH1_DQ26: now also U_A2.D25; no longer U_A2.F6
- net A2_CH1_DQ27: now also U_A2.D26; no longer U_A2.F7
- net A2_CH1_DQ28: now also U_A2.D27; no longer U_A2.F8
- net A2_CH1_DQ29: now also U_A2.D28; no longer U_A2.F9
- net A2_CH1_DQ3: now also U_A2.C18; no longer U_A2.D15
- net A2_CH1_DQ30: now also U_A2.E1; no longer U_A2.F10
- net A2_CH1_DQ31: now also U_A2.E2; no longer U_A2.F11
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
Commit message: Retarget the board to a host-attached 1U chassis
The energy model put the board at 0.5 to 1.6 kW of input across the
throughput range, which is a rack supply, not a PCIe slot.  The board is
now one 420 x 360 mm board in a 1U: two CRPS modules in a 1+1 pair, a
BMC with its own Ethernet, six front fans, and a SlimSAS 8i cable to the
host's PCIe.  With the room to carry it, the ASIC package is rated at the
50K tokens/s target (177 A core), which selects the 1225-ball 29 mm
package.

hw/board.yaml: 1U form factor, host cable, CRPS input, BMC, PSU, fan and
RJ45 parts and classes, 50K package rating.

hw/kicad_gen.py: form factors (1U default, card kept) that map the ring
frame onto the physical board with keep-outs (PSU bay, rear I/O, fans),
physical parts for the chassis connectors and BMC, a fit check, layout
derived from the package body, the FPGA beside H1 taking the ring on its
west edge (closing hop 74 mm instead of 95 mm with the 29 mm package),
PCIe pins on the FPGA's south edge, regulators spaced for the larger
package.  Every hop is within the 80 mm limit and pcbnew DRC reports only
the unrouted nets.

Tests cover both form factors, the keep-outs and the package rating;
docs describe the 1U, the rating decision and the floorplan findings.

Co-Authored-By: Claude Fable 5.1 <noreply@anthropic.com>
Claude-Session: https://claude.ai/code/session_01VmmvkZe8Ctg3RAykNGsQBn
Parts:
- U_A0, U_A1, U_A2, U_A3, U_A4, U_A5, U_A6, U_A7, U_H0, U_H1: footprint appliance:FCBGA784_28x28_P0.8 -> appliance:FCBGA1225_35x35_P0.8
Connections:
- net A0_CH0_CA0: now also U_A0.B14; no longer U_A0.B21
- net A0_CH0_CA1: now also U_A0.B15; no longer U_A0.B22
- net A0_CH0_CA10: now also U_A0.B24; no longer U_A0.C3
- net A0_CH0_CA11: now also U_A0.B25; no longer U_A0.C4
- net A0_CH0_CA12: now also U_A0.B26; no longer U_A0.C5
- net A0_CH0_CA13: now also U_A0.B27; no longer U_A0.C6
- net A0_CH0_CA2: now also U_A0.B16; no longer U_A0.B23
- net A0_CH0_CA3: now also U_A0.B17; no longer U_A0.B24
- net A0_CH0_CA4: now also U_A0.B18; no longer U_A0.B25
- net A0_CH0_CA5: now also U_A0.B19; no longer U_A0.B26
- net A0_CH0_CA6: now also U_A0.B20; no longer U_A0.B27
- net A0_CH0_CA7: now also U_A0.B21; no longer U_A0.B28
- net A0_CH0_CA8: now also U_A0.B22; no longer U_A0.C1
- net A0_CH0_CA9: now also U_A0.B23; no longer U_A0.C2
- net A0_CH0_CK0_N: now also U_A0.B31; no longer U_A0.C10
- net A0_CH0_CK0_P: now also U_A0.B30; no longer U_A0.C9
- net A0_CH0_CK1_N: now also U_A0.B33; no longer U_A0.C12
- net A0_CH0_CK1_P: now also U_A0.B32; no longer U_A0.C11
- net A0_CH0_CS0: now also U_A0.B28; no longer U_A0.C7
- net A0_CH0_CS1: now also U_A0.B29; no longer U_A0.C8
- net A0_CH0_DMI2: now also U_A0.A35; no longer U_A0.B7
- net A0_CH0_DMI3: now also U_A0.B12; no longer U_A0.B19
- net A0_CH0_DQ20: now also U_A0.A29; no longer U_A0.B1
- net A0_CH0_DQ21: now also U_A0.A30; no longer U_A0.B2
- net A0_CH0_DQ22: now also U_A0.A31; no longer U_A0.B3
- net A0_CH0_DQ23: now also U_A0.A32; no longer U_A0.B4
- net A0_CH0_DQ24: now also U_A0.B2; no longer U_A0.B9
- net A0_CH0_DQ25: now also U_A0.B3; no longer U_A0.B10
- net A0_CH0_DQ26: now also U_A0.B4; no longer U_A0.B11
- net A0_CH0_DQ27: now also U_A0.B5; no longer U_A0.B12
- net A0_CH0_DQ28: now also U_A0.B6; no longer U_A0.B13
- net A0_CH0_DQ29: now also U_A0.B7; no longer U_A0.B14
- net A0_CH0_DQ30: now also U_A0.B8; no longer U_A0.B15
- net A0_CH0_DQ31: now also U_A0.B9; no longer U_A0.B16
- net A0_CH0_DQS2_N: now also U_A0.A34; no longer U_A0.B6
- net A0_CH0_DQS2_P: now also U_A0.A33; no longer U_A0.B5
- net A0_CH0_DQS3_N: now also U_A0.B11; no longer U_A0.B18
- net A0_CH0_DQS3_P: now also U_A0.B10; no longer U_A0.B17
- net A0_CH0_RESET: now also U_A0.B34; no longer U_A0.C13
- net A0_CH1_CA0: now also U_A0.D14; no longer U_A0.E7
- net A0_CH1_CA1: now also U_A0.D15; no longer U_A0.E8
- net A0_CH1_CA10: now also U_A0.D24; no longer U_A0.E17
- net A0_CH1_CA11: now also U_A0.D25; no longer U_A0.E18
- net A0_CH1_CA12: now also U_A0.D26; no longer U_A0.E19
- net A0_CH1_CA13: now also U_A0.D27; no longer U_A0.E20
- net A0_CH1_CA2: now also U_A0.D16; no longer U_A0.E9
- net A0_CH1_CA3: now also U_A0.D17; no longer U_A0.E10
- net A0_CH1_CA4: now also U_A0.D18; no longer U_A0.E11
- net A0_CH1_CA5: now also U_A0.D19; no longer U_A0.E12
- net A0_CH1_CA6: now also U_A0.D20; no longer U_A0.E13
- net A0_CH1_CA7: now also U_A0.D21; no longer U_A0.E14
- net A0_CH1_CA8: now also U_A0.D22; no longer U_A0.E15
- net A0_CH1_CA9: now also U_A0.D23; no longer U_A0.E16
- net A0_CH1_CK0_N: now also U_A0.D31; no longer U_A0.E24
- net A0_CH1_CK0_P: now also U_A0.D30; no longer U_A0.E23
- net A0_CH1_CK1_N: now also U_A0.D33; no longer U_A0.E26
- net A0_CH1_CK1_P: now also U_A0.D32; no longer U_A0.E25
- net A0_CH1_CS0: now also U_A0.D28; no longer U_A0.E21
- net A0_CH1_CS1: now also U_A0.D29; no longer U_A0.E22
- net A0_CH1_DMI0: now also U_A0.C11; no longer U_A0.C25
- net A0_CH1_DMI1: now also U_A0.C23; no longer U_A0.D9
- net A0_CH1_DMI2: now also U_A0.C35; no longer U_A0.D21
- net A0_CH1_DMI3: now also U_A0.D12; no longer U_A0.E5
- net A0_CH1_DQ0: now also U_A0.C1; no longer U_A0.C15
- net A0_CH1_DQ1: now also U_A0.C2; no longer U_A0.C16
- net A0_CH1_DQ10: now also U_A0.C15; no longer U_A0.D1
- net A0_CH1_DQ11: now also U_A0.C16; no longer U_A0.D2
- net A0_CH1_DQ12: now also U_A0.C17; no longer U_A0.D3
- net A0_CH1_DQ13: now also U_A0.C18; no longer U_A0.D4
- net A0_CH1_DQ14: now also U_A0.C19; no longer U_A0.D5
- net A0_CH1_DQ15: now also U_A0.C20; no longer U_A0.D6
- net A0_CH1_DQ16: now also U_A0.C25; no longer U_A0.D11
- net A0_CH1_DQ17: now also U_A0.C26; no longer U_A0.D12
- net A0_CH1_DQ18: now also U_A0.C27; no longer U_A0.D13
- net A0_CH1_DQ19: now also U_A0.C28; no longer U_A0.D14
- net A0_CH1_DQ2: now also U_A0.C3; no longer U_A0.C17
- net A0_CH1_DQ20: now also U_A0.C29; no longer U_A0.D15
- net A0_CH1_DQ21: now also U_A0.C30; no longer U_A0.D16
- net A0_CH1_DQ22: now also U_A0.C31; no longer U_A0.D17
- net A0_CH1_DQ23: now also U_A0.C32; no longer U_A0.D18
- net A0_CH1_DQ24: now also U_A0.D2; no longer U_A0.D23
- net A0_CH1_DQ25: now also U_A0.D3; no longer U_A0.D24
- net A0_CH1_DQ26: now also U_A0.D4; no longer U_A0.D25
- net A0_CH1_DQ27: now also U_A0.D5; no longer U_A0.D26
- net A0_CH1_DQ28: now also U_A0.D6; no longer U_A0.D27
- net A0_CH1_DQ29: now also U_A0.D7; no longer U_A0.D28
- net A0_CH1_DQ3: now also U_A0.C4; no longer U_A0.C18
- net A0_CH1_DQ30: now also U_A0.D8; no longer U_A0.E1
- net A0_CH1_DQ31: now also U_A0.D9; no longer U_A0.E2
- net A0_CH1_DQ4: now also U_A0.C5; no longer U_A0.C19
- net A0_CH1_DQ5: now also U_A0.C6; no longer U_A0.C20
- net A0_CH1_DQ6: now also U_A0.C7; no longer U_A0.C21
- net A0_CH1_DQ7: now also U_A0.C8; no longer U_A0.C22
- net A0_CH1_DQ8: now also U_A0.C13; no longer U_A0.C27
- net A0_CH1_DQ9: now also U_A0.C14; no longer U_A0.C28
- net A0_CH1_DQS0_N: now also U_A0.C10; no longer U_A0.C24
- net A0_CH1_DQS0_P: now also U_A0.C9; no longer U_A0.C23
- net A0_CH1_DQS1_N: now also U_A0.C22; no longer U_A0.D8
- net A0_CH1_DQS1_P: now also U_A0.C21; no longer U_A0.D7
- net A0_CH1_DQS2_N: now also U_A0.C34; no longer U_A0.D20
- net A0_CH1_DQS2_P: now also U_A0.C33; no longer U_A0.D19
- net A0_CH1_DQS3_N: now also U_A0.D11; no longer U_A0.E4
- net A0_CH1_DQS3_P: now also U_A0.D10; no longer U_A0.E3
- net A0_CH1_RESET: now also U_A0.D34; no longer U_A0.E27
- net A1_CH0_CA0: now also U_A1.B14; no longer U_A1.B21
- net A1_CH0_CA1: now also U_A1.B15; no longer U_A1.B22
- net A1_CH0_CA10: now also U_A1.B24; no longer U_A1.C3
- net A1_CH0_CA11: now also U_A1.B25; no longer U_A1.C4
- net A1_CH0_CA12: now also U_A1.B26; no longer U_A1.C5
- net A1_CH0_CA13: now also U_A1.B27; no longer U_A1.C6
- net A1_CH0_CA2: now also U_A1.B16; no longer U_A1.B23
- net A1_CH0_CA3: now also U_A1.B17; no longer U_A1.B24
- net A1_CH0_CA4: now also U_A1.B18; no longer U_A1.B25
- net A1_CH0_CA5: now also U_A1.B19; no longer U_A1.B26
- net A1_CH0_CA6: now also U_A1.B20; no longer U_A1.B27
- net A1_CH0_CA7: now also U_A1.B21; no longer U_A1.B28
- net A1_CH0_CA8: now also U_A1.B22; no longer U_A1.C1
- net A1_CH0_CA9: now also U_A1.B23; no longer U_A1.C2
- net A1_CH0_CK0_N: now also U_A1.B31; no longer U_A1.C10
- net A1_CH0_CK0_P: now also U_A1.B30; no longer U_A1.C9
- net A1_CH0_CK1_N: now also U_A1.B33; no longer U_A1.C12
- net A1_CH0_CK1_P: now also U_A1.B32; no longer U_A1.C11
- net A1_CH0_CS0: now also U_A1.B28; no longer U_A1.C7
- net A1_CH0_CS1: now also U_A1.B29; no longer U_A1.C8
- net A1_CH0_DMI2: now also U_A1.A35; no longer U_A1.B7
- net A1_CH0_DMI3: now also U_A1.B12; no longer U_A1.B19
- net A1_CH0_DQ20: now also U_A1.A29; no longer U_A1.B1
- net A1_CH0_DQ21: now also U_A1.A30; no longer U_A1.B2
- net A1_CH0_DQ22: now also U_A1.A31; no longer U_A1.B3
- net A1_CH0_DQ23: now also U_A1.A32; no longer U_A1.B4
- net A1_CH0_DQ24: now also U_A1.B2; no longer U_A1.B9
- net A1_CH0_DQ25: now also U_A1.B3; no longer U_A1.B10
- net A1_CH0_DQ26: now also U_A1.B4; no longer U_A1.B11
- net A1_CH0_DQ27: now also U_A1.B5; no longer U_A1.B12
- net A1_CH0_DQ28: now also U_A1.B6; no longer U_A1.B13
- net A1_CH0_DQ29: now also U_A1.B7; no longer U_A1.B14
- net A1_CH0_DQ30: now also U_A1.B8; no longer U_A1.B15
- net A1_CH0_DQ31: now also U_A1.B9; no longer U_A1.B16
- net A1_CH0_DQS2_N: now also U_A1.A34; no longer U_A1.B6
- net A1_CH0_DQS2_P: now also U_A1.A33; no longer U_A1.B5
- net A1_CH0_DQS3_N: now also U_A1.B11; no longer U_A1.B18
- net A1_CH0_DQS3_P: now also U_A1.B10; no longer U_A1.B17
- net A1_CH0_RESET: now also U_A1.B34; no longer U_A1.C13
- net A1_CH1_CA0: now also U_A1.D14; no longer U_A1.E7
- net A1_CH1_CA1: now also U_A1.D15; no longer U_A1.E8
- net A1_CH1_CA10: now also U_A1.D24; no longer U_A1.E17
- net A1_CH1_CA11: now also U_A1.D25; no longer U_A1.E18
- net A1_CH1_CA12: now also U_A1.D26; no longer U_A1.E19
- net A1_CH1_CA13: now also U_A1.D27; no longer U_A1.E20
- net A1_CH1_CA2: now also U_A1.D16; no longer U_A1.E9
- net A1_CH1_CA3: now also U_A1.D17; no longer U_A1.E10
- net A1_CH1_CA4: now also U_A1.D18; no longer U_A1.E11
- net A1_CH1_CA5: now also U_A1.D19; no longer U_A1.E12
- net A1_CH1_CA6: now also U_A1.D20; no longer U_A1.E13
- net A1_CH1_CA7: now also U_A1.D21; no longer U_A1.E14
- net A1_CH1_CA8: now also U_A1.D22; no longer U_A1.E15
- net A1_CH1_CA9: now also U_A1.D23; no longer U_A1.E16
- net A1_CH1_CK0_N: now also U_A1.D31; no longer U_A1.E24
- net A1_CH1_CK0_P: now also U_A1.D30; no longer U_A1.E23
- net A1_CH1_CK1_N: now also U_A1.D33; no longer U_A1.E26
- net A1_CH1_CK1_P: now also U_A1.D32; no longer U_A1.E25
- net A1_CH1_CS0: now also U_A1.D28; no longer U_A1.E21
- net A1_CH1_CS1: now also U_A1.D29; no longer U_A1.E22
- net A1_CH1_DMI0: now also U_A1.C11; no longer U_A1.C25
- net A1_CH1_DMI1: now also U_A1.C23; no longer U_A1.D9
- net A1_CH1_DMI2: now also U_A1.C35; no longer U_A1.D21
- net A1_CH1_DMI3: now also U_A1.D12; no longer U_A1.E5
- net A1_CH1_DQ0: now also U_A1.C1; no longer U_A1.C15
- net A1_CH1_DQ1: now also U_A1.C2; no longer U_A1.C16
- net A1_CH1_DQ10: now also U_A1.C15; no longer U_A1.D1
- net A1_CH1_DQ11: now also U_A1.C16; no longer U_A1.D2
- net A1_CH1_DQ12: now also U_A1.C17; no longer U_A1.D3
- net A1_CH1_DQ13: now also U_A1.C18; no longer U_A1.D4
- net A1_CH1_DQ14: now also U_A1.C19; no longer U_A1.D5
- net A1_CH1_DQ15: now also U_A1.C20; no longer U_A1.D6
- net A1_CH1_DQ16: now also U_A1.C25; no longer U_A1.D11
- net A1_CH1_DQ17: now also U_A1.C26; no longer U_A1.D12
- net A1_CH1_DQ18: now also U_A1.C27; no longer U_A1.D13
- net A1_CH1_DQ19: now also U_A1.C28; no longer U_A1.D14
- net A1_CH1_DQ2: now also U_A1.C3; no longer U_A1.C17
- net A1_CH1_DQ20: now also U_A1.C29; no longer U_A1.D15
- net A1_CH1_DQ21: now also U_A1.C30; no longer U_A1.D16
- net A1_CH1_DQ22: now also U_A1.C31; no longer U_A1.D17
- net A1_CH1_DQ23: now also U_A1.C32; no longer U_A1.D18
- net A1_CH1_DQ24: now also U_A1.D2; no longer U_A1.D23
- net A1_CH1_DQ25: now also U_A1.D3; no longer U_A1.D24
- net A1_CH1_DQ26: now also U_A1.D4; no longer U_A1.D25
- net A1_CH1_DQ27: now also U_A1.D5; no longer U_A1.D26
- net A1_CH1_DQ28: now also U_A1.D6; no longer U_A1.D27
- net A1_CH1_DQ29: now also U_A1.D7; no longer U_A1.D28
- net A1_CH1_DQ3: now also U_A1.C4; no longer U_A1.C18
- net A1_CH1_DQ30: now also U_A1.D8; no longer U_A1.E1
- net A1_CH1_DQ31: now also U_A1.D9; no longer U_A1.E2
- net A1_CH1_DQ4: now also U_A1.C5; no longer U_A1.C19
- net A1_CH1_DQ5: now also U_A1.C6; no longer U_A1.C20
- net A1_CH1_DQ6: now also U_A1.C7; no longer U_A1.C21
- net A1_CH1_DQ7: now also U_A1.C8; no longer U_A1.C22
- net A1_CH1_DQ8: now also U_A1.C13; no longer U_A1.C27
- net A1_CH1_DQ9: now also U_A1.C14; no longer U_A1.C28
- net A1_CH1_DQS0_N: now also U_A1.C10; no longer U_A1.C24
- net A1_CH1_DQS0_P: now also U_A1.C9; no longer U_A1.C23
- net A1_CH1_DQS1_N: now also U_A1.C22; no longer U_A1.D8
- net A1_CH1_DQS1_P: now also U_A1.C21; no longer U_A1.D7
- net A1_CH1_DQS2_N: now also U_A1.C34; no longer U_A1.D20
- net A1_CH1_DQS2_P: now also U_A1.C33; no longer U_A1.D19
- net A1_CH1_DQS3_N: now also U_A1.D11; no longer U_A1.E4
- net A1_CH1_DQS3_P: now also U_A1.D10; no longer U_A1.E3
- net A1_CH1_RESET: now also U_A1.D34; no longer U_A1.E27
- net A2_CH0_CA0: now also U_A2.B14; no longer U_A2.B21
- net A2_CH0_CA1: now also U_A2.B15; no longer U_A2.B22
- net A2_CH0_CA10: now also U_A2.B24; no longer U_A2.C3
- net A2_CH0_CA11: now also U_A2.B25; no longer U_A2.C4
- net A2_CH0_CA12: now also U_A2.B26; no longer U_A2.C5
- net A2_CH0_CA13: now also U_A2.B27; no longer U_A2.C6
- net A2_CH0_CA2: now also U_A2.B16; no longer U_A2.B23
- net A2_CH0_CA3: now also U_A2.B17; no longer U_A2.B24
- net A2_CH0_CA4: now also U_A2.B18; no longer U_A2.B25
- net A2_CH0_CA5: now also U_A2.B19; no longer U_A2.B26
- net A2_CH0_CA6: now also U_A2.B20; no longer U_A2.B27
- net A2_CH0_CA7: now also U_A2.B21; no longer U_A2.B28
- net A2_CH0_CA8: now also U_A2.B22; no longer U_A2.C1
- net A2_CH0_CA9: now also U_A2.B23; no longer U_A2.C2
- net A2_CH0_CK0_N: now also U_A2.B31; no longer U_A2.C10
- net A2_CH0_CK0_P: now also U_A2.B30; no longer U_A2.C9
- net A2_CH0_CK1_N: now also U_A2.B33; no longer U_A2.C12
- net A2_CH0_CK1_P: now also U_A2.B32; no longer U_A2.C11
- net A2_CH0_CS0: now also U_A2.B28; no longer U_A2.C7
- net A2_CH0_CS1: now also U_A2.B29; no longer U_A2.C8
- net A2_CH0_DMI2: now also U_A2.A35; no longer U_A2.B7
- net A2_CH0_DMI3: now also U_A2.B12; no longer U_A2.B19
- net A2_CH0_DQ20: now also U_A2.A29; no longer U_A2.B1
- net A2_CH0_DQ21: now also U_A2.A30; no longer U_A2.B2
- net A2_CH0_DQ22: now also U_A2.A31; no longer U_A2.B3
- net A2_CH0_DQ23: now also U_A2.A32; no longer U_A2.B4
- net A2_CH0_DQ24: now also U_A2.B2; no longer U_A2.B9
- net A2_CH0_DQ25: now also U_A2.B3; no longer U_A2.B10
- net A2_CH0_DQ26: now also U_A2.B4; no longer U_A2.B11
- net A2_CH0_DQ27: now also U_A2.B5; no longer U_A2.B12
- net A2_CH0_DQ28: now also U_A2.B6; no longer U_A2.B13
- net A2_CH0_DQ29: now also U_A2.B7; no longer U_A2.B14
- net A2_CH0_DQ30: now also U_A2.B8; no longer U_A2.B15
- net A2_CH0_DQ31: now also U_A2.B9; no longer U_A2.B16
- net A2_CH0_DQS2_N: now also U_A2.A34; no longer U_A2.B6
- net A2_CH0_DQS2_P: now also U_A2.A33; no longer U_A2.B5
- net A2_CH0_DQS3_N: now also U_A2.B11; no longer U_A2.B18
- net A2_CH0_DQS3_P: now also U_A2.B10; no longer U_A2.B17
- net A2_CH0_RESET: now also U_A2.B34; no longer U_A2.C13
- net A2_CH1_CA0: now also U_A2.D14; no longer U_A2.E7
- net A2_CH1_CA1: now also U_A2.D15; no longer U_A2.E8
- net A2_CH1_CA10: now also U_A2.D24; no longer U_A2.E17
- net A2_CH1_CA11: now also U_A2.D25; no longer U_A2.E18
- net A2_CH1_CA12: now also U_A2.D26; no longer U_A2.E19
- net A2_CH1_CA13: now also U_A2.D27; no longer U_A2.E20
- net A2_CH1_CA2: now also U_A2.D16; no longer U_A2.E9
- net A2_CH1_CA3: now also U_A2.D17; no longer U_A2.E10
- net A2_CH1_CA4: now also U_A2.D18; no longer U_A2.E11
- net A2_CH1_CA5: now also U_A2.D19; no longer U_A2.E12
- net A2_CH1_CA6: now also U_A2.D20; no longer U_A2.E13
- net A2_CH1_CA7: now also U_A2.D21; no longer U_A2.E14
- net A2_CH1_CA8: now also U_A2.D22; no longer U_A2.E15
- net A2_CH1_CA9: now also U_A2.D23; no longer U_A2.E16
- net A2_CH1_CK0_N: now also U_A2.D31; no longer U_A2.E24
- net A2_CH1_CK0_P: now also U_A2.D30; no longer U_A2.E23
- net A2_CH1_CK1_N: now also U_A2.D33; no longer U_A2.E26
- net A2_CH1_CK1_P: now also U_A2.D32; no longer U_A2.E25
- net A2_CH1_CS0: now also U_A2.D28; no longer U_A2.E21
- net A2_CH1_CS1: now also U_A2.D29; no longer U_A2.E22
- net A2_CH1_DMI0: now also U_A2.C11; no longer U_A2.C25
- net A2_CH1_DMI1: now also U_A2.C23; no longer U_A2.D9
- net A2_CH1_DMI2: now also U_A2.C35; no longer U_A2.D21
- net A2_CH1_DMI3: now also U_A2.D12; no longer U_A2.E5
- net A2_CH1_DQ0: now also U_A2.C1; no longer U_A2.C15
- net A2_CH1_DQ1: now also U_A2.C2; no longer U_A2.C16
- net A2_CH1_DQ10: now also U_A2.C15; no longer U_A2.D1
- net A2_CH1_DQ11: now also U_A2.C16; no longer U_A2.D2
- net A2_CH1_DQ12: now also U_A2.C17; no longer U_A2.D3
- net A2_CH1_DQ13: now also U_A2.C18; no longer U_A2.D4
- net A2_CH1_DQ14: now also U_A2.C19; no longer U_A2.D5
- net A2_CH1_DQ15: now also U_A2.C20; no longer U_A2.D6
- net A2_CH1_DQ16: now also U_A2.C25; no longer U_A2.D11
- net A2_CH1_DQ17: now also U_A2.C26; no longer U_A2.D12
- net A2_CH1_DQ18: now also U_A2.C27; no longer U_A2.D13
- net A2_CH1_DQ19: now also U_A2.C28; no longer U_A2.D14
- net A2_CH1_DQ2: now also U_A2.C3; no longer U_A2.C17
- net A2_CH1_DQ20: now also U_A2.C29; no longer U_A2.D15
- net A2_CH1_DQ21: now also U_A2.C30; no longer U_A2.D16
- net A2_CH1_DQ22: now also U_A2.C31; no longer U_A2.D17
- net A2_CH1_DQ23: now also U_A2.C32; no longer U_A2.D18
- net A2_CH1_DQ24: now also U_A2.D2; no longer U_A2.D23
- net A2_CH1_DQ25: now also U_A2.D3; no longer U_A2.D24
- net A2_CH1_DQ26: now also U_A2.D4; no longer U_A2.D25
- net A2_CH1_DQ27: now also U_A2.D5; no longer U_A2.D26
- net A2_CH1_DQ28: now also U_A2.D6; no longer U_A2.D27
- net A2_CH1_DQ29: now also U_A2.D7; no longer U_A2.D28
- net A2_CH1_DQ3: now also U_A2.C4; no longer U_A2.C18
- net A2_CH1_DQ30: now also U_A2.D8; no longer U_A2.E1
- net A2_CH1_DQ31: now also U_A2.D9; no longer U_A2.E2
- net A2_CH1_DQ4: now also U_A2.C5; no longer U_A2.C19
- net A2_CH1_DQ5: now also U_A2.C6; no longer U_A2.C20
- net A2_CH1_DQ6: now also U_A2.C7; no longer U_A2.C21
- net A2_CH1_DQ7: now also U_A2.C8; no longer U_A2.C22
- net A2_CH1_DQ8: now also U_A2.C13; no longer U_A2.C27
- net A2_CH1_DQ9: now also U_A2.C14; no longer U_A2.C28
- net A2_CH1_DQS0_N: now also U_A2.C10; no longer U_A2.C24
- net A2_CH1_DQS0_P: now also U_A2.C9; no longer U_A2.C23
- net A2_CH1_DQS1_N: now also U_A2.C22; no longer U_A2.D8
- net A2_CH1_DQS1_P: now also U_A2.C21; no longer U_A2.D7
- net A2_CH1_DQS2_N: now also U_A2.C34; no longer U_A2.D20
- net A2_CH1_DQS2_P: now also U_A2.C33; no longer U_A2.D19
- net A2_CH1_DQS3_N: now also U_A2.D11; no longer U_A2.E4
- net A2_CH1_DQS3_P: now also U_A2.D10; no longer U_A2.E3
- net A2_CH1_RESET: now also U_A2.D34; no longer U_A2.E27
- net A3_CH0_CA0: now also U_A3.B14; no longer U_A3.B21
- net A3_CH0_CA1: now also U_A3.B15; no longer U_A3.B22
- net A3_CH0_CA10: now also U_A3.B24; no longer U_A3.C3
- net A3_CH0_CA11: now also U_A3.B25; no longer U_A3.C4
- net A3_CH0_CA12: now also U_A3.B26; no longer U_A3.C5
- net A3_CH0_CA13: now also U_A3.B27; no longer U_A3.C6
- net A3_CH0_CA2: now also U_A3.B16; no longer U_A3.B23
- net A3_CH0_CA3: now also U_A3.B17; no longer U_A3.B24
- net A3_CH0_CA4: now also U_A3.B18; no longer U_A3.B25
- net A3_CH0_CA5: now also U_A3.B19; no longer U_A3.B26
- net A3_CH0_CA6: now also U_A3.B20; no longer U_A3.B27
- net A3_CH0_CA7: now also U_A3.B21; no longer U_A3.B28
- net A3_CH0_CA8: now also U_A3.B22; no longer U_A3.C1
- net A3_CH0_CA9: now also U_A3.B23; no longer U_A3.C2
- net A3_CH0_CK0_N: now also U_A3.B31; no longer U_A3.C10
- net A3_CH0_CK0_P: now also U_A3.B30; no longer U_A3.C9
- net A3_CH0_CK1_N: now also U_A3.B33; no longer U_A3.C12
- net A3_CH0_CK1_P: now also U_A3.B32; no longer U_A3.C11
- net A3_CH0_CS0: now also U_A3.B28; no longer U_A3.C7
- net A3_CH0_CS1: now also U_A3.B29; no longer U_A3.C8
- net A3_CH0_DMI2: now also U_A3.A35; no longer U_A3.B7
- net A3_CH0_DMI3: now also U_A3.B12; no longer U_A3.B19
- net A3_CH0_DQ20: now also U_A3.A29; no longer U_A3.B1
- net A3_CH0_DQ21: now also U_A3.A30; no longer U_A3.B2
- net A3_CH0_DQ22: now also U_A3.A31; no longer U_A3.B3
- net A3_CH0_DQ23: now also U_A3.A32; no longer U_A3.B4
- net A3_CH0_DQ24: now also U_A3.B2; no longer U_A3.B9
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