File: hw/kicad/fpga.kicad_sch (KiCad schematic)
At the start: 4 parts

Commit message: Retarget the board to a host-attached 1U chassis
The energy model put the board at 0.5 to 1.6 kW of input across the
throughput range, which is a rack supply, not a PCIe slot.  The board is
now one 420 x 360 mm board in a 1U: two CRPS modules in a 1+1 pair, a
BMC with its own Ethernet, six front fans, and a SlimSAS 8i cable to the
host's PCIe.  With the room to carry it, the ASIC package is rated at the
50K tokens/s target (177 A core), which selects the 1225-ball 29 mm
package.

hw/board.yaml: 1U form factor, host cable, CRPS input, BMC, PSU, fan and
RJ45 parts and classes, 50K package rating.

hw/kicad_gen.py: form factors (1U default, card kept) that map the ring
frame onto the physical board with keep-outs (PSU bay, rear I/O, fans),
physical parts for the chassis connectors and BMC, a fit check, layout
derived from the package body, the FPGA beside H1 taking the ring on its
west edge (closing hop 74 mm instead of 95 mm with the 29 mm package),
PCIe pins on the FPGA's south edge, regulators spaced for the larger
package.  Every hop is within the 80 mm limit and pcbnew DRC reports only
the unrouted nets.

Tests cover both form factors, the keep-outs and the package rating;
docs describe the 1U, the rating decision and the floorplan findings.

Co-Authored-By: Claude Fable 5.1 <noreply@anthropic.com>
Claude-Session: https://claude.ai/code/session_01VmmvkZe8Ctg3RAykNGsQBn
Parts:
- removed J_PCIE: PCIe x8 edge, appliance:PCIE_X8_EDGE, symbol appliance:PCIE_X8_EDGE
- added J_BMC_NET: BMC Ethernet, appliance:RJ45_MAGJACK, symbol appliance:RJ45_MAGJACK
- added J_HOST: SlimSAS 8i host cable, appliance:SLIMSAS_8I, symbol appliance:SLIMSAS_8I
- added U_BMC: BMC SoC, appliance:BGA_BMC_21x21, symbol appliance:BGA_BMC_21x21
Connections:
- net DDR4_ADDR_CMD16: now also U_FPGA.E3; no longer U_FPGA.E1
- net DDR4_ADDR_CMD17: now also U_FPGA.E4; no longer U_FPGA.E2
- net DDR4_ADDR_CMD18: now also U_FPGA.E5; no longer U_FPGA.E3
- net DDR4_ADDR_CMD19: now also U_FPGA.E6; no longer U_FPGA.E4
- net DDR4_ADDR_CMD20: now also U_FPGA.E7; no longer U_FPGA.E5
- net DDR4_ADDR_CMD21: now also U_FPGA.E8; no longer U_FPGA.E6
- net DDR4_ADDR_CMD22: now also U_FPGA.E9; no longer U_FPGA.E7
- net DDR4_ADDR_CMD23: now also U_FPGA.E10; no longer U_FPGA.E8
- net DDR4_ADDR_CMD24: now also U_FPGA.E11; no longer U_FPGA.E9
- net DDR4_ADDR_CMD25: now also U_FPGA.E12; no longer U_FPGA.E10
- net DDR4_ADDR_CMD26: now also U_FPGA.E13; no longer U_FPGA.E11
- net DDR4_ADDR_CMD27: now also U_FPGA.E14; no longer U_FPGA.E12
- net DDR4_CK_N: now also U_FPGA.E16; no longer U_FPGA.E14
- net DDR4_CK_P: now also U_FPGA.E15; no longer U_FPGA.E13
- net DDR4_CTRL0: now also U_FPGA.E17; no longer U_FPGA.E15
- net DDR4_CTRL1: now also U_FPGA.E18; no longer U_FPGA.E16
- net DDR4_CTRL2: now also U_FPGA.E19; no longer U_FPGA.E17
- net DDR4_CTRL3: now also U_FPGA.E20; no longer U_FPGA.E18
- net DDR4_CTRL4: now also U_FPGA.E21; no longer U_FPGA.E19
- net DDR4_CTRL5: now also U_FPGA.E22; no longer U_FPGA.E20
- net GND: now also U_FPGA.AE1, U_FPGA.AE17, U_FPGA.AF2, J_BMC_NET.10, J_BMC_NET.11, J_BMC_NET.12, J_HOST.37, J_HOST.38, J_HOST.39, J_HOST.40, J_HOST.41, J_HOST.42, J_HOST.43, J_HOST.44, J_HOST.45, J_HOST.46, J_HOST.47, J_HOST.48, J_HOST.49, J_HOST.50, J_HOST.51, J_HOST.52, J_HOST.53, J_HOST.54, U_BMC.28, U_BMC.29; no longer U_FPGA.AF20, U_FPGA.AF22, U_FPGA.AF24, U_FPGA.E21
- net LINK10_CLOCK: now also U_FPGA.AA1; no longer U_FPGA.AF17
- net LINK10_DATA0: now also U_FPGA.E1; no longer U_FPGA.AF1
- net LINK10_DATA1: now also U_FPGA.E2; no longer U_FPGA.AE1
- net LINK10_DATA10: now also U_FPGA.K1; no longer U_FPGA.AF6
- net LINK10_DATA11: now also U_FPGA.K2; no longer U_FPGA.AE6
- net LINK10_DATA12: now also U_FPGA.L1; no longer U_FPGA.AF7
- net LINK10_DATA13: now also U_FPGA.L2; no longer U_FPGA.AE7
- net LINK10_DATA14: now also U_FPGA.M1; no longer U_FPGA.AF8
- net LINK10_DATA15: now also U_FPGA.M2; no longer U_FPGA.AE8
- net LINK10_DATA16: now also U_FPGA.N1; no longer U_FPGA.AF9
- net LINK10_DATA17: now also U_FPGA.N2; no longer U_FPGA.AE9
- net LINK10_DATA18: now also U_FPGA.P1; no longer U_FPGA.AF10
- net LINK10_DATA19: now also U_FPGA.P2; no longer U_FPGA.AE10
- net LINK10_DATA2: now also U_FPGA.F1; no longer U_FPGA.AF2
- net LINK10_DATA20: now also U_FPGA.R1; no longer U_FPGA.AF11
- net LINK10_DATA21: now also U_FPGA.R2; no longer U_FPGA.AE11
- net LINK10_DATA22: now also U_FPGA.T1; no longer U_FPGA.AF12
- net LINK10_DATA23: now also U_FPGA.T2; no longer U_FPGA.AE12
- net LINK10_DATA24: now also U_FPGA.U1; no longer U_FPGA.AF13
- net LINK10_DATA25: now also U_FPGA.U2; no longer U_FPGA.AE13
- net LINK10_DATA26: now also U_FPGA.V1; no longer U_FPGA.AF14
- net LINK10_DATA27: now also U_FPGA.V2; no longer U_FPGA.AE14
- net LINK10_DATA28: now also U_FPGA.W1; no longer U_FPGA.AF15
- net LINK10_DATA29: now also U_FPGA.W2; no longer U_FPGA.AE15
- net LINK10_DATA3: now also U_FPGA.F2; no longer U_FPGA.AE2
- net LINK10_DATA30: now also U_FPGA.Y1; no longer U_FPGA.AF16
- net LINK10_DATA31: now also U_FPGA.Y2; no longer U_FPGA.AE16
- net LINK10_DATA4: now also U_FPGA.G1; no longer U_FPGA.AF3
- net LINK10_DATA5: now also U_FPGA.G2; no longer U_FPGA.AE3
- net LINK10_DATA6: now also U_FPGA.H1; no longer U_FPGA.AF4
- net LINK10_DATA7: now also U_FPGA.H2; no longer U_FPGA.AE4
- net LINK10_DATA8: now also U_FPGA.J1; no longer U_FPGA.AF5
- net LINK10_DATA9: now also U_FPGA.J2; no longer U_FPGA.AE5
- net LINK10_READY_BACK: now also U_FPGA.AB1; no longer U_FPGA.AF18
- net LINK10_SOF: now also U_FPGA.AB2; no longer U_FPGA.AE18
- net LINK10_VALID: now also U_FPGA.AA2; no longer U_FPGA.AE17
- net MGTAVCC: now also U_FPGA.AE24
- net PCIE_REFCLK_N: now also U_FPGA.AE14, J_HOST.34; no longer U_FPGA.AB2
- net PCIE_REFCLK_P: now also U_FPGA.AE13, J_HOST.33; no longer U_FPGA.AB1
- net PCIE_RX0_N: now also U_FPGA.AF20, J_HOST.18; no longer U_FPGA.P2
- net PCIE_RX0_P: now also U_FPGA.AF19, J_HOST.17; no longer U_FPGA.P1
- net PCIE_RX1_N: now also U_FPGA.AF22, J_HOST.20; no longer U_FPGA.R2
- net PCIE_RX1_P: now also U_FPGA.AF21, J_HOST.19; no longer U_FPGA.R1
- net PCIE_RX2_N: now also U_FPGA.AF24, J_HOST.22; no longer U_FPGA.T2
- net PCIE_RX2_P: now also U_FPGA.AF23, J_HOST.21; no longer U_FPGA.T1
- net PCIE_RX3_N: now also U_FPGA.AE4, J_HOST.24; no longer U_FPGA.U2
- net PCIE_RX3_P: now also U_FPGA.AE3, J_HOST.23; no longer U_FPGA.U1
- net PCIE_RX4_N: now also U_FPGA.AE6, J_HOST.26; no longer U_FPGA.V2
- net PCIE_RX4_P: now also U_FPGA.AE5, J_HOST.25; no longer U_FPGA.V1
- net PCIE_RX5_N: now also U_FPGA.AE8, J_HOST.28; no longer U_FPGA.W2
- net PCIE_RX5_P: now also U_FPGA.AE7, J_HOST.27; no longer U_FPGA.W1
- net PCIE_RX6_N: now also U_FPGA.AE10, J_HOST.30; no longer U_FPGA.Y2
- net PCIE_RX6_P: now also U_FPGA.AE9, J_HOST.29; no longer U_FPGA.Y1
- net PCIE_RX7_N: now also U_FPGA.AE12, J_HOST.32; no longer U_FPGA.AA2
- net PCIE_RX7_P: now also U_FPGA.AE11, J_HOST.31; no longer U_FPGA.AA1
- net PCIE_TX0_N: now also U_FPGA.AF4, J_HOST.2; no longer U_FPGA.F2
- net PCIE_TX0_P: now also U_FPGA.AF3, J_HOST.1; no longer U_FPGA.F1
- net PCIE_TX1_N: now also U_FPGA.AF6, J_HOST.4; no longer U_FPGA.G2
- net PCIE_TX1_P: now also U_FPGA.AF5, J_HOST.3; no longer U_FPGA.G1
- net PCIE_TX2_N: now also U_FPGA.AF8, J_HOST.6; no longer U_FPGA.H2
- net PCIE_TX2_P: now also U_FPGA.AF7, J_HOST.5; no longer U_FPGA.H1
- net PCIE_TX3_N: now also U_FPGA.AF10, J_HOST.8; no longer U_FPGA.J2
- net PCIE_TX3_P: now also U_FPGA.AF9, J_HOST.7; no longer U_FPGA.J1
- net PCIE_TX4_N: now also U_FPGA.AF12, J_HOST.10; no longer U_FPGA.K2
- net PCIE_TX4_P: now also U_FPGA.AF11, J_HOST.9; no longer U_FPGA.K1
- net PCIE_TX5_N: now also U_FPGA.AF14, J_HOST.12; no longer U_FPGA.L2
- net PCIE_TX5_P: now also U_FPGA.AF13, J_HOST.11; no longer U_FPGA.L1
- net PCIE_TX6_N: now also U_FPGA.AF16, J_HOST.14; no longer U_FPGA.M2
- net PCIE_TX6_P: now also U_FPGA.AF15, J_HOST.13; no longer U_FPGA.M1
- net PCIE_TX7_N: now also U_FPGA.AF18, J_HOST.16; no longer U_FPGA.N2
- net PCIE_TX7_P: now also U_FPGA.AF17, J_HOST.15; no longer U_FPGA.N1
- net UART_RX: now also U_BMC.22
- net UART_TX: now also U_BMC.21
- net VCCINT_0V85: now also U_FPGA.AE2, U_FPGA.AF1; no longer U_FPGA.AF19, U_FPGA.AF21, U_FPGA.AF23, U_FPGA.E22
- net VCCO_1V2: now also U_FPGA.AE18; no longer U_FPGA.AE24
- net VDD_3V3: now also J_BMC_NET.9, U_BMC.26, U_BMC.27
- new net BMC_ETH0_N: J_BMC_NET.2, U_BMC.2
- new net BMC_ETH0_P: J_BMC_NET.1, U_BMC.1
- new net BMC_ETH1_N: J_BMC_NET.4, U_BMC.4
- new net BMC_ETH1_P: J_BMC_NET.3, U_BMC.3
- new net BMC_ETH2_N: J_BMC_NET.6, U_BMC.6
- new net BMC_ETH2_P: J_BMC_NET.5, U_BMC.5
- new net BMC_ETH3_N: J_BMC_NET.8, U_BMC.8
- new net BMC_ETH3_P: J_BMC_NET.7, U_BMC.7
- new net FAN_0_PWM: U_BMC.9
- new net FAN_0_TACH: U_BMC.10
- new net FAN_1_PWM: U_BMC.11
- new net FAN_1_TACH: U_BMC.12
- new net FAN_2_PWM: U_BMC.13
- new net FAN_2_TACH: U_BMC.14
- new net FAN_3_PWM: U_BMC.15
- new net FAN_3_TACH: U_BMC.16
- new net FAN_4_PWM: U_BMC.17
- new net FAN_4_TACH: U_BMC.18
- new net FAN_5_PWM: U_BMC.19
- new net FAN_5_TACH: U_BMC.20
- new net PCIE_PERST: J_HOST.35, U_FPGA.AE15
- new net PCIE_WAKE: J_HOST.36, U_FPGA.AE16
- new net PMB_SCL: U_BMC.23
- new net PMB_SDA: U_BMC.24
- new net PSU_ON: U_BMC.25
