File: hw/kicad/power.kicad_sch (KiCad schematic)
At the start: 18 parts

Commit message: Retarget the board to a host-attached 1U chassis
The energy model put the board at 0.5 to 1.6 kW of input across the
throughput range, which is a rack supply, not a PCIe slot.  The board is
now one 420 x 360 mm board in a 1U: two CRPS modules in a 1+1 pair, a
BMC with its own Ethernet, six front fans, and a SlimSAS 8i cable to the
host's PCIe.  With the room to carry it, the ASIC package is rated at the
50K tokens/s target (177 A core), which selects the 1225-ball 29 mm
package.

hw/board.yaml: 1U form factor, host cable, CRPS input, BMC, PSU, fan and
RJ45 parts and classes, 50K package rating.

hw/kicad_gen.py: form factors (1U default, card kept) that map the ring
frame onto the physical board with keep-outs (PSU bay, rear I/O, fans),
physical parts for the chassis connectors and BMC, a fit check, layout
derived from the package body, the FPGA beside H1 taking the ring on its
west edge (closing hop 74 mm instead of 95 mm with the 29 mm package),
PCIe pins on the FPGA's south edge, regulators spaced for the larger
package.  Every hop is within the 80 mm limit and pcbnew DRC reports only
the unrouted nets.

Tests cover both form factors, the keep-outs and the package rating;
docs describe the 1U, the rating decision and the floorplan findings.

Co-Authored-By: Claude Fable 5.1 <noreply@anthropic.com>
Claude-Session: https://claude.ai/code/session_01VmmvkZe8Ctg3RAykNGsQBn
Parts:
- removed J_AUX: 12V-2x6 aux, appliance:12V-2x6, symbol appliance:12V-2x6
- added J_FAN0, J_FAN1, J_FAN2, J_FAN3, J_FAN4, J_FAN5: fan header, appliance:FAN_4PIN, symbol appliance:FAN_4PIN
- added J_PSU0, J_PSU1: CRPS 12 V output, appliance:CRPS_BLADES, symbol appliance:CRPS_BLADES
Connections:
- net +12V: now also J_FAN0.1, J_FAN1.1, J_FAN2.1, J_FAN3.1, J_FAN4.1, J_FAN5.1, J_PSU0.1, J_PSU0.2, J_PSU0.3, J_PSU0.4, J_PSU0.5, J_PSU0.6, J_PSU1.1, J_PSU1.2, J_PSU1.3, J_PSU1.4, J_PSU1.5, J_PSU1.6
- net GND: now also J_FAN0.2, J_FAN1.2, J_FAN2.2, J_FAN3.2, J_FAN4.2, J_FAN5.2, J_PSU0.10, J_PSU0.11, J_PSU0.12, J_PSU0.16, J_PSU0.7, J_PSU0.8, J_PSU0.9, J_PSU1.10, J_PSU1.11, J_PSU1.12, J_PSU1.16, J_PSU1.7, J_PSU1.8, J_PSU1.9
- net PMB_SCL: now also J_PSU0.13, J_PSU1.13
- net PMB_SDA: now also J_PSU0.14, J_PSU1.14
- new net FAN_0_PWM: J_FAN0.3
- new net FAN_0_TACH: J_FAN0.4
- new net FAN_1_PWM: J_FAN1.3
- new net FAN_1_TACH: J_FAN1.4
- new net FAN_2_PWM: J_FAN2.3
- new net FAN_2_TACH: J_FAN2.4
- new net FAN_3_PWM: J_FAN3.3
- new net FAN_3_TACH: J_FAN3.4
- new net FAN_4_PWM: J_FAN4.3
- new net FAN_4_TACH: J_FAN4.4
- new net FAN_5_PWM: J_FAN5.3
- new net FAN_5_TACH: J_FAN5.4
- new net PSU_ON: J_PSU0.15, J_PSU1.15

Commit message: Add the four-plus-one high-end board variant with HBM in the package
hw/board_27b.yaml describes the 27B-class appliance on a 2 nm-class die:
four layer ASICs of sixteen layers, one head ASIC holding the whole LM
head, an HBM4 stack on each layer ASIC's interposer (no memory on the
board), direct-to-chip liquid cooling, a 1+1 pair of 3000 W CRPS modules,
rated at the 234K tokens/s fabric ceiling (525 W and 656 A per layer die,
a 55 x 55 package of 3025 balls, a hexagon ring of 85 mm side with 10 mm
between packages for the cold plates).  The simulator's 27B configs
become 4 + 1 too; throughput and board power are unchanged, per-die power
doubles.

To carry a second description the tools now take the memory channels
from the class's interfaces (none for in-package HBM), the rail ball
counts from the package rules, the regulators from the power tree (one
block per shared rail in the middle of the polygon, the FPGA's rails on
one block, DDR4 and 3.3 V beside the DDR4 row), a per-board ring gap, and
ball names past 40 rows; outputs are named after the source.  The
overlap test's margin had the wrong sign and let bodies touch by half a
millimetre; fixed, and both boards pass pcbnew DRC with only the unrouted
nets.  Tests cover the variant's hexagon, package, rails and fit.

Co-Authored-By: Claude Fable 5.1 <noreply@anthropic.com>
Claude-Session: https://claude.ai/code/session_01VmmvkZe8Ctg3RAykNGsQBn
Parts:
- added REG_IO_1V8: VDD_IO_1V8 regulator, appliance:REG_MODULE_20x6, symbol appliance:REG_MODULE_20x6
- REG_1V8: value VDD_IO_1V8 regulator -> VDD1_1V8 regulator
- REG_DDR: value VDD_1V2 regulator -> VDD_1V2, VPP_2V5 regulator
- REG_FPGA: value VCCINT_0V85 regulator -> VCCINT_0V85, VCCAUX_1V8, VCCO_1V8, VCCO_1V2, MGTAVCC, MGTAVTT regulator
Connections:
- net VDD_PLL_0V9 is gone; now on net VDD2L_0V9: REG_0V9.5
- net +12V: now also REG_IO_1V8.1, REG_IO_1V8.2, REG_IO_1V8.3
- net GND: now also REG_0V3.7, REG_0V9.7, REG_1V05.7, REG_1V8.7, REG_3V3.7, REG_FPGA.12, REG_FPGA.13, REG_FPGA.14, REG_IO_1V8.7, REG_IO_1V8.8, REG_IO_1V8.9; no longer REG_0V3.10, REG_0V9.10, REG_1V05.10, REG_1V8.10, REG_3V3.10, REG_FPGA.10, REG_FPGA.8, REG_FPGA.9
- net MGTAVCC: now also REG_FPGA.10; no longer REG_FPGA.6
- net MGTAVTT: now also REG_FPGA.11; no longer REG_FPGA.7
- net VCCAUX_1V8: now also REG_FPGA.7; no longer REG_FPGA.5
- net VCCINT_0V85: now also REG_FPGA.5, REG_FPGA.6
- net VCCO_1V2: now also REG_FPGA.9; no longer REG_1V05.5
- net VCCO_1V8: now also REG_FPGA.8; no longer REG_1V8.5
- net VDD1_1V8: now also REG_1V8.5, REG_1V8.6
- net VDD2H_1V05: now also REG_1V05.5; no longer REG_1V05.7
- net VDD2L_0V9: no longer REG_0V9.7
- net VDDQ_0V3: no longer REG_0V3.7
- net VDD_1V2: now also REG_DDR.6; no longer REG_DDR.7
- net VDD_3V3: no longer REG_3V3.7
- net VDD_IO_1V8: now also REG_IO_1V8.4, REG_IO_1V8.5, REG_IO_1V8.6; no longer REG_1V8.6, REG_1V8.7
- net VPP_2V5: now also REG_DDR.7; no longer REG_DDR.6
