File: hw/kicad_27b/appliance.kicad_pcb (KiCad board)
At the start: 12 copper layers, 420 x 360 mm, 34 parts

Commit message: Pipeline a layer's passes, and re-rate the 27B board to eight layer dies
Two things the last commit left open.

The simulator now separates a layer stage's latency from its initiation
interval.  A layer is a chain of passes and each pass has its own via-
programmed tiles, so nothing is reused between them: the first pass is free
the moment its token moves on, and the stage holds as many tokens as fit
between its latency and its interval.  layer_pass_cycles carries the pass,
a quarter of the layer in every shipped geometry, which is the same figure
the single-pass head die already used.

I expected that to be worth four times and it is worth almost nothing,
because after the memory corrections it is the memory and not the pass rate
that binds.  It is exactly neutral on every LPDDR5X and PSRAM configuration
at any context count, worth 4 to 8 percent on the 9B with HBM, and slightly
negative on the 27B, where more tokens per stage lengthen latency against a
fixed pool of contexts.  With the bandwidth raised tenfold it is worth 2.5
times, 240K to 597K tokens/s, so the lever is real and nothing in reach of
this design is close enough to the fabric to collect it.  Letting a token's
state write overlap the next token's state read, which the same change
allows, is what does move the HBM numbers: the 3 nm 9B goes from 190K to
244K.

The 27B board is now eight layer ASICs of eight layers and two head ASICs
splitting the LM head, at 153K tokens/s rather than the 234K that came from
the un-corrected model.  Halving the per-die load takes the core rail from
650 A to 249 A, the package from a 55 x 55 array to 35 x 35, the cold plate
from 525 W to 200 W, and puts the ring on the same 11-gon as the 9B board.
hw/README's open item is replaced by the re-rating itself.

The 9B board's design point follows the same correction, 14.5K to 8.2K, and
its per-die traffic is 7.35 MB per token rather than the 4.2 MB of retrieval
alone.  Generated files now name the board description they came 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
Parts:
- added U_A4: layer_asic, appliance:FCBGA1225_35x35_P0.8, F.Cu at (134.5, 103.2)
- added U_A5: layer_asic, appliance:FCBGA1225_35x35_P0.8, F.Cu at (185.5, 103.2)
- added U_A6: layer_asic, appliance:FCBGA1225_35x35_P0.8, F.Cu at (228.4, 130.7)
- added U_A7: layer_asic, appliance:FCBGA1225_35x35_P0.8, F.Cu at (249.6, 177.1)
- added U_H1: head_asic, appliance:FCBGA1225_35x35_P0.8, F.Cu at (208.9, 266.1)
- added VRM_A4: core VRM VDD_CORE_A4, appliance:VRM_MODULE_26x6, F.Cu at (140.1, 122.1)
- added VRM_A5: core VRM VDD_CORE_A5, appliance:VRM_MODULE_26x6, F.Cu at (179.9, 122.1)
- added VRM_A6: core VRM VDD_CORE_A6, appliance:VRM_MODULE_26x6, F.Cu at (213.5, 143.7)
- added VRM_A7: core VRM VDD_CORE_A7, appliance:VRM_MODULE_26x6, F.Cu at (230.0, 179.9)
- added VRM_H1: core VRM VDD_CORE_H1, appliance:VRM_MODULE_26x6, F.Cu at (198.3, 249.5)
- U_A0, U_A1, U_A2, U_A3, U_H0: footprint appliance:FCBGA3025_55x55_P1.0 -> appliance:FCBGA1225_35x35_P0.8
- moved U_A3 143.0 mm to (91.6, 130.7)
- moved U_A2 115.0 mm to (70.4, 177.1)
- moved VRM_A3 100.8 mm to (106.5, 143.7)
- moved VRM_A2 81.8 mm to (90.0, 179.9)
- moved U_A1 80.6 mm to (77.7, 227.6)
- moved VRM_A1 58.7 mm to (95.6, 219.4)
- moved U_A0 41.7 mm to (111.1, 266.1)
- moved VRM_A0 34.1 mm to (121.7, 249.5)
- moved VRM_H0 19.4 mm to (224.4, 219.4)
- moved U_H0 10.0 mm to (242.3, 227.6)
- moved REG_3V3 5.51 mm to (149.0, 311.9)
- moved REG_DDR 5.51 mm to (171.0, 311.9)
- moved REG_FPGA 5.51 mm to (160.0, 261.3)
- moved U_D0 5.51 mm to (172.8, 301.3)
- moved U_D1 5.51 mm to (164.2, 301.3)
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Connections:
- U_A0 pad AA1: LINK0_DATA4 -> LINK0_DATA24
- U_A0 pad AA2: LINK0_DATA5 -> LINK0_DATA25
- U_A0 pad AA34: VDD_CORE_A0 -> LINK1_DATA25
- U_A0 pad AA35: GND -> LINK1_DATA24
- U_A0 pad AB1: LINK0_DATA6 -> LINK0_DATA26
- U_A0 pad AB2: LINK0_DATA7 -> LINK0_DATA27
- U_A0 pad AB34: GND -> LINK1_DATA27
- U_A0 pad AB35: VDD_CORE_A0 -> LINK1_DATA26
- U_A0 pad AC1: LINK0_DATA8 -> LINK0_DATA28
- U_A0 pad AC2: LINK0_DATA9 -> LINK0_DATA29
- U_A0 pad AC34: VDD_CORE_A0 -> LINK1_DATA29
- U_A0 pad AC35: GND -> LINK1_DATA28
- U_A0 pad AD1: LINK0_DATA10 -> LINK0_DATA30
- U_A0 pad AD2: LINK0_DATA11 -> LINK0_DATA31
- U_A0 pad AD34: GND -> LINK1_DATA31
- U_A0 pad AD35: VDD_CORE_A0 -> LINK1_DATA30
- U_A0 pad AE1: LINK0_DATA12 -> LINK0_CLOCK
- U_A0 pad AE2: LINK0_DATA13 -> LINK0_VALID
- U_A0 pad AE34: VDD_CORE_A0 -> LINK1_VALID
- U_A0 pad AE35: GND -> LINK1_CLOCK
- U_A0 pad AF1: LINK0_DATA14 -> LINK0_READY_BACK
- U_A0 pad AF2: LINK0_DATA15 -> LINK0_SOF
- U_A0 pad AF34: GND -> LINK1_SOF
- U_A0 pad AF35: VDD_CORE_A0 -> LINK1_READY_BACK
- U_A0 pad AG1: LINK0_DATA16 -> GND
- U_A0 pad AG2: LINK0_DATA17 -> VDD_CORE_A0
- U_A0 pad AH1: LINK0_DATA18 -> VDD_CORE_A0
- U_A0 pad AH2: LINK0_DATA19 -> GND
- U_A0 pad AJ1: LINK0_DATA20 -> GND
- U_A0 pad AJ2: LINK0_DATA21 -> VDD_CORE_A0
- U_A0 pad AK1: LINK0_DATA22 -> VDD_CORE_A0
- U_A0 pad AK2: LINK0_DATA23 -> GND
- U_A0 pad AL1: LINK0_DATA24 -> GND
- U_A0 pad AL2: LINK0_DATA25 -> VDD_CORE_A0
- U_A0 pad AM1: LINK0_DATA26 -> VDD_CORE_A0
- U_A0 pad AM2: LINK0_DATA27 -> GND
- U_A0 pad AN1: LINK0_DATA28 -> GND
- U_A0 pad AN2: LINK0_DATA29 -> VDD_CORE_A0
- U_A0 pad AP1: LINK0_DATA30 -> VDD_CORE_A0
- U_A0 pad AP2: LINK0_DATA31 -> GND
- U_A0 pad AR1: LINK0_CLOCK -> GND
- U_A0 pad AR10: VDD_CORE_A0 -> JTAG_TMS
- U_A0 pad AR11: GND -> JTAG_TDO_FPGA
- U_A0 pad AR12: VDD_CORE_A0 -> GND
- U_A0 pad AR13: GND -> JTAG_TDO_A0
- U_A0 pad AR14: VDD_CORE_A0 -> JTAG_TRST
- U_A0 pad AR15: GND -> REFCLK_A0_P
- U_A0 pad AR16: VDD_CORE_A0 -> REFCLK_A0_N
- U_A0 pad AR18: VDD_CORE_A0 -> MODE0_A0
- U_A0 pad AR19: GND -> MODE1_A0
- U_A0 pad AR2: LINK0_VALID -> VDD_CORE_A0
- U_A0 pad AR3: GND -> MGMT_SCLK
- U_A0 pad AR4: VDD_CORE_A0 -> MGMT_MOSI
- U_A0 pad AR5: GND -> MGMT_MISO
- U_A0 pad AR6: VDD_CORE_A0 -> MGMT_CS_A0
- U_A0 pad AR8: VDD_CORE_A0 -> MGMT_IRQ_A0
- U_A0 pad AR9: GND -> JTAG_TCK
- U_A0 pad C18: VDD_HBM_1V1 -> VDD_IO_1V8
- U_A0 pad C28: VDD_HBM_1V1 -> VDD_PLL_0V9
- U_A0 pad C8: VDD_HBM_1V1 -> VDD_IO_1V8
- U_A0 pad D9: VDD_HBM_1V1 -> VDD_PLL_0V9
- U_A0 pad G32: VDDQ_HBM_0V4 -> VDD_HBM_1V1
- U_A0 pad H13: VDDQ_HBM_0V4 -> VDD_HBM_1V1
- U_A0 pad H23: VDDQ_HBM_0V4 -> VDD_HBM_1V1
- U_A0 pad H3: VDDQ_HBM_0V4 -> VDD_HBM_1V1
- U_A0 pad H33: VDDQ_HBM_0V4 -> VDD_HBM_1V1
- U_A0 pad J1: GND -> LINK0_DATA0
- U_A0 pad J14: VDDQ_HBM_0V4 -> VDD_HBM_1V1
- U_A0 pad J2: VDD_CORE_A0 -> LINK0_DATA1
- U_A0 pad J24: VDDQ_HBM_0V4 -> VDD_HBM_1V1
- U_A0 pad J34: VDD_CORE_A0 -> LINK1_DATA1
- U_A0 pad J35: GND -> LINK1_DATA0
- U_A0 pad J4: VDDQ_HBM_0V4 -> VDD_HBM_1V1
- U_A0 pad K1: VDD_CORE_A0 -> LINK0_DATA2
- U_A0 pad K15: VDD_CORE_A0 -> VDD_HBM_1V1
- U_A0 pad K2: GND -> LINK0_DATA3
- U_A0 pad K25: VDD_CORE_A0 -> VDD_HBM_1V1
- U_A0 pad K34: GND -> LINK1_DATA3
- U_A0 pad K35: VDD_CORE_A0 -> LINK1_DATA2
- U_A0 pad K5: VDD_CORE_A0 -> VDD_HBM_1V1
- U_A0 pad L1: GND -> LINK0_DATA4
- U_A0 pad L16: VDD_CORE_A0 -> VDDQ_HBM_0V4
- U_A0 pad L2: VDD_CORE_A0 -> LINK0_DATA5
- U_A0 pad L26: VDD_CORE_A0 -> VDDQ_HBM_0V4
- U_A0 pad L34: VDD_CORE_A0 -> LINK1_DATA5
- U_A0 pad L35: GND -> LINK1_DATA4
- U_A0 pad L6: VDD_CORE_A0 -> VDD_HBM_1V1
- U_A0 pad M1: VDD_CORE_A0 -> LINK0_DATA6
- U_A0 pad M17: VDD_CORE_A0 -> VDDQ_HBM_0V4
- U_A0 pad M2: GND -> LINK0_DATA7
- U_A0 pad M27: VDD_CORE_A0 -> VDDQ_HBM_0V4
- U_A0 pad M34: GND -> LINK1_DATA7
- U_A0 pad M35: VDD_CORE_A0 -> LINK1_DATA6
- U_A0 pad M7: VDD_CORE_A0 -> VDDQ_HBM_0V4
- U_A0 pad N1: GND -> LINK0_DATA8
- U_A0 pad N18: VDD_CORE_A0 -> VDDQ_HBM_0V4
- U_A0 pad N2: VDD_CORE_A0 -> LINK0_DATA9
- U_A0 pad N28: VDD_CORE_A0 -> VDDQ_HBM_0V4
- U_A0 pad N34: VDD_CORE_A0 -> LINK1_DATA9
- U_A0 pad N35: GND -> LINK1_DATA8
- U_A0 pad N8: VDD_CORE_A0 -> VDDQ_HBM_0V4
- U_A0 pad P1: VDD_CORE_A0 -> LINK0_DATA10
- U_A0 pad P19: VDD_CORE_A0 -> VDDQ_HBM_0V4
- U_A0 pad P2: GND -> LINK0_DATA11
- U_A0 pad P29: VDD_CORE_A0 -> VDDQ_HBM_0V4
- U_A0 pad P34: GND -> LINK1_DATA11
- U_A0 pad P35: VDD_CORE_A0 -> LINK1_DATA10
- U_A0 pad P9: VDD_CORE_A0 -> VDDQ_HBM_0V4
- U_A0 pad R1: GND -> LINK0_DATA12
- U_A0 pad R10: VDD_CORE_A0 -> VDDQ_HBM_0V4
- U_A0 pad R2: VDD_CORE_A0 -> LINK0_DATA13
- U_A0 pad R34: VDD_CORE_A0 -> LINK1_DATA13
- U_A0 pad R35: GND -> LINK1_DATA12
- U_A0 pad T1: VDD_CORE_A0 -> LINK0_DATA14
- U_A0 pad T2: GND -> LINK0_DATA15
- U_A0 pad T34: GND -> LINK1_DATA15
- U_A0 pad T35: VDD_CORE_A0 -> LINK1_DATA14
- U_A0 pad U1: GND -> LINK0_DATA16
- U_A0 pad U2: VDD_CORE_A0 -> LINK0_DATA17
- U_A0 pad U34: VDD_CORE_A0 -> LINK1_DATA17
- U_A0 pad U35: GND -> LINK1_DATA16
- U_A0 pad V1: VDD_CORE_A0 -> LINK0_DATA18
- U_A0 pad V2: GND -> LINK0_DATA19
- U_A0 pad V34: GND -> LINK1_DATA19
- U_A0 pad V35: VDD_CORE_A0 -> LINK1_DATA18
- U_A0 pad W1: LINK0_DATA0 -> LINK0_DATA20
- U_A0 pad W2: LINK0_DATA1 -> LINK0_DATA21
- U_A0 pad W34: VDD_CORE_A0 -> LINK1_DATA21
- U_A0 pad W35: GND -> LINK1_DATA20
- U_A0 pad Y1: LINK0_DATA2 -> LINK0_DATA22
- U_A0 pad Y2: LINK0_DATA3 -> LINK0_DATA23
- U_A0 pad Y34: GND -> LINK1_DATA23
- U_A0 pad Y35: VDD_CORE_A0 -> LINK1_DATA22
- U_A1 pad AA1: LINK1_DATA4 -> LINK1_DATA24
- U_A1 pad AA2: LINK1_DATA5 -> LINK1_DATA25
- U_A1 pad AA34: VDD_CORE_A1 -> LINK2_DATA25
- U_A1 pad AA35: GND -> LINK2_DATA24
- U_A1 pad AB1: LINK1_DATA6 -> LINK1_DATA26
- U_A1 pad AB2: LINK1_DATA7 -> LINK1_DATA27
- U_A1 pad AB34: GND -> LINK2_DATA27
- U_A1 pad AB35: VDD_CORE_A1 -> LINK2_DATA26
- U_A1 pad AC1: LINK1_DATA8 -> LINK1_DATA28
- U_A1 pad AC2: LINK1_DATA9 -> LINK1_DATA29
- U_A1 pad AC34: VDD_CORE_A1 -> LINK2_DATA29
- U_A1 pad AC35: GND -> LINK2_DATA28
- U_A1 pad AD1: LINK1_DATA10 -> LINK1_DATA30
- U_A1 pad AD2: LINK1_DATA11 -> LINK1_DATA31
- U_A1 pad AD34: GND -> LINK2_DATA31
- U_A1 pad AD35: VDD_CORE_A1 -> LINK2_DATA30
- U_A1 pad AE1: LINK1_DATA12 -> LINK1_CLOCK
- U_A1 pad AE2: LINK1_DATA13 -> LINK1_VALID
- U_A1 pad AE34: VDD_CORE_A1 -> LINK2_VALID
- U_A1 pad AE35: GND -> LINK2_CLOCK
- U_A1 pad AF1: LINK1_DATA14 -> LINK1_READY_BACK
- U_A1 pad AF2: LINK1_DATA15 -> LINK1_SOF
- U_A1 pad AF34: GND -> LINK2_SOF
- U_A1 pad AF35: VDD_CORE_A1 -> LINK2_READY_BACK
- U_A1 pad AG1: LINK1_DATA16 -> GND
- U_A1 pad AG2: LINK1_DATA17 -> VDD_CORE_A1
- U_A1 pad AH1: LINK1_DATA18 -> VDD_CORE_A1
- U_A1 pad AH2: LINK1_DATA19 -> GND
- U_A1 pad AJ1: LINK1_DATA20 -> GND
- U_A1 pad AJ2: LINK1_DATA21 -> VDD_CORE_A1
- U_A1 pad AK1: LINK1_DATA22 -> VDD_CORE_A1
- U_A1 pad AK2: LINK1_DATA23 -> GND
- U_A1 pad AL1: LINK1_DATA24 -> GND
- U_A1 pad AL2: LINK1_DATA25 -> VDD_CORE_A1
- U_A1 pad AM1: LINK1_DATA26 -> VDD_CORE_A1
- U_A1 pad AM2: LINK1_DATA27 -> GND
- U_A1 pad AN1: LINK1_DATA28 -> GND
- U_A1 pad AN2: LINK1_DATA29 -> VDD_CORE_A1
- U_A1 pad AP1: LINK1_DATA30 -> VDD_CORE_A1
- U_A1 pad AP2: LINK1_DATA31 -> GND
- U_A1 pad AR1: LINK1_CLOCK -> GND
- U_A1 pad AR10: VDD_CORE_A1 -> JTAG_TMS
- U_A1 pad AR11: GND -> JTAG_TDO_A0
- U_A1 pad AR12: VDD_CORE_A1 -> GND
- U_A1 pad AR13: GND -> JTAG_TDO_A1
- U_A1 pad AR14: VDD_CORE_A1 -> JTAG_TRST
- U_A1 pad AR15: GND -> REFCLK_A1_P
- U_A1 pad AR16: VDD_CORE_A1 -> REFCLK_A1_N
- U_A1 pad AR18: VDD_CORE_A1 -> MODE0_A1
- U_A1 pad AR19: GND -> MODE1_A1
- U_A1 pad AR2: LINK1_VALID -> VDD_CORE_A1
- U_A1 pad AR3: GND -> MGMT_SCLK
- U_A1 pad AR4: VDD_CORE_A1 -> MGMT_MOSI
- U_A1 pad AR5: GND -> MGMT_MISO
- U_A1 pad AR6: VDD_CORE_A1 -> MGMT_CS_A1
- U_A1 pad AR8: VDD_CORE_A1 -> MGMT_IRQ_A1
- U_A1 pad AR9: GND -> JTAG_TCK
- U_A1 pad C18: VDD_HBM_1V1 -> VDD_IO_1V8
- U_A1 pad C28: VDD_HBM_1V1 -> VDD_PLL_0V9
- U_A1 pad C8: VDD_HBM_1V1 -> VDD_IO_1V8
- U_A1 pad D9: VDD_HBM_1V1 -> VDD_PLL_0V9
- U_A1 pad G32: VDDQ_HBM_0V4 -> VDD_HBM_1V1
- U_A1 pad H13: VDDQ_HBM_0V4 -> VDD_HBM_1V1
- U_A1 pad H23: VDDQ_HBM_0V4 -> VDD_HBM_1V1
- U_A1 pad H3: VDDQ_HBM_0V4 -> VDD_HBM_1V1
- U_A1 pad H33: VDDQ_HBM_0V4 -> VDD_HBM_1V1
- U_A1 pad J1: GND -> LINK1_DATA0
- U_A1 pad J14: VDDQ_HBM_0V4 -> VDD_HBM_1V1
- U_A1 pad J2: VDD_CORE_A1 -> LINK1_DATA1
- U_A1 pad J24: VDDQ_HBM_0V4 -> VDD_HBM_1V1
- U_A1 pad J34: VDD_CORE_A1 -> LINK2_DATA1
- U_A1 pad J35: GND -> LINK2_DATA0
- U_A1 pad J4: VDDQ_HBM_0V4 -> VDD_HBM_1V1
- U_A1 pad K1: VDD_CORE_A1 -> LINK1_DATA2
- U_A1 pad K15: VDD_CORE_A1 -> VDD_HBM_1V1
- U_A1 pad K2: GND -> LINK1_DATA3
- U_A1 pad K25: VDD_CORE_A1 -> VDD_HBM_1V1
- U_A1 pad K34: GND -> LINK2_DATA3
- U_A1 pad K35: VDD_CORE_A1 -> LINK2_DATA2
- U_A1 pad K5: VDD_CORE_A1 -> VDD_HBM_1V1
- U_A1 pad L1: GND -> LINK1_DATA4
- U_A1 pad L16: VDD_CORE_A1 -> VDDQ_HBM_0V4
- U_A1 pad L2: VDD_CORE_A1 -> LINK1_DATA5
- U_A1 pad L26: VDD_CORE_A1 -> VDDQ_HBM_0V4
- U_A1 pad L34: VDD_CORE_A1 -> LINK2_DATA5
- U_A1 pad L35: GND -> LINK2_DATA4
- U_A1 pad L6: VDD_CORE_A1 -> VDD_HBM_1V1
- U_A1 pad M1: VDD_CORE_A1 -> LINK1_DATA6
- U_A1 pad M17: VDD_CORE_A1 -> VDDQ_HBM_0V4
- U_A1 pad M2: GND -> LINK1_DATA7
- U_A1 pad M27: VDD_CORE_A1 -> VDDQ_HBM_0V4
- U_A1 pad M34: GND -> LINK2_DATA7
- U_A1 pad M35: VDD_CORE_A1 -> LINK2_DATA6
- U_A1 pad M7: VDD_CORE_A1 -> VDDQ_HBM_0V4
- U_A1 pad N1: GND -> LINK1_DATA8
- U_A1 pad N18: VDD_CORE_A1 -> VDDQ_HBM_0V4
- U_A1 pad N2: VDD_CORE_A1 -> LINK1_DATA9
- U_A1 pad N28: VDD_CORE_A1 -> VDDQ_HBM_0V4
- U_A1 pad N34: VDD_CORE_A1 -> LINK2_DATA9
- U_A1 pad N35: GND -> LINK2_DATA8
- U_A1 pad N8: VDD_CORE_A1 -> VDDQ_HBM_0V4
- U_A1 pad P1: VDD_CORE_A1 -> LINK1_DATA10
- U_A1 pad P19: VDD_CORE_A1 -> VDDQ_HBM_0V4
- U_A1 pad P2: GND -> LINK1_DATA11
- U_A1 pad P29: VDD_CORE_A1 -> VDDQ_HBM_0V4
- U_A1 pad P34: GND -> LINK2_DATA11
- U_A1 pad P35: VDD_CORE_A1 -> LINK2_DATA10
- U_A1 pad P9: VDD_CORE_A1 -> VDDQ_HBM_0V4
- U_A1 pad R1: GND -> LINK1_DATA12
- U_A1 pad R10: VDD_CORE_A1 -> VDDQ_HBM_0V4
- U_A1 pad R2: VDD_CORE_A1 -> LINK1_DATA13
- U_A1 pad R34: VDD_CORE_A1 -> LINK2_DATA13
- U_A1 pad R35: GND -> LINK2_DATA12
- U_A1 pad T1: VDD_CORE_A1 -> LINK1_DATA14
- U_A1 pad T2: GND -> LINK1_DATA15
- U_A1 pad T34: GND -> LINK2_DATA15
- U_A1 pad T35: VDD_CORE_A1 -> LINK2_DATA14
- U_A1 pad U1: GND -> LINK1_DATA16
- U_A1 pad U2: VDD_CORE_A1 -> LINK1_DATA17
- U_A1 pad U34: VDD_CORE_A1 -> LINK2_DATA17
- U_A1 pad U35: GND -> LINK2_DATA16
- U_A1 pad V1: VDD_CORE_A1 -> LINK1_DATA18
- U_A1 pad V2: GND -> LINK1_DATA19
- U_A1 pad V34: GND -> LINK2_DATA19
- U_A1 pad V35: VDD_CORE_A1 -> LINK2_DATA18
- U_A1 pad W1: LINK1_DATA0 -> LINK1_DATA20
- U_A1 pad W2: LINK1_DATA1 -> LINK1_DATA21
- U_A1 pad W34: VDD_CORE_A1 -> LINK2_DATA21
- U_A1 pad W35: GND -> LINK2_DATA20
- U_A1 pad Y1: LINK1_DATA2 -> LINK1_DATA22
- U_A1 pad Y2: LINK1_DATA3 -> LINK1_DATA23
- U_A1 pad Y34: GND -> LINK2_DATA23
- U_A1 pad Y35: VDD_CORE_A1 -> LINK2_DATA22
- U_A2 pad AA1: LINK2_DATA4 -> LINK2_DATA24
- U_A2 pad AA2: LINK2_DATA5 -> LINK2_DATA25
- U_A2 pad AA34: VDD_CORE_A2 -> LINK3_DATA25
- U_A2 pad AA35: GND -> LINK3_DATA24
- U_A2 pad AB1: LINK2_DATA6 -> LINK2_DATA26
- U_A2 pad AB2: LINK2_DATA7 -> LINK2_DATA27
- U_A2 pad AB34: GND -> LINK3_DATA27
- U_A2 pad AB35: VDD_CORE_A2 -> LINK3_DATA26
- U_A2 pad AC1: LINK2_DATA8 -> LINK2_DATA28
- U_A2 pad AC2: LINK2_DATA9 -> LINK2_DATA29
- U_A2 pad AC34: VDD_CORE_A2 -> LINK3_DATA29
- U_A2 pad AC35: GND -> LINK3_DATA28
- U_A2 pad AD1: LINK2_DATA10 -> LINK2_DATA30
- U_A2 pad AD2: LINK2_DATA11 -> LINK2_DATA31
- U_A2 pad AD34: GND -> LINK3_DATA31
- U_A2 pad AD35: VDD_CORE_A2 -> LINK3_DATA30
- U_A2 pad AE1: LINK2_DATA12 -> LINK2_CLOCK
- U_A2 pad AE2: LINK2_DATA13 -> LINK2_VALID
- U_A2 pad AE34: VDD_CORE_A2 -> LINK3_VALID
- U_A2 pad AE35: GND -> LINK3_CLOCK
- U_A2 pad AF1: LINK2_DATA14 -> LINK2_READY_BACK
- U_A2 pad AF2: LINK2_DATA15 -> LINK2_SOF
- U_A2 pad AF34: GND -> LINK3_SOF
- U_A2 pad AF35: VDD_CORE_A2 -> LINK3_READY_BACK
- U_A2 pad AG1: LINK2_DATA16 -> GND
- U_A2 pad AG2: LINK2_DATA17 -> VDD_CORE_A2
- U_A2 pad AH1: LINK2_DATA18 -> VDD_CORE_A2
- U_A2 pad AH2: LINK2_DATA19 -> GND
- U_A2 pad AJ1: LINK2_DATA20 -> GND
- U_A2 pad AJ2: LINK2_DATA21 -> VDD_CORE_A2
- U_A2 pad AK1: LINK2_DATA22 -> VDD_CORE_A2
- U_A2 pad AK2: LINK2_DATA23 -> GND
- U_A2 pad AL1: LINK2_DATA24 -> GND
- U_A2 pad AL2: LINK2_DATA25 -> VDD_CORE_A2
- U_A2 pad AM1: LINK2_DATA26 -> VDD_CORE_A2
- U_A2 pad AM2: LINK2_DATA27 -> GND
- U_A2 pad AN1: LINK2_DATA28 -> GND
- U_A2 pad AN2: LINK2_DATA29 -> VDD_CORE_A2
- U_A2 pad AP1: LINK2_DATA30 -> VDD_CORE_A2
- U_A2 pad AP2: LINK2_DATA31 -> GND
- U_A2 pad AR1: LINK2_CLOCK -> GND
- U_A2 pad AR10: VDD_CORE_A2 -> JTAG_TMS
- U_A2 pad AR11: GND -> JTAG_TDO_A1
- U_A2 pad AR12: VDD_CORE_A2 -> GND
- U_A2 pad AR13: GND -> JTAG_TDO_A2
- U_A2 pad AR14: VDD_CORE_A2 -> JTAG_TRST
- U_A2 pad AR15: GND -> REFCLK_A2_P
- U_A2 pad AR16: VDD_CORE_A2 -> REFCLK_A2_N
- U_A2 pad AR18: VDD_CORE_A2 -> MODE0_A2
- U_A2 pad AR19: GND -> MODE1_A2
- U_A2 pad AR2: LINK2_VALID -> VDD_CORE_A2
- U_A2 pad AR3: GND -> MGMT_SCLK
- U_A2 pad AR4: VDD_CORE_A2 -> MGMT_MOSI
- U_A2 pad AR5: GND -> MGMT_MISO
- U_A2 pad AR6: VDD_CORE_A2 -> MGMT_CS_A2
- U_A2 pad AR8: VDD_CORE_A2 -> MGMT_IRQ_A2
- U_A2 pad AR9: GND -> JTAG_TCK
- U_A2 pad C18: VDD_HBM_1V1 -> VDD_IO_1V8
- U_A2 pad C28: VDD_HBM_1V1 -> VDD_PLL_0V9
- U_A2 pad C8: VDD_HBM_1V1 -> VDD_IO_1V8
- U_A2 pad D9: VDD_HBM_1V1 -> VDD_PLL_0V9
- U_A2 pad G32: VDDQ_HBM_0V4 -> VDD_HBM_1V1
- U_A2 pad H13: VDDQ_HBM_0V4 -> VDD_HBM_1V1
- U_A2 pad H23: VDDQ_HBM_0V4 -> VDD_HBM_1V1
- U_A2 pad H3: VDDQ_HBM_0V4 -> VDD_HBM_1V1
- U_A2 pad H33: VDDQ_HBM_0V4 -> VDD_HBM_1V1
- U_A2 pad J1: GND -> LINK2_DATA0
- U_A2 pad J14: VDDQ_HBM_0V4 -> VDD_HBM_1V1
- U_A2 pad J2: VDD_CORE_A2 -> LINK2_DATA1
- U_A2 pad J24: VDDQ_HBM_0V4 -> VDD_HBM_1V1
- U_A2 pad J34: VDD_CORE_A2 -> LINK3_DATA1
- U_A2 pad J35: GND -> LINK3_DATA0
- U_A2 pad J4: VDDQ_HBM_0V4 -> VDD_HBM_1V1
- U_A2 pad K1: VDD_CORE_A2 -> LINK2_DATA2
- U_A2 pad K15: VDD_CORE_A2 -> VDD_HBM_1V1
- U_A2 pad K2: GND -> LINK2_DATA3
- U_A2 pad K25: VDD_CORE_A2 -> VDD_HBM_1V1
- U_A2 pad K34: GND -> LINK3_DATA3
- U_A2 pad K35: VDD_CORE_A2 -> LINK3_DATA2
- U_A2 pad K5: VDD_CORE_A2 -> VDD_HBM_1V1
- U_A2 pad L1: GND -> LINK2_DATA4
- U_A2 pad L16: VDD_CORE_A2 -> VDDQ_HBM_0V4
- U_A2 pad L2: VDD_CORE_A2 -> LINK2_DATA5
- U_A2 pad L26: VDD_CORE_A2 -> VDDQ_HBM_0V4
- U_A2 pad L34: VDD_CORE_A2 -> LINK3_DATA5
- U_A2 pad L35: GND -> LINK3_DATA4
- U_A2 pad L6: VDD_CORE_A2 -> VDD_HBM_1V1
- U_A2 pad M1: VDD_CORE_A2 -> LINK2_DATA6
- U_A2 pad M17: VDD_CORE_A2 -> VDDQ_HBM_0V4
- U_A2 pad M2: GND -> LINK2_DATA7
- U_A2 pad M27: VDD_CORE_A2 -> VDDQ_HBM_0V4
- U_A2 pad M34: GND -> LINK3_DATA7
- U_A2 pad M35: VDD_CORE_A2 -> LINK3_DATA6
- U_A2 pad M7: VDD_CORE_A2 -> VDDQ_HBM_0V4
- U_A2 pad N1: GND -> LINK2_DATA8
- U_A2 pad N18: VDD_CORE_A2 -> VDDQ_HBM_0V4
- U_A2 pad N2: VDD_CORE_A2 -> LINK2_DATA9
- U_A2 pad N28: VDD_CORE_A2 -> VDDQ_HBM_0V4
- U_A2 pad N34: VDD_CORE_A2 -> LINK3_DATA9
- U_A2 pad N35: GND -> LINK3_DATA8
- U_A2 pad N8: VDD_CORE_A2 -> VDDQ_HBM_0V4
- U_A2 pad P1: VDD_CORE_A2 -> LINK2_DATA10
- U_A2 pad P19: VDD_CORE_A2 -> VDDQ_HBM_0V4
- U_A2 pad P2: GND -> LINK2_DATA11
- U_A2 pad P29: VDD_CORE_A2 -> VDDQ_HBM_0V4
- U_A2 pad P34: GND -> LINK3_DATA11
- U_A2 pad P35: VDD_CORE_A2 -> LINK3_DATA10
- U_A2 pad P9: VDD_CORE_A2 -> VDDQ_HBM_0V4
- U_A2 pad R1: GND -> LINK2_DATA12
- U_A2 pad R10: VDD_CORE_A2 -> VDDQ_HBM_0V4
- U_A2 pad R2: VDD_CORE_A2 -> LINK2_DATA13
- U_A2 pad R34: VDD_CORE_A2 -> LINK3_DATA13
- U_A2 pad R35: GND -> LINK3_DATA12
- U_A2 pad T1: VDD_CORE_A2 -> LINK2_DATA14
- U_A2 pad T2: GND -> LINK2_DATA15
- U_A2 pad T34: GND -> LINK3_DATA15
- U_A2 pad T35: VDD_CORE_A2 -> LINK3_DATA14
- U_A2 pad U1: GND -> LINK2_DATA16
- U_A2 pad U2: VDD_CORE_A2 -> LINK2_DATA17
- U_A2 pad U34: VDD_CORE_A2 -> LINK3_DATA17
- U_A2 pad U35: GND -> LINK3_DATA16
- U_A2 pad V1: VDD_CORE_A2 -> LINK2_DATA18
- U_A2 pad V2: GND -> LINK2_DATA19
- U_A2 pad V34: GND -> LINK3_DATA19
- U_A2 pad V35: VDD_CORE_A2 -> LINK3_DATA18
- U_A2 pad W1: LINK2_DATA0 -> LINK2_DATA20
- U_A2 pad W2: LINK2_DATA1 -> LINK2_DATA21
- U_A2 pad W34: VDD_CORE_A2 -> LINK3_DATA21
- U_A2 pad W35: GND -> LINK3_DATA20
- U_A2 pad Y1: LINK2_DATA2 -> LINK2_DATA22
- U_A2 pad Y2: LINK2_DATA3 -> LINK2_DATA23
- U_A2 pad Y34: GND -> LINK3_DATA23
- U_A2 pad Y35: VDD_CORE_A2 -> LINK3_DATA22
- U_A3 pad AA1: LINK3_DATA4 -> LINK3_DATA24
- U_A3 pad AA2: LINK3_DATA5 -> LINK3_DATA25
- U_A3 pad AA34: VDD_CORE_A3 -> LINK4_DATA25
- U_A3 pad AA35: GND -> LINK4_DATA24
- U_A3 pad AB1: LINK3_DATA6 -> LINK3_DATA26
- U_A3 pad AB2: LINK3_DATA7 -> LINK3_DATA27
- U_A3 pad AB34: GND -> LINK4_DATA27
- U_A3 pad AB35: VDD_CORE_A3 -> LINK4_DATA26
- U_A3 pad AC1: LINK3_DATA8 -> LINK3_DATA28
- U_A3 pad AC2: LINK3_DATA9 -> LINK3_DATA29
- U_A3 pad AC34: VDD_CORE_A3 -> LINK4_DATA29
- U_A3 pad AC35: GND -> LINK4_DATA28
- U_A3 pad AD1: LINK3_DATA10 -> LINK3_DATA30
- U_A3 pad AD2: LINK3_DATA11 -> LINK3_DATA31
- U_A3 pad AD34: GND -> LINK4_DATA31
- U_A3 pad AD35: VDD_CORE_A3 -> LINK4_DATA30
- U_A3 pad AE1: LINK3_DATA12 -> LINK3_CLOCK
- U_A3 pad AE2: LINK3_DATA13 -> LINK3_VALID
- U_A3 pad AE34: VDD_CORE_A3 -> LINK4_VALID
- U_A3 pad AE35: GND -> LINK4_CLOCK
- U_A3 pad AF1: LINK3_DATA14 -> LINK3_READY_BACK
- U_A3 pad AF2: LINK3_DATA15 -> LINK3_SOF
- U_A3 pad AF34: GND -> LINK4_SOF
- U_A3 pad AF35: VDD_CORE_A3 -> LINK4_READY_BACK
- U_A3 pad AG1: LINK3_DATA16 -> GND
- U_A3 pad AG2: LINK3_DATA17 -> VDD_CORE_A3
- U_A3 pad AH1: LINK3_DATA18 -> VDD_CORE_A3
- U_A3 pad AH2: LINK3_DATA19 -> GND
- U_A3 pad AJ1: LINK3_DATA20 -> GND
- U_A3 pad AJ2: LINK3_DATA21 -> VDD_CORE_A3
- U_A3 pad AK1: LINK3_DATA22 -> VDD_CORE_A3
- U_A3 pad AK2: LINK3_DATA23 -> GND
- U_A3 pad AL1: LINK3_DATA24 -> GND
- U_A3 pad AL2: LINK3_DATA25 -> VDD_CORE_A3
- U_A3 pad AM1: LINK3_DATA26 -> VDD_CORE_A3
- U_A3 pad AM2: LINK3_DATA27 -> GND
- U_A3 pad AN1: LINK3_DATA28 -> GND
- U_A3 pad AN2: LINK3_DATA29 -> VDD_CORE_A3
- U_A3 pad AP1: LINK3_DATA30 -> VDD_CORE_A3
- U_A3 pad AP2: LINK3_DATA31 -> GND
- U_A3 pad AR1: LINK3_CLOCK -> GND
- U_A3 pad AR10: VDD_CORE_A3 -> JTAG_TMS
- U_A3 pad AR11: GND -> JTAG_TDO_A2
- U_A3 pad AR12: VDD_CORE_A3 -> GND
- U_A3 pad AR13: GND -> JTAG_TDO_A3
- U_A3 pad AR14: VDD_CORE_A3 -> JTAG_TRST
- U_A3 pad AR15: GND -> REFCLK_A3_P
- U_A3 pad AR16: VDD_CORE_A3 -> REFCLK_A3_N
- U_A3 pad AR18: VDD_CORE_A3 -> MODE0_A3
- U_A3 pad AR19: GND -> MODE1_A3
- U_A3 pad AR2: LINK3_VALID -> VDD_CORE_A3
- U_A3 pad AR3: GND -> MGMT_SCLK
- U_A3 pad AR4: VDD_CORE_A3 -> MGMT_MOSI
- U_A3 pad AR5: GND -> MGMT_MISO
- U_A3 pad AR6: VDD_CORE_A3 -> MGMT_CS_A3
- U_A3 pad AR8: VDD_CORE_A3 -> MGMT_IRQ_A3
- U_A3 pad AR9: GND -> JTAG_TCK
- U_A3 pad C18: VDD_HBM_1V1 -> VDD_IO_1V8
- U_A3 pad C28: VDD_HBM_1V1 -> VDD_PLL_0V9
- U_A3 pad C8: VDD_HBM_1V1 -> VDD_IO_1V8
- U_A3 pad D9: VDD_HBM_1V1 -> VDD_PLL_0V9
- U_A3 pad G32: VDDQ_HBM_0V4 -> VDD_HBM_1V1
- U_A3 pad H13: VDDQ_HBM_0V4 -> VDD_HBM_1V1
- U_A3 pad H23: VDDQ_HBM_0V4 -> VDD_HBM_1V1
- U_A3 pad H3: VDDQ_HBM_0V4 -> VDD_HBM_1V1
- U_A3 pad H33: VDDQ_HBM_0V4 -> VDD_HBM_1V1
- U_A3 pad J1: GND -> LINK3_DATA0
- U_A3 pad J14: VDDQ_HBM_0V4 -> VDD_HBM_1V1
- U_A3 pad J2: VDD_CORE_A3 -> LINK3_DATA1
- U_A3 pad J24: VDDQ_HBM_0V4 -> VDD_HBM_1V1
- U_A3 pad J34: VDD_CORE_A3 -> LINK4_DATA1
- U_A3 pad J35: GND -> LINK4_DATA0
- U_A3 pad J4: VDDQ_HBM_0V4 -> VDD_HBM_1V1
- U_A3 pad K1: VDD_CORE_A3 -> LINK3_DATA2
- U_A3 pad K15: VDD_CORE_A3 -> VDD_HBM_1V1
- U_A3 pad K2: GND -> LINK3_DATA3
- U_A3 pad K25: VDD_CORE_A3 -> VDD_HBM_1V1
- U_A3 pad K34: GND -> LINK4_DATA3
- U_A3 pad K35: VDD_CORE_A3 -> LINK4_DATA2
- U_A3 pad K5: VDD_CORE_A3 -> VDD_HBM_1V1
- U_A3 pad L1: GND -> LINK3_DATA4
- U_A3 pad L16: VDD_CORE_A3 -> VDDQ_HBM_0V4
- U_A3 pad L2: VDD_CORE_A3 -> LINK3_DATA5
- U_A3 pad L26: VDD_CORE_A3 -> VDDQ_HBM_0V4
- U_A3 pad L34: VDD_CORE_A3 -> LINK4_DATA5
- U_A3 pad L35: GND -> LINK4_DATA4
- U_A3 pad L6: VDD_CORE_A3 -> VDD_HBM_1V1
- U_A3 pad M1: VDD_CORE_A3 -> LINK3_DATA6
- U_A3 pad M17: VDD_CORE_A3 -> VDDQ_HBM_0V4
- U_A3 pad M2: GND -> LINK3_DATA7
- U_A3 pad M27: VDD_CORE_A3 -> VDDQ_HBM_0V4
- U_A3 pad M34: GND -> LINK4_DATA7
- U_A3 pad M35: VDD_CORE_A3 -> LINK4_DATA6
- U_A3 pad M7: VDD_CORE_A3 -> VDDQ_HBM_0V4
- U_A3 pad N1: GND -> LINK3_DATA8
- U_A3 pad N18: VDD_CORE_A3 -> VDDQ_HBM_0V4
- U_A3 pad N2: VDD_CORE_A3 -> LINK3_DATA9
- U_A3 pad N28: VDD_CORE_A3 -> VDDQ_HBM_0V4
- U_A3 pad N34: VDD_CORE_A3 -> LINK4_DATA9
- U_A3 pad N35: GND -> LINK4_DATA8
- U_A3 pad N8: VDD_CORE_A3 -> VDDQ_HBM_0V4
- U_A3 pad P1: VDD_CORE_A3 -> LINK3_DATA10
- U_A3 pad P19: VDD_CORE_A3 -> VDDQ_HBM_0V4
- U_A3 pad P2: GND -> LINK3_DATA11
- U_A3 pad P29: VDD_CORE_A3 -> VDDQ_HBM_0V4
- U_A3 pad P34: GND -> LINK4_DATA11
- U_A3 pad P35: VDD_CORE_A3 -> LINK4_DATA10
- U_A3 pad P9: VDD_CORE_A3 -> VDDQ_HBM_0V4
- U_A3 pad R1: GND -> LINK3_DATA12
- U_A3 pad R10: VDD_CORE_A3 -> VDDQ_HBM_0V4
- U_A3 pad R2: VDD_CORE_A3 -> LINK3_DATA13
- U_A3 pad R34: VDD_CORE_A3 -> LINK4_DATA13
- U_A3 pad R35: GND -> LINK4_DATA12
- U_A3 pad T1: VDD_CORE_A3 -> LINK3_DATA14
- U_A3 pad T2: GND -> LINK3_DATA15
- U_A3 pad T34: GND -> LINK4_DATA15
- U_A3 pad T35: VDD_CORE_A3 -> LINK4_DATA14
- U_A3 pad U1: GND -> LINK3_DATA16
- U_A3 pad U2: VDD_CORE_A3 -> LINK3_DATA17
- U_A3 pad U34: VDD_CORE_A3 -> LINK4_DATA17
- U_A3 pad U35: GND -> LINK4_DATA16
- U_A3 pad V1: VDD_CORE_A3 -> LINK3_DATA18
- U_A3 pad V2: GND -> LINK3_DATA19
- U_A3 pad V34: GND -> LINK4_DATA19
- U_A3 pad V35: VDD_CORE_A3 -> LINK4_DATA18
- U_A3 pad W1: LINK3_DATA0 -> LINK3_DATA20
- U_A3 pad W2: LINK3_DATA1 -> LINK3_DATA21
- U_A3 pad W34: VDD_CORE_A3 -> LINK4_DATA21
- U_A3 pad W35: GND -> LINK4_DATA20
- U_A3 pad Y1: LINK3_DATA2 -> LINK3_DATA22
- U_A3 pad Y2: LINK3_DATA3 -> LINK3_DATA23
- U_A3 pad Y34: GND -> LINK4_DATA23
- U_A3 pad Y35: VDD_CORE_A3 -> LINK4_DATA22
- U_CLK pad 13: REFCLK_H0_P -> REFCLK_A4_P
- U_CLK pad 14: REFCLK_H0_N -> REFCLK_A4_N
- U_FPGA pad AA1: LINK5_CLOCK -> LINK10_CLOCK
- U_FPGA pad AA2: LINK5_VALID -> LINK10_VALID
- U_FPGA pad AB1: LINK5_READY_BACK -> LINK10_READY_BACK
- U_FPGA pad AB2: LINK5_SOF -> LINK10_SOF
- U_FPGA pad AC12: MGMT_CS_H0 -> MGMT_CS_A4
- U_FPGA pad AC13: MGMT_IRQ_H0 -> MGMT_IRQ_A4
- U_FPGA pad AC14: JTAG_TCK -> MGMT_CS_A5
- U_FPGA pad AC15: JTAG_TMS -> MGMT_IRQ_A5
- U_FPGA pad AC16: JTAG_TDI_FPGA -> MGMT_CS_A6
- U_FPGA pad AC17: JTAG_TDO_FPGA -> MGMT_IRQ_A6
- U_FPGA pad AC18: JTAG_TRST -> MGMT_CS_A7
- U_FPGA pad AC19: REFCLK_FPGA_P -> MGMT_IRQ_A7
- U_FPGA pad AC20: REFCLK_FPGA_N -> MGMT_CS_H0
- U_FPGA pad AC21: SFP_TX_P -> MGMT_IRQ_H0
- U_FPGA pad AC22: SFP_TX_N -> MGMT_CS_H1
- U_FPGA pad AC23: SFP_RX_P -> MGMT_IRQ_H1
- U_FPGA pad AC24: SFP_RX_N -> JTAG_TCK
- U_FPGA pad AD1: SFP_I2C0 -> JTAG_TMS
- U_FPGA pad AD10: QSPI3 -> SFP_RX_N
- U_FPGA pad AD11: QSPI4 -> SFP_I2C0
- U_FPGA pad AD12: QSPI5 -> SFP_I2C1
- U_FPGA pad AD13: UART_TX -> SFP_CTRL0
- U_FPGA pad AD14: UART_RX -> SFP_CTRL1
- U_FPGA pad AD15: VCCINT_0V85 -> SFP_CTRL2
- U_FPGA pad AD16: GND -> SFP_CTRL3
- U_FPGA pad AD17: VCCINT_0V85 -> QSPI0
- U_FPGA pad AD18: GND -> QSPI1
- U_FPGA pad AD19: VCCINT_0V85 -> QSPI2
- U_FPGA pad AD2: SFP_I2C1 -> JTAG_TDI_FPGA
- U_FPGA pad AD20: GND -> QSPI3
- U_FPGA pad AD21: VCCINT_0V85 -> QSPI4
- U_FPGA pad AD22: GND -> QSPI5
- U_FPGA pad AD23: VCCINT_0V85 -> UART_TX
- U_FPGA pad AD24: GND -> UART_RX
- U_FPGA pad AD3: SFP_CTRL0 -> JTAG_TDO_FPGA
- U_FPGA pad AD4: SFP_CTRL1 -> JTAG_TRST
- U_FPGA pad AD5: SFP_CTRL2 -> REFCLK_FPGA_P
- U_FPGA pad AD6: SFP_CTRL3 -> REFCLK_FPGA_N
- U_FPGA pad AD7: QSPI0 -> SFP_TX_P
- U_FPGA pad AD8: QSPI1 -> SFP_TX_N
- U_FPGA pad AD9: QSPI2 -> SFP_RX_P
- U_FPGA pad E1: LINK5_DATA0 -> LINK10_DATA0
- U_FPGA pad E2: LINK5_DATA1 -> LINK10_DATA1
- U_FPGA pad F1: LINK5_DATA2 -> LINK10_DATA2
- U_FPGA pad F2: LINK5_DATA3 -> LINK10_DATA3
- U_FPGA pad G1: LINK5_DATA4 -> LINK10_DATA4
- U_FPGA pad G2: LINK5_DATA5 -> LINK10_DATA5
- U_FPGA pad H1: LINK5_DATA6 -> LINK10_DATA6
- U_FPGA pad H2: LINK5_DATA7 -> LINK10_DATA7
- U_FPGA pad J1: LINK5_DATA8 -> LINK10_DATA8
- U_FPGA pad J2: LINK5_DATA9 -> LINK10_DATA9
- U_FPGA pad K1: LINK5_DATA10 -> LINK10_DATA10
- U_FPGA pad K2: LINK5_DATA11 -> LINK10_DATA11
- U_FPGA pad L1: LINK5_DATA12 -> LINK10_DATA12
- U_FPGA pad L2: LINK5_DATA13 -> LINK10_DATA13
- U_FPGA pad M1: LINK5_DATA14 -> LINK10_DATA14
- U_FPGA pad M2: LINK5_DATA15 -> LINK10_DATA15
- U_FPGA pad N1: LINK5_DATA16 -> LINK10_DATA16
- U_FPGA pad N2: LINK5_DATA17 -> LINK10_DATA17
- U_FPGA pad P1: LINK5_DATA18 -> LINK10_DATA18
- U_FPGA pad P2: LINK5_DATA19 -> LINK10_DATA19
- U_FPGA pad R1: LINK5_DATA20 -> LINK10_DATA20
- U_FPGA pad R2: LINK5_DATA21 -> LINK10_DATA21
- U_FPGA pad T1: LINK5_DATA22 -> LINK10_DATA22
- U_FPGA pad T2: LINK5_DATA23 -> LINK10_DATA23
- U_FPGA pad U1: LINK5_DATA24 -> LINK10_DATA24
- U_FPGA pad U2: LINK5_DATA25 -> LINK10_DATA25
- U_FPGA pad V1: LINK5_DATA26 -> LINK10_DATA26
- U_FPGA pad V2: LINK5_DATA27 -> LINK10_DATA27
- U_FPGA pad W1: LINK5_DATA28 -> LINK10_DATA28
- U_FPGA pad W2: LINK5_DATA29 -> LINK10_DATA29
- U_FPGA pad Y1: LINK5_DATA30 -> LINK10_DATA30
- U_FPGA pad Y2: LINK5_DATA31 -> LINK10_DATA31
- U_H0 pad AA1: LINK4_DATA4 -> LINK8_DATA24
- U_H0 pad AA2: LINK4_DATA5 -> LINK8_DATA25
- U_H0 pad AA34: VDD_CORE_H0 -> LINK9_DATA25
- U_H0 pad AA35: GND -> LINK9_DATA24
- U_H0 pad AB1: LINK4_DATA6 -> LINK8_DATA26
- U_H0 pad AB2: LINK4_DATA7 -> LINK8_DATA27
- U_H0 pad AB34: GND -> LINK9_DATA27
- U_H0 pad AB35: VDD_CORE_H0 -> LINK9_DATA26
- U_H0 pad AC1: LINK4_DATA8 -> LINK8_DATA28
- U_H0 pad AC2: LINK4_DATA9 -> LINK8_DATA29
- U_H0 pad AC34: VDD_CORE_H0 -> LINK9_DATA29
- U_H0 pad AC35: GND -> LINK9_DATA28
- U_H0 pad AD1: LINK4_DATA10 -> LINK8_DATA30
- U_H0 pad AD2: LINK4_DATA11 -> LINK8_DATA31
- U_H0 pad AD34: GND -> LINK9_DATA31
- U_H0 pad AD35: VDD_CORE_H0 -> LINK9_DATA30
- U_H0 pad AE1: LINK4_DATA12 -> LINK8_CLOCK
- U_H0 pad AE2: LINK4_DATA13 -> LINK8_VALID
- U_H0 pad AE34: VDD_CORE_H0 -> LINK9_VALID
- U_H0 pad AE35: GND -> LINK9_CLOCK
- U_H0 pad AF1: LINK4_DATA14 -> LINK8_READY_BACK
- U_H0 pad AF2: LINK4_DATA15 -> LINK8_SOF
- U_H0 pad AF34: GND -> LINK9_SOF
- U_H0 pad AF35: VDD_CORE_H0 -> LINK9_READY_BACK
- U_H0 pad AG1: LINK4_DATA16 -> GND
- U_H0 pad AG2: LINK4_DATA17 -> VDD_CORE_H0
- U_H0 pad AH1: LINK4_DATA18 -> VDD_CORE_H0
- U_H0 pad AH2: LINK4_DATA19 -> GND
- U_H0 pad AJ1: LINK4_DATA20 -> GND
- U_H0 pad AJ2: LINK4_DATA21 -> VDD_CORE_H0
- U_H0 pad AK1: LINK4_DATA22 -> VDD_CORE_H0
- U_H0 pad AK2: LINK4_DATA23 -> GND
- U_H0 pad AL1: LINK4_DATA24 -> GND
- U_H0 pad AL2: LINK4_DATA25 -> VDD_CORE_H0
- U_H0 pad AM1: LINK4_DATA26 -> VDD_CORE_H0
- U_H0 pad AM2: LINK4_DATA27 -> GND
- U_H0 pad AN1: LINK4_DATA28 -> GND
- U_H0 pad AN2: LINK4_DATA29 -> VDD_CORE_H0
- U_H0 pad AP1: LINK4_DATA30 -> VDD_CORE_H0
- U_H0 pad AP2: LINK4_DATA31 -> GND
- U_H0 pad AR1: LINK4_CLOCK -> GND
- U_H0 pad AR10: VDD_CORE_H0 -> JTAG_TMS
- U_H0 pad AR11: GND -> JTAG_TDO_A7
- U_H0 pad AR12: VDD_CORE_H0 -> GND
- U_H0 pad AR13: GND -> JTAG_TDO_H0
- U_H0 pad AR14: VDD_CORE_H0 -> JTAG_TRST
- U_H0 pad AR15: GND -> REFCLK_H0_P
- U_H0 pad AR16: VDD_CORE_H0 -> REFCLK_H0_N
- U_H0 pad AR18: VDD_CORE_H0 -> MODE0_H0
- U_H0 pad AR19: GND -> MODE1_H0
- U_H0 pad AR2: LINK4_VALID -> VDD_CORE_H0
- U_H0 pad AR3: GND -> MGMT_SCLK
- U_H0 pad AR4: VDD_CORE_H0 -> MGMT_MOSI
- U_H0 pad AR5: GND -> MGMT_MISO
- U_H0 pad AR6: VDD_CORE_H0 -> MGMT_CS_H0
- U_H0 pad AR8: VDD_CORE_H0 -> MGMT_IRQ_H0
- U_H0 pad AR9: GND -> JTAG_TCK
- U_H0 pad C18: (no net) -> VDD_IO_1V8
- U_H0 pad C28: (no net) -> VDD_PLL_0V9
- U_H0 pad C8: (no net) -> VDD_IO_1V8
- U_H0 pad D9: (no net) -> VDD_PLL_0V9
- U_H0 pad J1: GND -> LINK8_DATA0
- U_H0 pad J2: VDD_CORE_H0 -> LINK8_DATA1
- U_H0 pad J34: VDD_CORE_H0 -> LINK9_DATA1
- U_H0 pad J35: GND -> LINK9_DATA0
- U_H0 pad K1: VDD_CORE_H0 -> LINK8_DATA2
- U_H0 pad K15: VDD_CORE_H0 -> (no net)
- U_H0 pad K2: GND -> LINK8_DATA3
- U_H0 pad K25: VDD_CORE_H0 -> (no net)
- U_H0 pad K34: GND -> LINK9_DATA3
- U_H0 pad K35: VDD_CORE_H0 -> LINK9_DATA2
- U_H0 pad K5: VDD_CORE_H0 -> (no net)
- U_H0 pad L1: GND -> LINK8_DATA4
- U_H0 pad L16: VDD_CORE_H0 -> (no net)
- U_H0 pad L2: VDD_CORE_H0 -> LINK8_DATA5
- U_H0 pad L26: VDD_CORE_H0 -> (no net)
- U_H0 pad L34: VDD_CORE_H0 -> LINK9_DATA5
- U_H0 pad L35: GND -> LINK9_DATA4
- U_H0 pad L6: VDD_CORE_H0 -> (no net)
- U_H0 pad M1: VDD_CORE_H0 -> LINK8_DATA6
- U_H0 pad M17: VDD_CORE_H0 -> (no net)
- U_H0 pad M2: GND -> LINK8_DATA7
- U_H0 pad M27: VDD_CORE_H0 -> (no net)
- U_H0 pad M34: GND -> LINK9_DATA7
- U_H0 pad M35: VDD_CORE_H0 -> LINK9_DATA6
- U_H0 pad M7: VDD_CORE_H0 -> (no net)
- U_H0 pad N1: GND -> LINK8_DATA8
- U_H0 pad N18: VDD_CORE_H0 -> (no net)
- U_H0 pad N2: VDD_CORE_H0 -> LINK8_DATA9
- U_H0 pad N28: VDD_CORE_H0 -> (no net)
- U_H0 pad N34: VDD_CORE_H0 -> LINK9_DATA9
- U_H0 pad N35: GND -> LINK9_DATA8
- U_H0 pad N8: VDD_CORE_H0 -> (no net)
- U_H0 pad P1: VDD_CORE_H0 -> LINK8_DATA10
- U_H0 pad P19: VDD_CORE_H0 -> (no net)
- U_H0 pad P2: GND -> LINK8_DATA11
- U_H0 pad P29: VDD_CORE_H0 -> (no net)
- U_H0 pad P34: GND -> LINK9_DATA11
- U_H0 pad P35: VDD_CORE_H0 -> LINK9_DATA10
- U_H0 pad P9: VDD_CORE_H0 -> (no net)
- U_H0 pad R1: GND -> LINK8_DATA12
- U_H0 pad R10: VDD_CORE_H0 -> (no net)
- U_H0 pad R2: VDD_CORE_H0 -> LINK8_DATA13
- U_H0 pad R34: VDD_CORE_H0 -> LINK9_DATA13
- U_H0 pad R35: GND -> LINK9_DATA12
- U_H0 pad T1: VDD_CORE_H0 -> LINK8_DATA14
- U_H0 pad T2: GND -> LINK8_DATA15
- U_H0 pad T34: GND -> LINK9_DATA15
- U_H0 pad T35: VDD_CORE_H0 -> LINK9_DATA14
- U_H0 pad U1: GND -> LINK8_DATA16
- U_H0 pad U2: VDD_CORE_H0 -> LINK8_DATA17
- U_H0 pad U34: VDD_CORE_H0 -> LINK9_DATA17
- U_H0 pad U35: GND -> LINK9_DATA16
- U_H0 pad V1: VDD_CORE_H0 -> LINK8_DATA18
- U_H0 pad V2: GND -> LINK8_DATA19
- U_H0 pad V34: GND -> LINK9_DATA19
- U_H0 pad V35: VDD_CORE_H0 -> LINK9_DATA18
- U_H0 pad W1: LINK4_DATA0 -> LINK8_DATA20
- U_H0 pad W2: LINK4_DATA1 -> LINK8_DATA21
- U_H0 pad W34: VDD_CORE_H0 -> LINK9_DATA21
- U_H0 pad W35: GND -> LINK9_DATA20
- U_H0 pad Y1: LINK4_DATA2 -> LINK8_DATA22
- U_H0 pad Y2: LINK4_DATA3 -> LINK8_DATA23
- U_H0 pad Y34: GND -> LINK9_DATA23
- U_H0 pad Y35: VDD_CORE_H0 -> LINK9_DATA22
Routing:
- net LINK5_DATA1: track 66.2 -> 31.9 mm
- net LINK5_DATA3: track 65.1 -> 31.4 mm
- net LINK5_DATA0: track 63.2 -> 29.7 mm
- net LINK10_DATA1: track 0.00 -> 33.4 mm, vias 0 -> 2
- net LINK5_DATA5: track 64.0 -> 30.9 mm
- net LINK5_DATA2: track 62.2 -> 29.2 mm
- net LINK0_DATA1: track 66.2 -> 33.4 mm
- net LINK10_DATA3: track 0.00 -> 32.8 mm, vias 0 -> 2
- net LINK5_DATA7: track 63.0 -> 30.5 mm
- net LINK10_DATA5: track 0.00 -> 32.3 mm, vias 0 -> 2
- net LINK0_DATA0: track 63.2 -> 30.9 mm
- net LINK5_DATA4: track 61.1 -> 28.8 mm
- net LINK0_DATA3: track 65.1 -> 32.8 mm
- net LINK8_DATA1: track 0.00 -> 31.9 mm, vias 0 -> 2
- net LINK7_DATA1: track 0.00 -> 31.9 mm, vias 0 -> 2
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- added copper zone on In8.Cu, net VDD_CORE_A4
- added copper zone on In8.Cu, net VDD_CORE_A5
- added copper zone on In8.Cu, net VDD_CORE_A6
- added copper zone on In8.Cu, net VDD_CORE_A7
- added copper zone on In8.Cu, net VDD_CORE_H1
Other:
- board text added: "appliance: 1U rack chassis, single board, host-attached, floorplan generated from hw/board_27b.yaml"
- board text removed: "appliance: 1U rack chassis, single board, host-attached, floorplan generated from hw/board.yaml"
