File: hw/kicad_27b/asics.kicad_sch (KiCad schematic)
At the start: 5 parts

Commit message: Pipeline a layer's passes, and re-rate the 27B board to eight layer dies
Two things the last commit left open.

The simulator now separates a layer stage's latency from its initiation
interval.  A layer is a chain of passes and each pass has its own via-
programmed tiles, so nothing is reused between them: the first pass is free
the moment its token moves on, and the stage holds as many tokens as fit
between its latency and its interval.  layer_pass_cycles carries the pass,
a quarter of the layer in every shipped geometry, which is the same figure
the single-pass head die already used.

I expected that to be worth four times and it is worth almost nothing,
because after the memory corrections it is the memory and not the pass rate
that binds.  It is exactly neutral on every LPDDR5X and PSRAM configuration
at any context count, worth 4 to 8 percent on the 9B with HBM, and slightly
negative on the 27B, where more tokens per stage lengthen latency against a
fixed pool of contexts.  With the bandwidth raised tenfold it is worth 2.5
times, 240K to 597K tokens/s, so the lever is real and nothing in reach of
this design is close enough to the fabric to collect it.  Letting a token's
state write overlap the next token's state read, which the same change
allows, is what does move the HBM numbers: the 3 nm 9B goes from 190K to
244K.

The 27B board is now eight layer ASICs of eight layers and two head ASICs
splitting the LM head, at 153K tokens/s rather than the 234K that came from
the un-corrected model.  Halving the per-die load takes the core rail from
650 A to 249 A, the package from a 55 x 55 array to 35 x 35, the cold plate
from 525 W to 200 W, and puts the ring on the same 11-gon as the 9B board.
hw/README's open item is replaced by the re-rating itself.

The 9B board's design point follows the same correction, 14.5K to 8.2K, and
its per-die traffic is 7.35 MB per token rather than the 4.2 MB of retrieval
alone.  Generated files now name the board description they came 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
Parts:
- added U_A4, U_A5, U_A6, U_A7: layer_asic, appliance:FCBGA1225_35x35_P0.8, symbol appliance:layer_asic
- added U_H1: head_asic, appliance:FCBGA1225_35x35_P0.8, symbol appliance:head_asic
- U_A0, U_A1, U_A2, U_A3, U_H0: footprint appliance:FCBGA3025_55x55_P1.0 -> appliance:FCBGA1225_35x35_P0.8
Connections:
- net GND: now also U_A0.AG1, U_A0.AH2, U_A0.AJ1, U_A0.AK2, U_A0.AL1, U_A0.AM2, U_A0.AN1, U_A0.AP2, U_A0.AR1, U_A0.AR12, U_A1.AG1, U_A1.AH2, U_A1.AJ1, U_A1.AK2, U_A1.AL1, U_A1.AM2, U_A1.AN1, U_A1.AP2, U_A1.AR1, U_A1.AR12, U_A2.AG1, U_A2.AH2, U_A2.AJ1, U_A2.AK2, U_A2.AL1, U_A2.AM2, U_A2.AN1, U_A2.AP2, U_A2.AR1, U_A2.AR12, U_A3.AG1, U_A3.AH2, U_A3.AJ1, U_A3.AK2, U_A3.AL1, U_A3.AM2, U_A3.AN1, U_A3.AP2, U_A3.AR1, U_A3.AR12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; no longer U_A0.A37, U_A0.A39, U_A0.A41, U_A0.A43, U_A0.A45, U_A0.A47, U_A0.A49, U_A0.A51, U_A0.A53, U_A0.A55, U_A0.AA35, U_A0.AA37, U_A0.AA39, U_A0.AA41, U_A0.AA43, U_A0.AA45, U_A0.AA47, U_A0.AA49, U_A0.AA51, U_A0.AA53, U_A0.AB34, U_A0.AB36, U_A0.AB38, U_A0.AB40, U_A0.AB42, U_A0.AB44, U_A0.AB46, U_A0.AB48, U_A0.AB50, U_A0.AB52, U_A0.AC35, U_A0.AC37, U_A0.AC39, U_A0.AC41, U_A0.AC43, U_A0.AC45, U_A0.AC47, U_A0.AC49, U_A0.AC51, U_A0.AC53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
- net JTAG_TCK: now also U_A0.AR9, U_A1.AR9, U_A2.AR9, U_A3.AR9, U_H0.AR9, U_A4.AR9, U_A5.AR9, U_A6.AR9, U_A7.AR9, U_H1.AR9; no longer U_A0.BR9, U_A1.BR9, U_A2.BR9, U_A3.BR9, U_H0.BR9
- net JTAG_TDO_A0: now also U_A0.AR13, U_A1.AR11; no longer U_A0.BR13, U_A1.BR11
- net JTAG_TDO_A1: now also U_A1.AR13, U_A2.AR11; no longer U_A1.BR13, U_A2.BR11
- net JTAG_TDO_A2: now also U_A2.AR13, U_A3.AR11; no longer U_A2.BR13, U_A3.BR11
- net JTAG_TDO_A3: now also U_A3.AR13, U_A4.AR11; no longer U_A3.BR13, U_H0.BR11
- net JTAG_TDO_FPGA: now also U_A0.AR11; no longer U_A0.BR11
- net JTAG_TDO_H0: now also U_H0.AR13, U_H1.AR11; no longer U_H0.BR13
- net JTAG_TMS: now also U_A0.AR10, U_A1.AR10, U_A2.AR10, U_A3.AR10, U_H0.AR10, U_A4.AR10, U_A5.AR10, U_A6.AR10, U_A7.AR10, U_H1.AR10; no longer U_A0.BR10, U_A1.BR10, U_A2.BR10, U_A3.BR10, U_H0.BR10
- net JTAG_TRST: now also U_A0.AR14, U_A1.AR14, U_A2.AR14, U_A3.AR14, U_H0.AR14, U_A4.AR14, U_A5.AR14, U_A6.AR14, U_A7.AR14, U_H1.AR14; no longer U_A0.BR14, U_A1.BR14, U_A2.BR14, U_A3.BR14, U_H0.BR14
- net LINK0_CLOCK: now also U_A0.AE1; no longer U_A0.AR1
- net LINK0_DATA0: now also U_A0.J1; no longer U_A0.W1
- net LINK0_DATA1: now also U_A0.J2; no longer U_A0.W2
- net LINK0_DATA10: now also U_A0.P1; no longer U_A0.AD1
- net LINK0_DATA11: now also U_A0.P2; no longer U_A0.AD2
- net LINK0_DATA12: now also U_A0.R1; no longer U_A0.AE1
- net LINK0_DATA13: now also U_A0.R2; no longer U_A0.AE2
- net LINK0_DATA14: now also U_A0.T1; no longer U_A0.AF1
- net LINK0_DATA15: now also U_A0.T2; no longer U_A0.AF2
- net LINK0_DATA16: now also U_A0.U1; no longer U_A0.AG1
- net LINK0_DATA17: now also U_A0.U2; no longer U_A0.AG2
- net LINK0_DATA18: now also U_A0.V1; no longer U_A0.AH1
- net LINK0_DATA19: now also U_A0.V2; no longer U_A0.AH2
- net LINK0_DATA2: now also U_A0.K1; no longer U_A0.Y1
- net LINK0_DATA20: now also U_A0.W1; no longer U_A0.AJ1
- net LINK0_DATA21: now also U_A0.W2; no longer U_A0.AJ2
- net LINK0_DATA22: now also U_A0.Y1; no longer U_A0.AK1
- net LINK0_DATA23: now also U_A0.Y2; no longer U_A0.AK2
- net LINK0_DATA24: now also U_A0.AA1; no longer U_A0.AL1
- net LINK0_DATA25: now also U_A0.AA2; no longer U_A0.AL2
- net LINK0_DATA26: now also U_A0.AB1; no longer U_A0.AM1
- net LINK0_DATA27: now also U_A0.AB2; no longer U_A0.AM2
- net LINK0_DATA28: now also U_A0.AC1; no longer U_A0.AN1
- net LINK0_DATA29: now also U_A0.AC2; no longer U_A0.AN2
- net LINK0_DATA3: now also U_A0.K2; no longer U_A0.Y2
- net LINK0_DATA30: now also U_A0.AD1; no longer U_A0.AP1
- net LINK0_DATA31: now also U_A0.AD2; no longer U_A0.AP2
- net LINK0_DATA4: now also U_A0.L1; no longer U_A0.AA1
- net LINK0_DATA5: now also U_A0.L2; no longer U_A0.AA2
- net LINK0_DATA6: now also U_A0.M1; no longer U_A0.AB1
- net LINK0_DATA7: now also U_A0.M2; no longer U_A0.AB2
- net LINK0_DATA8: now also U_A0.N1; no longer U_A0.AC1
- net LINK0_DATA9: now also U_A0.N2; no longer U_A0.AC2
- net LINK0_READY_BACK: now also U_A0.AF1; no longer U_A0.AT1
- net LINK0_SOF: now also U_A0.AF2; no longer U_A0.AT2
- net LINK0_VALID: now also U_A0.AE2; no longer U_A0.AR2
- net LINK1_CLOCK: now also U_A0.AE35, U_A1.AE1; no longer U_A0.AR55, U_A1.AR1
- net LINK1_DATA0: now also U_A0.J35, U_A1.J1; no longer U_A0.W55, U_A1.W1
- net LINK1_DATA1: now also U_A0.J34, U_A1.J2; no longer U_A0.W54, U_A1.W2
- net LINK1_DATA10: now also U_A0.P35, U_A1.P1; no longer U_A0.AD55, U_A1.AD1
- net LINK1_DATA11: now also U_A0.P34, U_A1.P2; no longer U_A0.AD54, U_A1.AD2
- net LINK1_DATA12: now also U_A0.R35, U_A1.R1; no longer U_A0.AE55, U_A1.AE1
- net LINK1_DATA13: now also U_A0.R34, U_A1.R2; no longer U_A0.AE54, U_A1.AE2
- net LINK1_DATA14: now also U_A0.T35, U_A1.T1; no longer U_A0.AF55, U_A1.AF1
- net LINK1_DATA15: now also U_A0.T34, U_A1.T2; no longer U_A0.AF54, U_A1.AF2
- net LINK1_DATA16: now also U_A0.U35, U_A1.U1; no longer U_A0.AG55, U_A1.AG1
- net LINK1_DATA17: now also U_A0.U34, U_A1.U2; no longer U_A0.AG54, U_A1.AG2
- net LINK1_DATA18: now also U_A0.V35, U_A1.V1; no longer U_A0.AH55, U_A1.AH1
- net LINK1_DATA19: now also U_A0.V34, U_A1.V2; no longer U_A0.AH54, U_A1.AH2
- net LINK1_DATA2: now also U_A0.K35, U_A1.K1; no longer U_A0.Y55, U_A1.Y1
- net LINK1_DATA20: now also U_A0.W35, U_A1.W1; no longer U_A0.AJ55, U_A1.AJ1
- net LINK1_DATA21: now also U_A0.W34, U_A1.W2; no longer U_A0.AJ54, U_A1.AJ2
- net LINK1_DATA22: now also U_A0.Y35, U_A1.Y1; no longer U_A0.AK55, U_A1.AK1
- net LINK1_DATA23: now also U_A0.Y34, U_A1.Y2; no longer U_A0.AK54, U_A1.AK2
- net LINK1_DATA24: now also U_A0.AA35, U_A1.AA1; no longer U_A0.AL55, U_A1.AL1
- net LINK1_DATA25: now also U_A0.AA34, U_A1.AA2; no longer U_A0.AL54, U_A1.AL2
- net LINK1_DATA26: now also U_A0.AB35, U_A1.AB1; no longer U_A0.AM55, U_A1.AM1
- net LINK1_DATA27: now also U_A0.AB34, U_A1.AB2; no longer U_A0.AM54, U_A1.AM2
- net LINK1_DATA28: now also U_A0.AC35, U_A1.AC1; no longer U_A0.AN55, U_A1.AN1
- net LINK1_DATA29: now also U_A0.AC34, U_A1.AC2; no longer U_A0.AN54, U_A1.AN2
- net LINK1_DATA3: now also U_A0.K34, U_A1.K2; no longer U_A0.Y54, U_A1.Y2
- net LINK1_DATA30: now also U_A0.AD35, U_A1.AD1; no longer U_A0.AP55, U_A1.AP1
- net LINK1_DATA31: now also U_A0.AD34, U_A1.AD2; no longer U_A0.AP54, U_A1.AP2
- net LINK1_DATA4: now also U_A0.L35, U_A1.L1; no longer U_A0.AA55, U_A1.AA1
- net LINK1_DATA5: now also U_A0.L34, U_A1.L2; no longer U_A0.AA54, U_A1.AA2
- net LINK1_DATA6: now also U_A0.M35, U_A1.M1; no longer U_A0.AB55, U_A1.AB1
- net LINK1_DATA7: now also U_A0.M34, U_A1.M2; no longer U_A0.AB54, U_A1.AB2
- net LINK1_DATA8: now also U_A0.N35, U_A1.N1; no longer U_A0.AC55, U_A1.AC1
- net LINK1_DATA9: now also U_A0.N34, U_A1.N2; no longer U_A0.AC54, U_A1.AC2
- net LINK1_READY_BACK: now also U_A0.AF35, U_A1.AF1; no longer U_A0.AT55, U_A1.AT1
- net LINK1_SOF: now also U_A0.AF34, U_A1.AF2; no longer U_A0.AT54, U_A1.AT2
- net LINK1_VALID: now also U_A0.AE34, U_A1.AE2; no longer U_A0.AR54, U_A1.AR2
- net LINK2_CLOCK: now also U_A1.AE35, U_A2.AE1; no longer U_A1.AR55, U_A2.AR1
- net LINK2_DATA0: now also U_A1.J35, U_A2.J1; no longer U_A1.W55, U_A2.W1
- net LINK2_DATA1: now also U_A1.J34, U_A2.J2; no longer U_A1.W54, U_A2.W2
- net LINK2_DATA10: now also U_A1.P35, U_A2.P1; no longer U_A1.AD55, U_A2.AD1
- net LINK2_DATA11: now also U_A1.P34, U_A2.P2; no longer U_A1.AD54, U_A2.AD2
- net LINK2_DATA12: now also U_A1.R35, U_A2.R1; no longer U_A1.AE55, U_A2.AE1
- net LINK2_DATA13: now also U_A1.R34, U_A2.R2; no longer U_A1.AE54, U_A2.AE2
- net LINK2_DATA14: now also U_A1.T35, U_A2.T1; no longer U_A1.AF55, U_A2.AF1
- net LINK2_DATA15: now also U_A1.T34, U_A2.T2; no longer U_A1.AF54, U_A2.AF2
- net LINK2_DATA16: now also U_A1.U35, U_A2.U1; no longer U_A1.AG55, U_A2.AG1
- net LINK2_DATA17: now also U_A1.U34, U_A2.U2; no longer U_A1.AG54, U_A2.AG2
- net LINK2_DATA18: now also U_A1.V35, U_A2.V1; no longer U_A1.AH55, U_A2.AH1
- net LINK2_DATA19: now also U_A1.V34, U_A2.V2; no longer U_A1.AH54, U_A2.AH2
- net LINK2_DATA2: now also U_A1.K35, U_A2.K1; no longer U_A1.Y55, U_A2.Y1
- net LINK2_DATA20: now also U_A1.W35, U_A2.W1; no longer U_A1.AJ55, U_A2.AJ1
- net LINK2_DATA21: now also U_A1.W34, U_A2.W2; no longer U_A1.AJ54, U_A2.AJ2
- net LINK2_DATA22: now also U_A1.Y35, U_A2.Y1; no longer U_A1.AK55, U_A2.AK1
- net LINK2_DATA23: now also U_A1.Y34, U_A2.Y2; no longer U_A1.AK54, U_A2.AK2
- net LINK2_DATA24: now also U_A1.AA35, U_A2.AA1; no longer U_A1.AL55, U_A2.AL1
- net LINK2_DATA25: now also U_A1.AA34, U_A2.AA2; no longer U_A1.AL54, U_A2.AL2
- net LINK2_DATA26: now also U_A1.AB35, U_A2.AB1; no longer U_A1.AM55, U_A2.AM1
- net LINK2_DATA27: now also U_A1.AB34, U_A2.AB2; no longer U_A1.AM54, U_A2.AM2
- net LINK2_DATA28: now also U_A1.AC35, U_A2.AC1; no longer U_A1.AN55, U_A2.AN1
- net LINK2_DATA29: now also U_A1.AC34, U_A2.AC2; no longer U_A1.AN54, U_A2.AN2
- net LINK2_DATA3: now also U_A1.K34, U_A2.K2; no longer U_A1.Y54, U_A2.Y2
- net LINK2_DATA30: now also U_A1.AD35, U_A2.AD1; no longer U_A1.AP55, U_A2.AP1
- net LINK2_DATA31: now also U_A1.AD34, U_A2.AD2; no longer U_A1.AP54, U_A2.AP2
- net LINK2_DATA4: now also U_A1.L35, U_A2.L1; no longer U_A1.AA55, U_A2.AA1
- net LINK2_DATA5: now also U_A1.L34, U_A2.L2; no longer U_A1.AA54, U_A2.AA2
- net LINK2_DATA6: now also U_A1.M35, U_A2.M1; no longer U_A1.AB55, U_A2.AB1
- net LINK2_DATA7: now also U_A1.M34, U_A2.M2; no longer U_A1.AB54, U_A2.AB2
- net LINK2_DATA8: now also U_A1.N35, U_A2.N1; no longer U_A1.AC55, U_A2.AC1
- net LINK2_DATA9: now also U_A1.N34, U_A2.N2; no longer U_A1.AC54, U_A2.AC2
- net LINK2_READY_BACK: now also U_A1.AF35, U_A2.AF1; no longer U_A1.AT55, U_A2.AT1
- net LINK2_SOF: now also U_A1.AF34, U_A2.AF2; no longer U_A1.AT54, U_A2.AT2
- net LINK2_VALID: now also U_A1.AE34, U_A2.AE2; no longer U_A1.AR54, U_A2.AR2
- net LINK3_CLOCK: now also U_A2.AE35, U_A3.AE1; no longer U_A2.AR55, U_A3.AR1
- net LINK3_DATA0: now also U_A2.J35, U_A3.J1; no longer U_A2.W55, U_A3.W1
- net LINK3_DATA1: now also U_A2.J34, U_A3.J2; no longer U_A2.W54, U_A3.W2
- net LINK3_DATA10: now also U_A2.P35, U_A3.P1; no longer U_A2.AD55, U_A3.AD1
- net LINK3_DATA11: now also U_A2.P34, U_A3.P2; no longer U_A2.AD54, U_A3.AD2
- net LINK3_DATA12: now also U_A2.R35, U_A3.R1; no longer U_A2.AE55, U_A3.AE1
- net LINK3_DATA13: now also U_A2.R34, U_A3.R2; no longer U_A2.AE54, U_A3.AE2
- net LINK3_DATA14: now also U_A2.T35, U_A3.T1; no longer U_A2.AF55, U_A3.AF1
- net LINK3_DATA15: now also U_A2.T34, U_A3.T2; no longer U_A2.AF54, U_A3.AF2
- net LINK3_DATA16: now also U_A2.U35, U_A3.U1; no longer U_A2.AG55, U_A3.AG1
- net LINK3_DATA17: now also U_A2.U34, U_A3.U2; no longer U_A2.AG54, U_A3.AG2
- net LINK3_DATA18: now also U_A2.V35, U_A3.V1; no longer U_A2.AH55, U_A3.AH1
- net LINK3_DATA19: now also U_A2.V34, U_A3.V2; no longer U_A2.AH54, U_A3.AH2
- net LINK3_DATA2: now also U_A2.K35, U_A3.K1; no longer U_A2.Y55, U_A3.Y1
- net LINK3_DATA20: now also U_A2.W35, U_A3.W1; no longer U_A2.AJ55, U_A3.AJ1
- net LINK3_DATA21: now also U_A2.W34, U_A3.W2; no longer U_A2.AJ54, U_A3.AJ2
- net LINK3_DATA22: now also U_A2.Y35, U_A3.Y1; no longer U_A2.AK55, U_A3.AK1
- net LINK3_DATA23: now also U_A2.Y34, U_A3.Y2; no longer U_A2.AK54, U_A3.AK2
- net LINK3_DATA24: now also U_A2.AA35, U_A3.AA1; no longer U_A2.AL55, U_A3.AL1
- net LINK3_DATA25: now also U_A2.AA34, U_A3.AA2; no longer U_A2.AL54, U_A3.AL2
- net LINK3_DATA26: now also U_A2.AB35, U_A3.AB1; no longer U_A2.AM55, U_A3.AM1
- net LINK3_DATA27: now also U_A2.AB34, U_A3.AB2; no longer U_A2.AM54, U_A3.AM2
- net LINK3_DATA28: now also U_A2.AC35, U_A3.AC1; no longer U_A2.AN55, U_A3.AN1
- net LINK3_DATA29: now also U_A2.AC34, U_A3.AC2; no longer U_A2.AN54, U_A3.AN2
- net LINK3_DATA3: now also U_A2.K34, U_A3.K2; no longer U_A2.Y54, U_A3.Y2
- net LINK3_DATA30: now also U_A2.AD35, U_A3.AD1; no longer U_A2.AP55, U_A3.AP1
- net LINK3_DATA31: now also U_A2.AD34, U_A3.AD2; no longer U_A2.AP54, U_A3.AP2
- net LINK3_DATA4: now also U_A2.L35, U_A3.L1; no longer U_A2.AA55, U_A3.AA1
- net LINK3_DATA5: now also U_A2.L34, U_A3.L2; no longer U_A2.AA54, U_A3.AA2
- net LINK3_DATA6: now also U_A2.M35, U_A3.M1; no longer U_A2.AB55, U_A3.AB1
- net LINK3_DATA7: now also U_A2.M34, U_A3.M2; no longer U_A2.AB54, U_A3.AB2
- net LINK3_DATA8: now also U_A2.N35, U_A3.N1; no longer U_A2.AC55, U_A3.AC1
- net LINK3_DATA9: now also U_A2.N34, U_A3.N2; no longer U_A2.AC54, U_A3.AC2
- net LINK3_READY_BACK: now also U_A2.AF35, U_A3.AF1; no longer U_A2.AT55, U_A3.AT1
- net LINK3_SOF: now also U_A2.AF34, U_A3.AF2; no longer U_A2.AT54, U_A3.AT2
- net LINK3_VALID: now also U_A2.AE34, U_A3.AE2; no longer U_A2.AR54, U_A3.AR2
- net LINK4_CLOCK: now also U_A3.AE35, U_A4.AE1; no longer U_A3.AR55, U_H0.AR1
- net LINK4_DATA0: now also U_A3.J35, U_A4.J1; no longer U_A3.W55, U_H0.W1
- net LINK4_DATA1: now also U_A3.J34, U_A4.J2; no longer U_A3.W54, U_H0.W2
- net LINK4_DATA10: now also U_A3.P35, U_A4.P1; no longer U_A3.AD55, U_H0.AD1
- net LINK4_DATA11: now also U_A3.P34, U_A4.P2; no longer U_A3.AD54, U_H0.AD2
- net LINK4_DATA12: now also U_A3.R35, U_A4.R1; no longer U_A3.AE55, U_H0.AE1
- net LINK4_DATA13: now also U_A3.R34, U_A4.R2; no longer U_A3.AE54, U_H0.AE2
- net LINK4_DATA14: now also U_A3.T35, U_A4.T1; no longer U_A3.AF55, U_H0.AF1
- net LINK4_DATA15: now also U_A3.T34, U_A4.T2; no longer U_A3.AF54, U_H0.AF2
- net LINK4_DATA16: now also U_A3.U35, U_A4.U1; no longer U_A3.AG55, U_H0.AG1
- net LINK4_DATA17: now also U_A3.U34, U_A4.U2; no longer U_A3.AG54, U_H0.AG2
- net LINK4_DATA18: now also U_A3.V35, U_A4.V1; no longer U_A3.AH55, U_H0.AH1
- net LINK4_DATA19: now also U_A3.V34, U_A4.V2; no longer U_A3.AH54, U_H0.AH2
- net LINK4_DATA2: now also U_A3.K35, U_A4.K1; no longer U_A3.Y55, U_H0.Y1
- net LINK4_DATA20: now also U_A3.W35, U_A4.W1; no longer U_A3.AJ55, U_H0.AJ1
- net LINK4_DATA21: now also U_A3.W34, U_A4.W2; no longer U_A3.AJ54, U_H0.AJ2
- net LINK4_DATA22: now also U_A3.Y35, U_A4.Y1; no longer U_A3.AK55, U_H0.AK1
- net LINK4_DATA23: now also U_A3.Y34, U_A4.Y2; no longer U_A3.AK54, U_H0.AK2
- net LINK4_DATA24: now also U_A3.AA35, U_A4.AA1; no longer U_A3.AL55, U_H0.AL1
- net LINK4_DATA25: now also U_A3.AA34, U_A4.AA2; no longer U_A3.AL54, U_H0.AL2
- net LINK4_DATA26: now also U_A3.AB35, U_A4.AB1; no longer U_A3.AM55, U_H0.AM1
- net LINK4_DATA27: now also U_A3.AB34, U_A4.AB2; no longer U_A3.AM54, U_H0.AM2
- net LINK4_DATA28: now also U_A3.AC35, U_A4.AC1; no longer U_A3.AN55, U_H0.AN1
- net LINK4_DATA29: now also U_A3.AC34, U_A4.AC2; no longer U_A3.AN54, U_H0.AN2
- net LINK4_DATA3: now also U_A3.K34, U_A4.K2; no longer U_A3.Y54, U_H0.Y2
- net LINK4_DATA30: now also U_A3.AD35, U_A4.AD1; no longer U_A3.AP55, U_H0.AP1
- net LINK4_DATA31: now also U_A3.AD34, U_A4.AD2; no longer U_A3.AP54, U_H0.AP2
- net LINK4_DATA4: now also U_A3.L35, U_A4.L1; no longer U_A3.AA55, U_H0.AA1
- net LINK4_DATA5: now also U_A3.L34, U_A4.L2; no longer U_A3.AA54, U_H0.AA2
- net LINK4_DATA6: now also U_A3.M35, U_A4.M1; no longer U_A3.AB55, U_H0.AB1
- net LINK4_DATA7: now also U_A3.M34, U_A4.M2; no longer U_A3.AB54, U_H0.AB2
- net LINK4_DATA8: now also U_A3.N35, U_A4.N1; no longer U_A3.AC55, U_H0.AC1
- net LINK4_DATA9: now also U_A3.N34, U_A4.N2; no longer U_A3.AC54, U_H0.AC2
- net LINK4_READY_BACK: now also U_A3.AF35, U_A4.AF1; no longer U_A3.AT55, U_H0.AT1
- net LINK4_SOF: now also U_A3.AF34, U_A4.AF2; no longer U_A3.AT54, U_H0.AT2
- net LINK4_VALID: now also U_A3.AE34, U_A4.AE2; no longer U_A3.AR54, U_H0.AR2
- net LINK5_CLOCK: now also U_A4.AE35, U_A5.AE1; no longer U_H0.AR55
- net LINK5_DATA0: now also U_A4.J35, U_A5.J1; no longer U_H0.W55
- net LINK5_DATA1: now also U_A4.J34, U_A5.J2; no longer U_H0.W54
- net LINK5_DATA10: now also U_A4.P35, U_A5.P1; no longer U_H0.AD55
- net LINK5_DATA11: now also U_A4.P34, U_A5.P2; no longer U_H0.AD54
- net LINK5_DATA12: now also U_A4.R35, U_A5.R1; no longer U_H0.AE55
- net LINK5_DATA13: now also U_A4.R34, U_A5.R2; no longer U_H0.AE54
- net LINK5_DATA14: now also U_A4.T35, U_A5.T1; no longer U_H0.AF55
- net LINK5_DATA15: now also U_A4.T34, U_A5.T2; no longer U_H0.AF54
- net LINK5_DATA16: now also U_A4.U35, U_A5.U1; no longer U_H0.AG55
- net LINK5_DATA17: now also U_A4.U34, U_A5.U2; no longer U_H0.AG54
- net LINK5_DATA18: now also U_A4.V35, U_A5.V1; no longer U_H0.AH55
- net LINK5_DATA19: now also U_A4.V34, U_A5.V2; no longer U_H0.AH54
- net LINK5_DATA2: now also U_A4.K35, U_A5.K1; no longer U_H0.Y55
- net LINK5_DATA20: now also U_A4.W35, U_A5.W1; no longer U_H0.AJ55
- net LINK5_DATA21: now also U_A4.W34, U_A5.W2; no longer U_H0.AJ54
- net LINK5_DATA22: now also U_A4.Y35, U_A5.Y1; no longer U_H0.AK55
- net LINK5_DATA23: now also U_A4.Y34, U_A5.Y2; no longer U_H0.AK54
- net LINK5_DATA24: now also U_A4.AA35, U_A5.AA1; no longer U_H0.AL55
- net LINK5_DATA25: now also U_A4.AA34, U_A5.AA2; no longer U_H0.AL54
- net LINK5_DATA26: now also U_A4.AB35, U_A5.AB1; no longer U_H0.AM55
- net LINK5_DATA27: now also U_A4.AB34, U_A5.AB2; no longer U_H0.AM54
- net LINK5_DATA28: now also U_A4.AC35, U_A5.AC1; no longer U_H0.AN55
- net LINK5_DATA29: now also U_A4.AC34, U_A5.AC2; no longer U_H0.AN54
- net LINK5_DATA3: now also U_A4.K34, U_A5.K2; no longer U_H0.Y54
- net LINK5_DATA30: now also U_A4.AD35, U_A5.AD1; no longer U_H0.AP55
- net LINK5_DATA31: now also U_A4.AD34, U_A5.AD2; no longer U_H0.AP54
- net LINK5_DATA4: now also U_A4.L35, U_A5.L1; no longer U_H0.AA55
- net LINK5_DATA5: now also U_A4.L34, U_A5.L2; no longer U_H0.AA54
- net LINK5_DATA6: now also U_A4.M35, U_A5.M1; no longer U_H0.AB55
- net LINK5_DATA7: now also U_A4.M34, U_A5.M2; no longer U_H0.AB54
- net LINK5_DATA8: now also U_A4.N35, U_A5.N1; no longer U_H0.AC55
- net LINK5_DATA9: now also U_A4.N34, U_A5.N2; no longer U_H0.AC54
- net LINK5_READY_BACK: now also U_A4.AF35, U_A5.AF1; no longer U_H0.AT55
- net LINK5_SOF: now also U_A4.AF34, U_A5.AF2; no longer U_H0.AT54
- net LINK5_VALID: now also U_A4.AE34, U_A5.AE2; no longer U_H0.AR54
- net MGMT_CS_A0: now also U_A0.AR6; no longer U_A0.BR6
- net MGMT_CS_A1: now also U_A1.AR6; no longer U_A1.BR6
- net MGMT_CS_A2: now also U_A2.AR6; no longer U_A2.BR6
- net MGMT_CS_A3: now also U_A3.AR6; no longer U_A3.BR6
- net MGMT_CS_H0: now also U_H0.AR6; no longer U_H0.BR6
- net MGMT_IRQ_A0: now also U_A0.AR8; no longer U_A0.BR8
- net MGMT_IRQ_A1: now also U_A1.AR8; no longer U_A1.BR8
- net MGMT_IRQ_A2: now also U_A2.AR8; no longer U_A2.BR8
- net MGMT_IRQ_A3: now also U_A3.AR8; no longer U_A3.BR8
- net MGMT_IRQ_H0: now also U_H0.AR8; no longer U_H0.BR8
- net MGMT_MISO: now also U_A0.AR5, U_A1.AR5, U_A2.AR5, U_A3.AR5, U_H0.AR5, U_A4.AR5, U_A5.AR5, U_A6.AR5, U_A7.AR5, U_H1.AR5; no longer U_A0.BR5, U_A1.BR5, U_A2.BR5, U_A3.BR5, U_H0.BR5
- net MGMT_MOSI: now also U_A0.AR4, U_A1.AR4, U_A2.AR4, U_A3.AR4, U_H0.AR4, U_A4.AR4, U_A5.AR4, U_A6.AR4, U_A7.AR4, U_H1.AR4; no longer U_A0.BR4, U_A1.BR4, U_A2.BR4, U_A3.BR4, U_H0.BR4
- net MGMT_SCLK: now also U_A0.AR3, U_A1.AR3, U_A2.AR3, U_A3.AR3, U_H0.AR3, U_A4.AR3, U_A5.AR3, U_A6.AR3, U_A7.AR3, U_H1.AR3; no longer U_A0.BR3, U_A1.BR3, U_A2.BR3, U_A3.BR3, U_H0.BR3
- net MODE0_A0: now also U_A0.AR18; no longer U_A0.BR18
- net MODE0_A1: now also U_A1.AR18; no longer U_A1.BR18
- net MODE0_A2: now also U_A2.AR18; no longer U_A2.BR18
- net MODE0_A3: now also U_A3.AR18; no longer U_A3.BR18
- net MODE0_H0: now also U_H0.AR18; no longer U_H0.BR18
- net MODE1_A0: now also U_A0.AR19; no longer U_A0.BR19
- net MODE1_A1: now also U_A1.AR19; no longer U_A1.BR19
- net MODE1_A2: now also U_A2.AR19; no longer U_A2.BR19
- net MODE1_A3: now also U_A3.AR19; no longer U_A3.BR19
- net MODE1_H0: now also U_H0.AR19; no longer U_H0.BR19
- net REFCLK_A0_N: now also U_A0.AR16; no longer U_A0.BR16
- net REFCLK_A0_P: now also U_A0.AR15; no longer U_A0.BR15
- net REFCLK_A1_N: now also U_A1.AR16; no longer U_A1.BR16
- net REFCLK_A1_P: now also U_A1.AR15; no longer U_A1.BR15
- net REFCLK_A2_N: now also U_A2.AR16; no longer U_A2.BR16
- net REFCLK_A2_P: now also U_A2.AR15; no longer U_A2.BR15
- net REFCLK_A3_N: now also U_A3.AR16; no longer U_A3.BR16
- net REFCLK_A3_P: now also U_A3.AR15; no longer U_A3.BR15
- net REFCLK_H0_N: now also U_H0.AR16; no longer U_H0.BR16
- net REFCLK_H0_P: now also U_H0.AR15; no longer U_H0.BR15
- net VDDQ_HBM_0V4: now also U_A0.L16, U_A0.L26, U_A0.M17, U_A0.M27, U_A0.M7, U_A0.N18, U_A0.N28, U_A0.N8, U_A0.P19, U_A0.P29, U_A0.P9, U_A0.R10, U_A1.L16, U_A1.L26, U_A1.M17, U_A1.M27, U_A1.M7, U_A1.N18, U_A1.N28, U_A1.N8, U_A1.P19, U_A1.P29, U_A1.P9, U_A1.R10, U_A2.L16, U_A2.L26, U_A2.M17, U_A2.M27, U_A2.M7, U_A2.N18, U_A2.N28, U_A2.N8, U_A2.P19, U_A2.P29, U_A2.P9, U_A2.R10, U_A3.L16, U_A3.L26, U_A3.M17, U_A3.M27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; no longer U_A0.G32, U_A0.G42, U_A0.G52, U_A0.H13, U_A0.H23, U_A0.H3, U_A0.H33, U_A0.H43, U_A0.H53, U_A0.J14, U_A0.J24, U_A0.J4, U_A1.G32, U_A1.G42, U_A1.G52, U_A1.H13, U_A1.H23, U_A1.H3, U_A1.H33, U_A1.H43, U_A1.H53, U_A1.J14, U_A1.J24, U_A1.J4, U_A2.G32, U_A2.G42, U_A2.G52, U_A2.H13, U_A2.H23, U_A2.H3, U_A2.H33, U_A2.H43, U_A2.H53, U_A2.J14, U_A2.J24, U_A2.J4, U_A3.G32, U_A3.G42, U_A3.G52, U_A3.H13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
- net VDD_CORE_A0: now also U_A0.AG2, U_A0.AH1, U_A0.AJ2, U_A0.AK1, U_A0.AL2, U_A0.AM1, U_A0.AN2, U_A0.AP1, U_A0.AR2; no longer U_A0.A38, U_A0.A40, U_A0.A42, U_A0.A44, U_A0.A48, U_A0.A50, U_A0.A52, U_A0.A54, U_A0.AA34, U_A0.AA36, U_A0.AA38, U_A0.AA40, U_A0.AA42, U_A0.AA44, U_A0.AA46, U_A0.AA48, U_A0.AA50, U_A0.AA52, U_A0.AB35, U_A0.AB37, U_A0.AB39, U_A0.AB41, U_A0.AB43, U_A0.AB45, U_A0.AB47, U_A0.AB49, U_A0.AB51, U_A0.AB53, U_A0.AC34, U_A0.AC36, U_A0.AC38, U_A0.AC40, U_A0.AC42, U_A0.AC44, U_A0.AC46, U_A0.AC48, U_A0.AC50, U_A0.AC52, U_A0.AD35, U_A0.AD37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
- net VDD_CORE_A1: now also U_A1.AG2, U_A1.AH1, U_A1.AJ2, U_A1.AK1, U_A1.AL2, U_A1.AM1, U_A1.AN2, U_A1.AP1, U_A1.AR2; no longer U_A1.A38, U_A1.A40, U_A1.A42, U_A1.A44, U_A1.A48, U_A1.A50, U_A1.A52, U_A1.A54, U_A1.AA34, U_A1.AA36, U_A1.AA38, U_A1.AA40, U_A1.AA42, U_A1.AA44, U_A1.AA46, U_A1.AA48, U_A1.AA50, U_A1.AA52, U_A1.AB35, U_A1.AB37, U_A1.AB39, U_A1.AB41, U_A1.AB43, U_A1.AB45, U_A1.AB47, U_A1.AB49, U_A1.AB51, U_A1.AB53, U_A1.AC34, U_A1.AC36, U_A1.AC38, U_A1.AC40, U_A1.AC42, U_A1.AC44, U_A1.AC46, U_A1.AC48, U_A1.AC50, U_A1.AC52, U_A1.AD35, U_A1.AD37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
- net VDD_CORE_A2: now also U_A2.AG2, U_A2.AH1, U_A2.AJ2, U_A2.AK1, U_A2.AL2, U_A2.AM1, U_A2.AN2, U_A2.AP1, U_A2.AR2; no longer U_A2.A38, U_A2.A40, U_A2.A42, U_A2.A44, U_A2.A48, U_A2.A50, U_A2.A52, U_A2.A54, U_A2.AA34, U_A2.AA36, U_A2.AA38, U_A2.AA40, U_A2.AA42, U_A2.AA44, U_A2.AA46, U_A2.AA48, U_A2.AA50, U_A2.AA52, U_A2.AB35, U_A2.AB37, U_A2.AB39, U_A2.AB41, U_A2.AB43, U_A2.AB45, U_A2.AB47, U_A2.AB49, U_A2.AB51, U_A2.AB53, U_A2.AC34, U_A2.AC36, U_A2.AC38, U_A2.AC40, U_A2.AC42, U_A2.AC44, U_A2.AC46, U_A2.AC48, U_A2.AC50, U_A2.AC52, U_A2.AD35, U_A2.AD37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
- net VDD_CORE_A3: now also U_A3.AG2, U_A3.AH1, U_A3.AJ2, U_A3.AK1, U_A3.AL2, U_A3.AM1, U_A3.AN2, U_A3.AP1, U_A3.AR2; no longer U_A3.A38, U_A3.A40, U_A3.A42, U_A3.A44, U_A3.A48, U_A3.A50, U_A3.A52, U_A3.A54, U_A3.AA34, U_A3.AA36, U_A3.AA38, U_A3.AA40, U_A3.AA42, U_A3.AA44, U_A3.AA46, U_A3.AA48, U_A3.AA50, U_A3.AA52, U_A3.AB35, U_A3.AB37, U_A3.AB39, U_A3.AB41, U_A3.AB43, U_A3.AB45, U_A3.AB47, U_A3.AB49, U_A3.AB51, U_A3.AB53, U_A3.AC34, U_A3.AC36, U_A3.AC38, U_A3.AC40, U_A3.AC42, U_A3.AC44, U_A3.AC46, U_A3.AC48, U_A3.AC50, U_A3.AC52, U_A3.AD35, U_A3.AD37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
- net VDD_CORE_H0: now also U_H0.AG2, U_H0.AH1, U_H0.AJ2, U_H0.AK1, U_H0.AL2, U_H0.AM1, U_H0.AN2, U_H0.AP1, U_H0.AR2; no longer U_H0.A38, U_H0.A40, U_H0.A42, U_H0.A44, U_H0.A48, U_H0.A50, U_H0.A52, U_H0.A54, U_H0.AA34, U_H0.AA36, U_H0.AA38, U_H0.AA40, U_H0.AA42, U_H0.AA44, U_H0.AA46, U_H0.AA48, U_H0.AA50, U_H0.AA52, U_H0.AB35, U_H0.AB37, U_H0.AB39, U_H0.AB41, U_H0.AB43, U_H0.AB45, U_H0.AB47, U_H0.AB49, U_H0.AB51, U_H0.AB53, U_H0.AC34, U_H0.AC36, U_H0.AC38, U_H0.AC40, U_H0.AC42, U_H0.AC44, U_H0.AC46, U_H0.AC48, U_H0.AC50, U_H0.AC52, U_H0.AD35, U_H0.AD37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
- net VDD_HBM_1V1: now also U_A0.G32, U_A0.H13, U_A0.H23, U_A0.H3, U_A0.H33, U_A0.J14, U_A0.J24, U_A0.J4, U_A0.K15, U_A0.K25, U_A0.K5, U_A0.L6, U_A1.G32, U_A1.H13, U_A1.H23, U_A1.H3, U_A1.H33, U_A1.J14, U_A1.J24, U_A1.J4, U_A1.K15, U_A1.K25, U_A1.K5, U_A1.L6, U_A2.G32, U_A2.H13, U_A2.H23, U_A2.H3, U_A2.H33, U_A2.J14, U_A2.J24, U_A2.J4, U_A2.K15, U_A2.K25, U_A2.K5, U_A2.L6, U_A3.G32, U_A3.H13, U_A3.H23, U_A3.H3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; no longer U_A0.C18, U_A0.C28, U_A0.C38, U_A0.C48, U_A0.C8, U_A0.D39, U_A0.D49, U_A0.D9, U_A0.E40, U_A0.E50, U_A0.F41, U_A0.F51, U_A1.C18, U_A1.C28, U_A1.C38, U_A1.C48, U_A1.C8, U_A1.D39, U_A1.D49, U_A1.D9, U_A1.E40, U_A1.E50, U_A1.F41, U_A1.F51, U_A2.C18, U_A2.C28, U_A2.C38, U_A2.C48, U_A2.C8, U_A2.D39, U_A2.D49, U_A2.D9, U_A2.E40, U_A2.E50, U_A2.F41, U_A2.F51, U_A3.C18, U_A3.C28, U_A3.C38, U_A3.C48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
- net VDD_IO_1V8: now also U_A0.C18, U_A0.C8, U_A1.C18, U_A1.C8, U_A2.C18, U_A2.C8, U_A3.C18, U_A3.C8, U_H0.C18, U_H0.C8, U_A4.A16, U_A4.A26, U_A4.A6, U_A4.B17, U_A4.B27, U_A4.B7, U_A4.C18, U_A4.C8, U_A5.A16, U_A5.A26, U_A5.A6, U_A5.B17, U_A5.B27, U_A5.B7, U_A5.C18, U_A5.C8, U_A6.A16, U_A6.A26, U_A6.A6, U_A6.B17, U_A6.B27, U_A6.B7, U_A6.C18, U_A6.C8, U_A7.A16, U_A7.A26, U_A7.A6, U_A7.B17, U_A7.B27, U_A7.B7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; no longer U_A0.A36, U_A0.A46, U_A1.A36, U_A1.A46, U_A2.A36, U_A2.A46, U_A3.A36, U_A3.A46, U_H0.A36, U_H0.A46
- net VDD_PLL_0V9: now also U_A0.C28, U_A0.D9, U_A1.C28, U_A1.D9, U_A2.C28, U_A2.D9, U_A3.C28, U_A3.D9, U_H0.C28, U_H0.D9, U_A4.C28, U_A4.D9, U_A5.C28, U_A5.D9, U_A6.C28, U_A6.D9, U_A7.C28, U_A7.D9, U_H1.C28, U_H1.D9; no longer U_A0.B37, U_A0.B47, U_A1.B37, U_A1.B47, U_A2.B37, U_A2.B47, U_A3.B37, U_A3.B47, U_H0.B37, U_H0.B47
- new net JTAG_TDO_A4: U_A4.AR13, U_A5.AR11
- new net JTAG_TDO_A5: U_A5.AR13, U_A6.AR11
- new net JTAG_TDO_A6: U_A6.AR13, U_A7.AR11
- new net JTAG_TDO_A7: U_A7.AR13, U_H0.AR11
- new net JTAG_TDO_H1: U_H1.AR13
- new net LINK10_CLOCK: U_H1.AE35
- new net LINK10_DATA0: U_H1.J35
- new net LINK10_DATA1: U_H1.J34
- new net LINK10_DATA10: U_H1.P35
- new net LINK10_DATA11: U_H1.P34
- new net LINK10_DATA12: U_H1.R35
- new net LINK10_DATA13: U_H1.R34
- new net LINK10_DATA14: U_H1.T35
- new net LINK10_DATA15: U_H1.T34
- new net LINK10_DATA16: U_H1.U35
- new net LINK10_DATA17: U_H1.U34
- new net LINK10_DATA18: U_H1.V35
- new net LINK10_DATA19: U_H1.V34
- new net LINK10_DATA2: U_H1.K35
- new net LINK10_DATA20: U_H1.W35
- new net LINK10_DATA21: U_H1.W34
- new net LINK10_DATA22: U_H1.Y35
- new net LINK10_DATA23: U_H1.Y34
- new net LINK10_DATA24: U_H1.AA35
- new net LINK10_DATA25: U_H1.AA34
- new net LINK10_DATA26: U_H1.AB35
- new net LINK10_DATA27: U_H1.AB34
- new net LINK10_DATA28: U_H1.AC35
- new net LINK10_DATA29: U_H1.AC34
- new net LINK10_DATA3: U_H1.K34
- new net LINK10_DATA30: U_H1.AD35
- new net LINK10_DATA31: U_H1.AD34
- new net LINK10_DATA4: U_H1.L35
- new net LINK10_DATA5: U_H1.L34
- new net LINK10_DATA6: U_H1.M35
- new net LINK10_DATA7: U_H1.M34
- new net LINK10_DATA8: U_H1.N35
- new net LINK10_DATA9: U_H1.N34
- new net LINK10_READY_BACK: U_H1.AF35
- new net LINK10_SOF: U_H1.AF34
- new net LINK10_VALID: U_H1.AE34
- new net LINK6_CLOCK: U_A5.AE35, U_A6.AE1
- new net LINK6_DATA0: U_A5.J35, U_A6.J1
- new net LINK6_DATA1: U_A5.J34, U_A6.J2
- new net LINK6_DATA10: U_A5.P35, U_A6.P1
- new net LINK6_DATA11: U_A5.P34, U_A6.P2
- new net LINK6_DATA12: U_A5.R35, U_A6.R1
- new net LINK6_DATA13: U_A5.R34, U_A6.R2
- new net LINK6_DATA14: U_A5.T35, U_A6.T1
- new net LINK6_DATA15: U_A5.T34, U_A6.T2
- new net LINK6_DATA16: U_A5.U35, U_A6.U1
- new net LINK6_DATA17: U_A5.U34, U_A6.U2
- new net LINK6_DATA18: U_A5.V35, U_A6.V1
- new net LINK6_DATA19: U_A5.V34, U_A6.V2
- new net LINK6_DATA2: U_A5.K35, U_A6.K1
- new net LINK6_DATA20: U_A5.W35, U_A6.W1
- new net LINK6_DATA21: U_A5.W34, U_A6.W2
- new net LINK6_DATA22: U_A5.Y35, U_A6.Y1
- new net LINK6_DATA23: U_A5.Y34, U_A6.Y2
- new net LINK6_DATA24: U_A5.AA35, U_A6.AA1
- new net LINK6_DATA25: U_A5.AA34, U_A6.AA2
- new net LINK6_DATA26: U_A5.AB35, U_A6.AB1
- new net LINK6_DATA27: U_A5.AB34, U_A6.AB2
- new net LINK6_DATA28: U_A5.AC35, U_A6.AC1
- new net LINK6_DATA29: U_A5.AC34, U_A6.AC2
- new net LINK6_DATA3: U_A5.K34, U_A6.K2
- new net LINK6_DATA30: U_A5.AD35, U_A6.AD1
- new net LINK6_DATA31: U_A5.AD34, U_A6.AD2
- new net LINK6_DATA4: U_A5.L35, U_A6.L1
- new net LINK6_DATA5: U_A5.L34, U_A6.L2
- new net LINK6_DATA6: U_A5.M35, U_A6.M1
- new net LINK6_DATA7: U_A5.M34, U_A6.M2
- new net LINK6_DATA8: U_A5.N35, U_A6.N1
- new net LINK6_DATA9: U_A5.N34, U_A6.N2
- new net LINK6_READY_BACK: U_A5.AF35, U_A6.AF1
- new net LINK6_SOF: U_A5.AF34, U_A6.AF2
- new net LINK6_VALID: U_A5.AE34, U_A6.AE2
- new net LINK7_CLOCK: U_A6.AE35, U_A7.AE1
- new net LINK7_DATA0: U_A6.J35, U_A7.J1
- new net LINK7_DATA1: U_A6.J34, U_A7.J2
- new net LINK7_DATA10: U_A6.P35, U_A7.P1
- new net LINK7_DATA11: U_A6.P34, U_A7.P2
- new net LINK7_DATA12: U_A6.R35, U_A7.R1
- new net LINK7_DATA13: U_A6.R34, U_A7.R2
- new net LINK7_DATA14: U_A6.T35, U_A7.T1
- new net LINK7_DATA15: U_A6.T34, U_A7.T2
- new net LINK7_DATA16: U_A6.U35, U_A7.U1
- new net LINK7_DATA17: U_A6.U34, U_A7.U2
- new net LINK7_DATA18: U_A6.V35, U_A7.V1
- new net LINK7_DATA19: U_A6.V34, U_A7.V2
- new net LINK7_DATA2: U_A6.K35, U_A7.K1
- new net LINK7_DATA20: U_A6.W35, U_A7.W1
- new net LINK7_DATA21: U_A6.W34, U_A7.W2
- new net LINK7_DATA22: U_A6.Y35, U_A7.Y1
- new net LINK7_DATA23: U_A6.Y34, U_A7.Y2
- new net LINK7_DATA24: U_A6.AA35, U_A7.AA1
- new net LINK7_DATA25: U_A6.AA34, U_A7.AA2
- new net LINK7_DATA26: U_A6.AB35, U_A7.AB1
- new net LINK7_DATA27: U_A6.AB34, U_A7.AB2
- new net LINK7_DATA28: U_A6.AC35, U_A7.AC1
- new net LINK7_DATA29: U_A6.AC34, U_A7.AC2
- new net LINK7_DATA3: U_A6.K34, U_A7.K2
- new net LINK7_DATA30: U_A6.AD35, U_A7.AD1
- new net LINK7_DATA31: U_A6.AD34, U_A7.AD2
- new net LINK7_DATA4: U_A6.L35, U_A7.L1
- new net LINK7_DATA5: U_A6.L34, U_A7.L2
- new net LINK7_DATA6: U_A6.M35, U_A7.M1
- new net LINK7_DATA7: U_A6.M34, U_A7.M2
- new net LINK7_DATA8: U_A6.N35, U_A7.N1
- new net LINK7_DATA9: U_A6.N34, U_A7.N2
- new net LINK7_READY_BACK: U_A6.AF35, U_A7.AF1
- new net LINK7_SOF: U_A6.AF34, U_A7.AF2
- new net LINK7_VALID: U_A6.AE34, U_A7.AE2
- new net LINK8_CLOCK: U_A7.AE35, U_H0.AE1
- new net LINK8_DATA0: U_A7.J35, U_H0.J1
- new net LINK8_DATA1: U_A7.J34, U_H0.J2
- new net LINK8_DATA10: U_A7.P35, U_H0.P1
- new net LINK8_DATA11: U_A7.P34, U_H0.P2
- new net LINK8_DATA12: U_A7.R35, U_H0.R1
- new net LINK8_DATA13: U_A7.R34, U_H0.R2
- new net LINK8_DATA14: U_A7.T35, U_H0.T1
- new net LINK8_DATA15: U_A7.T34, U_H0.T2
- new net LINK8_DATA16: U_A7.U35, U_H0.U1
- new net LINK8_DATA17: U_A7.U34, U_H0.U2
- new net LINK8_DATA18: U_A7.V35, U_H0.V1
- new net LINK8_DATA19: U_A7.V34, U_H0.V2
- new net LINK8_DATA2: U_A7.K35, U_H0.K1
- new net LINK8_DATA20: U_A7.W35, U_H0.W1
- new net LINK8_DATA21: U_A7.W34, U_H0.W2
- new net LINK8_DATA22: U_A7.Y35, U_H0.Y1
- new net LINK8_DATA23: U_A7.Y34, U_H0.Y2
- new net LINK8_DATA24: U_A7.AA35, U_H0.AA1
- new net LINK8_DATA25: U_A7.AA34, U_H0.AA2
- new net LINK8_DATA26: U_A7.AB35, U_H0.AB1
- new net LINK8_DATA27: U_A7.AB34, U_H0.AB2
- new net LINK8_DATA28: U_A7.AC35, U_H0.AC1
- new net LINK8_DATA29: U_A7.AC34, U_H0.AC2
- new net LINK8_DATA3: U_A7.K34, U_H0.K2
- new net LINK8_DATA30: U_A7.AD35, U_H0.AD1
- new net LINK8_DATA31: U_A7.AD34, U_H0.AD2
- new net LINK8_DATA4: U_A7.L35, U_H0.L1
- new net LINK8_DATA5: U_A7.L34, U_H0.L2
- new net LINK8_DATA6: U_A7.M35, U_H0.M1
- new net LINK8_DATA7: U_A7.M34, U_H0.M2
- new net LINK8_DATA8: U_A7.N35, U_H0.N1
- new net LINK8_DATA9: U_A7.N34, U_H0.N2
- new net LINK8_READY_BACK: U_A7.AF35, U_H0.AF1
- new net LINK8_SOF: U_A7.AF34, U_H0.AF2
- new net LINK8_VALID: U_A7.AE34, U_H0.AE2
- new net LINK9_CLOCK: U_H0.AE35, U_H1.AE1
- new net LINK9_DATA0: U_H0.J35, U_H1.J1
- new net LINK9_DATA1: U_H0.J34, U_H1.J2
- new net LINK9_DATA10: U_H0.P35, U_H1.P1
- new net LINK9_DATA11: U_H0.P34, U_H1.P2
- new net LINK9_DATA12: U_H0.R35, U_H1.R1
- new net LINK9_DATA13: U_H0.R34, U_H1.R2
- new net LINK9_DATA14: U_H0.T35, U_H1.T1
- new net LINK9_DATA15: U_H0.T34, U_H1.T2
- new net LINK9_DATA16: U_H0.U35, U_H1.U1
- new net LINK9_DATA17: U_H0.U34, U_H1.U2
- new net LINK9_DATA18: U_H0.V35, U_H1.V1
- new net LINK9_DATA19: U_H0.V34, U_H1.V2
- new net LINK9_DATA2: U_H0.K35, U_H1.K1
- new net LINK9_DATA20: U_H0.W35, U_H1.W1
- new net LINK9_DATA21: U_H0.W34, U_H1.W2
- new net LINK9_DATA22: U_H0.Y35, U_H1.Y1
- new net LINK9_DATA23: U_H0.Y34, U_H1.Y2
- new net LINK9_DATA24: U_H0.AA35, U_H1.AA1
- new net LINK9_DATA25: U_H0.AA34, U_H1.AA2
- new net LINK9_DATA26: U_H0.AB35, U_H1.AB1
- new net LINK9_DATA27: U_H0.AB34, U_H1.AB2
- new net LINK9_DATA28: U_H0.AC35, U_H1.AC1
- new net LINK9_DATA29: U_H0.AC34, U_H1.AC2
- new net LINK9_DATA3: U_H0.K34, U_H1.K2
- new net LINK9_DATA30: U_H0.AD35, U_H1.AD1
- new net LINK9_DATA31: U_H0.AD34, U_H1.AD2
- new net LINK9_DATA4: U_H0.L35, U_H1.L1
- new net LINK9_DATA5: U_H0.L34, U_H1.L2
- new net LINK9_DATA6: U_H0.M35, U_H1.M1
- new net LINK9_DATA7: U_H0.M34, U_H1.M2
- new net LINK9_DATA8: U_H0.N35, U_H1.N1
- new net LINK9_DATA9: U_H0.N34, U_H1.N2
- new net LINK9_READY_BACK: U_H0.AF35, U_H1.AF1
- new net LINK9_SOF: U_H0.AF34, U_H1.AF2
- new net LINK9_VALID: U_H0.AE34, U_H1.AE2
- new net MGMT_CS_A4: U_A4.AR6
- new net MGMT_CS_A5: U_A5.AR6
- new net MGMT_CS_A6: U_A6.AR6
- new net MGMT_CS_A7: U_A7.AR6
- new net MGMT_CS_H1: U_H1.AR6
- new net MGMT_IRQ_A4: U_A4.AR8
- new net MGMT_IRQ_A5: U_A5.AR8
- new net MGMT_IRQ_A6: U_A6.AR8
- new net MGMT_IRQ_A7: U_A7.AR8
- new net MGMT_IRQ_H1: U_H1.AR8
- new net MODE0_A4: U_A4.AR18
- new net MODE0_A5: U_A5.AR18
- new net MODE0_A6: U_A6.AR18
- new net MODE0_A7: U_A7.AR18
- new net MODE0_H1: U_H1.AR18
- new net MODE1_A4: U_A4.AR19
- new net MODE1_A5: U_A5.AR19
- new net MODE1_A6: U_A6.AR19
- new net MODE1_A7: U_A7.AR19
- new net MODE1_H1: U_H1.AR19
- new net REFCLK_A4_N: U_A4.AR16
- new net REFCLK_A4_P: U_A4.AR15
- new net REFCLK_A5_N: U_A5.AR16
- new net REFCLK_A5_P: U_A5.AR15
- new net REFCLK_A6_N: U_A6.AR16
- new net REFCLK_A6_P: U_A6.AR15
- new net REFCLK_A7_N: U_A7.AR16
- new net REFCLK_A7_P: U_A7.AR15
- new net REFCLK_H1_N: U_H1.AR16
- new net REFCLK_H1_P: U_H1.AR15
- new net VDD_CORE_A4: U_A4.A10, U_A4.A12, U_A4.A14, U_A4.A18, U_A4.A2, U_A4.A20, U_A4.A22, U_A4.A24, U_A4.A28, U_A4.A30, U_A4.A32, U_A4.A34, U_A4.A4, U_A4.A8, U_A4.AA10, U_A4.AA12, U_A4.AA14, U_A4.AA16, U_A4.AA18, U_A4.AA20, U_A4.AA22, U_A4.AA24, U_A4.AA26, U_A4.AA28, U_A4.AA30, U_A4.AA32, U_A4.AA4, U_A4.AA6, U_A4.AA8, U_A4.AB11, U_A4.AB13, U_A4.AB15, U_A4.AB17, U_A4.AB19, U_A4.AB21, U_A4.AB23, U_A4.AB25, U_A4.AB27, U_A4.AB29, U_A4.AB3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
- new net VDD_CORE_A5: U_A5.A10, U_A5.A12, U_A5.A14, U_A5.A18, U_A5.A2, U_A5.A20, U_A5.A22, U_A5.A24, U_A5.A28, U_A5.A30, U_A5.A32, U_A5.A34, U_A5.A4, U_A5.A8, U_A5.AA10, U_A5.AA12, U_A5.AA14, U_A5.AA16, U_A5.AA18, U_A5.AA20, U_A5.AA22, U_A5.AA24, U_A5.AA26, U_A5.AA28, U_A5.AA30, U_A5.AA32, U_A5.AA4, U_A5.AA6, U_A5.AA8, U_A5.AB11, U_A5.AB13, U_A5.AB15, U_A5.AB17, U_A5.AB19, U_A5.AB21, U_A5.AB23, U_A5.AB25, U_A5.AB27, U_A5.AB29, U_A5.AB3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
- new net VDD_CORE_A6: U_A6.A10, U_A6.A12, U_A6.A14, U_A6.A18, U_A6.A2, U_A6.A20, U_A6.A22, U_A6.A24, U_A6.A28, U_A6.A30, U_A6.A32, U_A6.A34, U_A6.A4, U_A6.A8, U_A6.AA10, U_A6.AA12, U_A6.AA14, U_A6.AA16, U_A6.AA18, U_A6.AA20, U_A6.AA22, U_A6.AA24, U_A6.AA26, U_A6.AA28, U_A6.AA30, U_A6.AA32, U_A6.AA4, U_A6.AA6, U_A6.AA8, U_A6.AB11, U_A6.AB13, U_A6.AB15, U_A6.AB17, U_A6.AB19, U_A6.AB21, U_A6.AB23, U_A6.AB25, U_A6.AB27, U_A6.AB29, U_A6.AB3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
- new net VDD_CORE_A7: U_A7.A10, U_A7.A12, U_A7.A14, U_A7.A18, U_A7.A2, U_A7.A20, U_A7.A22, U_A7.A24, U_A7.A28, U_A7.A30, U_A7.A32, U_A7.A34, U_A7.A4, U_A7.A8, U_A7.AA10, U_A7.AA12, U_A7.AA14, U_A7.AA16, U_A7.AA18, U_A7.AA20, U_A7.AA22, U_A7.AA24, U_A7.AA26, U_A7.AA28, U_A7.AA30, U_A7.AA32, U_A7.AA4, U_A7.AA6, U_A7.AA8, U_A7.AB11, U_A7.AB13, U_A7.AB15, U_A7.AB17, U_A7.AB19, U_A7.AB21, U_A7.AB23, U_A7.AB25, U_A7.AB27, U_A7.AB29, U_A7.AB3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
- new net VDD_CORE_H1: U_H1.A10, U_H1.A12, U_H1.A14, U_H1.A18, U_H1.A2, U_H1.A20, U_H1.A22, U_H1.A24, U_H1.A28, U_H1.A30, U_H1.A32, U_H1.A34, U_H1.A4, U_H1.A8, U_H1.AA10, U_H1.AA12, U_H1.AA14, U_H1.AA16, U_H1.AA18, U_H1.AA20, U_H1.AA22, U_H1.AA24, U_H1.AA26, U_H1.AA28, U_H1.AA30, U_H1.AA32, U_H1.AA4, U_H1.AA6, U_H1.AA8, U_H1.AB11, U_H1.AB13, U_H1.AB15, U_H1.AB17, U_H1.AB19, U_H1.AB21, U_H1.AB23, U_H1.AB25, U_H1.AB27, U_H1.AB29, U_H1.AB3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
