File: hw/kicad_27b/fpga.kicad_sch (KiCad schematic)
At the start: 6 parts

Commit message: Pipeline a layer's passes, and re-rate the 27B board to eight layer dies
Two things the last commit left open.

The simulator now separates a layer stage's latency from its initiation
interval.  A layer is a chain of passes and each pass has its own via-
programmed tiles, so nothing is reused between them: the first pass is free
the moment its token moves on, and the stage holds as many tokens as fit
between its latency and its interval.  layer_pass_cycles carries the pass,
a quarter of the layer in every shipped geometry, which is the same figure
the single-pass head die already used.

I expected that to be worth four times and it is worth almost nothing,
because after the memory corrections it is the memory and not the pass rate
that binds.  It is exactly neutral on every LPDDR5X and PSRAM configuration
at any context count, worth 4 to 8 percent on the 9B with HBM, and slightly
negative on the 27B, where more tokens per stage lengthen latency against a
fixed pool of contexts.  With the bandwidth raised tenfold it is worth 2.5
times, 240K to 597K tokens/s, so the lever is real and nothing in reach of
this design is close enough to the fabric to collect it.  Letting a token's
state write overlap the next token's state read, which the same change
allows, is what does move the HBM numbers: the 3 nm 9B goes from 190K to
244K.

The 27B board is now eight layer ASICs of eight layers and two head ASICs
splitting the LM head, at 153K tokens/s rather than the 234K that came from
the un-corrected model.  Halving the per-die load takes the core rail from
650 A to 249 A, the package from a 55 x 55 array to 35 x 35, the cold plate
from 525 W to 200 W, and puts the ring on the same 11-gon as the 9B board.
hw/README's open item is replaced by the re-rating itself.

The 9B board's design point follows the same correction, 14.5K to 8.2K, and
its per-die traffic is 7.35 MB per token rather than the 4.2 MB of retrieval
alone.  Generated files now name the board description they came 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
Connections:
- net GND: no longer U_FPGA.AD16, U_FPGA.AD18, U_FPGA.AD20, U_FPGA.AD22, U_FPGA.AD24
- net JTAG_TCK: now also U_FPGA.AC24; no longer U_FPGA.AC14
- net JTAG_TDI_FPGA: now also U_FPGA.AD2; no longer U_FPGA.AC16
- net JTAG_TDO_FPGA: now also U_FPGA.AD3; no longer U_FPGA.AC17
- net JTAG_TMS: now also U_FPGA.AD1; no longer U_FPGA.AC15
- net JTAG_TRST: now also U_FPGA.AD4; no longer U_FPGA.AC18
- net MGMT_CS_H0: now also U_FPGA.AC20; no longer U_FPGA.AC12
- net MGMT_IRQ_H0: now also U_FPGA.AC21; no longer U_FPGA.AC13
- net QSPI0: now also U_FPGA.AD17; no longer U_FPGA.AD7
- net QSPI1: now also U_FPGA.AD18; no longer U_FPGA.AD8
- net QSPI2: now also U_FPGA.AD19; no longer U_FPGA.AD9
- net QSPI3: now also U_FPGA.AD20; no longer U_FPGA.AD10
- net QSPI4: now also U_FPGA.AD21; no longer U_FPGA.AD11
- net QSPI5: now also U_FPGA.AD22; no longer U_FPGA.AD12
- net REFCLK_FPGA_N: now also U_FPGA.AD6; no longer U_FPGA.AC20
- net REFCLK_FPGA_P: now also U_FPGA.AD5; no longer U_FPGA.AC19
- net REFCLK_H0_N: now also U_CLK.22; no longer U_CLK.14
- net REFCLK_H0_P: now also U_CLK.21; no longer U_CLK.13
- net SFP_CTRL0: now also U_FPGA.AD13; no longer U_FPGA.AD3
- net SFP_CTRL1: now also U_FPGA.AD14; no longer U_FPGA.AD4
- net SFP_CTRL2: now also U_FPGA.AD15; no longer U_FPGA.AD5
- net SFP_CTRL3: now also U_FPGA.AD16; no longer U_FPGA.AD6
- net SFP_I2C0: now also U_FPGA.AD11; no longer U_FPGA.AD1
- net SFP_I2C1: now also U_FPGA.AD12; no longer U_FPGA.AD2
- net SFP_RX_N: now also U_FPGA.AD10; no longer U_FPGA.AC24
- net SFP_RX_P: now also U_FPGA.AD9; no longer U_FPGA.AC23
- net SFP_TX_N: now also U_FPGA.AD8; no longer U_FPGA.AC22
- net SFP_TX_P: now also U_FPGA.AD7; no longer U_FPGA.AC21
- net UART_RX: now also U_FPGA.AD24; no longer U_FPGA.AD14
- net UART_TX: now also U_FPGA.AD23; no longer U_FPGA.AD13
- net VCCINT_0V85: no longer U_FPGA.AD15, U_FPGA.AD17, U_FPGA.AD19, U_FPGA.AD21, U_FPGA.AD23
- net LINK5_CLOCK renamed LINK10_CLOCK
- net LINK5_DATA0 renamed LINK10_DATA0
- net LINK5_DATA1 renamed LINK10_DATA1
- net LINK5_DATA10 renamed LINK10_DATA10
- net LINK5_DATA11 renamed LINK10_DATA11
- net LINK5_DATA12 renamed LINK10_DATA12
- net LINK5_DATA13 renamed LINK10_DATA13
- net LINK5_DATA14 renamed LINK10_DATA14
- net LINK5_DATA15 renamed LINK10_DATA15
- net LINK5_DATA16 renamed LINK10_DATA16
- net LINK5_DATA17 renamed LINK10_DATA17
- net LINK5_DATA18 renamed LINK10_DATA18
- net LINK5_DATA19 renamed LINK10_DATA19
- net LINK5_DATA2 renamed LINK10_DATA2
- net LINK5_DATA20 renamed LINK10_DATA20
- net LINK5_DATA21 renamed LINK10_DATA21
- net LINK5_DATA22 renamed LINK10_DATA22
- net LINK5_DATA23 renamed LINK10_DATA23
- net LINK5_DATA24 renamed LINK10_DATA24
- net LINK5_DATA25 renamed LINK10_DATA25
- net LINK5_DATA26 renamed LINK10_DATA26
- net LINK5_DATA27 renamed LINK10_DATA27
- net LINK5_DATA28 renamed LINK10_DATA28
- net LINK5_DATA29 renamed LINK10_DATA29
- net LINK5_DATA3 renamed LINK10_DATA3
- net LINK5_DATA30 renamed LINK10_DATA30
- net LINK5_DATA31 renamed LINK10_DATA31
- net LINK5_DATA4 renamed LINK10_DATA4
- net LINK5_DATA5 renamed LINK10_DATA5
- net LINK5_DATA6 renamed LINK10_DATA6
- net LINK5_DATA7 renamed LINK10_DATA7
- net LINK5_DATA8 renamed LINK10_DATA8
- net LINK5_DATA9 renamed LINK10_DATA9
- net LINK5_READY_BACK renamed LINK10_READY_BACK
- net LINK5_SOF renamed LINK10_SOF
- net LINK5_VALID renamed LINK10_VALID
- new net MGMT_CS_A4: U_FPGA.AC12
- new net MGMT_CS_A5: U_FPGA.AC14
- new net MGMT_CS_A6: U_FPGA.AC16
- new net MGMT_CS_A7: U_FPGA.AC18
- new net MGMT_CS_H1: U_FPGA.AC22
- new net MGMT_IRQ_A4: U_FPGA.AC13
- new net MGMT_IRQ_A5: U_FPGA.AC15
- new net MGMT_IRQ_A6: U_FPGA.AC17
- new net MGMT_IRQ_A7: U_FPGA.AC19
- new net MGMT_IRQ_H1: U_FPGA.AC23
- new net REFCLK_A4_N: U_CLK.14
- new net REFCLK_A4_P: U_CLK.13
- new net REFCLK_A5_N: U_CLK.16
- new net REFCLK_A5_P: U_CLK.15
- new net REFCLK_A6_N: U_CLK.18
- new net REFCLK_A6_P: U_CLK.17
- new net REFCLK_A7_N: U_CLK.20
- new net REFCLK_A7_P: U_CLK.19
- new net REFCLK_H1_N: U_CLK.24
- new net REFCLK_H1_P: U_CLK.23
