File: hw/kicad_27b/power.kicad_sch (KiCad schematic)
At the start: 19 parts

Commit message: Pipeline a layer's passes, and re-rate the 27B board to eight layer dies
Two things the last commit left open.

The simulator now separates a layer stage's latency from its initiation
interval.  A layer is a chain of passes and each pass has its own via-
programmed tiles, so nothing is reused between them: the first pass is free
the moment its token moves on, and the stage holds as many tokens as fit
between its latency and its interval.  layer_pass_cycles carries the pass,
a quarter of the layer in every shipped geometry, which is the same figure
the single-pass head die already used.

I expected that to be worth four times and it is worth almost nothing,
because after the memory corrections it is the memory and not the pass rate
that binds.  It is exactly neutral on every LPDDR5X and PSRAM configuration
at any context count, worth 4 to 8 percent on the 9B with HBM, and slightly
negative on the 27B, where more tokens per stage lengthen latency against a
fixed pool of contexts.  With the bandwidth raised tenfold it is worth 2.5
times, 240K to 597K tokens/s, so the lever is real and nothing in reach of
this design is close enough to the fabric to collect it.  Letting a token's
state write overlap the next token's state read, which the same change
allows, is what does move the HBM numbers: the 3 nm 9B goes from 190K to
244K.

The 27B board is now eight layer ASICs of eight layers and two head ASICs
splitting the LM head, at 153K tokens/s rather than the 234K that came from
the un-corrected model.  Halving the per-die load takes the core rail from
650 A to 249 A, the package from a 55 x 55 array to 35 x 35, the cold plate
from 525 W to 200 W, and puts the ring on the same 11-gon as the 9B board.
hw/README's open item is replaced by the re-rating itself.

The 9B board's design point follows the same correction, 14.5K to 8.2K, and
its per-die traffic is 7.35 MB per token rather than the 4.2 MB of retrieval
alone.  Generated files now name the board description they came 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
Parts:
- added VRM_A4: core VRM VDD_CORE_A4, appliance:VRM_MODULE_26x6, symbol appliance:VRM_MODULE_26x6
- added VRM_A5: core VRM VDD_CORE_A5, appliance:VRM_MODULE_26x6, symbol appliance:VRM_MODULE_26x6
- added VRM_A6: core VRM VDD_CORE_A6, appliance:VRM_MODULE_26x6, symbol appliance:VRM_MODULE_26x6
- added VRM_A7: core VRM VDD_CORE_A7, appliance:VRM_MODULE_26x6, symbol appliance:VRM_MODULE_26x6
- added VRM_H1: core VRM VDD_CORE_H1, appliance:VRM_MODULE_26x6, symbol appliance:VRM_MODULE_26x6
Connections:
- net +12V: now also VRM_A4.1, VRM_A4.2, VRM_A4.3, VRM_A4.4, VRM_A5.1, VRM_A5.2, VRM_A5.3, VRM_A5.4, VRM_A6.1, VRM_A6.2, VRM_A6.3, VRM_A6.4, VRM_A7.1, VRM_A7.2, VRM_A7.3, VRM_A7.4, VRM_H1.1, VRM_H1.2, VRM_H1.3, VRM_H1.4
- net GND: now also VRM_A4.11, VRM_A4.12, VRM_A4.13, VRM_A4.14, VRM_A4.15, VRM_A4.16, VRM_A5.11, VRM_A5.12, VRM_A5.13, VRM_A5.14, VRM_A5.15, VRM_A5.16, VRM_A6.11, VRM_A6.12, VRM_A6.13, VRM_A6.14, VRM_A6.15, VRM_A6.16, VRM_A7.11, VRM_A7.12, VRM_A7.13, VRM_A7.14, VRM_A7.15, VRM_A7.16, VRM_H1.11, VRM_H1.12, VRM_H1.13, VRM_H1.14, VRM_H1.15, VRM_H1.16
- net PMB_SCL: now also VRM_A4.17, VRM_A5.17, VRM_A6.17, VRM_A7.17, VRM_H1.17
- net PMB_SDA: now also VRM_A4.18, VRM_A5.18, VRM_A6.18, VRM_A7.18, VRM_H1.18
- new net VDD_CORE_A4: VRM_A4.10, VRM_A4.5, VRM_A4.6, VRM_A4.7, VRM_A4.8, VRM_A4.9
- new net VDD_CORE_A5: VRM_A5.10, VRM_A5.5, VRM_A5.6, VRM_A5.7, VRM_A5.8, VRM_A5.9
- new net VDD_CORE_A6: VRM_A6.10, VRM_A6.5, VRM_A6.6, VRM_A6.7, VRM_A6.8, VRM_A6.9
- new net VDD_CORE_A7: VRM_A7.10, VRM_A7.5, VRM_A7.6, VRM_A7.7, VRM_A7.8, VRM_A7.9
- new net VDD_CORE_H1: VRM_H1.10, VRM_H1.5, VRM_H1.6, VRM_H1.7, VRM_H1.8, VRM_H1.9
- new net VRM_EN_A4: VRM_A4.19
- new net VRM_EN_A5: VRM_A5.19
- new net VRM_EN_A6: VRM_A6.19
- new net VRM_EN_A7: VRM_A7.19
- new net VRM_EN_H1: VRM_H1.19
