File: hw/kicad_psram/appliance.kicad_pcb (KiCad board)
At the start: 6 copper layers, 420 x 360 mm, 32 parts

Commit message: Fold the module row onto a short-depth 2U with surface-mount slots
The two facing rows of slots existed only to keep the closing hop short.
One row does the same: the outbound cards in the even positions running
away from the FPGA, the returning cards in the odd positions between them,
so ring order 0..9 sits at positions 0,2,4,6,8 and 9,7,5,3,1, every hop
skips one slot, the turn is a square U round the last slot and the ring
closes on the FPGA's east edge, which now carries both link ports side by
side as a card's die does.  The slots are surface-mount, so a ribbon on the
link layer passes beneath the slot it skips instead of weaving between
pins; their ground and 12 V pads get no via-in-pad, reaching the planes by
stubs clear of the ribbon corridor.

The slot field is then the card's 89 mm and the board drops from 420 x 360
to 420 x 160 mm, a short-depth 2U (2u_short) whose CRPS modules overhang
the board's front edge.  Hops end to end: 72 mm slot to slot at 34
degrees, 130 mm at the turn, 46 and 67 mm into and out of the FPGA.  The
two-row layout stays selectable (layout: two_rows on the 2u) and is kept
under test.

Co-Authored-By: Claude Fable 5.1 <noreply@anthropic.com>
Claude-Session: https://claude.ai/code/session_01VmmvkZe8Ctg3RAykNGsQBn
Parts:
- J_SLOT0, J_SLOT1, J_SLOT2, J_SLOT3, J_SLOT4, J_SLOT5, J_SLOT6, J_SLOT7, J_SLOT8, J_SLOT9: footprint appliance:PCIE_X16_SLOT -> appliance:PCIE_X16_SLOT_SMT
- moved U_BMC 232.0 mm to (50.0, 88.0)
- moved J_SLOT4 205.6 mm to (108.0, 122.0)
- moved J_SFP 201.4 mm to (56.0, 153.0)
- moved J_BMC_NET 200.4 mm to (38.0, 167.0)
- moved J_HOST 200.4 mm to (293.2, 174.0)
- moved J_SLOT3 200.0 mm to (152.0, 122.0)
- moved J_SLOT0 197.7 mm to (284.0, 122.0)
- moved J_SLOT2 196.8 mm to (196.0, 122.0)
- moved J_SLOT1 196.0 mm to (240.0, 122.0)
- moved REG_3V3 180.9 mm to (358.6, 103.5)
- moved REG_DDR 180.9 mm to (358.6, 125.5)
- moved REG_FPGA 180.9 mm to (327.2, 133.8)
- moved U_D0 180.9 mm to (348.1, 101.8)
- moved U_D1 180.9 mm to (348.1, 110.2)
- moved U_D2 180.9 mm to (348.1, 118.8)
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Connections:
- U_FPGA pad AA25: GND -> LINK0_DATA7
- U_FPGA pad AA26: VCCINT_0V85 -> LINK0_DATA6
- U_FPGA pad AB11: MGTAVTT -> VCCAUX_1V8
- U_FPGA pad AB17: VCCAUX_1V8 -> VCCO_1V8
- U_FPGA pad AB23: VCCO_1V8 -> VCCO_1V2
- U_FPGA pad AB25: VCCINT_0V85 -> LINK0_DATA5
- U_FPGA pad AB26: GND -> LINK0_DATA4
- U_FPGA pad AC25: GND -> LINK0_DATA3
- U_FPGA pad AC26: VCCINT_0V85 -> LINK0_DATA2
- U_FPGA pad AD25: VCCINT_0V85 -> LINK0_DATA1
- U_FPGA pad AD26: GND -> LINK0_DATA0
- U_FPGA pad AE11: LINK10_READY_BACK -> GND
- U_FPGA pad AE12: LINK10_CLOCK -> MGTAVTT
- U_FPGA pad AE13: LINK10_DATA6 -> GND
- U_FPGA pad AE14: LINK10_DATA4 -> VCCINT_0V85
- U_FPGA pad AE15: LINK10_DATA2 -> GND
- U_FPGA pad AE16: LINK10_DATA0 -> VCCINT_0V85
- U_FPGA pad AE18: MGTAVCC -> VCCAUX_1V8
- U_FPGA pad AE24: MGTAVTT -> VCCO_1V8
- U_FPGA pad AE6: VCCO_1V2 -> MGTAVCC
- U_FPGA pad AF11: LINK10_SOF -> VCCINT_0V85
- U_FPGA pad AF12: LINK10_VALID -> GND
- U_FPGA pad AF13: LINK10_DATA7 -> VCCINT_0V85
- U_FPGA pad AF14: LINK10_DATA5 -> GND
- U_FPGA pad AF15: LINK10_DATA3 -> VCCINT_0V85
- U_FPGA pad AF16: LINK10_DATA1 -> GND
- U_FPGA pad D25: VCCINT_0V85 -> LINK10_DATA0
- U_FPGA pad D26: GND -> LINK10_DATA1
- U_FPGA pad E25: GND -> LINK10_DATA2
- U_FPGA pad E26: VCCINT_0V85 -> LINK10_DATA3
- U_FPGA pad F25: VCCINT_0V85 -> LINK10_DATA4
- U_FPGA pad F26: GND -> LINK10_DATA5
- U_FPGA pad G25: GND -> LINK10_DATA6
- U_FPGA pad G26: VCCINT_0V85 -> LINK10_DATA7
- U_FPGA pad H25: VCCINT_0V85 -> LINK10_CLOCK
- U_FPGA pad H26: GND -> LINK10_VALID
- U_FPGA pad J25: GND -> LINK10_READY_BACK
- U_FPGA pad J26: VCCINT_0V85 -> LINK10_SOF
- U_FPGA pad L25: LINK0_SOF -> GND
- U_FPGA pad L26: LINK0_READY_BACK -> VCCINT_0V85
- U_FPGA pad M25: LINK0_VALID -> VCCINT_0V85
- U_FPGA pad M26: LINK0_CLOCK -> GND
- U_FPGA pad N25: LINK0_DATA7 -> GND
- U_FPGA pad N26: LINK0_DATA6 -> MGTAVCC
- U_FPGA pad P25: LINK0_DATA5 -> VCCINT_0V85
- U_FPGA pad P26: LINK0_DATA4 -> GND
- U_FPGA pad R25: LINK0_DATA3 -> GND
- U_FPGA pad R26: LINK0_DATA2 -> VCCINT_0V85
- U_FPGA pad T15: MGTAVTT -> VCCAUX_1V8
- U_FPGA pad T21: VCCAUX_1V8 -> VCCO_1V8
- U_FPGA pad T25: LINK0_DATA1 -> VCCINT_0V85
- U_FPGA pad T26: LINK0_DATA0 -> GND
- U_FPGA pad T9: MGTAVCC -> MGTAVTT
- U_FPGA pad W10: VCCO_1V8 -> VCCO_1V2
- U_FPGA pad W16: VCCO_1V2 -> MGTAVCC
- U_FPGA pad W22: MGTAVCC -> MGTAVTT
- U_FPGA pad W25: GND -> LINK0_SOF
- U_FPGA pad W26: VCCINT_0V85 -> LINK0_READY_BACK
- U_FPGA pad Y25: VCCINT_0V85 -> LINK0_VALID
- U_FPGA pad Y26: GND -> LINK0_CLOCK
Routing:
- net LINK5_SOF: track 104.2 -> 53.6 mm, vias 0 -> 2
- net LINK5_READY_BACK: track 100.2 -> 57.6 mm, vias 0 -> 2
- net LINK10_SOF: track 92.2 -> 50.1 mm, vias 1 -> 2
- net LINK10_READY_BACK: track 91.6 -> 51.1 mm, vias 1 -> 2
- net LINK10_VALID: track 88.7 -> 49.6 mm, vias 1 -> 2
- net LINK10_CLOCK: track 88.1 -> 50.6 mm, vias 1 -> 2
- net LINK5_DATA0: track 60.2 -> 97.6 mm, vias 0 -> 2
- net LINK10_DATA7: track 85.2 -> 49.3 mm, vias 1 -> 2
- net LINK5_VALID: track 96.2 -> 61.6 mm, vias 0 -> 2
- net LINK10_DATA6: track 84.7 -> 50.4 mm, vias 1 -> 2
- net LINK10_DATA5: track 81.9 -> 49.2 mm, vias 1 -> 2
- net LINK10_DATA4: track 81.5 -> 50.5 mm, vias 1 -> 2
- net LINK5_DATA1: track 64.2 -> 93.6 mm, vias 0 -> 2
- net LINK10_DATA3: track 78.7 -> 49.5 mm, vias 1 -> 2
- net LINK10_DATA2: track 78.3 -> 50.9 mm, vias 1 -> 2
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Other:
- board size 420 x 360 mm -> 420 x 160 mm
- board text added: "PSU bay (two CRPS, stacked, overhanging)"
- board text added: "appliance: short-depth 2U rack chassis, motherboard with a folded row of module slots, host-attached, floorplan generated from hw/board_psram.yaml"
- board text removed: "PSU bay (two CRPS, stacked)"
- board text removed: "appliance: 2U rack chassis, motherboard with module slots, host-attached, floorplan generated from hw/board_psram.yaml"

Commit message: Through-hole slots on the folded row, the two sets staggered past each other
A surface-mount x16 card-edge slot is not the commodity part, and the fold
only needed the skip-one ribbons to miss the skipped slot's pins.  Each
set's ribbon band runs at its link end, so shifting the two sets along the
cards by half a slot plus the band's clearance, 52 mm, puts every band past
the far end of the other set's pins with no weaving.  The stagger is derived
from the geometry and reported; slot_kind: smt keeps the single-line
arrangement for a surface-mount part.  The board is 420 x 180 mm, hops 83 mm
slot to slot, 183 mm at the turn, 73 and 89 mm at the FPGA.

Co-Authored-By: Claude Fable 5.1 <noreply@anthropic.com>
Claude-Session: https://claude.ai/code/session_01VmmvkZe8Ctg3RAykNGsQBn
Parts:
- J_SLOT0, J_SLOT1, J_SLOT2, J_SLOT3, J_SLOT4, J_SLOT5, J_SLOT6, J_SLOT7, J_SLOT8, J_SLOT9: footprint appliance:PCIE_X16_SLOT_SMT -> appliance:PCIE_X16_SLOT
- moved REG_IO 124.1 mm to (70.0, 70.0)
- moved U_CLK 124.1 mm to (50.0, 70.0)
- moved J_SLOT0 32.8 mm to (284.0, 89.2)
- moved J_SLOT1 32.8 mm to (240.0, 89.2)
- moved J_SLOT2 32.8 mm to (196.0, 89.2)
- moved J_SLOT3 32.8 mm to (152.0, 89.2)
- moved J_SLOT4 32.8 mm to (108.0, 89.2)
- moved J_HOST 20.4 mm to (297.2, 194.0)
- moved J_BMC_NET 20.0 mm to (38.0, 187.0)
- moved J_SFP 20.0 mm to (56.0, 173.0)
- moved J_SLOT5 20.0 mm to (86.0, 142.0)
- moved J_SLOT6 20.0 mm to (130.0, 142.0)
- moved J_SLOT7 20.0 mm to (174.0, 142.0)
- moved J_SLOT8 20.0 mm to (218.0, 142.0)
- moved J_SLOT9 20.0 mm to (262.0, 142.0)
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Routing:
- net LINK5_DATA4: track 81.6 -> 129.0 mm, vias 2 -> 0
- net LINK5_DATA3: track 85.6 -> 133.0 mm, vias 2 -> 0
- net LINK5_DATA2: track 89.6 -> 137.0 mm, vias 2 -> 0
- net LINK5_DATA1: track 93.6 -> 141.0 mm, vias 2 -> 0
- net LINK5_VALID: track 61.6 -> 109.0 mm, vias 2 -> 0
- net LINK5_SOF: track 53.6 -> 101.0 mm, vias 2 -> 0
- net LINK5_READY_BACK: track 57.6 -> 105.0 mm, vias 2 -> 0
- net LINK5_DATA7: track 69.6 -> 117.0 mm, vias 2 -> 0
- net LINK5_DATA6: track 73.6 -> 121.0 mm, vias 2 -> 0
- net LINK5_DATA5: track 77.6 -> 125.0 mm, vias 2 -> 0
- net LINK5_CLOCK: track 65.6 -> 113.0 mm, vias 2 -> 0
- net LINK5_DATA0: track 97.6 -> 145.0 mm, vias 2 -> 0
- net LINK0_DATA0: track 29.9 -> 54.2 mm, vias 2 -> 1
- net LINK0_DATA1: track 30.6 -> 54.5 mm, vias 2 -> 1
- net LINK0_DATA2: track 28.9 -> 52.5 mm, vias 2 -> 1
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Other:
- board size 420 x 160 mm -> 420 x 180 mm

Commit message: Link in and out on the same finger positions: straight slot-to-slot hops
link_in sits on side A and link_out on side B of the same twelve edge
positions, so a slot's out-row pin faces the next slot's in-row pin and
every skip-one hop is a straight ribbon.  On the card the two drops from
the die's south-edge blocks lean towards one finger span from either side
and cross, so the out drop takes In3 and the two faces' vias interleave
half a position apart above the fingers.  The ribbon band narrows from
27 mm to 12, the stagger from 52 mm to 38, and the short board from 180 to
170 mm deep.  finger_layout: offset keeps the earlier separate spans.

Co-Authored-By: Claude Fable 5.1 <noreply@anthropic.com>
Claude-Session: https://claude.ai/code/session_01VmmvkZe8Ctg3RAykNGsQBn
Parts:
- moved J_BMC_NET 10.0 mm to (38.0, 177.0)
- moved J_HOST 10.0 mm to (297.2, 184.0)
- moved J_SFP 10.0 mm to (56.0, 163.0)
- moved J_SLOT5 10.0 mm to (86.0, 132.0)
- moved J_SLOT6 10.0 mm to (130.0, 132.0)
- moved J_SLOT7 10.0 mm to (174.0, 132.0)
- moved J_SLOT8 10.0 mm to (218.0, 132.0)
- moved J_SLOT9 10.0 mm to (262.0, 132.0)
- moved REG_IO 10.0 mm to (70.0, 60.0)
- moved U_BMC 10.0 mm to (50.0, 98.0)
- moved U_CLK 10.0 mm to (50.0, 60.0)
- moved J_SLOT0 5.00 mm to (284.0, 94.2)
- moved J_SLOT1 5.00 mm to (240.0, 94.2)
- moved J_SLOT2 5.00 mm to (196.0, 94.2)
- moved J_SLOT3 5.00 mm to (152.0, 94.2)
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Connections:
- J_SLOT0 pad B12: GND -> LINK1_DATA0
- J_SLOT0 pad B13: GND -> LINK1_DATA1
- J_SLOT0 pad B14: GND -> LINK1_DATA2
- J_SLOT0 pad B15: GND -> LINK1_DATA3
- J_SLOT0 pad B16: GND -> LINK1_DATA4
- J_SLOT0 pad B17: GND -> LINK1_DATA5
- J_SLOT0 pad B18: GND -> LINK1_DATA6
- J_SLOT0 pad B19: GND -> LINK1_DATA7
- J_SLOT0 pad B20: GND -> LINK1_CLOCK
- J_SLOT0 pad B21: GND -> LINK1_VALID
- J_SLOT0 pad B22: GND -> LINK1_READY_BACK
- J_SLOT0 pad B23: GND -> LINK1_SOF
- J_SLOT0 pad B27: LINK1_DATA0 -> GND
- J_SLOT0 pad B28: LINK1_DATA1 -> GND
- J_SLOT0 pad B29: LINK1_DATA2 -> GND
- J_SLOT0 pad B30: LINK1_DATA3 -> GND
- J_SLOT0 pad B31: LINK1_DATA4 -> GND
- J_SLOT0 pad B32: LINK1_DATA5 -> GND
- J_SLOT0 pad B33: LINK1_DATA6 -> GND
- J_SLOT0 pad B34: LINK1_DATA7 -> GND
- J_SLOT0 pad B35: LINK1_CLOCK -> GND
- J_SLOT0 pad B36: LINK1_VALID -> GND
- J_SLOT0 pad B37: LINK1_READY_BACK -> GND
- J_SLOT0 pad B38: LINK1_SOF -> GND
- J_SLOT1 pad B12: GND -> LINK2_DATA0
- J_SLOT1 pad B13: GND -> LINK2_DATA1
- J_SLOT1 pad B14: GND -> LINK2_DATA2
- J_SLOT1 pad B15: GND -> LINK2_DATA3
- J_SLOT1 pad B16: GND -> LINK2_DATA4
- J_SLOT1 pad B17: GND -> LINK2_DATA5
- J_SLOT1 pad B18: GND -> LINK2_DATA6
- J_SLOT1 pad B19: GND -> LINK2_DATA7
- J_SLOT1 pad B20: GND -> LINK2_CLOCK
- J_SLOT1 pad B21: GND -> LINK2_VALID
- J_SLOT1 pad B22: GND -> LINK2_READY_BACK
- J_SLOT1 pad B23: GND -> LINK2_SOF
- J_SLOT1 pad B27: LINK2_DATA0 -> GND
- J_SLOT1 pad B28: LINK2_DATA1 -> GND
- J_SLOT1 pad B29: LINK2_DATA2 -> GND
- J_SLOT1 pad B30: LINK2_DATA3 -> GND
- J_SLOT1 pad B31: LINK2_DATA4 -> GND
- J_SLOT1 pad B32: LINK2_DATA5 -> GND
- J_SLOT1 pad B33: LINK2_DATA6 -> GND
- J_SLOT1 pad B34: LINK2_DATA7 -> GND
- J_SLOT1 pad B35: LINK2_CLOCK -> GND
- J_SLOT1 pad B36: LINK2_VALID -> GND
- J_SLOT1 pad B37: LINK2_READY_BACK -> GND
- J_SLOT1 pad B38: LINK2_SOF -> GND
- J_SLOT2 pad B12: GND -> LINK3_DATA0
- J_SLOT2 pad B13: GND -> LINK3_DATA1
- J_SLOT2 pad B14: GND -> LINK3_DATA2
- J_SLOT2 pad B15: GND -> LINK3_DATA3
- J_SLOT2 pad B16: GND -> LINK3_DATA4
- J_SLOT2 pad B17: GND -> LINK3_DATA5
- J_SLOT2 pad B18: GND -> LINK3_DATA6
- J_SLOT2 pad B19: GND -> LINK3_DATA7
- J_SLOT2 pad B20: GND -> LINK3_CLOCK
- J_SLOT2 pad B21: GND -> LINK3_VALID
- J_SLOT2 pad B22: GND -> LINK3_READY_BACK
- J_SLOT2 pad B23: GND -> LINK3_SOF
- J_SLOT2 pad B27: LINK3_DATA0 -> GND
- J_SLOT2 pad B28: LINK3_DATA1 -> GND
- J_SLOT2 pad B29: LINK3_DATA2 -> GND
- J_SLOT2 pad B30: LINK3_DATA3 -> GND
- J_SLOT2 pad B31: LINK3_DATA4 -> GND
- J_SLOT2 pad B32: LINK3_DATA5 -> GND
- J_SLOT2 pad B33: LINK3_DATA6 -> GND
- J_SLOT2 pad B34: LINK3_DATA7 -> GND
- J_SLOT2 pad B35: LINK3_CLOCK -> GND
- J_SLOT2 pad B36: LINK3_VALID -> GND
- J_SLOT2 pad B37: LINK3_READY_BACK -> GND
- J_SLOT2 pad B38: LINK3_SOF -> GND
- J_SLOT3 pad B12: GND -> LINK4_DATA0
- J_SLOT3 pad B13: GND -> LINK4_DATA1
- J_SLOT3 pad B14: GND -> LINK4_DATA2
- J_SLOT3 pad B15: GND -> LINK4_DATA3
- J_SLOT3 pad B16: GND -> LINK4_DATA4
- J_SLOT3 pad B17: GND -> LINK4_DATA5
- J_SLOT3 pad B18: GND -> LINK4_DATA6
- J_SLOT3 pad B19: GND -> LINK4_DATA7
- J_SLOT3 pad B20: GND -> LINK4_CLOCK
- J_SLOT3 pad B21: GND -> LINK4_VALID
- J_SLOT3 pad B22: GND -> LINK4_READY_BACK
- J_SLOT3 pad B23: GND -> LINK4_SOF
- J_SLOT3 pad B27: LINK4_DATA0 -> GND
- J_SLOT3 pad B28: LINK4_DATA1 -> GND
- J_SLOT3 pad B29: LINK4_DATA2 -> GND
- J_SLOT3 pad B30: LINK4_DATA3 -> GND
- J_SLOT3 pad B31: LINK4_DATA4 -> GND
- J_SLOT3 pad B32: LINK4_DATA5 -> GND
- J_SLOT3 pad B33: LINK4_DATA6 -> GND
- J_SLOT3 pad B34: LINK4_DATA7 -> GND
- J_SLOT3 pad B35: LINK4_CLOCK -> GND
- J_SLOT3 pad B36: LINK4_VALID -> GND
- J_SLOT3 pad B37: LINK4_READY_BACK -> GND
- J_SLOT3 pad B38: LINK4_SOF -> GND
- J_SLOT4 pad B12: GND -> LINK5_DATA0
- J_SLOT4 pad B13: GND -> LINK5_DATA1
- J_SLOT4 pad B14: GND -> LINK5_DATA2
- J_SLOT4 pad B15: GND -> LINK5_DATA3
- J_SLOT4 pad B16: GND -> LINK5_DATA4
- J_SLOT4 pad B17: GND -> LINK5_DATA5
- J_SLOT4 pad B18: GND -> LINK5_DATA6
- J_SLOT4 pad B19: GND -> LINK5_DATA7
- J_SLOT4 pad B20: GND -> LINK5_CLOCK
- J_SLOT4 pad B21: GND -> LINK5_VALID
- J_SLOT4 pad B22: GND -> LINK5_READY_BACK
- J_SLOT4 pad B23: GND -> LINK5_SOF
- J_SLOT4 pad B27: LINK5_DATA0 -> GND
- J_SLOT4 pad B28: LINK5_DATA1 -> GND
- J_SLOT4 pad B29: LINK5_DATA2 -> GND
- J_SLOT4 pad B30: LINK5_DATA3 -> GND
- J_SLOT4 pad B31: LINK5_DATA4 -> GND
- J_SLOT4 pad B32: LINK5_DATA5 -> GND
- J_SLOT4 pad B33: LINK5_DATA6 -> GND
- J_SLOT4 pad B34: LINK5_DATA7 -> GND
- J_SLOT4 pad B35: LINK5_CLOCK -> GND
- J_SLOT4 pad B36: LINK5_VALID -> GND
- J_SLOT4 pad B37: LINK5_READY_BACK -> GND
- J_SLOT4 pad B38: LINK5_SOF -> GND
- J_SLOT5 pad B12: GND -> LINK6_DATA0
- J_SLOT5 pad B13: GND -> LINK6_DATA1
- J_SLOT5 pad B14: GND -> LINK6_DATA2
- J_SLOT5 pad B15: GND -> LINK6_DATA3
- J_SLOT5 pad B16: GND -> LINK6_DATA4
- J_SLOT5 pad B17: GND -> LINK6_DATA5
- J_SLOT5 pad B18: GND -> LINK6_DATA6
- J_SLOT5 pad B19: GND -> LINK6_DATA7
- J_SLOT5 pad B20: GND -> LINK6_CLOCK
- J_SLOT5 pad B21: GND -> LINK6_VALID
- J_SLOT5 pad B22: GND -> LINK6_READY_BACK
- J_SLOT5 pad B23: GND -> LINK6_SOF
- J_SLOT5 pad B27: LINK6_DATA0 -> GND
- J_SLOT5 pad B28: LINK6_DATA1 -> GND
- J_SLOT5 pad B29: LINK6_DATA2 -> GND
- J_SLOT5 pad B30: LINK6_DATA3 -> GND
- J_SLOT5 pad B31: LINK6_DATA4 -> GND
- J_SLOT5 pad B32: LINK6_DATA5 -> GND
- J_SLOT5 pad B33: LINK6_DATA6 -> GND
- J_SLOT5 pad B34: LINK6_DATA7 -> GND
- J_SLOT5 pad B35: LINK6_CLOCK -> GND
- J_SLOT5 pad B36: LINK6_VALID -> GND
- J_SLOT5 pad B37: LINK6_READY_BACK -> GND
- J_SLOT5 pad B38: LINK6_SOF -> GND
- J_SLOT6 pad B12: GND -> LINK7_DATA0
- J_SLOT6 pad B13: GND -> LINK7_DATA1
- J_SLOT6 pad B14: GND -> LINK7_DATA2
- J_SLOT6 pad B15: GND -> LINK7_DATA3
- J_SLOT6 pad B16: GND -> LINK7_DATA4
- J_SLOT6 pad B17: GND -> LINK7_DATA5
- J_SLOT6 pad B18: GND -> LINK7_DATA6
- J_SLOT6 pad B19: GND -> LINK7_DATA7
- J_SLOT6 pad B20: GND -> LINK7_CLOCK
- J_SLOT6 pad B21: GND -> LINK7_VALID
- J_SLOT6 pad B22: GND -> LINK7_READY_BACK
- J_SLOT6 pad B23: GND -> LINK7_SOF
- J_SLOT6 pad B27: LINK7_DATA0 -> GND
- J_SLOT6 pad B28: LINK7_DATA1 -> GND
- J_SLOT6 pad B29: LINK7_DATA2 -> GND
- J_SLOT6 pad B30: LINK7_DATA3 -> GND
- J_SLOT6 pad B31: LINK7_DATA4 -> GND
- J_SLOT6 pad B32: LINK7_DATA5 -> GND
- J_SLOT6 pad B33: LINK7_DATA6 -> GND
- J_SLOT6 pad B34: LINK7_DATA7 -> GND
- J_SLOT6 pad B35: LINK7_CLOCK -> GND
- J_SLOT6 pad B36: LINK7_VALID -> GND
- J_SLOT6 pad B37: LINK7_READY_BACK -> GND
- J_SLOT6 pad B38: LINK7_SOF -> GND
- J_SLOT7 pad B12: GND -> LINK8_DATA0
- J_SLOT7 pad B13: GND -> LINK8_DATA1
- J_SLOT7 pad B14: GND -> LINK8_DATA2
- J_SLOT7 pad B15: GND -> LINK8_DATA3
- J_SLOT7 pad B16: GND -> LINK8_DATA4
- J_SLOT7 pad B17: GND -> LINK8_DATA5
- J_SLOT7 pad B18: GND -> LINK8_DATA6
- J_SLOT7 pad B19: GND -> LINK8_DATA7
- J_SLOT7 pad B20: GND -> LINK8_CLOCK
- J_SLOT7 pad B21: GND -> LINK8_VALID
- J_SLOT7 pad B22: GND -> LINK8_READY_BACK
- J_SLOT7 pad B23: GND -> LINK8_SOF
- J_SLOT7 pad B27: LINK8_DATA0 -> GND
- J_SLOT7 pad B28: LINK8_DATA1 -> GND
- J_SLOT7 pad B29: LINK8_DATA2 -> GND
- J_SLOT7 pad B30: LINK8_DATA3 -> GND
- J_SLOT7 pad B31: LINK8_DATA4 -> GND
- J_SLOT7 pad B32: LINK8_DATA5 -> GND
- J_SLOT7 pad B33: LINK8_DATA6 -> GND
- J_SLOT7 pad B34: LINK8_DATA7 -> GND
- J_SLOT7 pad B35: LINK8_CLOCK -> GND
- J_SLOT7 pad B36: LINK8_VALID -> GND
- J_SLOT7 pad B37: LINK8_READY_BACK -> GND
- J_SLOT7 pad B38: LINK8_SOF -> GND
- J_SLOT8 pad B12: GND -> LINK9_DATA0
- J_SLOT8 pad B13: GND -> LINK9_DATA1
- J_SLOT8 pad B14: GND -> LINK9_DATA2
- J_SLOT8 pad B15: GND -> LINK9_DATA3
- J_SLOT8 pad B16: GND -> LINK9_DATA4
- J_SLOT8 pad B17: GND -> LINK9_DATA5
- J_SLOT8 pad B18: GND -> LINK9_DATA6
- J_SLOT8 pad B19: GND -> LINK9_DATA7
- J_SLOT8 pad B20: GND -> LINK9_CLOCK
- J_SLOT8 pad B21: GND -> LINK9_VALID
- J_SLOT8 pad B22: GND -> LINK9_READY_BACK
- J_SLOT8 pad B23: GND -> LINK9_SOF
- J_SLOT8 pad B27: LINK9_DATA0 -> GND
- J_SLOT8 pad B28: LINK9_DATA1 -> GND
- J_SLOT8 pad B29: LINK9_DATA2 -> GND
- J_SLOT8 pad B30: LINK9_DATA3 -> GND
- J_SLOT8 pad B31: LINK9_DATA4 -> GND
- J_SLOT8 pad B32: LINK9_DATA5 -> GND
- J_SLOT8 pad B33: LINK9_DATA6 -> GND
- J_SLOT8 pad B34: LINK9_DATA7 -> GND
- J_SLOT8 pad B35: LINK9_CLOCK -> GND
- J_SLOT8 pad B36: LINK9_VALID -> GND
- J_SLOT8 pad B37: LINK9_READY_BACK -> GND
- J_SLOT8 pad B38: LINK9_SOF -> GND
- J_SLOT9 pad B12: GND -> LINK10_DATA0
- J_SLOT9 pad B13: GND -> LINK10_DATA1
- J_SLOT9 pad B14: GND -> LINK10_DATA2
- J_SLOT9 pad B15: GND -> LINK10_DATA3
- J_SLOT9 pad B16: GND -> LINK10_DATA4
- J_SLOT9 pad B17: GND -> LINK10_DATA5
- J_SLOT9 pad B18: GND -> LINK10_DATA6
- J_SLOT9 pad B19: GND -> LINK10_DATA7
- J_SLOT9 pad B20: GND -> LINK10_CLOCK
- J_SLOT9 pad B21: GND -> LINK10_VALID
- J_SLOT9 pad B22: GND -> LINK10_READY_BACK
- J_SLOT9 pad B23: GND -> LINK10_SOF
- J_SLOT9 pad B27: LINK10_DATA0 -> GND
- J_SLOT9 pad B28: LINK10_DATA1 -> GND
- J_SLOT9 pad B29: LINK10_DATA2 -> GND
- J_SLOT9 pad B30: LINK10_DATA3 -> GND
- J_SLOT9 pad B31: LINK10_DATA4 -> GND
- J_SLOT9 pad B32: LINK10_DATA5 -> GND
- J_SLOT9 pad B33: LINK10_DATA6 -> GND
- J_SLOT9 pad B34: LINK10_DATA7 -> GND
- J_SLOT9 pad B35: LINK10_CLOCK -> GND
- J_SLOT9 pad B36: LINK10_VALID -> GND
- J_SLOT9 pad B37: LINK10_READY_BACK -> GND
- J_SLOT9 pad B38: LINK10_SOF -> GND
Routing:
- net LINK9_VALID: track 45.1 -> 42.0 mm
- net LINK9_SOF: track 45.1 -> 42.0 mm
- net LINK9_READY_BACK: track 45.1 -> 42.0 mm
- net LINK9_DATA7: track 45.1 -> 42.0 mm
- net LINK9_DATA6: track 45.1 -> 42.0 mm
- net LINK9_DATA5: track 45.1 -> 42.0 mm
- net LINK9_DATA4: track 45.1 -> 42.0 mm
- net LINK9_DATA3: track 45.1 -> 42.0 mm
- net LINK9_DATA2: track 45.1 -> 42.0 mm
- net LINK9_DATA1: track 45.1 -> 42.0 mm
- net LINK9_DATA0: track 45.1 -> 42.0 mm
- net LINK9_CLOCK: track 45.1 -> 42.0 mm
- net LINK8_VALID: track 45.1 -> 42.0 mm
- net LINK8_SOF: track 45.1 -> 42.0 mm
- net LINK8_READY_BACK: track 45.1 -> 42.0 mm
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Other:
- board size 420 x 180 mm -> 420 x 170 mm

Commit message: Shorten the folded-row stagger and turn the FPGA to face the slot row
The through-hole slot stagger counted an escape allowance the ribbon band
never uses; deriving it from the slot's half body, the pin clearance and
the band's offset gives 29 mm instead of 38, and the short 2U board drops
from 170 to 160 mm deep.

The FPGA now sits at rotation 0 with link_out on its north edge into the
outbound set's band and link_in on its south edge beside PCIe, so neither
FPGA hop wraps round the package.  Its core regulator moves to the west
edge and the DDR4 with its regulators to the east, against the PSU bay.
fpga_ball_map takes an edge per port and place_fpga_neighbours takes the
DDR side and the regulator side; the two-row layout uses the shared helper
with its old placement.  The report quotes one rounded stagger figure.

Tests, README and the generated PSRAM outputs follow.

Co-Authored-By: Claude Fable 5.1 <noreply@anthropic.com>
Claude-Session: https://claude.ai/code/session_01VmmvkZe8Ctg3RAykNGsQBn
Parts:
- moved REG_FPGA 31.3 mm to (312.0, 107.7)
- moved U_D3 30.9 mm to (352.1, 95.0)
- moved REG_DDR 27.4 mm to (362.6, 96.7)
- moved U_D0 20.1 mm to (352.1, 120.5)
- moved REG_3V3 16.6 mm to (362.6, 118.7)
- moved U_D2 13.9 mm to (352.1, 103.5)
- moved J_BMC_NET 10.0 mm to (38.0, 167.0)
- moved J_HOST 10.0 mm to (297.2, 174.0)
- moved J_SFP 10.0 mm to (56.0, 153.0)
- moved J_SLOT5 10.0 mm to (86.0, 122.0)
- moved J_SLOT6 10.0 mm to (130.0, 122.0)
- moved J_SLOT7 10.0 mm to (174.0, 122.0)
- moved J_SLOT8 10.0 mm to (218.0, 122.0)
- moved J_SLOT9 10.0 mm to (262.0, 122.0)
- moved REG_IO 10.0 mm to (70.0, 50.0)
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Connections:
- U_FPGA pad A10: PCIE_TX3_N -> VCCO_1V8
- U_FPGA pad A11: PCIE_TX4_P -> LINK0_SOF
- U_FPGA pad A12: PCIE_TX4_N -> LINK0_VALID
- U_FPGA pad A13: PCIE_TX5_P -> LINK0_DATA7
- U_FPGA pad A14: PCIE_TX5_N -> LINK0_DATA5
- U_FPGA pad A15: PCIE_TX6_P -> LINK0_DATA3
- U_FPGA pad A16: PCIE_TX6_N -> LINK0_DATA1
- U_FPGA pad A17: PCIE_TX7_P -> GND
- U_FPGA pad A18: PCIE_TX7_N -> VCCINT_0V85
- U_FPGA pad A19: PCIE_RX0_P -> GND
- U_FPGA pad A20: PCIE_RX0_N -> VCCINT_0V85
- U_FPGA pad A21: PCIE_RX1_P -> GND
- U_FPGA pad A22: PCIE_RX1_N -> VCCO_1V2
- U_FPGA pad A23: PCIE_RX2_P -> GND
- U_FPGA pad A24: PCIE_RX2_N -> VCCINT_0V85
- U_FPGA pad A3: PCIE_TX0_P -> GND
- U_FPGA pad A4: PCIE_TX0_N -> VCCAUX_1V8
- U_FPGA pad A5: PCIE_TX1_P -> GND
- U_FPGA pad A6: PCIE_TX1_N -> VCCINT_0V85
- U_FPGA pad A7: PCIE_TX2_P -> GND
- U_FPGA pad A8: PCIE_TX2_N -> VCCINT_0V85
- U_FPGA pad A9: PCIE_TX3_P -> GND
- U_FPGA pad AA1: DDR4_DQ18 -> GND
- U_FPGA pad AA2: DDR4_DQ38 -> VCCINT_0V85
- U_FPGA pad AA20: VCCINT_0V85 -> DDR4_DQ18
- U_FPGA pad AA21: GND -> DDR4_DQ38
- U_FPGA pad AA22: VCCINT_0V85 -> DDR4_DQ58
- U_FPGA pad AA23: GND -> DDR4_DQS7_P
- U_FPGA pad AA24: VCCINT_0V85 -> DDR4_ADDR_CMD10
- U_FPGA pad AA25: LINK0_DATA7 -> DDR4_CTRL0
- U_FPGA pad AA26: LINK0_DATA6 -> VCCINT_0V85
- U_FPGA pad AA3: DDR4_DQ58 -> GND
- U_FPGA pad AA4: DDR4_DQS7_P -> VCCINT_0V85
- U_FPGA pad AA5: DDR4_ADDR_CMD10 -> GND
- U_FPGA pad AA6: DDR4_CTRL0 -> VCCINT_0V85
- U_FPGA pad AB1: DDR4_DQ19 -> VCCINT_0V85
- U_FPGA pad AB11: VCCAUX_1V8 -> MGTAVTT
- U_FPGA pad AB17: VCCO_1V8 -> VCCAUX_1V8
- U_FPGA pad AB2: DDR4_DQ39 -> GND
- U_FPGA pad AB20: GND -> DDR4_DQ19
- U_FPGA pad AB21: VCCINT_0V85 -> DDR4_DQ39
- U_FPGA pad AB22: GND -> DDR4_DQ59
- U_FPGA pad AB23: VCCO_1V2 -> DDR4_DQS7_N
- U_FPGA pad AB24: GND -> DDR4_ADDR_CMD11
- U_FPGA pad AB25: LINK0_DATA5 -> DDR4_CTRL1
- U_FPGA pad AB26: LINK0_DATA4 -> GND
- U_FPGA pad AB3: DDR4_DQ59 -> VCCINT_0V85
- U_FPGA pad AB4: DDR4_DQS7_N -> GND
- U_FPGA pad AB5: DDR4_ADDR_CMD11 -> MGTAVCC
- U_FPGA pad AB6: DDR4_CTRL1 -> GND
- U_FPGA pad AC25: LINK0_DATA3 -> GND
- U_FPGA pad AC26: LINK0_DATA2 -> VCCINT_0V85
- U_FPGA pad AD25: LINK0_DATA1 -> VCCINT_0V85
- U_FPGA pad AD26: LINK0_DATA0 -> GND
- U_FPGA pad AE1: GND -> PCIE_RX2_P
- U_FPGA pad AE10: VCCINT_0V85 -> PCIE_RX6_N
- U_FPGA pad AE11: GND -> LINK10_READY_BACK
- U_FPGA pad AE12: MGTAVTT -> LINK10_CLOCK
- U_FPGA pad AE13: GND -> LINK10_DATA6
- U_FPGA pad AE14: VCCINT_0V85 -> LINK10_DATA4
- U_FPGA pad AE15: GND -> LINK10_DATA2
- U_FPGA pad AE16: VCCINT_0V85 -> LINK10_DATA0
- U_FPGA pad AE17: GND -> PCIE_RX7_P
- U_FPGA pad AE18: VCCAUX_1V8 -> PCIE_RX7_N
- U_FPGA pad AE19: GND -> PCIE_REFCLK_P
- U_FPGA pad AE2: VCCINT_0V85 -> PCIE_RX2_N
- U_FPGA pad AE20: VCCINT_0V85 -> PCIE_REFCLK_N
- U_FPGA pad AE21: GND -> PCIE_PERST
- U_FPGA pad AE22: VCCINT_0V85 -> PCIE_WAKE
- U_FPGA pad AE3: GND -> PCIE_RX3_P
- U_FPGA pad AE4: VCCINT_0V85 -> PCIE_RX3_N
- U_FPGA pad AE5: GND -> PCIE_RX4_P
- U_FPGA pad AE6: MGTAVCC -> PCIE_RX4_N
- U_FPGA pad AE7: GND -> PCIE_RX5_P
- U_FPGA pad AE8: VCCINT_0V85 -> PCIE_RX5_N
- U_FPGA pad AE9: GND -> PCIE_RX6_P
- U_FPGA pad AF1: VCCINT_0V85 -> PCIE_TX0_P
- U_FPGA pad AF10: GND -> PCIE_TX4_N
- U_FPGA pad AF11: VCCINT_0V85 -> LINK10_SOF
- U_FPGA pad AF12: GND -> LINK10_VALID
- U_FPGA pad AF13: VCCINT_0V85 -> LINK10_DATA7
- U_FPGA pad AF14: GND -> LINK10_DATA5
- U_FPGA pad AF15: VCCINT_0V85 -> LINK10_DATA3
- U_FPGA pad AF16: GND -> LINK10_DATA1
- U_FPGA pad AF17: VCCINT_0V85 -> PCIE_TX5_P
- U_FPGA pad AF18: GND -> PCIE_TX5_N
- U_FPGA pad AF19: VCCINT_0V85 -> PCIE_TX6_P
- U_FPGA pad AF2: GND -> PCIE_TX0_N
- U_FPGA pad AF20: GND -> PCIE_TX6_N
- U_FPGA pad AF21: VCCINT_0V85 -> PCIE_TX7_P
- U_FPGA pad AF22: GND -> PCIE_TX7_N
- U_FPGA pad AF23: VCCINT_0V85 -> PCIE_RX0_P
- U_FPGA pad AF24: GND -> PCIE_RX0_N
- U_FPGA pad AF25: VCCINT_0V85 -> PCIE_RX1_P
- U_FPGA pad AF26: GND -> PCIE_RX1_N
- U_FPGA pad AF3: VCCINT_0V85 -> PCIE_TX1_P
- U_FPGA pad AF4: GND -> PCIE_TX1_N
- U_FPGA pad AF5: VCCINT_0V85 -> PCIE_TX2_P
- U_FPGA pad AF6: GND -> PCIE_TX2_N
- U_FPGA pad AF7: VCCINT_0V85 -> PCIE_TX3_P
- U_FPGA pad AF8: GND -> PCIE_TX3_N
- U_FPGA pad AF9: VCCINT_0V85 -> PCIE_TX4_P
- U_FPGA pad B10: PCIE_RX6_N -> GND
- U_FPGA pad B11: PCIE_RX7_P -> LINK0_READY_BACK
- U_FPGA pad B12: PCIE_RX7_N -> LINK0_CLOCK
- U_FPGA pad B13: PCIE_REFCLK_P -> LINK0_DATA6
- U_FPGA pad B14: PCIE_REFCLK_N -> LINK0_DATA4
- U_FPGA pad B15: PCIE_PERST -> LINK0_DATA2
- U_FPGA pad B16: PCIE_WAKE -> LINK0_DATA0
- U_FPGA pad B3: PCIE_RX3_P -> VCCINT_0V85
- U_FPGA pad B4: PCIE_RX3_N -> GND
- U_FPGA pad B5: PCIE_RX4_P -> VCCINT_0V85
- U_FPGA pad B6: PCIE_RX4_N -> GND
- U_FPGA pad B7: PCIE_RX5_P -> VCCINT_0V85
- U_FPGA pad B8: PCIE_RX5_N -> GND
- U_FPGA pad B9: PCIE_RX6_P -> VCCINT_0V85
- U_FPGA pad C1: DDR4_DQ0 -> GND
- U_FPGA pad C2: DDR4_DQ20 -> VCCINT_0V85
- U_FPGA pad C20: VCCINT_0V85 -> DDR4_DQ0
- U_FPGA pad C21: GND -> DDR4_DQ20
- U_FPGA pad C22: VCCINT_0V85 -> DDR4_DQ40
- U_FPGA pad C23: GND -> DDR4_DQ60
- U_FPGA pad C24: VCCINT_0V85 -> DDR4_DM0
- U_FPGA pad C25: GND -> DDR4_ADDR_CMD12
- U_FPGA pad C26: VCCINT_0V85 -> DDR4_CTRL2
- U_FPGA pad C3: DDR4_DQ40 -> GND
- U_FPGA pad C4: DDR4_DQ60 -> VCCINT_0V85
- U_FPGA pad C5: DDR4_DM0 -> GND
- U_FPGA pad C6: DDR4_ADDR_CMD12 -> VCCINT_0V85
- U_FPGA pad C7: DDR4_CTRL2 -> GND
- U_FPGA pad D1: DDR4_DQ1 -> VCCINT_0V85
- U_FPGA pad D11: VCCAUX_1V8 -> MGTAVTT
- U_FPGA pad D17: VCCO_1V8 -> VCCAUX_1V8
- U_FPGA pad D2: DDR4_DQ21 -> GND
- U_FPGA pad D20: GND -> DDR4_DQ1
- U_FPGA pad D21: VCCINT_0V85 -> DDR4_DQ21
- U_FPGA pad D22: GND -> DDR4_DQ41
- U_FPGA pad D23: VCCO_1V2 -> DDR4_DQ61
- U_FPGA pad D24: GND -> DDR4_DM1
- U_FPGA pad D25: LINK10_DATA0 -> DDR4_ADDR_CMD13
- U_FPGA pad D26: LINK10_DATA1 -> DDR4_CTRL3
- U_FPGA pad D3: DDR4_DQ41 -> VCCINT_0V85
- U_FPGA pad D4: DDR4_DQ61 -> GND
- U_FPGA pad D5: DDR4_DM1 -> MGTAVCC
- U_FPGA pad D6: DDR4_ADDR_CMD13 -> GND
- U_FPGA pad D7: DDR4_CTRL3 -> VCCINT_0V85
- U_FPGA pad E1: DDR4_DQ2 -> GND
- U_FPGA pad E2: DDR4_DQ22 -> VCCINT_0V85
- U_FPGA pad E20: VCCINT_0V85 -> DDR4_DQ2
- U_FPGA pad E21: GND -> DDR4_DQ22
- U_FPGA pad E22: VCCINT_0V85 -> DDR4_DQ42
- U_FPGA pad E23: GND -> DDR4_DQ62
- U_FPGA pad E24: VCCINT_0V85 -> DDR4_DM2
- U_FPGA pad E25: LINK10_DATA2 -> DDR4_ADDR_CMD14
- U_FPGA pad E26: LINK10_DATA3 -> DDR4_CTRL4
- U_FPGA pad E3: DDR4_DQ42 -> GND
- U_FPGA pad E4: DDR4_DQ62 -> VCCINT_0V85
- U_FPGA pad E5: DDR4_DM2 -> GND
- U_FPGA pad E6: DDR4_ADDR_CMD14 -> VCCINT_0V85
- U_FPGA pad E7: DDR4_CTRL4 -> GND
- U_FPGA pad F1: DDR4_DQ3 -> VCCINT_0V85
- U_FPGA pad F2: DDR4_DQ23 -> GND
- U_FPGA pad F20: GND -> DDR4_DQ3
- U_FPGA pad F21: VCCINT_0V85 -> DDR4_DQ23
- U_FPGA pad F22: GND -> DDR4_DQ43
- U_FPGA pad F23: VCCINT_0V85 -> DDR4_DQ63
- U_FPGA pad F24: GND -> DDR4_DM3
- U_FPGA pad F25: LINK10_DATA4 -> DDR4_ADDR_CMD15
- U_FPGA pad F26: LINK10_DATA5 -> DDR4_CTRL5
- U_FPGA pad F3: DDR4_DQ43 -> VCCINT_0V85
- U_FPGA pad F4: DDR4_DQ63 -> GND
- U_FPGA pad F5: DDR4_DM3 -> VCCINT_0V85
- U_FPGA pad F6: DDR4_ADDR_CMD15 -> GND
- U_FPGA pad F7: DDR4_CTRL5 -> VCCINT_0V85
- U_FPGA pad G1: DDR4_DQ4 -> GND
- U_FPGA pad G12: MGTAVCC -> VCCO_1V2
- U_FPGA pad G18: MGTAVTT -> MGTAVCC
- U_FPGA pad G2: DDR4_DQ24 -> VCCINT_0V85
- U_FPGA pad G20: VCCINT_0V85 -> DDR4_DQ4
- U_FPGA pad G21: GND -> DDR4_DQ24
- U_FPGA pad G22: VCCINT_0V85 -> DDR4_DQ44
- U_FPGA pad G23: GND -> DDR4_DQS0_P
- U_FPGA pad G24: VCCAUX_1V8 -> DDR4_DM4
- U_FPGA pad G25: LINK10_DATA6 -> DDR4_ADDR_CMD16
- U_FPGA pad G26: LINK10_DATA7 -> VCCINT_0V85
- U_FPGA pad G3: DDR4_DQ44 -> GND
- U_FPGA pad G4: DDR4_DQS0_P -> VCCINT_0V85
- U_FPGA pad G5: DDR4_DM4 -> GND
- U_FPGA pad G6: DDR4_ADDR_CMD16 -> VCCO_1V8
- U_FPGA pad H1: DDR4_DQ5 -> VCCINT_0V85
- U_FPGA pad H2: DDR4_DQ25 -> GND
- U_FPGA pad H20: GND -> DDR4_DQ5
- U_FPGA pad H21: VCCINT_0V85 -> DDR4_DQ25
- U_FPGA pad H22: GND -> DDR4_DQ45
- U_FPGA pad H23: VCCINT_0V85 -> DDR4_DQS0_N
- U_FPGA pad H24: GND -> DDR4_DM5
- U_FPGA pad H25: LINK10_CLOCK -> DDR4_ADDR_CMD17
- U_FPGA pad H26: LINK10_VALID -> GND
- U_FPGA pad H3: DDR4_DQ45 -> VCCINT_0V85
- U_FPGA pad H4: DDR4_DQS0_N -> GND
- U_FPGA pad H5: DDR4_DM5 -> VCCINT_0V85
- U_FPGA pad H6: DDR4_ADDR_CMD17 -> GND
- U_FPGA pad J1: DDR4_DQ6 -> GND
- U_FPGA pad J2: DDR4_DQ26 -> VCCINT_0V85
- U_FPGA pad J20: VCCINT_0V85 -> DDR4_DQ6
- U_FPGA pad J21: GND -> DDR4_DQ26
- U_FPGA pad J22: VCCINT_0V85 -> DDR4_DQ46
- U_FPGA pad J23: GND -> DDR4_DQS1_P
- U_FPGA pad J24: VCCINT_0V85 -> DDR4_DM6
- U_FPGA pad J25: LINK10_READY_BACK -> DDR4_ADDR_CMD18
- U_FPGA pad J26: LINK10_SOF -> VCCINT_0V85
- U_FPGA pad J3: DDR4_DQ46 -> GND
- U_FPGA pad J4: DDR4_DQS1_P -> VCCINT_0V85
- U_FPGA pad J5: DDR4_DM6 -> GND
- U_FPGA pad J6: DDR4_ADDR_CMD18 -> VCCINT_0V85
- U_FPGA pad K1: DDR4_DQ7 -> MGTAVTT
- U_FPGA pad K13: VCCO_1V2 -> VCCO_1V8
- U_FPGA pad K19: MGTAVCC -> VCCO_1V2
- U_FPGA pad K2: DDR4_DQ27 -> GND
- U_FPGA pad K20: GND -> DDR4_DQ7
- U_FPGA pad K21: VCCINT_0V85 -> DDR4_DQ27
- U_FPGA pad K22: GND -> DDR4_DQ47
- U_FPGA pad K23: VCCINT_0V85 -> DDR4_DQS1_N
- U_FPGA pad K24: GND -> DDR4_DM7
- U_FPGA pad K25: MGTAVTT -> DDR4_ADDR_CMD19
- U_FPGA pad K3: DDR4_DQ47 -> VCCINT_0V85
- U_FPGA pad K4: DDR4_DQS1_N -> GND
- U_FPGA pad K5: DDR4_DM7 -> VCCINT_0V85
- U_FPGA pad K6: DDR4_ADDR_CMD19 -> GND
- U_FPGA pad K7: VCCO_1V8 -> VCCAUX_1V8
- U_FPGA pad L1: DDR4_DQ8 -> GND
- U_FPGA pad L2: DDR4_DQ28 -> VCCINT_0V85
- U_FPGA pad L20: VCCINT_0V85 -> DDR4_DQ8
- U_FPGA pad L21: GND -> DDR4_DQ28
- U_FPGA pad L22: VCCINT_0V85 -> DDR4_DQ48
- U_FPGA pad L23: GND -> DDR4_DQS2_P
- U_FPGA pad L24: VCCINT_0V85 -> DDR4_ADDR_CMD0
- U_FPGA pad L25: GND -> DDR4_ADDR_CMD20
- U_FPGA pad L3: DDR4_DQ48 -> GND
- U_FPGA pad L4: DDR4_DQS2_P -> VCCINT_0V85
- U_FPGA pad L5: DDR4_ADDR_CMD0 -> GND
- U_FPGA pad L6: DDR4_ADDR_CMD20 -> VCCINT_0V85
- U_FPGA pad M1: DDR4_DQ9 -> VCCINT_0V85
- U_FPGA pad M2: DDR4_DQ29 -> GND
- U_FPGA pad M20: GND -> DDR4_DQ9
- U_FPGA pad M21: VCCINT_0V85 -> DDR4_DQ29
- U_FPGA pad M22: GND -> DDR4_DQ49
- U_FPGA pad M23: VCCINT_0V85 -> DDR4_DQS2_N
- U_FPGA pad M24: GND -> DDR4_ADDR_CMD1
- U_FPGA pad M25: VCCINT_0V85 -> DDR4_ADDR_CMD21
- U_FPGA pad M3: DDR4_DQ49 -> VCCINT_0V85
- U_FPGA pad M4: DDR4_DQS2_N -> GND
- U_FPGA pad M5: DDR4_ADDR_CMD1 -> VCCINT_0V85
- U_FPGA pad M6: DDR4_ADDR_CMD21 -> GND
- U_FPGA pad N1: DDR4_DQ10 -> GND
- U_FPGA pad N14: VCCO_1V8 -> VCCAUX_1V8
- U_FPGA pad N2: DDR4_DQ30 -> MGTAVCC
- U_FPGA pad N20: VCCO_1V2 -> DDR4_DQ10
- U_FPGA pad N21: GND -> DDR4_DQ30
- U_FPGA pad N22: VCCINT_0V85 -> DDR4_DQ50
- U_FPGA pad N23: GND -> DDR4_DQS3_P
- U_FPGA pad N24: VCCINT_0V85 -> DDR4_ADDR_CMD2
- U_FPGA pad N25: GND -> DDR4_ADDR_CMD22
- U_FPGA pad N26: MGTAVCC -> VCCO_1V8
- U_FPGA pad N3: DDR4_DQ50 -> GND
- U_FPGA pad N4: DDR4_DQS3_P -> VCCINT_0V85
- U_FPGA pad N5: DDR4_ADDR_CMD2 -> GND
- U_FPGA pad N6: DDR4_ADDR_CMD22 -> VCCINT_0V85
- U_FPGA pad N8: VCCAUX_1V8 -> MGTAVTT
- U_FPGA pad P1: DDR4_DQ11 -> VCCINT_0V85
- U_FPGA pad P2: DDR4_DQ31 -> GND
- U_FPGA pad P20: GND -> DDR4_DQ11
- U_FPGA pad P21: VCCINT_0V85 -> DDR4_DQ31
- U_FPGA pad P22: GND -> DDR4_DQ51
- U_FPGA pad P23: VCCINT_0V85 -> DDR4_DQS3_N
- U_FPGA pad P24: GND -> DDR4_ADDR_CMD3
- U_FPGA pad P25: VCCINT_0V85 -> DDR4_ADDR_CMD23
- U_FPGA pad P3: DDR4_DQ51 -> VCCINT_0V85
- U_FPGA pad P4: DDR4_DQS3_N -> GND
- U_FPGA pad P5: DDR4_ADDR_CMD3 -> VCCINT_0V85
- U_FPGA pad P6: DDR4_ADDR_CMD23 -> GND
- U_FPGA pad R1: DDR4_DQ12 -> GND
- U_FPGA pad R2: DDR4_DQ32 -> VCCINT_0V85
- U_FPGA pad R20: VCCINT_0V85 -> DDR4_DQ12
- U_FPGA pad R21: GND -> DDR4_DQ32
- U_FPGA pad R22: VCCINT_0V85 -> DDR4_DQ52
- U_FPGA pad R23: GND -> DDR4_DQS4_P
- U_FPGA pad R24: VCCINT_0V85 -> DDR4_ADDR_CMD4
- U_FPGA pad R25: GND -> DDR4_ADDR_CMD24
- U_FPGA pad R3: DDR4_DQ52 -> GND
- U_FPGA pad R4: DDR4_DQS4_P -> VCCINT_0V85
- U_FPGA pad R5: DDR4_ADDR_CMD4 -> GND
- U_FPGA pad R6: DDR4_ADDR_CMD24 -> VCCINT_0V85
- U_FPGA pad T1: DDR4_DQ13 -> VCCINT_0V85
- U_FPGA pad T15: VCCAUX_1V8 -> MGTAVTT
- U_FPGA pad T2: DDR4_DQ33 -> GND
- U_FPGA pad T20: GND -> DDR4_DQ13
- U_FPGA pad T21: VCCO_1V8 -> DDR4_DQ33
- U_FPGA pad T22: GND -> DDR4_DQ53
- U_FPGA pad T23: VCCINT_0V85 -> DDR4_DQS4_N
- U_FPGA pad T24: GND -> DDR4_ADDR_CMD5
- U_FPGA pad T25: VCCINT_0V85 -> DDR4_ADDR_CMD25
- U_FPGA pad T3: DDR4_DQ53 -> VCCO_1V2
- U_FPGA pad T4: DDR4_DQS4_N -> GND
- U_FPGA pad T5: DDR4_ADDR_CMD5 -> VCCINT_0V85
- U_FPGA pad T6: DDR4_ADDR_CMD25 -> GND
- U_FPGA pad T9: MGTAVTT -> MGTAVCC
- U_FPGA pad U1: DDR4_DQ14 -> GND
- U_FPGA pad U2: DDR4_DQ34 -> VCCINT_0V85
- U_FPGA pad U20: VCCINT_0V85 -> DDR4_DQ14
- U_FPGA pad U21: GND -> DDR4_DQ34
- U_FPGA pad U22: VCCINT_0V85 -> DDR4_DQ54
- U_FPGA pad U23: GND -> DDR4_DQS5_P
- U_FPGA pad U24: VCCINT_0V85 -> DDR4_ADDR_CMD6
- U_FPGA pad U25: GND -> DDR4_ADDR_CMD26
- U_FPGA pad U3: DDR4_DQ54 -> GND
- U_FPGA pad U4: DDR4_DQS5_P -> VCCINT_0V85
- U_FPGA pad U5: DDR4_ADDR_CMD6 -> GND
- U_FPGA pad U6: DDR4_ADDR_CMD26 -> VCCINT_0V85
- U_FPGA pad V1: DDR4_DQ15 -> VCCINT_0V85
- U_FPGA pad V2: DDR4_DQ35 -> GND
- U_FPGA pad V20: GND -> DDR4_DQ15
- U_FPGA pad V21: VCCINT_0V85 -> DDR4_DQ35
- U_FPGA pad V22: GND -> DDR4_DQ55
- U_FPGA pad V23: VCCINT_0V85 -> DDR4_DQS5_N
- U_FPGA pad V24: GND -> DDR4_ADDR_CMD7
- U_FPGA pad V25: VCCINT_0V85 -> DDR4_ADDR_CMD27
- U_FPGA pad V3: DDR4_DQ55 -> VCCINT_0V85
- U_FPGA pad V4: DDR4_DQS5_N -> GND
- U_FPGA pad V5: DDR4_ADDR_CMD7 -> VCCINT_0V85
- U_FPGA pad V6: DDR4_ADDR_CMD27 -> GND
- U_FPGA pad W1: DDR4_DQ16 -> GND
- U_FPGA pad W10: VCCO_1V2 -> VCCO_1V8
- U_FPGA pad W16: MGTAVCC -> VCCO_1V2
- U_FPGA pad W2: DDR4_DQ36 -> VCCINT_0V85
- U_FPGA pad W20: VCCINT_0V85 -> DDR4_DQ16
- U_FPGA pad W21: GND -> DDR4_DQ36
- U_FPGA pad W22: MGTAVTT -> DDR4_DQ56
- U_FPGA pad W23: GND -> DDR4_DQS6_P
- U_FPGA pad W24: VCCINT_0V85 -> DDR4_ADDR_CMD8
- U_FPGA pad W25: LINK0_SOF -> DDR4_CK_P
- U_FPGA pad W26: LINK0_READY_BACK -> VCCINT_0V85
- U_FPGA pad W3: DDR4_DQ56 -> GND
- U_FPGA pad W4: DDR4_DQS6_P -> VCCAUX_1V8
- U_FPGA pad W5: DDR4_ADDR_CMD8 -> GND
- U_FPGA pad W6: DDR4_CK_P -> VCCINT_0V85
- U_FPGA pad Y1: DDR4_DQ17 -> VCCINT_0V85
- U_FPGA pad Y2: DDR4_DQ37 -> GND
- U_FPGA pad Y20: GND -> DDR4_DQ17
- U_FPGA pad Y21: VCCINT_0V85 -> DDR4_DQ37
- U_FPGA pad Y22: GND -> DDR4_DQ57
- U_FPGA pad Y23: VCCINT_0V85 -> DDR4_DQS6_N
- U_FPGA pad Y24: GND -> DDR4_ADDR_CMD9
- U_FPGA pad Y25: LINK0_VALID -> DDR4_CK_N
- U_FPGA pad Y26: LINK0_CLOCK -> GND
- U_FPGA pad Y3: DDR4_DQ57 -> VCCINT_0V85
- U_FPGA pad Y4: DDR4_DQS6_N -> GND
- U_FPGA pad Y5: DDR4_ADDR_CMD9 -> VCCINT_0V85
- U_FPGA pad Y6: DDR4_CK_N -> GND
Routing:
- net LINK10_DATA0: track 70.4 -> 88.9 mm
- net LINK10_DATA1: track 68.6 -> 85.8 mm
- net LINK10_DATA2: track 69.3 -> 85.1 mm
- net LINK10_DATA3: track 67.7 -> 82.0 mm
- net LINK0_DATA0: track 54.2 -> 67.9 mm
- net LINK10_DATA4: track 68.7 -> 81.3 mm
- net LINK0_DATA2: track 52.5 -> 64.1 mm
- net LINK10_DATA5: track 67.4 -> 78.3 mm
- net LINK0_DATA1: track 54.5 -> 64.8 mm
- net LINK5_DATA4: track 129.0 -> 119.7 mm
- net LINK5_DATA3: track 133.0 -> 123.7 mm
- net LINK5_DATA2: track 137.0 -> 127.7 mm
- net LINK5_VALID: track 109.0 -> 99.7 mm
- net LINK5_SOF: track 101.0 -> 91.7 mm
- net LINK5_READY_BACK: track 105.0 -> 95.7 mm
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Other:
- board size 420 x 170 mm -> 420 x 160 mm
