File: hw/kicad_psram/appliance.kicad_pcb (KiCad board)
At the start: 6 copper layers, 420 x 160 mm, 32 parts

Commit message: Choose the PSRAM board's FPGA: XCAU15P-2FFVB676E, with the fit checked
The controller FPGA is the AMD Artix UltraScale+ AU15P in FFVB676, the
one Artix UltraScale+ package whose transceivers run at 16.3 Gb/s and
whose PCIe block is Gen4 x8, so the host link stays as specified.  The
class records the part's resources and an io_plan (DDR4 on the HP
banks, the transceiver pairs on the GTH quads, the rest on HD), and
board.py checks and reports the fit: 124 of 156 HP I/O, 52 of 72 HD,
9 of 12 lanes.  The KiCad FPGA symbol carries the part number when the
class names one.

Co-Authored-By: Claude Fable 5.1 <noreply@anthropic.com>
Claude-Session: https://claude.ai/code/session_01VmmvkZe8Ctg3RAykNGsQBn
Parts:
- U_FPGA: value FPGA -> XCAU15P-2FFVB676E
Changed lines of the file:
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@@
     (attr smd)
     (fp_text reference "U_FPGA" (at 0 0) (layer "F.SilkS") (effects (font (size 1.5 1.5) (thickness 0.2))))
-    (fp_text value "FPGA" (at 0 2) (layer "F.Fab") (effects (font (size 1 1) (thickness 0.15))))
+    (fp_text value "XCAU15P-2FFVB676E" (at 0 2) (layer "F.Fab") (effects (font (size 1 1) (thickness 0.15))))
     (fp_poly (pts (xy -13.5 13.5) (xy 13.5 13.5) (xy 13.5 -13.5) (xy -13.5 -13.5)) (stroke (width 0.1) (type default)) (fill none) (layer "F.SilkS"))
     (fp_poly (pts (xy -14 14) (xy 14 14) (xy 14 -14) (xy -14 -14)) (stroke (width 0.1) (type default)) (fill none) (layer "F.CrtYd"))
