File: hw/kicad_psram/asics.kicad_sch (KiCad schematic)
At the start: 10 parts

Commit message: Fold the module row onto a short-depth 2U with surface-mount slots
The two facing rows of slots existed only to keep the closing hop short.
One row does the same: the outbound cards in the even positions running
away from the FPGA, the returning cards in the odd positions between them,
so ring order 0..9 sits at positions 0,2,4,6,8 and 9,7,5,3,1, every hop
skips one slot, the turn is a square U round the last slot and the ring
closes on the FPGA's east edge, which now carries both link ports side by
side as a card's die does.  The slots are surface-mount, so a ribbon on the
link layer passes beneath the slot it skips instead of weaving between
pins; their ground and 12 V pads get no via-in-pad, reaching the planes by
stubs clear of the ribbon corridor.

The slot field is then the card's 89 mm and the board drops from 420 x 360
to 420 x 160 mm, a short-depth 2U (2u_short) whose CRPS modules overhang
the board's front edge.  Hops end to end: 72 mm slot to slot at 34
degrees, 130 mm at the turn, 46 and 67 mm into and out of the FPGA.  The
two-row layout stays selectable (layout: two_rows on the 2u) and is kept
under test.

Co-Authored-By: Claude Fable 5.1 <noreply@anthropic.com>
Claude-Session: https://claude.ai/code/session_01VmmvkZe8Ctg3RAykNGsQBn
Parts:
- removed J_SLOT0: slot for U_A0, appliance:PCIE_X16_SLOT, symbol appliance:PCIE_X16_SLOT
- removed J_SLOT1: slot for U_A1, appliance:PCIE_X16_SLOT, symbol appliance:PCIE_X16_SLOT
- removed J_SLOT2: slot for U_A2, appliance:PCIE_X16_SLOT, symbol appliance:PCIE_X16_SLOT
- removed J_SLOT3: slot for U_A3, appliance:PCIE_X16_SLOT, symbol appliance:PCIE_X16_SLOT
- removed J_SLOT4: slot for U_A4, appliance:PCIE_X16_SLOT, symbol appliance:PCIE_X16_SLOT
- removed J_SLOT5: slot for U_A5, appliance:PCIE_X16_SLOT, symbol appliance:PCIE_X16_SLOT
- removed J_SLOT6: slot for U_A6, appliance:PCIE_X16_SLOT, symbol appliance:PCIE_X16_SLOT
- removed J_SLOT7: slot for U_A7, appliance:PCIE_X16_SLOT, symbol appliance:PCIE_X16_SLOT
- removed J_SLOT8: slot for U_H0, appliance:PCIE_X16_SLOT, symbol appliance:PCIE_X16_SLOT
- removed J_SLOT9: slot for U_H1, appliance:PCIE_X16_SLOT, symbol appliance:PCIE_X16_SLOT
- added J_SLOT0: slot for U_A0, appliance:PCIE_X16_SLOT_SMT, symbol appliance:PCIE_X16_SLOT_SMT
- added J_SLOT1: slot for U_A1, appliance:PCIE_X16_SLOT_SMT, symbol appliance:PCIE_X16_SLOT_SMT
- added J_SLOT2: slot for U_A2, appliance:PCIE_X16_SLOT_SMT, symbol appliance:PCIE_X16_SLOT_SMT
- added J_SLOT3: slot for U_A3, appliance:PCIE_X16_SLOT_SMT, symbol appliance:PCIE_X16_SLOT_SMT
- added J_SLOT4: slot for U_A4, appliance:PCIE_X16_SLOT_SMT, symbol appliance:PCIE_X16_SLOT_SMT
- added J_SLOT5: slot for U_A5, appliance:PCIE_X16_SLOT_SMT, symbol appliance:PCIE_X16_SLOT_SMT
- added J_SLOT6: slot for U_A6, appliance:PCIE_X16_SLOT_SMT, symbol appliance:PCIE_X16_SLOT_SMT
- added J_SLOT7: slot for U_A7, appliance:PCIE_X16_SLOT_SMT, symbol appliance:PCIE_X16_SLOT_SMT
- added J_SLOT8: slot for U_H0, appliance:PCIE_X16_SLOT_SMT, symbol appliance:PCIE_X16_SLOT_SMT
- added J_SLOT9: slot for U_H1, appliance:PCIE_X16_SLOT_SMT, symbol appliance:PCIE_X16_SLOT_SMT
Connections:
- net +12V: now also J_SLOT0.A1, J_SLOT0.A2, J_SLOT0.A3, J_SLOT0.A4, J_SLOT0.A5, J_SLOT0.A6, J_SLOT0.B1, J_SLOT0.B2, J_SLOT0.B3, J_SLOT0.B4, J_SLOT0.B5, J_SLOT0.B6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
- net GND: now also J_SLOT0.A10, J_SLOT0.A11, J_SLOT0.A24, J_SLOT0.A25, J_SLOT0.A26, J_SLOT0.A27, J_SLOT0.A28, J_SLOT0.A29, J_SLOT0.A30, J_SLOT0.A31, J_SLOT0.A32, J_SLOT0.A33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
- net JTAG_TCK: now also J_SLOT0.A55, J_SLOT1.A55, J_SLOT2.A55, J_SLOT3.A55, J_SLOT4.A55, J_SLOT5.A55, J_SLOT6.A55, J_SLOT7.A55, J_SLOT8.A55, J_SLOT9.A55
- net JTAG_TDO_A0: now also J_SLOT0.A58, J_SLOT1.A57
- net JTAG_TDO_A1: now also J_SLOT1.A58, J_SLOT2.A57
- net JTAG_TDO_A2: now also J_SLOT2.A58, J_SLOT3.A57
- net JTAG_TDO_A3: now also J_SLOT3.A58, J_SLOT4.A57
- net JTAG_TDO_A4: now also J_SLOT4.A58, J_SLOT5.A57
- net JTAG_TDO_A5: now also J_SLOT5.A58, J_SLOT6.A57
- net JTAG_TDO_A6: now also J_SLOT6.A58, J_SLOT7.A57
- net JTAG_TDO_A7: now also J_SLOT7.A58, J_SLOT8.A57
- net JTAG_TDO_FPGA: now also J_SLOT0.A57
- net JTAG_TDO_H0: now also J_SLOT8.A58, J_SLOT9.A57
- net JTAG_TDO_H1: now also J_SLOT9.A58
- net JTAG_TMS: now also J_SLOT0.A56, J_SLOT1.A56, J_SLOT2.A56, J_SLOT3.A56, J_SLOT4.A56, J_SLOT5.A56, J_SLOT6.A56, J_SLOT7.A56, J_SLOT8.A56, J_SLOT9.A56
- net JTAG_TRST: now also J_SLOT0.A59, J_SLOT1.A59, J_SLOT2.A59, J_SLOT3.A59, J_SLOT4.A59, J_SLOT5.A59, J_SLOT6.A59, J_SLOT7.A59, J_SLOT8.A59, J_SLOT9.A59
- net LINK0_CLOCK: now also J_SLOT0.A20
- net LINK0_DATA0: now also J_SLOT0.A12
- net LINK0_DATA1: now also J_SLOT0.A13
- net LINK0_DATA2: now also J_SLOT0.A14
- net LINK0_DATA3: now also J_SLOT0.A15
- net LINK0_DATA4: now also J_SLOT0.A16
- net LINK0_DATA5: now also J_SLOT0.A17
- net LINK0_DATA6: now also J_SLOT0.A18
- net LINK0_DATA7: now also J_SLOT0.A19
- net LINK0_READY_BACK: now also J_SLOT0.A22
- net LINK0_SOF: now also J_SLOT0.A23
- net LINK0_VALID: now also J_SLOT0.A21
- net LINK10_CLOCK: now also J_SLOT9.B35
- net LINK10_DATA0: now also J_SLOT9.B27
- net LINK10_DATA1: now also J_SLOT9.B28
- net LINK10_DATA2: now also J_SLOT9.B29
- net LINK10_DATA3: now also J_SLOT9.B30
- net LINK10_DATA4: now also J_SLOT9.B31
- net LINK10_DATA5: now also J_SLOT9.B32
- net LINK10_DATA6: now also J_SLOT9.B33
- net LINK10_DATA7: now also J_SLOT9.B34
- net LINK10_READY_BACK: now also J_SLOT9.B37
- net LINK10_SOF: now also J_SLOT9.B38
- net LINK10_VALID: now also J_SLOT9.B36
- net LINK1_CLOCK: now also J_SLOT0.B35, J_SLOT1.A20
- net LINK1_DATA0: now also J_SLOT0.B27, J_SLOT1.A12
- net LINK1_DATA1: now also J_SLOT0.B28, J_SLOT1.A13
- net LINK1_DATA2: now also J_SLOT0.B29, J_SLOT1.A14
- net LINK1_DATA3: now also J_SLOT0.B30, J_SLOT1.A15
- net LINK1_DATA4: now also J_SLOT0.B31, J_SLOT1.A16
- net LINK1_DATA5: now also J_SLOT0.B32, J_SLOT1.A17
- net LINK1_DATA6: now also J_SLOT0.B33, J_SLOT1.A18
- net LINK1_DATA7: now also J_SLOT0.B34, J_SLOT1.A19
- net LINK1_READY_BACK: now also J_SLOT0.B37, J_SLOT1.A22
- net LINK1_SOF: now also J_SLOT0.B38, J_SLOT1.A23
- net LINK1_VALID: now also J_SLOT0.B36, J_SLOT1.A21
- net LINK2_CLOCK: now also J_SLOT1.B35, J_SLOT2.A20
- net LINK2_DATA0: now also J_SLOT1.B27, J_SLOT2.A12
- net LINK2_DATA1: now also J_SLOT1.B28, J_SLOT2.A13
- net LINK2_DATA2: now also J_SLOT1.B29, J_SLOT2.A14
- net LINK2_DATA3: now also J_SLOT1.B30, J_SLOT2.A15
- net LINK2_DATA4: now also J_SLOT1.B31, J_SLOT2.A16
- net LINK2_DATA5: now also J_SLOT1.B32, J_SLOT2.A17
- net LINK2_DATA6: now also J_SLOT1.B33, J_SLOT2.A18
- net LINK2_DATA7: now also J_SLOT1.B34, J_SLOT2.A19
- net LINK2_READY_BACK: now also J_SLOT1.B37, J_SLOT2.A22
- net LINK2_SOF: now also J_SLOT1.B38, J_SLOT2.A23
- net LINK2_VALID: now also J_SLOT1.B36, J_SLOT2.A21
- net LINK3_CLOCK: now also J_SLOT2.B35, J_SLOT3.A20
- net LINK3_DATA0: now also J_SLOT2.B27, J_SLOT3.A12
- net LINK3_DATA1: now also J_SLOT2.B28, J_SLOT3.A13
- net LINK3_DATA2: now also J_SLOT2.B29, J_SLOT3.A14
- net LINK3_DATA3: now also J_SLOT2.B30, J_SLOT3.A15
- net LINK3_DATA4: now also J_SLOT2.B31, J_SLOT3.A16
- net LINK3_DATA5: now also J_SLOT2.B32, J_SLOT3.A17
- net LINK3_DATA6: now also J_SLOT2.B33, J_SLOT3.A18
- net LINK3_DATA7: now also J_SLOT2.B34, J_SLOT3.A19
- net LINK3_READY_BACK: now also J_SLOT2.B37, J_SLOT3.A22
- net LINK3_SOF: now also J_SLOT2.B38, J_SLOT3.A23
- net LINK3_VALID: now also J_SLOT2.B36, J_SLOT3.A21
- net LINK4_CLOCK: now also J_SLOT3.B35, J_SLOT4.A20
- net LINK4_DATA0: now also J_SLOT3.B27, J_SLOT4.A12
- net LINK4_DATA1: now also J_SLOT3.B28, J_SLOT4.A13
- net LINK4_DATA2: now also J_SLOT3.B29, J_SLOT4.A14
- net LINK4_DATA3: now also J_SLOT3.B30, J_SLOT4.A15
- net LINK4_DATA4: now also J_SLOT3.B31, J_SLOT4.A16
- net LINK4_DATA5: now also J_SLOT3.B32, J_SLOT4.A17
- net LINK4_DATA6: now also J_SLOT3.B33, J_SLOT4.A18
- net LINK4_DATA7: now also J_SLOT3.B34, J_SLOT4.A19
- net LINK4_READY_BACK: now also J_SLOT3.B37, J_SLOT4.A22
- net LINK4_SOF: now also J_SLOT3.B38, J_SLOT4.A23
- net LINK4_VALID: now also J_SLOT3.B36, J_SLOT4.A21
- net LINK5_CLOCK: now also J_SLOT4.B35, J_SLOT5.A20
- net LINK5_DATA0: now also J_SLOT4.B27, J_SLOT5.A12
- net LINK5_DATA1: now also J_SLOT4.B28, J_SLOT5.A13
- net LINK5_DATA2: now also J_SLOT4.B29, J_SLOT5.A14
- net LINK5_DATA3: now also J_SLOT4.B30, J_SLOT5.A15
- net LINK5_DATA4: now also J_SLOT4.B31, J_SLOT5.A16
- net LINK5_DATA5: now also J_SLOT4.B32, J_SLOT5.A17
- net LINK5_DATA6: now also J_SLOT4.B33, J_SLOT5.A18
- net LINK5_DATA7: now also J_SLOT4.B34, J_SLOT5.A19
- net LINK5_READY_BACK: now also J_SLOT4.B37, J_SLOT5.A22
- net LINK5_SOF: now also J_SLOT4.B38, J_SLOT5.A23
- net LINK5_VALID: now also J_SLOT4.B36, J_SLOT5.A21
- net LINK6_CLOCK: now also J_SLOT5.B35, J_SLOT6.A20
- net LINK6_DATA0: now also J_SLOT5.B27, J_SLOT6.A12
- net LINK6_DATA1: now also J_SLOT5.B28, J_SLOT6.A13
- net LINK6_DATA2: now also J_SLOT5.B29, J_SLOT6.A14
- net LINK6_DATA3: now also J_SLOT5.B30, J_SLOT6.A15
- net LINK6_DATA4: now also J_SLOT5.B31, J_SLOT6.A16
- net LINK6_DATA5: now also J_SLOT5.B32, J_SLOT6.A17
- net LINK6_DATA6: now also J_SLOT5.B33, J_SLOT6.A18
- net LINK6_DATA7: now also J_SLOT5.B34, J_SLOT6.A19
- net LINK6_READY_BACK: now also J_SLOT5.B37, J_SLOT6.A22
- net LINK6_SOF: now also J_SLOT5.B38, J_SLOT6.A23
- net LINK6_VALID: now also J_SLOT5.B36, J_SLOT6.A21
- net LINK7_CLOCK: now also J_SLOT6.B35, J_SLOT7.A20
- net LINK7_DATA0: now also J_SLOT6.B27, J_SLOT7.A12
- net LINK7_DATA1: now also J_SLOT6.B28, J_SLOT7.A13
- net LINK7_DATA2: now also J_SLOT6.B29, J_SLOT7.A14
- net LINK7_DATA3: now also J_SLOT6.B30, J_SLOT7.A15
- net LINK7_DATA4: now also J_SLOT6.B31, J_SLOT7.A16
- net LINK7_DATA5: now also J_SLOT6.B32, J_SLOT7.A17
- net LINK7_DATA6: now also J_SLOT6.B33, J_SLOT7.A18
- net LINK7_DATA7: now also J_SLOT6.B34, J_SLOT7.A19
- net LINK7_READY_BACK: now also J_SLOT6.B37, J_SLOT7.A22
- net LINK7_SOF: now also J_SLOT6.B38, J_SLOT7.A23
- net LINK7_VALID: now also J_SLOT6.B36, J_SLOT7.A21
- net LINK8_CLOCK: now also J_SLOT7.B35, J_SLOT8.A20
- net LINK8_DATA0: now also J_SLOT7.B27, J_SLOT8.A12
- net LINK8_DATA1: now also J_SLOT7.B28, J_SLOT8.A13
- net LINK8_DATA2: now also J_SLOT7.B29, J_SLOT8.A14
- net LINK8_DATA3: now also J_SLOT7.B30, J_SLOT8.A15
- net LINK8_DATA4: now also J_SLOT7.B31, J_SLOT8.A16
- net LINK8_DATA5: now also J_SLOT7.B32, J_SLOT8.A17
- net LINK8_DATA6: now also J_SLOT7.B33, J_SLOT8.A18
- net LINK8_DATA7: now also J_SLOT7.B34, J_SLOT8.A19
- net LINK8_READY_BACK: now also J_SLOT7.B37, J_SLOT8.A22
- net LINK8_SOF: now also J_SLOT7.B38, J_SLOT8.A23
- net LINK8_VALID: now also J_SLOT7.B36, J_SLOT8.A21
- net LINK9_CLOCK: now also J_SLOT8.B35, J_SLOT9.A20
- net LINK9_DATA0: now also J_SLOT8.B27, J_SLOT9.A12
- net LINK9_DATA1: now also J_SLOT8.B28, J_SLOT9.A13
- net LINK9_DATA2: now also J_SLOT8.B29, J_SLOT9.A14
- net LINK9_DATA3: now also J_SLOT8.B30, J_SLOT9.A15
- net LINK9_DATA4: now also J_SLOT8.B31, J_SLOT9.A16
- net LINK9_DATA5: now also J_SLOT8.B32, J_SLOT9.A17
- net LINK9_DATA6: now also J_SLOT8.B33, J_SLOT9.A18
- net LINK9_DATA7: now also J_SLOT8.B34, J_SLOT9.A19
- net LINK9_READY_BACK: now also J_SLOT8.B37, J_SLOT9.A22
- net LINK9_SOF: now also J_SLOT8.B38, J_SLOT9.A23
- net LINK9_VALID: now also J_SLOT8.B36, J_SLOT9.A21
- net MGMT_CS_A0: now also J_SLOT0.A53
- net MGMT_CS_A1: now also J_SLOT1.A53
- net MGMT_CS_A2: now also J_SLOT2.A53
- net MGMT_CS_A3: now also J_SLOT3.A53
- net MGMT_CS_A4: now also J_SLOT4.A53
- net MGMT_CS_A5: now also J_SLOT5.A53
- net MGMT_CS_A6: now also J_SLOT6.A53
- net MGMT_CS_A7: now also J_SLOT7.A53
- net MGMT_CS_H0: now also J_SLOT8.A53
- net MGMT_CS_H1: now also J_SLOT9.A53
- net MGMT_IRQ_A0: now also J_SLOT0.A54
- net MGMT_IRQ_A1: now also J_SLOT1.A54
- net MGMT_IRQ_A2: now also J_SLOT2.A54
- net MGMT_IRQ_A3: now also J_SLOT3.A54
- net MGMT_IRQ_A4: now also J_SLOT4.A54
- net MGMT_IRQ_A5: now also J_SLOT5.A54
- net MGMT_IRQ_A6: now also J_SLOT6.A54
- net MGMT_IRQ_A7: now also J_SLOT7.A54
- net MGMT_IRQ_H0: now also J_SLOT8.A54
- net MGMT_IRQ_H1: now also J_SLOT9.A54
- net MGMT_MISO: now also J_SLOT0.A52, J_SLOT1.A52, J_SLOT2.A52, J_SLOT3.A52, J_SLOT4.A52, J_SLOT5.A52, J_SLOT6.A52, J_SLOT7.A52, J_SLOT8.A52, J_SLOT9.A52
- net MGMT_MOSI: now also J_SLOT0.A51, J_SLOT1.A51, J_SLOT2.A51, J_SLOT3.A51, J_SLOT4.A51, J_SLOT5.A51, J_SLOT6.A51, J_SLOT7.A51, J_SLOT8.A51, J_SLOT9.A51
- net MGMT_SCLK: now also J_SLOT0.A50, J_SLOT1.A50, J_SLOT2.A50, J_SLOT3.A50, J_SLOT4.A50, J_SLOT5.A50, J_SLOT6.A50, J_SLOT7.A50, J_SLOT8.A50, J_SLOT9.A50
- net MODE0_A0: now also J_SLOT0.A62
- net MODE0_A1: now also J_SLOT1.A62
- net MODE0_A2: now also J_SLOT2.A62
- net MODE0_A3: now also J_SLOT3.A62
- net MODE0_A4: now also J_SLOT4.A62
- net MODE0_A5: now also J_SLOT5.A62
- net MODE0_A6: now also J_SLOT6.A62
- net MODE0_A7: now also J_SLOT7.A62
- net MODE0_H0: now also J_SLOT8.A62
- net MODE0_H1: now also J_SLOT9.A62
- net MODE1_A0: now also J_SLOT0.A63
- net MODE1_A1: now also J_SLOT1.A63
- net MODE1_A2: now also J_SLOT2.A63
- net MODE1_A3: now also J_SLOT3.A63
- net MODE1_A4: now also J_SLOT4.A63
- net MODE1_A5: now also J_SLOT5.A63
- net MODE1_A6: now also J_SLOT6.A63
- net MODE1_A7: now also J_SLOT7.A63
- net MODE1_H0: now also J_SLOT8.A63
- net MODE1_H1: now also J_SLOT9.A63
- net PMB_SCL: now also J_SLOT0.B50, J_SLOT1.B50, J_SLOT2.B50, J_SLOT3.B50, J_SLOT4.B50, J_SLOT5.B50, J_SLOT6.B50, J_SLOT7.B50, J_SLOT8.B50, J_SLOT9.B50
- net PMB_SDA: now also J_SLOT0.B51, J_SLOT1.B51, J_SLOT2.B51, J_SLOT3.B51, J_SLOT4.B51, J_SLOT5.B51, J_SLOT6.B51, J_SLOT7.B51, J_SLOT8.B51, J_SLOT9.B51
- net PRSNT_A0: now also J_SLOT0.B53
- net PRSNT_A1: now also J_SLOT1.B53
- net PRSNT_A2: now also J_SLOT2.B53
- net PRSNT_A3: now also J_SLOT3.B53
- net PRSNT_A4: now also J_SLOT4.B53
- net PRSNT_A5: now also J_SLOT5.B53
- net PRSNT_A6: now also J_SLOT6.B53
- net PRSNT_A7: now also J_SLOT7.B53
- net PRSNT_H0: now also J_SLOT8.B53
- net PRSNT_H1: now also J_SLOT9.B53
- net REFCLK_A0_N: now also J_SLOT0.A61
- net REFCLK_A0_P: now also J_SLOT0.A60
- net REFCLK_A1_N: now also J_SLOT1.A61
- net REFCLK_A1_P: now also J_SLOT1.A60
- net REFCLK_A2_N: now also J_SLOT2.A61
- net REFCLK_A2_P: now also J_SLOT2.A60
- net REFCLK_A3_N: now also J_SLOT3.A61
- net REFCLK_A3_P: now also J_SLOT3.A60
- net REFCLK_A4_N: now also J_SLOT4.A61
- net REFCLK_A4_P: now also J_SLOT4.A60
- net REFCLK_A5_N: now also J_SLOT5.A61
- net REFCLK_A5_P: now also J_SLOT5.A60
- net REFCLK_A6_N: now also J_SLOT6.A61
- net REFCLK_A6_P: now also J_SLOT6.A60
- net REFCLK_A7_N: now also J_SLOT7.A61
- net REFCLK_A7_P: now also J_SLOT7.A60
- net REFCLK_H0_N: now also J_SLOT8.A61
- net REFCLK_H0_P: now also J_SLOT8.A60
- net REFCLK_H1_N: now also J_SLOT9.A61
- net REFCLK_H1_P: now also J_SLOT9.A60
- net VRM_EN_A0: now also J_SLOT0.B52
- net VRM_EN_A1: now also J_SLOT1.B52
- net VRM_EN_A2: now also J_SLOT2.B52
- net VRM_EN_A3: now also J_SLOT3.B52
- net VRM_EN_A4: now also J_SLOT4.B52
- net VRM_EN_A5: now also J_SLOT5.B52
- net VRM_EN_A6: now also J_SLOT6.B52
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
Commit message: Through-hole slots on the folded row, the two sets staggered past each other
A surface-mount x16 card-edge slot is not the commodity part, and the fold
only needed the skip-one ribbons to miss the skipped slot's pins.  Each
set's ribbon band runs at its link end, so shifting the two sets along the
cards by half a slot plus the band's clearance, 52 mm, puts every band past
the far end of the other set's pins with no weaving.  The stagger is derived
from the geometry and reported; slot_kind: smt keeps the single-line
arrangement for a surface-mount part.  The board is 420 x 180 mm, hops 83 mm
slot to slot, 183 mm at the turn, 73 and 89 mm at the FPGA.

Co-Authored-By: Claude Fable 5.1 <noreply@anthropic.com>
Claude-Session: https://claude.ai/code/session_01VmmvkZe8Ctg3RAykNGsQBn
Parts:
- removed J_SLOT0: slot for U_A0, appliance:PCIE_X16_SLOT_SMT, symbol appliance:PCIE_X16_SLOT_SMT
- removed J_SLOT1: slot for U_A1, appliance:PCIE_X16_SLOT_SMT, symbol appliance:PCIE_X16_SLOT_SMT
- removed J_SLOT2: slot for U_A2, appliance:PCIE_X16_SLOT_SMT, symbol appliance:PCIE_X16_SLOT_SMT
- removed J_SLOT3: slot for U_A3, appliance:PCIE_X16_SLOT_SMT, symbol appliance:PCIE_X16_SLOT_SMT
- removed J_SLOT4: slot for U_A4, appliance:PCIE_X16_SLOT_SMT, symbol appliance:PCIE_X16_SLOT_SMT
- removed J_SLOT5: slot for U_A5, appliance:PCIE_X16_SLOT_SMT, symbol appliance:PCIE_X16_SLOT_SMT
- removed J_SLOT6: slot for U_A6, appliance:PCIE_X16_SLOT_SMT, symbol appliance:PCIE_X16_SLOT_SMT
- removed J_SLOT7: slot for U_A7, appliance:PCIE_X16_SLOT_SMT, symbol appliance:PCIE_X16_SLOT_SMT
- removed J_SLOT8: slot for U_H0, appliance:PCIE_X16_SLOT_SMT, symbol appliance:PCIE_X16_SLOT_SMT
- removed J_SLOT9: slot for U_H1, appliance:PCIE_X16_SLOT_SMT, symbol appliance:PCIE_X16_SLOT_SMT
- added J_SLOT0: slot for U_A0, appliance:PCIE_X16_SLOT, symbol appliance:PCIE_X16_SLOT
- added J_SLOT1: slot for U_A1, appliance:PCIE_X16_SLOT, symbol appliance:PCIE_X16_SLOT
- added J_SLOT2: slot for U_A2, appliance:PCIE_X16_SLOT, symbol appliance:PCIE_X16_SLOT
- added J_SLOT3: slot for U_A3, appliance:PCIE_X16_SLOT, symbol appliance:PCIE_X16_SLOT
- added J_SLOT4: slot for U_A4, appliance:PCIE_X16_SLOT, symbol appliance:PCIE_X16_SLOT
- added J_SLOT5: slot for U_A5, appliance:PCIE_X16_SLOT, symbol appliance:PCIE_X16_SLOT
- added J_SLOT6: slot for U_A6, appliance:PCIE_X16_SLOT, symbol appliance:PCIE_X16_SLOT
- added J_SLOT7: slot for U_A7, appliance:PCIE_X16_SLOT, symbol appliance:PCIE_X16_SLOT
- added J_SLOT8: slot for U_H0, appliance:PCIE_X16_SLOT, symbol appliance:PCIE_X16_SLOT
- added J_SLOT9: slot for U_H1, appliance:PCIE_X16_SLOT, symbol appliance:PCIE_X16_SLOT
Connections:
- net +12V: now also J_SLOT0.A1, J_SLOT0.A2, J_SLOT0.A3, J_SLOT0.A4, J_SLOT0.A5, J_SLOT0.A6, J_SLOT0.B1, J_SLOT0.B2, J_SLOT0.B3, J_SLOT0.B4, J_SLOT0.B5, J_SLOT0.B6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
- net GND: now also J_SLOT0.A10, J_SLOT0.A11, J_SLOT0.A24, J_SLOT0.A25, J_SLOT0.A26, J_SLOT0.A27, J_SLOT0.A28, J_SLOT0.A29, J_SLOT0.A30, J_SLOT0.A31, J_SLOT0.A32, J_SLOT0.A33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
- net JTAG_TCK: now also J_SLOT0.A55, J_SLOT1.A55, J_SLOT2.A55, J_SLOT3.A55, J_SLOT4.A55, J_SLOT5.A55, J_SLOT6.A55, J_SLOT7.A55, J_SLOT8.A55, J_SLOT9.A55
- net JTAG_TDO_A0: now also J_SLOT0.A58, J_SLOT1.A57
- net JTAG_TDO_A1: now also J_SLOT1.A58, J_SLOT2.A57
- net JTAG_TDO_A2: now also J_SLOT2.A58, J_SLOT3.A57
- net JTAG_TDO_A3: now also J_SLOT3.A58, J_SLOT4.A57
- net JTAG_TDO_A4: now also J_SLOT4.A58, J_SLOT5.A57
- net JTAG_TDO_A5: now also J_SLOT5.A58, J_SLOT6.A57
- net JTAG_TDO_A6: now also J_SLOT6.A58, J_SLOT7.A57
- net JTAG_TDO_A7: now also J_SLOT7.A58, J_SLOT8.A57
- net JTAG_TDO_FPGA: now also J_SLOT0.A57
- net JTAG_TDO_H0: now also J_SLOT8.A58, J_SLOT9.A57
- net JTAG_TDO_H1: now also J_SLOT9.A58
- net JTAG_TMS: now also J_SLOT0.A56, J_SLOT1.A56, J_SLOT2.A56, J_SLOT3.A56, J_SLOT4.A56, J_SLOT5.A56, J_SLOT6.A56, J_SLOT7.A56, J_SLOT8.A56, J_SLOT9.A56
- net JTAG_TRST: now also J_SLOT0.A59, J_SLOT1.A59, J_SLOT2.A59, J_SLOT3.A59, J_SLOT4.A59, J_SLOT5.A59, J_SLOT6.A59, J_SLOT7.A59, J_SLOT8.A59, J_SLOT9.A59
- net LINK0_CLOCK: now also J_SLOT0.A20
- net LINK0_DATA0: now also J_SLOT0.A12
- net LINK0_DATA1: now also J_SLOT0.A13
- net LINK0_DATA2: now also J_SLOT0.A14
- net LINK0_DATA3: now also J_SLOT0.A15
- net LINK0_DATA4: now also J_SLOT0.A16
- net LINK0_DATA5: now also J_SLOT0.A17
- net LINK0_DATA6: now also J_SLOT0.A18
- net LINK0_DATA7: now also J_SLOT0.A19
- net LINK0_READY_BACK: now also J_SLOT0.A22
- net LINK0_SOF: now also J_SLOT0.A23
- net LINK0_VALID: now also J_SLOT0.A21
- net LINK10_CLOCK: now also J_SLOT9.B35
- net LINK10_DATA0: now also J_SLOT9.B27
- net LINK10_DATA1: now also J_SLOT9.B28
- net LINK10_DATA2: now also J_SLOT9.B29
- net LINK10_DATA3: now also J_SLOT9.B30
- net LINK10_DATA4: now also J_SLOT9.B31
- net LINK10_DATA5: now also J_SLOT9.B32
- net LINK10_DATA6: now also J_SLOT9.B33
- net LINK10_DATA7: now also J_SLOT9.B34
- net LINK10_READY_BACK: now also J_SLOT9.B37
- net LINK10_SOF: now also J_SLOT9.B38
- net LINK10_VALID: now also J_SLOT9.B36
- net LINK1_CLOCK: now also J_SLOT0.B35, J_SLOT1.A20
- net LINK1_DATA0: now also J_SLOT0.B27, J_SLOT1.A12
- net LINK1_DATA1: now also J_SLOT0.B28, J_SLOT1.A13
- net LINK1_DATA2: now also J_SLOT0.B29, J_SLOT1.A14
- net LINK1_DATA3: now also J_SLOT0.B30, J_SLOT1.A15
- net LINK1_DATA4: now also J_SLOT0.B31, J_SLOT1.A16
- net LINK1_DATA5: now also J_SLOT0.B32, J_SLOT1.A17
- net LINK1_DATA6: now also J_SLOT0.B33, J_SLOT1.A18
- net LINK1_DATA7: now also J_SLOT0.B34, J_SLOT1.A19
- net LINK1_READY_BACK: now also J_SLOT0.B37, J_SLOT1.A22
- net LINK1_SOF: now also J_SLOT0.B38, J_SLOT1.A23
- net LINK1_VALID: now also J_SLOT0.B36, J_SLOT1.A21
- net LINK2_CLOCK: now also J_SLOT1.B35, J_SLOT2.A20
- net LINK2_DATA0: now also J_SLOT1.B27, J_SLOT2.A12
- net LINK2_DATA1: now also J_SLOT1.B28, J_SLOT2.A13
- net LINK2_DATA2: now also J_SLOT1.B29, J_SLOT2.A14
- net LINK2_DATA3: now also J_SLOT1.B30, J_SLOT2.A15
- net LINK2_DATA4: now also J_SLOT1.B31, J_SLOT2.A16
- net LINK2_DATA5: now also J_SLOT1.B32, J_SLOT2.A17
- net LINK2_DATA6: now also J_SLOT1.B33, J_SLOT2.A18
- net LINK2_DATA7: now also J_SLOT1.B34, J_SLOT2.A19
- net LINK2_READY_BACK: now also J_SLOT1.B37, J_SLOT2.A22
- net LINK2_SOF: now also J_SLOT1.B38, J_SLOT2.A23
- net LINK2_VALID: now also J_SLOT1.B36, J_SLOT2.A21
- net LINK3_CLOCK: now also J_SLOT2.B35, J_SLOT3.A20
- net LINK3_DATA0: now also J_SLOT2.B27, J_SLOT3.A12
- net LINK3_DATA1: now also J_SLOT2.B28, J_SLOT3.A13
- net LINK3_DATA2: now also J_SLOT2.B29, J_SLOT3.A14
- net LINK3_DATA3: now also J_SLOT2.B30, J_SLOT3.A15
- net LINK3_DATA4: now also J_SLOT2.B31, J_SLOT3.A16
- net LINK3_DATA5: now also J_SLOT2.B32, J_SLOT3.A17
- net LINK3_DATA6: now also J_SLOT2.B33, J_SLOT3.A18
- net LINK3_DATA7: now also J_SLOT2.B34, J_SLOT3.A19
- net LINK3_READY_BACK: now also J_SLOT2.B37, J_SLOT3.A22
- net LINK3_SOF: now also J_SLOT2.B38, J_SLOT3.A23
- net LINK3_VALID: now also J_SLOT2.B36, J_SLOT3.A21
- net LINK4_CLOCK: now also J_SLOT3.B35, J_SLOT4.A20
- net LINK4_DATA0: now also J_SLOT3.B27, J_SLOT4.A12
- net LINK4_DATA1: now also J_SLOT3.B28, J_SLOT4.A13
- net LINK4_DATA2: now also J_SLOT3.B29, J_SLOT4.A14
- net LINK4_DATA3: now also J_SLOT3.B30, J_SLOT4.A15
- net LINK4_DATA4: now also J_SLOT3.B31, J_SLOT4.A16
- net LINK4_DATA5: now also J_SLOT3.B32, J_SLOT4.A17
- net LINK4_DATA6: now also J_SLOT3.B33, J_SLOT4.A18
- net LINK4_DATA7: now also J_SLOT3.B34, J_SLOT4.A19
- net LINK4_READY_BACK: now also J_SLOT3.B37, J_SLOT4.A22
- net LINK4_SOF: now also J_SLOT3.B38, J_SLOT4.A23
- net LINK4_VALID: now also J_SLOT3.B36, J_SLOT4.A21
- net LINK5_CLOCK: now also J_SLOT4.B35, J_SLOT5.A20
- net LINK5_DATA0: now also J_SLOT4.B27, J_SLOT5.A12
- net LINK5_DATA1: now also J_SLOT4.B28, J_SLOT5.A13
- net LINK5_DATA2: now also J_SLOT4.B29, J_SLOT5.A14
- net LINK5_DATA3: now also J_SLOT4.B30, J_SLOT5.A15
- net LINK5_DATA4: now also J_SLOT4.B31, J_SLOT5.A16
- net LINK5_DATA5: now also J_SLOT4.B32, J_SLOT5.A17
- net LINK5_DATA6: now also J_SLOT4.B33, J_SLOT5.A18
- net LINK5_DATA7: now also J_SLOT4.B34, J_SLOT5.A19
- net LINK5_READY_BACK: now also J_SLOT4.B37, J_SLOT5.A22
- net LINK5_SOF: now also J_SLOT4.B38, J_SLOT5.A23
- net LINK5_VALID: now also J_SLOT4.B36, J_SLOT5.A21
- net LINK6_CLOCK: now also J_SLOT5.B35, J_SLOT6.A20
- net LINK6_DATA0: now also J_SLOT5.B27, J_SLOT6.A12
- net LINK6_DATA1: now also J_SLOT5.B28, J_SLOT6.A13
- net LINK6_DATA2: now also J_SLOT5.B29, J_SLOT6.A14
- net LINK6_DATA3: now also J_SLOT5.B30, J_SLOT6.A15
- net LINK6_DATA4: now also J_SLOT5.B31, J_SLOT6.A16
- net LINK6_DATA5: now also J_SLOT5.B32, J_SLOT6.A17
- net LINK6_DATA6: now also J_SLOT5.B33, J_SLOT6.A18
- net LINK6_DATA7: now also J_SLOT5.B34, J_SLOT6.A19
- net LINK6_READY_BACK: now also J_SLOT5.B37, J_SLOT6.A22
- net LINK6_SOF: now also J_SLOT5.B38, J_SLOT6.A23
- net LINK6_VALID: now also J_SLOT5.B36, J_SLOT6.A21
- net LINK7_CLOCK: now also J_SLOT6.B35, J_SLOT7.A20
- net LINK7_DATA0: now also J_SLOT6.B27, J_SLOT7.A12
- net LINK7_DATA1: now also J_SLOT6.B28, J_SLOT7.A13
- net LINK7_DATA2: now also J_SLOT6.B29, J_SLOT7.A14
- net LINK7_DATA3: now also J_SLOT6.B30, J_SLOT7.A15
- net LINK7_DATA4: now also J_SLOT6.B31, J_SLOT7.A16
- net LINK7_DATA5: now also J_SLOT6.B32, J_SLOT7.A17
- net LINK7_DATA6: now also J_SLOT6.B33, J_SLOT7.A18
- net LINK7_DATA7: now also J_SLOT6.B34, J_SLOT7.A19
- net LINK7_READY_BACK: now also J_SLOT6.B37, J_SLOT7.A22
- net LINK7_SOF: now also J_SLOT6.B38, J_SLOT7.A23
- net LINK7_VALID: now also J_SLOT6.B36, J_SLOT7.A21
- net LINK8_CLOCK: now also J_SLOT7.B35, J_SLOT8.A20
- net LINK8_DATA0: now also J_SLOT7.B27, J_SLOT8.A12
- net LINK8_DATA1: now also J_SLOT7.B28, J_SLOT8.A13
- net LINK8_DATA2: now also J_SLOT7.B29, J_SLOT8.A14
- net LINK8_DATA3: now also J_SLOT7.B30, J_SLOT8.A15
- net LINK8_DATA4: now also J_SLOT7.B31, J_SLOT8.A16
- net LINK8_DATA5: now also J_SLOT7.B32, J_SLOT8.A17
- net LINK8_DATA6: now also J_SLOT7.B33, J_SLOT8.A18
- net LINK8_DATA7: now also J_SLOT7.B34, J_SLOT8.A19
- net LINK8_READY_BACK: now also J_SLOT7.B37, J_SLOT8.A22
- net LINK8_SOF: now also J_SLOT7.B38, J_SLOT8.A23
- net LINK8_VALID: now also J_SLOT7.B36, J_SLOT8.A21
- net LINK9_CLOCK: now also J_SLOT8.B35, J_SLOT9.A20
- net LINK9_DATA0: now also J_SLOT8.B27, J_SLOT9.A12
- net LINK9_DATA1: now also J_SLOT8.B28, J_SLOT9.A13
- net LINK9_DATA2: now also J_SLOT8.B29, J_SLOT9.A14
- net LINK9_DATA3: now also J_SLOT8.B30, J_SLOT9.A15
- net LINK9_DATA4: now also J_SLOT8.B31, J_SLOT9.A16
- net LINK9_DATA5: now also J_SLOT8.B32, J_SLOT9.A17
- net LINK9_DATA6: now also J_SLOT8.B33, J_SLOT9.A18
- net LINK9_DATA7: now also J_SLOT8.B34, J_SLOT9.A19
- net LINK9_READY_BACK: now also J_SLOT8.B37, J_SLOT9.A22
- net LINK9_SOF: now also J_SLOT8.B38, J_SLOT9.A23
- net LINK9_VALID: now also J_SLOT8.B36, J_SLOT9.A21
- net MGMT_CS_A0: now also J_SLOT0.A53
- net MGMT_CS_A1: now also J_SLOT1.A53
- net MGMT_CS_A2: now also J_SLOT2.A53
- net MGMT_CS_A3: now also J_SLOT3.A53
- net MGMT_CS_A4: now also J_SLOT4.A53
- net MGMT_CS_A5: now also J_SLOT5.A53
- net MGMT_CS_A6: now also J_SLOT6.A53
- net MGMT_CS_A7: now also J_SLOT7.A53
- net MGMT_CS_H0: now also J_SLOT8.A53
- net MGMT_CS_H1: now also J_SLOT9.A53
- net MGMT_IRQ_A0: now also J_SLOT0.A54
- net MGMT_IRQ_A1: now also J_SLOT1.A54
- net MGMT_IRQ_A2: now also J_SLOT2.A54
- net MGMT_IRQ_A3: now also J_SLOT3.A54
- net MGMT_IRQ_A4: now also J_SLOT4.A54
- net MGMT_IRQ_A5: now also J_SLOT5.A54
- net MGMT_IRQ_A6: now also J_SLOT6.A54
- net MGMT_IRQ_A7: now also J_SLOT7.A54
- net MGMT_IRQ_H0: now also J_SLOT8.A54
- net MGMT_IRQ_H1: now also J_SLOT9.A54
- net MGMT_MISO: now also J_SLOT0.A52, J_SLOT1.A52, J_SLOT2.A52, J_SLOT3.A52, J_SLOT4.A52, J_SLOT5.A52, J_SLOT6.A52, J_SLOT7.A52, J_SLOT8.A52, J_SLOT9.A52
- net MGMT_MOSI: now also J_SLOT0.A51, J_SLOT1.A51, J_SLOT2.A51, J_SLOT3.A51, J_SLOT4.A51, J_SLOT5.A51, J_SLOT6.A51, J_SLOT7.A51, J_SLOT8.A51, J_SLOT9.A51
- net MGMT_SCLK: now also J_SLOT0.A50, J_SLOT1.A50, J_SLOT2.A50, J_SLOT3.A50, J_SLOT4.A50, J_SLOT5.A50, J_SLOT6.A50, J_SLOT7.A50, J_SLOT8.A50, J_SLOT9.A50
- net MODE0_A0: now also J_SLOT0.A62
- net MODE0_A1: now also J_SLOT1.A62
- net MODE0_A2: now also J_SLOT2.A62
- net MODE0_A3: now also J_SLOT3.A62
- net MODE0_A4: now also J_SLOT4.A62
- net MODE0_A5: now also J_SLOT5.A62
- net MODE0_A6: now also J_SLOT6.A62
- net MODE0_A7: now also J_SLOT7.A62
- net MODE0_H0: now also J_SLOT8.A62
- net MODE0_H1: now also J_SLOT9.A62
- net MODE1_A0: now also J_SLOT0.A63
- net MODE1_A1: now also J_SLOT1.A63
- net MODE1_A2: now also J_SLOT2.A63
- net MODE1_A3: now also J_SLOT3.A63
- net MODE1_A4: now also J_SLOT4.A63
- net MODE1_A5: now also J_SLOT5.A63
- net MODE1_A6: now also J_SLOT6.A63
- net MODE1_A7: now also J_SLOT7.A63
- net MODE1_H0: now also J_SLOT8.A63
- net MODE1_H1: now also J_SLOT9.A63
- net PMB_SCL: now also J_SLOT0.B50, J_SLOT1.B50, J_SLOT2.B50, J_SLOT3.B50, J_SLOT4.B50, J_SLOT5.B50, J_SLOT6.B50, J_SLOT7.B50, J_SLOT8.B50, J_SLOT9.B50
- net PMB_SDA: now also J_SLOT0.B51, J_SLOT1.B51, J_SLOT2.B51, J_SLOT3.B51, J_SLOT4.B51, J_SLOT5.B51, J_SLOT6.B51, J_SLOT7.B51, J_SLOT8.B51, J_SLOT9.B51
- net PRSNT_A0: now also J_SLOT0.B53
- net PRSNT_A1: now also J_SLOT1.B53
- net PRSNT_A2: now also J_SLOT2.B53
- net PRSNT_A3: now also J_SLOT3.B53
- net PRSNT_A4: now also J_SLOT4.B53
- net PRSNT_A5: now also J_SLOT5.B53
- net PRSNT_A6: now also J_SLOT6.B53
- net PRSNT_A7: now also J_SLOT7.B53
- net PRSNT_H0: now also J_SLOT8.B53
- net PRSNT_H1: now also J_SLOT9.B53
- net REFCLK_A0_N: now also J_SLOT0.A61
- net REFCLK_A0_P: now also J_SLOT0.A60
- net REFCLK_A1_N: now also J_SLOT1.A61
- net REFCLK_A1_P: now also J_SLOT1.A60
- net REFCLK_A2_N: now also J_SLOT2.A61
- net REFCLK_A2_P: now also J_SLOT2.A60
- net REFCLK_A3_N: now also J_SLOT3.A61
- net REFCLK_A3_P: now also J_SLOT3.A60
- net REFCLK_A4_N: now also J_SLOT4.A61
- net REFCLK_A4_P: now also J_SLOT4.A60
- net REFCLK_A5_N: now also J_SLOT5.A61
- net REFCLK_A5_P: now also J_SLOT5.A60
- net REFCLK_A6_N: now also J_SLOT6.A61
- net REFCLK_A6_P: now also J_SLOT6.A60
- net REFCLK_A7_N: now also J_SLOT7.A61
- net REFCLK_A7_P: now also J_SLOT7.A60
- net REFCLK_H0_N: now also J_SLOT8.A61
- net REFCLK_H0_P: now also J_SLOT8.A60
- net REFCLK_H1_N: now also J_SLOT9.A61
- net REFCLK_H1_P: now also J_SLOT9.A60
- net VRM_EN_A0: now also J_SLOT0.B52
- net VRM_EN_A1: now also J_SLOT1.B52
- net VRM_EN_A2: now also J_SLOT2.B52
- net VRM_EN_A3: now also J_SLOT3.B52
- net VRM_EN_A4: now also J_SLOT4.B52
- net VRM_EN_A5: now also J_SLOT5.B52
- net VRM_EN_A6: now also J_SLOT6.B52
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
Commit message: Link in and out on the same finger positions: straight slot-to-slot hops
link_in sits on side A and link_out on side B of the same twelve edge
positions, so a slot's out-row pin faces the next slot's in-row pin and
every skip-one hop is a straight ribbon.  On the card the two drops from
the die's south-edge blocks lean towards one finger span from either side
and cross, so the out drop takes In3 and the two faces' vias interleave
half a position apart above the fingers.  The ribbon band narrows from
27 mm to 12, the stagger from 52 mm to 38, and the short board from 180 to
170 mm deep.  finger_layout: offset keeps the earlier separate spans.

Co-Authored-By: Claude Fable 5.1 <noreply@anthropic.com>
Claude-Session: https://claude.ai/code/session_01VmmvkZe8Ctg3RAykNGsQBn
Connections:
- net GND: now also J_SLOT0.B27, J_SLOT0.B28, J_SLOT0.B29, J_SLOT0.B30, J_SLOT0.B31, J_SLOT0.B32, J_SLOT0.B33, J_SLOT0.B34, J_SLOT0.B35, J_SLOT0.B36, J_SLOT0.B37, J_SLOT0.B38, J_SLOT1.B27, J_SLOT1.B28, J_SLOT1.B29, J_SLOT1.B30, J_SLOT1.B31, J_SLOT1.B32, J_SLOT1.B33, J_SLOT1.B34, J_SLOT1.B35, J_SLOT1.B36, J_SLOT1.B37, J_SLOT1.B38, J_SLOT2.B27, J_SLOT2.B28, J_SLOT2.B29, J_SLOT2.B30, J_SLOT2.B31, J_SLOT2.B32, J_SLOT2.B33, J_SLOT2.B34, J_SLOT2.B35, J_SLOT2.B36, J_SLOT2.B37, J_SLOT2.B38, J_SLOT3.B27, J_SLOT3.B28, J_SLOT3.B29, J_SLOT3.B30, J_SLOT3.B31, J_SLOT3.B32, J_SLOT3.B33, J_SLOT3.B34, J_SLOT3.B35, J_SLOT3.B36, J_SLOT3.B37, J_SLOT3.B38, J_SLOT4.B27, J_SLOT4.B28, J_SLOT4.B29, J_SLOT4.B30, J_SLOT4.B31, J_SLOT4.B32, J_SLOT4.B33, J_SLOT4.B34, J_SLOT4.B35, J_SLOT4.B36, J_SLOT4.B37, J_SLOT4.B38, J_SLOT5.B27, J_SLOT5.B28, J_SLOT5.B29, J_SLOT5.B30, J_SLOT5.B31, J_SLOT5.B32, J_SLOT5.B33, J_SLOT5.B34, J_SLOT5.B35, J_SLOT5.B36, J_SLOT5.B37, J_SLOT5.B38, J_SLOT6.B27, J_SLOT6.B28, J_SLOT6.B29, J_SLOT6.B30, J_SLOT6.B31, J_SLOT6.B32, J_SLOT6.B33, J_SLOT6.B34, J_SLOT6.B35, J_SLOT6.B36, J_SLOT6.B37, J_SLOT6.B38, J_SLOT7.B27, J_SLOT7.B28, J_SLOT7.B29, J_SLOT7.B30, J_SLOT7.B31, J_SLOT7.B32, J_SLOT7.B33, J_SLOT7.B34, J_SLOT7.B35, J_SLOT7.B36, J_SLOT7.B37, J_SLOT7.B38, J_SLOT8.B27, J_SLOT8.B28, J_SLOT8.B29, J_SLOT8.B30, J_SLOT8.B31, J_SLOT8.B32, J_SLOT8.B33, J_SLOT8.B34, J_SLOT8.B35, J_SLOT8.B36, J_SLOT8.B37, J_SLOT8.B38, J_SLOT9.B27, J_SLOT9.B28, J_SLOT9.B29, J_SLOT9.B30, J_SLOT9.B31, J_SLOT9.B32, J_SLOT9.B33, J_SLOT9.B34, J_SLOT9.B35, J_SLOT9.B36, J_SLOT9.B37, J_SLOT9.B38; no longer J_SLOT0.B12, J_SLOT0.B13, J_SLOT0.B14, J_SLOT0.B15, J_SLOT0.B16, J_SLOT0.B17, J_SLOT0.B18, J_SLOT0.B19, J_SLOT0.B20, J_SLOT0.B21, J_SLOT0.B22, J_SLOT0.B23, J_SLOT1.B12, J_SLOT1.B13, J_SLOT1.B14, J_SLOT1.B15, J_SLOT1.B16, J_SLOT1.B17, J_SLOT1.B18, J_SLOT1.B19, J_SLOT1.B20, J_SLOT1.B21, J_SLOT1.B22, J_SLOT1.B23, J_SLOT2.B12, J_SLOT2.B13, J_SLOT2.B14, J_SLOT2.B15, J_SLOT2.B16, J_SLOT2.B17, J_SLOT2.B18, J_SLOT2.B19, J_SLOT2.B20, J_SLOT2.B21, J_SLOT2.B22, J_SLOT2.B23, J_SLOT3.B12, J_SLOT3.B13, J_SLOT3.B14, J_SLOT3.B15, J_SLOT3.B16, J_SLOT3.B17, J_SLOT3.B18, J_SLOT3.B19, J_SLOT3.B20, J_SLOT3.B21, J_SLOT3.B22, J_SLOT3.B23, J_SLOT4.B12, J_SLOT4.B13, J_SLOT4.B14, J_SLOT4.B15, J_SLOT4.B16, J_SLOT4.B17, J_SLOT4.B18, J_SLOT4.B19, J_SLOT4.B20, J_SLOT4.B21, J_SLOT4.B22, J_SLOT4.B23, J_SLOT5.B12, J_SLOT5.B13, J_SLOT5.B14, J_SLOT5.B15, J_SLOT5.B16, J_SLOT5.B17, J_SLOT5.B18, J_SLOT5.B19, J_SLOT5.B20, J_SLOT5.B21, J_SLOT5.B22, J_SLOT5.B23, J_SLOT6.B12, J_SLOT6.B13, J_SLOT6.B14, J_SLOT6.B15, J_SLOT6.B16, J_SLOT6.B17, J_SLOT6.B18, J_SLOT6.B19, J_SLOT6.B20, J_SLOT6.B21, J_SLOT6.B22, J_SLOT6.B23, J_SLOT7.B12, J_SLOT7.B13, J_SLOT7.B14, J_SLOT7.B15, J_SLOT7.B16, J_SLOT7.B17, J_SLOT7.B18, J_SLOT7.B19, J_SLOT7.B20, J_SLOT7.B21, J_SLOT7.B22, J_SLOT7.B23, J_SLOT8.B12, J_SLOT8.B13, J_SLOT8.B14, J_SLOT8.B15, J_SLOT8.B16, J_SLOT8.B17, J_SLOT8.B18, J_SLOT8.B19, J_SLOT8.B20, J_SLOT8.B21, J_SLOT8.B22, J_SLOT8.B23, J_SLOT9.B12, J_SLOT9.B13, J_SLOT9.B14, J_SLOT9.B15, J_SLOT9.B16, J_SLOT9.B17, J_SLOT9.B18, J_SLOT9.B19, J_SLOT9.B20, J_SLOT9.B21, J_SLOT9.B22, J_SLOT9.B23
- net LINK10_CLOCK: now also J_SLOT9.B20; no longer J_SLOT9.B35
- net LINK10_DATA0: now also J_SLOT9.B12; no longer J_SLOT9.B27
- net LINK10_DATA1: now also J_SLOT9.B13; no longer J_SLOT9.B28
- net LINK10_DATA2: now also J_SLOT9.B14; no longer J_SLOT9.B29
- net LINK10_DATA3: now also J_SLOT9.B15; no longer J_SLOT9.B30
- net LINK10_DATA4: now also J_SLOT9.B16; no longer J_SLOT9.B31
- net LINK10_DATA5: now also J_SLOT9.B17; no longer J_SLOT9.B32
- net LINK10_DATA6: now also J_SLOT9.B18; no longer J_SLOT9.B33
- net LINK10_DATA7: now also J_SLOT9.B19; no longer J_SLOT9.B34
- net LINK10_READY_BACK: now also J_SLOT9.B22; no longer J_SLOT9.B37
- net LINK10_SOF: now also J_SLOT9.B23; no longer J_SLOT9.B38
- net LINK10_VALID: now also J_SLOT9.B21; no longer J_SLOT9.B36
- net LINK1_CLOCK: now also J_SLOT0.B20; no longer J_SLOT0.B35
- net LINK1_DATA0: now also J_SLOT0.B12; no longer J_SLOT0.B27
- net LINK1_DATA1: now also J_SLOT0.B13; no longer J_SLOT0.B28
- net LINK1_DATA2: now also J_SLOT0.B14; no longer J_SLOT0.B29
- net LINK1_DATA3: now also J_SLOT0.B15; no longer J_SLOT0.B30
- net LINK1_DATA4: now also J_SLOT0.B16; no longer J_SLOT0.B31
- net LINK1_DATA5: now also J_SLOT0.B17; no longer J_SLOT0.B32
- net LINK1_DATA6: now also J_SLOT0.B18; no longer J_SLOT0.B33
- net LINK1_DATA7: now also J_SLOT0.B19; no longer J_SLOT0.B34
- net LINK1_READY_BACK: now also J_SLOT0.B22; no longer J_SLOT0.B37
- net LINK1_SOF: now also J_SLOT0.B23; no longer J_SLOT0.B38
- net LINK1_VALID: now also J_SLOT0.B21; no longer J_SLOT0.B36
- net LINK2_CLOCK: now also J_SLOT1.B20; no longer J_SLOT1.B35
- net LINK2_DATA0: now also J_SLOT1.B12; no longer J_SLOT1.B27
- net LINK2_DATA1: now also J_SLOT1.B13; no longer J_SLOT1.B28
- net LINK2_DATA2: now also J_SLOT1.B14; no longer J_SLOT1.B29
- net LINK2_DATA3: now also J_SLOT1.B15; no longer J_SLOT1.B30
- net LINK2_DATA4: now also J_SLOT1.B16; no longer J_SLOT1.B31
- net LINK2_DATA5: now also J_SLOT1.B17; no longer J_SLOT1.B32
- net LINK2_DATA6: now also J_SLOT1.B18; no longer J_SLOT1.B33
- net LINK2_DATA7: now also J_SLOT1.B19; no longer J_SLOT1.B34
- net LINK2_READY_BACK: now also J_SLOT1.B22; no longer J_SLOT1.B37
- net LINK2_SOF: now also J_SLOT1.B23; no longer J_SLOT1.B38
- net LINK2_VALID: now also J_SLOT1.B21; no longer J_SLOT1.B36
- net LINK3_CLOCK: now also J_SLOT2.B20; no longer J_SLOT2.B35
- net LINK3_DATA0: now also J_SLOT2.B12; no longer J_SLOT2.B27
- net LINK3_DATA1: now also J_SLOT2.B13; no longer J_SLOT2.B28
- net LINK3_DATA2: now also J_SLOT2.B14; no longer J_SLOT2.B29
- net LINK3_DATA3: now also J_SLOT2.B15; no longer J_SLOT2.B30
- net LINK3_DATA4: now also J_SLOT2.B16; no longer J_SLOT2.B31
- net LINK3_DATA5: now also J_SLOT2.B17; no longer J_SLOT2.B32
- net LINK3_DATA6: now also J_SLOT2.B18; no longer J_SLOT2.B33
- net LINK3_DATA7: now also J_SLOT2.B19; no longer J_SLOT2.B34
- net LINK3_READY_BACK: now also J_SLOT2.B22; no longer J_SLOT2.B37
- net LINK3_SOF: now also J_SLOT2.B23; no longer J_SLOT2.B38
- net LINK3_VALID: now also J_SLOT2.B21; no longer J_SLOT2.B36
- net LINK4_CLOCK: now also J_SLOT3.B20; no longer J_SLOT3.B35
- net LINK4_DATA0: now also J_SLOT3.B12; no longer J_SLOT3.B27
- net LINK4_DATA1: now also J_SLOT3.B13; no longer J_SLOT3.B28
- net LINK4_DATA2: now also J_SLOT3.B14; no longer J_SLOT3.B29
- net LINK4_DATA3: now also J_SLOT3.B15; no longer J_SLOT3.B30
- net LINK4_DATA4: now also J_SLOT3.B16; no longer J_SLOT3.B31
- net LINK4_DATA5: now also J_SLOT3.B17; no longer J_SLOT3.B32
- net LINK4_DATA6: now also J_SLOT3.B18; no longer J_SLOT3.B33
- net LINK4_DATA7: now also J_SLOT3.B19; no longer J_SLOT3.B34
- net LINK4_READY_BACK: now also J_SLOT3.B22; no longer J_SLOT3.B37
- net LINK4_SOF: now also J_SLOT3.B23; no longer J_SLOT3.B38
- net LINK4_VALID: now also J_SLOT3.B21; no longer J_SLOT3.B36
- net LINK5_CLOCK: now also J_SLOT4.B20; no longer J_SLOT4.B35
- net LINK5_DATA0: now also J_SLOT4.B12; no longer J_SLOT4.B27
- net LINK5_DATA1: now also J_SLOT4.B13; no longer J_SLOT4.B28
- net LINK5_DATA2: now also J_SLOT4.B14; no longer J_SLOT4.B29
- net LINK5_DATA3: now also J_SLOT4.B15; no longer J_SLOT4.B30
- net LINK5_DATA4: now also J_SLOT4.B16; no longer J_SLOT4.B31
- net LINK5_DATA5: now also J_SLOT4.B17; no longer J_SLOT4.B32
- net LINK5_DATA6: now also J_SLOT4.B18; no longer J_SLOT4.B33
- net LINK5_DATA7: now also J_SLOT4.B19; no longer J_SLOT4.B34
- net LINK5_READY_BACK: now also J_SLOT4.B22; no longer J_SLOT4.B37
- net LINK5_SOF: now also J_SLOT4.B23; no longer J_SLOT4.B38
- net LINK5_VALID: now also J_SLOT4.B21; no longer J_SLOT4.B36
- net LINK6_CLOCK: now also J_SLOT5.B20; no longer J_SLOT5.B35
- net LINK6_DATA0: now also J_SLOT5.B12; no longer J_SLOT5.B27
- net LINK6_DATA1: now also J_SLOT5.B13; no longer J_SLOT5.B28
- net LINK6_DATA2: now also J_SLOT5.B14; no longer J_SLOT5.B29
- net LINK6_DATA3: now also J_SLOT5.B15; no longer J_SLOT5.B30
- net LINK6_DATA4: now also J_SLOT5.B16; no longer J_SLOT5.B31
- net LINK6_DATA5: now also J_SLOT5.B17; no longer J_SLOT5.B32
- net LINK6_DATA6: now also J_SLOT5.B18; no longer J_SLOT5.B33
- net LINK6_DATA7: now also J_SLOT5.B19; no longer J_SLOT5.B34
- net LINK6_READY_BACK: now also J_SLOT5.B22; no longer J_SLOT5.B37
- net LINK6_SOF: now also J_SLOT5.B23; no longer J_SLOT5.B38
- net LINK6_VALID: now also J_SLOT5.B21; no longer J_SLOT5.B36
- net LINK7_CLOCK: now also J_SLOT6.B20; no longer J_SLOT6.B35
- net LINK7_DATA0: now also J_SLOT6.B12; no longer J_SLOT6.B27
- net LINK7_DATA1: now also J_SLOT6.B13; no longer J_SLOT6.B28
- net LINK7_DATA2: now also J_SLOT6.B14; no longer J_SLOT6.B29
- net LINK7_DATA3: now also J_SLOT6.B15; no longer J_SLOT6.B30
- net LINK7_DATA4: now also J_SLOT6.B16; no longer J_SLOT6.B31
- net LINK7_DATA5: now also J_SLOT6.B17; no longer J_SLOT6.B32
- net LINK7_DATA6: now also J_SLOT6.B18; no longer J_SLOT6.B33
- net LINK7_DATA7: now also J_SLOT6.B19; no longer J_SLOT6.B34
- net LINK7_READY_BACK: now also J_SLOT6.B22; no longer J_SLOT6.B37
- net LINK7_SOF: now also J_SLOT6.B23; no longer J_SLOT6.B38
- net LINK7_VALID: now also J_SLOT6.B21; no longer J_SLOT6.B36
- net LINK8_CLOCK: now also J_SLOT7.B20; no longer J_SLOT7.B35
- net LINK8_DATA0: now also J_SLOT7.B12; no longer J_SLOT7.B27
- net LINK8_DATA1: now also J_SLOT7.B13; no longer J_SLOT7.B28
- net LINK8_DATA2: now also J_SLOT7.B14; no longer J_SLOT7.B29
- net LINK8_DATA3: now also J_SLOT7.B15; no longer J_SLOT7.B30
- net LINK8_DATA4: now also J_SLOT7.B16; no longer J_SLOT7.B31
- net LINK8_DATA5: now also J_SLOT7.B17; no longer J_SLOT7.B32
- net LINK8_DATA6: now also J_SLOT7.B18; no longer J_SLOT7.B33
- net LINK8_DATA7: now also J_SLOT7.B19; no longer J_SLOT7.B34
- net LINK8_READY_BACK: now also J_SLOT7.B22; no longer J_SLOT7.B37
- net LINK8_SOF: now also J_SLOT7.B23; no longer J_SLOT7.B38
- net LINK8_VALID: now also J_SLOT7.B21; no longer J_SLOT7.B36
- net LINK9_CLOCK: now also J_SLOT8.B20; no longer J_SLOT8.B35
- net LINK9_DATA0: now also J_SLOT8.B12; no longer J_SLOT8.B27
- net LINK9_DATA1: now also J_SLOT8.B13; no longer J_SLOT8.B28
- net LINK9_DATA2: now also J_SLOT8.B14; no longer J_SLOT8.B29
- net LINK9_DATA3: now also J_SLOT8.B15; no longer J_SLOT8.B30
- net LINK9_DATA4: now also J_SLOT8.B16; no longer J_SLOT8.B31
- net LINK9_DATA5: now also J_SLOT8.B17; no longer J_SLOT8.B32
- net LINK9_DATA6: now also J_SLOT8.B18; no longer J_SLOT8.B33
- net LINK9_DATA7: now also J_SLOT8.B19; no longer J_SLOT8.B34
- net LINK9_READY_BACK: now also J_SLOT8.B22; no longer J_SLOT8.B37
- net LINK9_SOF: now also J_SLOT8.B23; no longer J_SLOT8.B38
- net LINK9_VALID: now also J_SLOT8.B21; no longer J_SLOT8.B36
