File: hw/kicad_psram/fpga.kicad_sch (KiCad schematic)
At the start: 6 parts

Commit message: Fold the module row onto a short-depth 2U with surface-mount slots
The two facing rows of slots existed only to keep the closing hop short.
One row does the same: the outbound cards in the even positions running
away from the FPGA, the returning cards in the odd positions between them,
so ring order 0..9 sits at positions 0,2,4,6,8 and 9,7,5,3,1, every hop
skips one slot, the turn is a square U round the last slot and the ring
closes on the FPGA's east edge, which now carries both link ports side by
side as a card's die does.  The slots are surface-mount, so a ribbon on the
link layer passes beneath the slot it skips instead of weaving between
pins; their ground and 12 V pads get no via-in-pad, reaching the planes by
stubs clear of the ribbon corridor.

The slot field is then the card's 89 mm and the board drops from 420 x 360
to 420 x 160 mm, a short-depth 2U (2u_short) whose CRPS modules overhang
the board's front edge.  Hops end to end: 72 mm slot to slot at 34
degrees, 130 mm at the turn, 46 and 67 mm into and out of the FPGA.  The
two-row layout stays selectable (layout: two_rows on the 2u) and is kept
under test.

Co-Authored-By: Claude Fable 5.1 <noreply@anthropic.com>
Claude-Session: https://claude.ai/code/session_01VmmvkZe8Ctg3RAykNGsQBn
Connections:
- net GND: now also U_FPGA.AE11, U_FPGA.AE13, U_FPGA.AE15, U_FPGA.AF12, U_FPGA.AF14, U_FPGA.AF16, U_FPGA.L25, U_FPGA.M26, U_FPGA.N25, U_FPGA.P26, U_FPGA.R25, U_FPGA.T26; no longer U_FPGA.AA25, U_FPGA.AB26, U_FPGA.AC25, U_FPGA.AD26, U_FPGA.D26, U_FPGA.E25, U_FPGA.F26, U_FPGA.G25, U_FPGA.H26, U_FPGA.J25, U_FPGA.W25, U_FPGA.Y26
- net LINK0_CLOCK: now also U_FPGA.Y26; no longer U_FPGA.M26
- net LINK0_DATA0: now also U_FPGA.AD26; no longer U_FPGA.T26
- net LINK0_DATA1: now also U_FPGA.AD25; no longer U_FPGA.T25
- net LINK0_DATA2: now also U_FPGA.AC26; no longer U_FPGA.R26
- net LINK0_DATA3: now also U_FPGA.AC25; no longer U_FPGA.R25
- net LINK0_DATA4: now also U_FPGA.AB26; no longer U_FPGA.P26
- net LINK0_DATA5: now also U_FPGA.AB25; no longer U_FPGA.P25
- net LINK0_DATA6: now also U_FPGA.AA26; no longer U_FPGA.N26
- net LINK0_DATA7: now also U_FPGA.AA25; no longer U_FPGA.N25
- net LINK0_READY_BACK: now also U_FPGA.W26; no longer U_FPGA.L26
- net LINK0_SOF: now also U_FPGA.W25; no longer U_FPGA.L25
- net LINK0_VALID: now also U_FPGA.Y25; no longer U_FPGA.M25
- net LINK10_CLOCK: now also U_FPGA.H25; no longer U_FPGA.AE12
- net LINK10_DATA0: now also U_FPGA.D25; no longer U_FPGA.AE16
- net LINK10_DATA1: now also U_FPGA.D26; no longer U_FPGA.AF16
- net LINK10_DATA2: now also U_FPGA.E25; no longer U_FPGA.AE15
- net LINK10_DATA3: now also U_FPGA.E26; no longer U_FPGA.AF15
- net LINK10_DATA4: now also U_FPGA.F25; no longer U_FPGA.AE14
- net LINK10_DATA5: now also U_FPGA.F26; no longer U_FPGA.AF14
- net LINK10_DATA6: now also U_FPGA.G25; no longer U_FPGA.AE13
- net LINK10_DATA7: now also U_FPGA.G26; no longer U_FPGA.AF13
- net LINK10_READY_BACK: now also U_FPGA.J25; no longer U_FPGA.AE11
- net LINK10_SOF: now also U_FPGA.J26; no longer U_FPGA.AF11
- net LINK10_VALID: now also U_FPGA.H26; no longer U_FPGA.AF12
- net MGTAVCC: now also U_FPGA.AE6, U_FPGA.N26, U_FPGA.W16; no longer U_FPGA.AE18, U_FPGA.T9, U_FPGA.W22
- net MGTAVTT: now also U_FPGA.AE12, U_FPGA.T9, U_FPGA.W22; no longer U_FPGA.AB11, U_FPGA.AE24, U_FPGA.T15
- net VCCAUX_1V8: now also U_FPGA.AB11, U_FPGA.AE18, U_FPGA.T15; no longer U_FPGA.AB17, U_FPGA.T21
- net VCCINT_0V85: now also U_FPGA.AE14, U_FPGA.AE16, U_FPGA.AF11, U_FPGA.AF13, U_FPGA.AF15, U_FPGA.L26, U_FPGA.M25, U_FPGA.P25, U_FPGA.R26, U_FPGA.T25; no longer U_FPGA.AA26, U_FPGA.AB25, U_FPGA.AC26, U_FPGA.AD25, U_FPGA.D25, U_FPGA.E26, U_FPGA.F25, U_FPGA.G26, U_FPGA.H25, U_FPGA.J26, U_FPGA.W26, U_FPGA.Y25
- net VCCO_1V2: now also U_FPGA.AB23, U_FPGA.W10; no longer U_FPGA.AE6, U_FPGA.W16
- net VCCO_1V8: now also U_FPGA.AB17, U_FPGA.AE24, U_FPGA.T21; no longer U_FPGA.AB23, U_FPGA.W10

Commit message: Shorten the folded-row stagger and turn the FPGA to face the slot row
The through-hole slot stagger counted an escape allowance the ribbon band
never uses; deriving it from the slot's half body, the pin clearance and
the band's offset gives 29 mm instead of 38, and the short 2U board drops
from 170 to 160 mm deep.

The FPGA now sits at rotation 0 with link_out on its north edge into the
outbound set's band and link_in on its south edge beside PCIe, so neither
FPGA hop wraps round the package.  Its core regulator moves to the west
edge and the DDR4 with its regulators to the east, against the PSU bay.
fpga_ball_map takes an edge per port and place_fpga_neighbours takes the
DDR side and the regulator side; the two-row layout uses the shared helper
with its old placement.  The report quotes one rounded stagger figure.

Tests, README and the generated PSRAM outputs follow.

Co-Authored-By: Claude Fable 5.1 <noreply@anthropic.com>
Claude-Session: https://claude.ai/code/session_01VmmvkZe8Ctg3RAykNGsQBn
Connections:
- net DDR4_ADDR_CMD0: now also U_FPGA.L24; no longer U_FPGA.L5
- net DDR4_ADDR_CMD1: now also U_FPGA.M24; no longer U_FPGA.M5
- net DDR4_ADDR_CMD10: now also U_FPGA.AA24; no longer U_FPGA.AA5
- net DDR4_ADDR_CMD11: now also U_FPGA.AB24; no longer U_FPGA.AB5
- net DDR4_ADDR_CMD12: now also U_FPGA.C25; no longer U_FPGA.C6
- net DDR4_ADDR_CMD13: now also U_FPGA.D25; no longer U_FPGA.D6
- net DDR4_ADDR_CMD14: now also U_FPGA.E25; no longer U_FPGA.E6
- net DDR4_ADDR_CMD15: now also U_FPGA.F25; no longer U_FPGA.F6
- net DDR4_ADDR_CMD16: now also U_FPGA.G25; no longer U_FPGA.G6
- net DDR4_ADDR_CMD17: now also U_FPGA.H25; no longer U_FPGA.H6
- net DDR4_ADDR_CMD18: now also U_FPGA.J25; no longer U_FPGA.J6
- net DDR4_ADDR_CMD19: now also U_FPGA.K25; no longer U_FPGA.K6
- net DDR4_ADDR_CMD2: now also U_FPGA.N24; no longer U_FPGA.N5
- net DDR4_ADDR_CMD20: now also U_FPGA.L25; no longer U_FPGA.L6
- net DDR4_ADDR_CMD21: now also U_FPGA.M25; no longer U_FPGA.M6
- net DDR4_ADDR_CMD22: now also U_FPGA.N25; no longer U_FPGA.N6
- net DDR4_ADDR_CMD23: now also U_FPGA.P25; no longer U_FPGA.P6
- net DDR4_ADDR_CMD24: now also U_FPGA.R25; no longer U_FPGA.R6
- net DDR4_ADDR_CMD25: now also U_FPGA.T25; no longer U_FPGA.T6
- net DDR4_ADDR_CMD26: now also U_FPGA.U25; no longer U_FPGA.U6
- net DDR4_ADDR_CMD27: now also U_FPGA.V25; no longer U_FPGA.V6
- net DDR4_ADDR_CMD3: now also U_FPGA.P24; no longer U_FPGA.P5
- net DDR4_ADDR_CMD4: now also U_FPGA.R24; no longer U_FPGA.R5
- net DDR4_ADDR_CMD5: now also U_FPGA.T24; no longer U_FPGA.T5
- net DDR4_ADDR_CMD6: now also U_FPGA.U24; no longer U_FPGA.U5
- net DDR4_ADDR_CMD7: now also U_FPGA.V24; no longer U_FPGA.V5
- net DDR4_ADDR_CMD8: now also U_FPGA.W24; no longer U_FPGA.W5
- net DDR4_ADDR_CMD9: now also U_FPGA.Y24; no longer U_FPGA.Y5
- net DDR4_CK_N: now also U_FPGA.Y25; no longer U_FPGA.Y6
- net DDR4_CK_P: now also U_FPGA.W25; no longer U_FPGA.W6
- net DDR4_CTRL0: now also U_FPGA.AA25; no longer U_FPGA.AA6
- net DDR4_CTRL1: now also U_FPGA.AB25; no longer U_FPGA.AB6
- net DDR4_CTRL2: now also U_FPGA.C26; no longer U_FPGA.C7
- net DDR4_CTRL3: now also U_FPGA.D26; no longer U_FPGA.D7
- net DDR4_CTRL4: now also U_FPGA.E26; no longer U_FPGA.E7
- net DDR4_CTRL5: now also U_FPGA.F26; no longer U_FPGA.F7
- net DDR4_DM0: now also U_FPGA.C24; no longer U_FPGA.C5
- net DDR4_DM1: now also U_FPGA.D24; no longer U_FPGA.D5
- net DDR4_DM2: now also U_FPGA.E24; no longer U_FPGA.E5
- net DDR4_DM3: now also U_FPGA.F24; no longer U_FPGA.F5
- net DDR4_DM4: now also U_FPGA.G24; no longer U_FPGA.G5
- net DDR4_DM5: now also U_FPGA.H24; no longer U_FPGA.H5
- net DDR4_DM6: now also U_FPGA.J24; no longer U_FPGA.J5
- net DDR4_DM7: now also U_FPGA.K24; no longer U_FPGA.K5
- net DDR4_DQ0: now also U_FPGA.C20; no longer U_FPGA.C1
- net DDR4_DQ1: now also U_FPGA.D20; no longer U_FPGA.D1
- net DDR4_DQ10: now also U_FPGA.N20; no longer U_FPGA.N1
- net DDR4_DQ11: now also U_FPGA.P20; no longer U_FPGA.P1
- net DDR4_DQ12: now also U_FPGA.R20; no longer U_FPGA.R1
- net DDR4_DQ13: now also U_FPGA.T20; no longer U_FPGA.T1
- net DDR4_DQ14: now also U_FPGA.U20; no longer U_FPGA.U1
- net DDR4_DQ15: now also U_FPGA.V20; no longer U_FPGA.V1
- net DDR4_DQ16: now also U_FPGA.W20; no longer U_FPGA.W1
- net DDR4_DQ17: now also U_FPGA.Y20; no longer U_FPGA.Y1
- net DDR4_DQ18: now also U_FPGA.AA20; no longer U_FPGA.AA1
- net DDR4_DQ19: now also U_FPGA.AB20; no longer U_FPGA.AB1
- net DDR4_DQ2: now also U_FPGA.E20; no longer U_FPGA.E1
- net DDR4_DQ20: now also U_FPGA.C21; no longer U_FPGA.C2
- net DDR4_DQ21: now also U_FPGA.D21; no longer U_FPGA.D2
- net DDR4_DQ22: now also U_FPGA.E21; no longer U_FPGA.E2
- net DDR4_DQ23: now also U_FPGA.F21; no longer U_FPGA.F2
- net DDR4_DQ24: now also U_FPGA.G21; no longer U_FPGA.G2
- net DDR4_DQ25: now also U_FPGA.H21; no longer U_FPGA.H2
- net DDR4_DQ26: now also U_FPGA.J21; no longer U_FPGA.J2
- net DDR4_DQ27: now also U_FPGA.K21; no longer U_FPGA.K2
- net DDR4_DQ28: now also U_FPGA.L21; no longer U_FPGA.L2
- net DDR4_DQ29: now also U_FPGA.M21; no longer U_FPGA.M2
- net DDR4_DQ3: now also U_FPGA.F20; no longer U_FPGA.F1
- net DDR4_DQ30: now also U_FPGA.N21; no longer U_FPGA.N2
- net DDR4_DQ31: now also U_FPGA.P21; no longer U_FPGA.P2
- net DDR4_DQ32: now also U_FPGA.R21; no longer U_FPGA.R2
- net DDR4_DQ33: now also U_FPGA.T21; no longer U_FPGA.T2
- net DDR4_DQ34: now also U_FPGA.U21; no longer U_FPGA.U2
- net DDR4_DQ35: now also U_FPGA.V21; no longer U_FPGA.V2
- net DDR4_DQ36: now also U_FPGA.W21; no longer U_FPGA.W2
- net DDR4_DQ37: now also U_FPGA.Y21; no longer U_FPGA.Y2
- net DDR4_DQ38: now also U_FPGA.AA21; no longer U_FPGA.AA2
- net DDR4_DQ39: now also U_FPGA.AB21; no longer U_FPGA.AB2
- net DDR4_DQ4: now also U_FPGA.G20; no longer U_FPGA.G1
- net DDR4_DQ40: now also U_FPGA.C22; no longer U_FPGA.C3
- net DDR4_DQ41: now also U_FPGA.D22; no longer U_FPGA.D3
- net DDR4_DQ42: now also U_FPGA.E22; no longer U_FPGA.E3
- net DDR4_DQ43: now also U_FPGA.F22; no longer U_FPGA.F3
- net DDR4_DQ44: now also U_FPGA.G22; no longer U_FPGA.G3
- net DDR4_DQ45: now also U_FPGA.H22; no longer U_FPGA.H3
- net DDR4_DQ46: now also U_FPGA.J22; no longer U_FPGA.J3
- net DDR4_DQ47: now also U_FPGA.K22; no longer U_FPGA.K3
- net DDR4_DQ48: now also U_FPGA.L22; no longer U_FPGA.L3
- net DDR4_DQ49: now also U_FPGA.M22; no longer U_FPGA.M3
- net DDR4_DQ5: now also U_FPGA.H20; no longer U_FPGA.H1
- net DDR4_DQ50: now also U_FPGA.N22; no longer U_FPGA.N3
- net DDR4_DQ51: now also U_FPGA.P22; no longer U_FPGA.P3
- net DDR4_DQ52: now also U_FPGA.R22; no longer U_FPGA.R3
- net DDR4_DQ53: now also U_FPGA.T22; no longer U_FPGA.T3
- net DDR4_DQ54: now also U_FPGA.U22; no longer U_FPGA.U3
- net DDR4_DQ55: now also U_FPGA.V22; no longer U_FPGA.V3
- net DDR4_DQ56: now also U_FPGA.W22; no longer U_FPGA.W3
- net DDR4_DQ57: now also U_FPGA.Y22; no longer U_FPGA.Y3
- net DDR4_DQ58: now also U_FPGA.AA22; no longer U_FPGA.AA3
- net DDR4_DQ59: now also U_FPGA.AB22; no longer U_FPGA.AB3
- net DDR4_DQ6: now also U_FPGA.J20; no longer U_FPGA.J1
- net DDR4_DQ60: now also U_FPGA.C23; no longer U_FPGA.C4
- net DDR4_DQ61: now also U_FPGA.D23; no longer U_FPGA.D4
- net DDR4_DQ62: now also U_FPGA.E23; no longer U_FPGA.E4
- net DDR4_DQ63: now also U_FPGA.F23; no longer U_FPGA.F4
- net DDR4_DQ7: now also U_FPGA.K20; no longer U_FPGA.K1
- net DDR4_DQ8: now also U_FPGA.L20; no longer U_FPGA.L1
- net DDR4_DQ9: now also U_FPGA.M20; no longer U_FPGA.M1
- net DDR4_DQS0_N: now also U_FPGA.H23; no longer U_FPGA.H4
- net DDR4_DQS0_P: now also U_FPGA.G23; no longer U_FPGA.G4
- net DDR4_DQS1_N: now also U_FPGA.K23; no longer U_FPGA.K4
- net DDR4_DQS1_P: now also U_FPGA.J23; no longer U_FPGA.J4
- net DDR4_DQS2_N: now also U_FPGA.M23; no longer U_FPGA.M4
- net DDR4_DQS2_P: now also U_FPGA.L23; no longer U_FPGA.L4
- net DDR4_DQS3_N: now also U_FPGA.P23; no longer U_FPGA.P4
- net DDR4_DQS3_P: now also U_FPGA.N23; no longer U_FPGA.N4
- net DDR4_DQS4_N: now also U_FPGA.T23; no longer U_FPGA.T4
- net DDR4_DQS4_P: now also U_FPGA.R23; no longer U_FPGA.R4
- net DDR4_DQS5_N: now also U_FPGA.V23; no longer U_FPGA.V4
- net DDR4_DQS5_P: now also U_FPGA.U23; no longer U_FPGA.U4
- net DDR4_DQS6_N: now also U_FPGA.Y23; no longer U_FPGA.Y4
- net DDR4_DQS6_P: now also U_FPGA.W23; no longer U_FPGA.W4
- net DDR4_DQS7_N: now also U_FPGA.AB23; no longer U_FPGA.AB4
- net DDR4_DQS7_P: now also U_FPGA.AA23; no longer U_FPGA.AA4
- net GND: now also U_FPGA.A17, U_FPGA.A19, U_FPGA.A21, U_FPGA.A23, U_FPGA.A3, U_FPGA.A5, U_FPGA.A7, U_FPGA.A9, U_FPGA.AA1, U_FPGA.AA3, U_FPGA.AA5, U_FPGA.AB2, U_FPGA.AB26, U_FPGA.AB4, U_FPGA.AB6, U_FPGA.AC25, U_FPGA.AD26, U_FPGA.B10, U_FPGA.B4, U_FPGA.B6, U_FPGA.B8, U_FPGA.C1, U_FPGA.C3, U_FPGA.C5, U_FPGA.C7, U_FPGA.D2, U_FPGA.D4, U_FPGA.D6, U_FPGA.E1, U_FPGA.E3, U_FPGA.E5, U_FPGA.E7, U_FPGA.F2, U_FPGA.F4, U_FPGA.F6, U_FPGA.G1, U_FPGA.G3, U_FPGA.G5, U_FPGA.H2, U_FPGA.H26, U_FPGA.H4, U_FPGA.H6, U_FPGA.J1, U_FPGA.J3, U_FPGA.J5, U_FPGA.K2, U_FPGA.K4, U_FPGA.K6, U_FPGA.L1, U_FPGA.L3, U_FPGA.L5, U_FPGA.M2, U_FPGA.M4, U_FPGA.M6, U_FPGA.N1, U_FPGA.N3, U_FPGA.N5, U_FPGA.P2, U_FPGA.P4, U_FPGA.P6, U_FPGA.R1, U_FPGA.R3, U_FPGA.R5, U_FPGA.T2, U_FPGA.T4, U_FPGA.T6, U_FPGA.U1, U_FPGA.U3, U_FPGA.U5, U_FPGA.V2, U_FPGA.V4, U_FPGA.V6, U_FPGA.W1, U_FPGA.W3, U_FPGA.W5, U_FPGA.Y2, U_FPGA.Y26, U_FPGA.Y4, U_FPGA.Y6; no longer U_FPGA.AA21, U_FPGA.AA23, U_FPGA.AB20, U_FPGA.AB22, U_FPGA.AB24, U_FPGA.AE1, U_FPGA.AE11, U_FPGA.AE13, U_FPGA.AE15, U_FPGA.AE17, U_FPGA.AE19, U_FPGA.AE21, U_FPGA.AE3, U_FPGA.AE5, U_FPGA.AE7, U_FPGA.AE9, U_FPGA.AF10, U_FPGA.AF12, U_FPGA.AF14, U_FPGA.AF16, U_FPGA.AF18, U_FPGA.AF2, U_FPGA.AF20, U_FPGA.AF22, U_FPGA.AF24, U_FPGA.AF26, U_FPGA.AF4, U_FPGA.AF6, U_FPGA.AF8, U_FPGA.C21, U_FPGA.C23, U_FPGA.C25, U_FPGA.D20, U_FPGA.D22, U_FPGA.D24, U_FPGA.E21, U_FPGA.E23, U_FPGA.F20, U_FPGA.F22, U_FPGA.F24, U_FPGA.G21, U_FPGA.G23, U_FPGA.H20, U_FPGA.H22, U_FPGA.H24, U_FPGA.J21, U_FPGA.J23, U_FPGA.K20, U_FPGA.K22, U_FPGA.K24, U_FPGA.L21, U_FPGA.L23, U_FPGA.L25, U_FPGA.M20, U_FPGA.M22, U_FPGA.M24, U_FPGA.N21, U_FPGA.N23, U_FPGA.N25, U_FPGA.P20, U_FPGA.P22, U_FPGA.P24, U_FPGA.R21, U_FPGA.R23, U_FPGA.R25, U_FPGA.T20, U_FPGA.T22, U_FPGA.T24, U_FPGA.U21, U_FPGA.U23, U_FPGA.U25, U_FPGA.V20, U_FPGA.V22, U_FPGA.V24, U_FPGA.W21, U_FPGA.W23, U_FPGA.Y20, U_FPGA.Y22, U_FPGA.Y24
- net LINK0_CLOCK: now also U_FPGA.B12; no longer U_FPGA.Y26
- net LINK0_DATA0: now also U_FPGA.B16; no longer U_FPGA.AD26
- net LINK0_DATA1: now also U_FPGA.A16; no longer U_FPGA.AD25
- net LINK0_DATA2: now also U_FPGA.B15; no longer U_FPGA.AC26
- net LINK0_DATA3: now also U_FPGA.A15; no longer U_FPGA.AC25
- net LINK0_DATA4: now also U_FPGA.B14; no longer U_FPGA.AB26
- net LINK0_DATA5: now also U_FPGA.A14; no longer U_FPGA.AB25
- net LINK0_DATA6: now also U_FPGA.B13; no longer U_FPGA.AA26
- net LINK0_DATA7: now also U_FPGA.A13; no longer U_FPGA.AA25
- net LINK0_READY_BACK: now also U_FPGA.B11; no longer U_FPGA.W26
- net LINK0_SOF: now also U_FPGA.A11; no longer U_FPGA.W25
- net LINK0_VALID: now also U_FPGA.A12; no longer U_FPGA.Y25
- net LINK10_CLOCK: now also U_FPGA.AE12; no longer U_FPGA.H25
- net LINK10_DATA0: now also U_FPGA.AE16; no longer U_FPGA.D25
- net LINK10_DATA1: now also U_FPGA.AF16; no longer U_FPGA.D26
- net LINK10_DATA2: now also U_FPGA.AE15; no longer U_FPGA.E25
- net LINK10_DATA3: now also U_FPGA.AF15; no longer U_FPGA.E26
- net LINK10_DATA4: now also U_FPGA.AE14; no longer U_FPGA.F25
- net LINK10_DATA5: now also U_FPGA.AF14; no longer U_FPGA.F26
- net LINK10_DATA6: now also U_FPGA.AE13; no longer U_FPGA.G25
- net LINK10_DATA7: now also U_FPGA.AF13; no longer U_FPGA.G26
- net LINK10_READY_BACK: now also U_FPGA.AE11; no longer U_FPGA.J25
- net LINK10_SOF: now also U_FPGA.AF11; no longer U_FPGA.J26
- net LINK10_VALID: now also U_FPGA.AF12; no longer U_FPGA.H26
- net MGTAVCC: now also U_FPGA.AB5, U_FPGA.D5, U_FPGA.G18, U_FPGA.N2, U_FPGA.T9; no longer U_FPGA.AE6, U_FPGA.G12, U_FPGA.K19, U_FPGA.N26, U_FPGA.W16
- net MGTAVTT: now also U_FPGA.AB11, U_FPGA.D11, U_FPGA.K1, U_FPGA.N8, U_FPGA.T15; no longer U_FPGA.AE12, U_FPGA.G18, U_FPGA.K25, U_FPGA.T9, U_FPGA.W22
- net PCIE_PERST: now also U_FPGA.AE21; no longer U_FPGA.B15
- net PCIE_REFCLK_N: now also U_FPGA.AE20; no longer U_FPGA.B14
- net PCIE_REFCLK_P: now also U_FPGA.AE19; no longer U_FPGA.B13
- net PCIE_RX0_N: now also U_FPGA.AF24; no longer U_FPGA.A20
- net PCIE_RX0_P: now also U_FPGA.AF23; no longer U_FPGA.A19
- net PCIE_RX1_N: now also U_FPGA.AF26; no longer U_FPGA.A22
- net PCIE_RX1_P: now also U_FPGA.AF25; no longer U_FPGA.A21
- net PCIE_RX2_N: now also U_FPGA.AE2; no longer U_FPGA.A24
- net PCIE_RX2_P: now also U_FPGA.AE1; no longer U_FPGA.A23
- net PCIE_RX3_N: now also U_FPGA.AE4; no longer U_FPGA.B4
- net PCIE_RX3_P: now also U_FPGA.AE3; no longer U_FPGA.B3
- net PCIE_RX4_N: now also U_FPGA.AE6; no longer U_FPGA.B6
- net PCIE_RX4_P: now also U_FPGA.AE5; no longer U_FPGA.B5
- net PCIE_RX5_N: now also U_FPGA.AE8; no longer U_FPGA.B8
- net PCIE_RX5_P: now also U_FPGA.AE7; no longer U_FPGA.B7
- net PCIE_RX6_N: now also U_FPGA.AE10; no longer U_FPGA.B10
- net PCIE_RX6_P: now also U_FPGA.AE9; no longer U_FPGA.B9
- net PCIE_RX7_N: now also U_FPGA.AE18; no longer U_FPGA.B12
- net PCIE_RX7_P: now also U_FPGA.AE17; no longer U_FPGA.B11
- net PCIE_TX0_N: now also U_FPGA.AF2; no longer U_FPGA.A4
- net PCIE_TX0_P: now also U_FPGA.AF1; no longer U_FPGA.A3
- net PCIE_TX1_N: now also U_FPGA.AF4; no longer U_FPGA.A6
- net PCIE_TX1_P: now also U_FPGA.AF3; no longer U_FPGA.A5
- net PCIE_TX2_N: now also U_FPGA.AF6; no longer U_FPGA.A8
- net PCIE_TX2_P: now also U_FPGA.AF5; no longer U_FPGA.A7
- net PCIE_TX3_N: now also U_FPGA.AF8; no longer U_FPGA.A10
- net PCIE_TX3_P: now also U_FPGA.AF7; no longer U_FPGA.A9
- net PCIE_TX4_N: now also U_FPGA.AF10; no longer U_FPGA.A12
- net PCIE_TX4_P: now also U_FPGA.AF9; no longer U_FPGA.A11
- net PCIE_TX5_N: now also U_FPGA.AF18; no longer U_FPGA.A14
- net PCIE_TX5_P: now also U_FPGA.AF17; no longer U_FPGA.A13
- net PCIE_TX6_N: now also U_FPGA.AF20; no longer U_FPGA.A16
- net PCIE_TX6_P: now also U_FPGA.AF19; no longer U_FPGA.A15
- net PCIE_TX7_N: now also U_FPGA.AF22; no longer U_FPGA.A18
- net PCIE_TX7_P: now also U_FPGA.AF21; no longer U_FPGA.A17
- net PCIE_WAKE: now also U_FPGA.AE22; no longer U_FPGA.B16
- net VCCAUX_1V8: now also U_FPGA.A4, U_FPGA.AB17, U_FPGA.D17, U_FPGA.K7, U_FPGA.N14, U_FPGA.W4; no longer U_FPGA.AB11, U_FPGA.AE18, U_FPGA.D11, U_FPGA.G24, U_FPGA.N8, U_FPGA.T15
- net VCCINT_0V85: now also U_FPGA.A18, U_FPGA.A20, U_FPGA.A24, U_FPGA.A6, U_FPGA.A8, U_FPGA.AA2, U_FPGA.AA26, U_FPGA.AA4, U_FPGA.AA6, U_FPGA.AB1, U_FPGA.AB3, U_FPGA.AC26, U_FPGA.AD25, U_FPGA.B3, U_FPGA.B5, U_FPGA.B7, U_FPGA.B9, U_FPGA.C2, U_FPGA.C4, U_FPGA.C6, U_FPGA.D1, U_FPGA.D3, U_FPGA.D7, U_FPGA.E2, U_FPGA.E4, U_FPGA.E6, U_FPGA.F1, U_FPGA.F3, U_FPGA.F5, U_FPGA.F7, U_FPGA.G2, U_FPGA.G26, U_FPGA.G4, U_FPGA.H1, U_FPGA.H3, U_FPGA.H5, U_FPGA.J2, U_FPGA.J26, U_FPGA.J4, U_FPGA.J6, U_FPGA.K3, U_FPGA.K5, U_FPGA.L2, U_FPGA.L4, U_FPGA.L6, U_FPGA.M1, U_FPGA.M3, U_FPGA.M5, U_FPGA.N4, U_FPGA.N6, U_FPGA.P1, U_FPGA.P3, U_FPGA.P5, U_FPGA.R2, U_FPGA.R4, U_FPGA.R6, U_FPGA.T1, U_FPGA.T5, U_FPGA.U2, U_FPGA.U4, U_FPGA.U6, U_FPGA.V1, U_FPGA.V3, U_FPGA.V5, U_FPGA.W2, U_FPGA.W26, U_FPGA.W6, U_FPGA.Y1, U_FPGA.Y3, U_FPGA.Y5; no longer U_FPGA.AA20, U_FPGA.AA22, U_FPGA.AA24, U_FPGA.AB21, U_FPGA.AE10, U_FPGA.AE14, U_FPGA.AE16, U_FPGA.AE2, U_FPGA.AE20, U_FPGA.AE22, U_FPGA.AE4, U_FPGA.AE8, U_FPGA.AF1, U_FPGA.AF11, U_FPGA.AF13, U_FPGA.AF15, U_FPGA.AF17, U_FPGA.AF19, U_FPGA.AF21, U_FPGA.AF23, U_FPGA.AF25, U_FPGA.AF3, U_FPGA.AF5, U_FPGA.AF7, U_FPGA.AF9, U_FPGA.C20, U_FPGA.C22, U_FPGA.C24, U_FPGA.C26, U_FPGA.D21, U_FPGA.E20, U_FPGA.E22, U_FPGA.E24, U_FPGA.F21, U_FPGA.F23, U_FPGA.G20, U_FPGA.G22, U_FPGA.H21, U_FPGA.H23, U_FPGA.J20, U_FPGA.J22, U_FPGA.J24, U_FPGA.K21, U_FPGA.K23, U_FPGA.L20, U_FPGA.L22, U_FPGA.L24, U_FPGA.M21, U_FPGA.M23, U_FPGA.M25, U_FPGA.N22, U_FPGA.N24, U_FPGA.P21, U_FPGA.P23, U_FPGA.P25, U_FPGA.R20, U_FPGA.R22, U_FPGA.R24, U_FPGA.T23, U_FPGA.T25, U_FPGA.U20, U_FPGA.U22, U_FPGA.U24, U_FPGA.V21, U_FPGA.V23, U_FPGA.V25, U_FPGA.W20, U_FPGA.W24, U_FPGA.Y21, U_FPGA.Y23
- net VCCO_1V2: now also U_FPGA.A22, U_FPGA.G12, U_FPGA.K19, U_FPGA.T3, U_FPGA.W16; no longer U_FPGA.AB23, U_FPGA.D23, U_FPGA.K13, U_FPGA.N20, U_FPGA.W10
- net VCCO_1V8: now also U_FPGA.A10, U_FPGA.G6, U_FPGA.K13, U_FPGA.N26, U_FPGA.W10; no longer U_FPGA.AB17, U_FPGA.D17, U_FPGA.K7, U_FPGA.N14, U_FPGA.T21

Commit message: Choose the PSRAM board's FPGA: XCAU15P-2FFVB676E, with the fit checked
The controller FPGA is the AMD Artix UltraScale+ AU15P in FFVB676, the
one Artix UltraScale+ package whose transceivers run at 16.3 Gb/s and
whose PCIe block is Gen4 x8, so the host link stays as specified.  The
class records the part's resources and an io_plan (DDR4 on the HP
banks, the transceiver pairs on the GTH quads, the rest on HD), and
board.py checks and reports the fit: 124 of 156 HP I/O, 52 of 72 HD,
9 of 12 lanes.  The KiCad FPGA symbol carries the part number when the
class names one.

Co-Authored-By: Claude Fable 5.1 <noreply@anthropic.com>
Claude-Session: https://claude.ai/code/session_01VmmvkZe8Ctg3RAykNGsQBn
Parts:
- U_FPGA: value FPGA -> XCAU15P-2FFVB676E
Changed lines of the file:
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@@
   (symbol (lib_id "appliance:fpga") (at 309.63 309.63 0) (unit 1) (in_bom yes) (on_board yes) (dnp no)
     (property "Reference" "U_FPGA" (at 309.63 87 0) (effects (font (size 2 2))))
-    (property "Value" "FPGA" (at 309.63 532.26 0) (effects (font (size 1.5 1.5))))
+    (property "Value" "XCAU15P-2FFVB676E" (at 309.63 532.26 0) (effects (font (size 1.5 1.5))))
     (property "Footprint" "appliance:FFVB676_26x26_P1.0" (at 309.63 309.63 0) (effects (font (size 1.27 1.27)) hide))
     (pin "A1")
@@
     (pin "AF25")
     (pin "AF26")
-    (instances (project "appliance" (path "/b363f2b7-d82b-4060-bc2e-dd969050e0e4/6b62cff2-c0c4-4134-9de9-7646bb73b1d8" (reference "U_FPGA") (unit 1))))
+    (instances (project "appliance" (path "/43d7ae43-76b3-4aac-9135-e49f10a8b944/45c89e01-2854-4607-8c7d-441e36c6bf5c" (reference "U_FPGA") (unit 1))))
   )
   (global_label "GND" (shape input) (at 87.46 522.99 180) (effects (font (size 0.8 0.8)) (justify right)) (property "Intersheetrefs" "${INTERSHEET_REFS}" (at 0 0 0) (effects (font (size 0.8 0.8)) hide)))
@@
     (pin "23")
     (pin "24")
-    (instances (project "appliance" (path "/b363f2b7-d82b-4060-bc2e-dd969050e0e4/6b62cff2-c0c4-4134-9de9-7646bb73b1d8" (reference "U_CLK") (unit 1))))
+    (instances (project "appliance" (path "/43d7ae43-76b3-4aac-9135-e49f10a8b944/45c89e01-2854-4607-8c7d-441e36c6bf5c" (reference "U_CLK") (unit 1))))
   )
   (global_label "VDD_IO_1V8" (shape input) (at 586.72 108.97 180) (effects (font (size 0.8 0.8)) (justify right)) (property "Intersheetrefs" "${INTERSHEET_REFS}" (at 0 0 0) (effects (font (size 0.8 0.8)) hide)))
@@
     (pin "53")
     (pin "54")
-    (instances (project "appliance" (path "/b363f2b7-d82b-4060-bc2e-dd969050e0e4/6b62cff2-c0c4-4134-9de9-7646bb73b1d8" (reference "J_HOST") (unit 1))))
+    (instances (project "appliance" (path "/43d7ae43-76b3-4aac-9135-e49f10a8b944/45c89e01-2854-4607-8c7d-441e36c6bf5c" (reference "J_HOST") (unit 1))))
   )
   (global_label "PCIE_TX0_P" (shape input) (at 676.72 129.29 180) (effects (font (size 0.8 0.8)) (justify right)) (property "Intersheetrefs" "${INTERSHEET_REFS}" (at 0 0 0) (effects (font (size 0.8 0.8)) hide)))
@@
     (pin "15")
     (pin "16")
-    (instances (project "appliance" (path "/b363f2b7-d82b-4060-bc2e-dd969050e0e4/6b62cff2-c0c4-4134-9de9-7646bb73b1d8" (reference "J_SFP") (unit 1))))
+    (instances (project "appliance" (path "/43d7ae43-76b3-4aac-9135-e49f10a8b944/45c89e01-2854-4607-8c7d-441e36c6bf5c" (reference "J_SFP") (unit 1))))
   )
   (global_label "SFP_TX_P" (shape input) (at 782.28 103.89 180) (effects (font (size 0.8 0.8)) (justify right)) (property "Intersheetrefs" "${INTERSHEET_REFS}" (at 0 0 0) (effects (font (size 0.8 0.8)) hide)))
@@
     (pin "11")
     (pin "12")
-    (instances (project "appliance" (path "/b363f2b7-d82b-4060-bc2e-dd969050e0e4/6b62cff2-c0c4-4134-9de9-7646bb73b1d8" (reference "J_BMC_NET") (unit 1))))
+    (instances (project "appliance" (path "/43d7ae43-76b3-4aac-9135-e49f10a8b944/45c89e01-2854-4607-8c7d-441e36c6bf5c" (reference "J_BMC_NET") (unit 1))))
   )
   (global_label "BMC_ETH0_P" (shape input) (at 872.28 102.54 180) (effects (font (size 0.8 0.8)) (justify right)) (property "Intersheetrefs" "${INTERSHEET_REFS}" (at 0 0 0) (effects (font (size 0.8 0.8)) hide)))
@@
     (pin "28")
     (pin "29")
-    (instances (project "appliance" (path "/b363f2b7-d82b-4060-bc2e-dd969050e0e4/6b62cff2-c0c4-4134-9de9-7646bb73b1d8" (reference "U_BMC") (unit 1))))
+    (instances (project "appliance" (path "/43d7ae43-76b3-4aac-9135-e49f10a8b944/45c89e01-2854-4607-8c7d-441e36c6bf5c" (reference "U_BMC") (unit 1))))
   )
   (global_label "BMC_ETH0_P" (shape input) (at 962.28 114.05 180) (effects (font (size 0.8 0.8)) (justify right)) (property "Intersheetrefs" "${INTERSHEET_REFS}" (at 0 0 0) (effects (font (size 0.8 0.8)) hide)))
