File: hw/kicad_psram/module_asics.kicad_sch (KiCad schematic)
At the start: 2 parts

Commit message: Link in and out on the same finger positions: straight slot-to-slot hops
link_in sits on side A and link_out on side B of the same twelve edge
positions, so a slot's out-row pin faces the next slot's in-row pin and
every skip-one hop is a straight ribbon.  On the card the two drops from
the die's south-edge blocks lean towards one finger span from either side
and cross, so the out drop takes In3 and the two faces' vias interleave
half a position apart above the fingers.  The ribbon band narrows from
27 mm to 12, the stagger from 52 mm to 38, and the short board from 180 to
170 mm deep.  finger_layout: offset keeps the earlier separate spans.

Co-Authored-By: Claude Fable 5.1 <noreply@anthropic.com>
Claude-Session: https://claude.ai/code/session_01VmmvkZe8Ctg3RAykNGsQBn
Connections:
- net GND: now also J_EDGE.B27, J_EDGE.B28, J_EDGE.B29, J_EDGE.B30, J_EDGE.B31, J_EDGE.B32, J_EDGE.B33, J_EDGE.B34, J_EDGE.B35, J_EDGE.B36, J_EDGE.B37, J_EDGE.B38; no longer J_EDGE.B12, J_EDGE.B13, J_EDGE.B14, J_EDGE.B15, J_EDGE.B16, J_EDGE.B17, J_EDGE.B18, J_EDGE.B19, J_EDGE.B20, J_EDGE.B21, J_EDGE.B22, J_EDGE.B23
- net LINK_OUT_CLOCK: now also J_EDGE.B20; no longer J_EDGE.B35
- net LINK_OUT_DATA0: now also J_EDGE.B12; no longer J_EDGE.B27
- net LINK_OUT_DATA1: now also J_EDGE.B13; no longer J_EDGE.B28
- net LINK_OUT_DATA2: now also J_EDGE.B14; no longer J_EDGE.B29
- net LINK_OUT_DATA3: now also J_EDGE.B15; no longer J_EDGE.B30
- net LINK_OUT_DATA4: now also J_EDGE.B16; no longer J_EDGE.B31
- net LINK_OUT_DATA5: now also J_EDGE.B17; no longer J_EDGE.B32
- net LINK_OUT_DATA6: now also J_EDGE.B18; no longer J_EDGE.B33
- net LINK_OUT_DATA7: now also J_EDGE.B19; no longer J_EDGE.B34
- net LINK_OUT_READY_BACK: now also J_EDGE.B22; no longer J_EDGE.B37
- net LINK_OUT_SOF: now also J_EDGE.B23; no longer J_EDGE.B38
- net LINK_OUT_VALID: now also J_EDGE.B21; no longer J_EDGE.B36

Commit message: Choose the PSRAM and write its HPI controller
The PSRAM board's device is the AP Memory APS512XXN-OB9-BG: 512 Mb, the
Xccela DDR interface in x16 (HPI) mode, 250 MHz, 1.8 V, a 24-ball 6 x 8
mm BGA.  fabric/hpi.py carries its geometry, the mode-register
encodings, the command frame and the striping of the die's memory port
over sixteen devices in page-sized stripes; fabric_hpi.sv is the
controller: a per-device channel with the power-up sequence, global
reset, mode registers and an identity check, the command phase on both
clock edges, fixed-latency writes with data mask, and reads captured by
the device's strobe through a gray-pointer ring so refresh push-out
costs nothing; and a stripe unit that splits a burst into concurrent
per-device chunks, returns read data in order and completes a write
only when every chunk is in the device.  A behavioural device model
checks the protocol (tCEM, tCPH, even addresses, x16 mode) and the
testbench runs random bursts over one, two, four and sixteen devices
against the striped image.

The memory port's burst count widens to 12 bits so a head's state is
one burst across all devices, and the map aligns regions to a page.
The board gains the real part, its DQS/DM naming, and the four shared
clocks as a small interface the pinout places with the management
signals and the card wires to its devices; the connector count is
unchanged.

Co-Authored-By: Claude Fable 5.1 <noreply@anthropic.com>
Claude-Session: https://claude.ai/code/session_01VmmvkZe8Ctg3RAykNGsQBn
Connections:
- net GND: no longer U_CHIP.AG13, U_CHIP.AG17
- net VDD_CORE: no longer U_CHIP.AG14, U_CHIP.AG16
- net PSRAM_0_CS renamed PSRAM_0_CE
- net PSRAM_0_RWDS0 renamed PSRAM_0_DQS0
- net PSRAM_0_RWDS1 renamed PSRAM_0_DQS1
- net PSRAM_10_CS renamed PSRAM_10_CE
- net PSRAM_10_RWDS0 renamed PSRAM_10_DQS0
- net PSRAM_10_RWDS1 renamed PSRAM_10_DQS1
- net PSRAM_11_CS renamed PSRAM_11_CE
- net PSRAM_11_RWDS0 renamed PSRAM_11_DQS0
- net PSRAM_11_RWDS1 renamed PSRAM_11_DQS1
- net PSRAM_12_CS renamed PSRAM_12_CE
- net PSRAM_12_RWDS0 renamed PSRAM_12_DQS0
- net PSRAM_12_RWDS1 renamed PSRAM_12_DQS1
- net PSRAM_13_CS renamed PSRAM_13_CE
- net PSRAM_13_RWDS0 renamed PSRAM_13_DQS0
- net PSRAM_13_RWDS1 renamed PSRAM_13_DQS1
- net PSRAM_14_CS renamed PSRAM_14_CE
- net PSRAM_14_RWDS0 renamed PSRAM_14_DQS0
- net PSRAM_14_RWDS1 renamed PSRAM_14_DQS1
- net PSRAM_15_CS renamed PSRAM_15_CE
- net PSRAM_15_RWDS0 renamed PSRAM_15_DQS0
- net PSRAM_15_RWDS1 renamed PSRAM_15_DQS1
- net PSRAM_1_CS renamed PSRAM_1_CE
- net PSRAM_1_RWDS0 renamed PSRAM_1_DQS0
- net PSRAM_1_RWDS1 renamed PSRAM_1_DQS1
- net PSRAM_2_CS renamed PSRAM_2_CE
- net PSRAM_2_RWDS0 renamed PSRAM_2_DQS0
- net PSRAM_2_RWDS1 renamed PSRAM_2_DQS1
- net PSRAM_3_CS renamed PSRAM_3_CE
- net PSRAM_3_RWDS0 renamed PSRAM_3_DQS0
- net PSRAM_3_RWDS1 renamed PSRAM_3_DQS1
- net PSRAM_4_CS renamed PSRAM_4_CE
- net PSRAM_4_RWDS0 renamed PSRAM_4_DQS0
- net PSRAM_4_RWDS1 renamed PSRAM_4_DQS1
- net PSRAM_5_CS renamed PSRAM_5_CE
- net PSRAM_5_RWDS0 renamed PSRAM_5_DQS0
- net PSRAM_5_RWDS1 renamed PSRAM_5_DQS1
- net PSRAM_6_CS renamed PSRAM_6_CE
- net PSRAM_6_RWDS0 renamed PSRAM_6_DQS0
- net PSRAM_6_RWDS1 renamed PSRAM_6_DQS1
- net PSRAM_7_CS renamed PSRAM_7_CE
- net PSRAM_7_RWDS0 renamed PSRAM_7_DQS0
- net PSRAM_7_RWDS1 renamed PSRAM_7_DQS1
- net PSRAM_8_CS renamed PSRAM_8_CE
- net PSRAM_8_RWDS0 renamed PSRAM_8_DQS0
- net PSRAM_8_RWDS1 renamed PSRAM_8_DQS1
- net PSRAM_9_CS renamed PSRAM_9_CE
- net PSRAM_9_RWDS0 renamed PSRAM_9_DQS0
- net PSRAM_9_RWDS1 renamed PSRAM_9_DQS1
- new net PSRAM_CLK0: U_CHIP.AG13
- new net PSRAM_CLK1: U_CHIP.AG14
- new net PSRAM_CLK2: U_CHIP.AG16
- new net PSRAM_CLK3: U_CHIP.AG17

Commit message: Add the PHY delay lines with their DLL, and settle the PSRAM clock by simulation
fabric_phy.sv is the PHY: a behavioural 256-tap delay line and a master
DLL that measures the clock period in taps with a replica line and a
phase detector, walking the code through one period and then dithering
a tap either side of it; the quarter code drives the slave lines (the
device clock and the two DQS strobes per channel), which take a new
code only while every channel has CE# high.  A line that cannot span
the period is reported rather than searched forever.  The channel
waits for the lock before starting the device, and tb_hpi and
tb_mem_bridge run the whole controller through the delay lines at taps
of 25 to 90 ps in place of the ideal quarter-period delays.

hw/si.py is a small time-domain solver for lossless transmission-line
networks (LC ladder, 1 mm segments, 2 ps steps, Thevenin driver, the
datasheet's 5 pF package input per receiver) and hw/si_psram_clock.md
its answer to whether four devices can share one 250 MHz clock: the
star of four and the fly-by, terminated or not, cannot meet the
device's 0.6 ns edge without ringing past its absolute maximum, two per
clock passes only in a narrow band, and one clock per device passes
from 33 to 50 ohm at every length on the card.  The board takes a
clock per device: sixteen psram_clk balls, the small interfaces
allowed a third row on the south edge, the card's nets one per device,
the derived pinout and KiCad outputs regenerated.

Co-Authored-By: Claude Fable 5.1 <noreply@anthropic.com>
Claude-Session: https://claude.ai/code/session_01VmmvkZe8Ctg3RAykNGsQBn
Connections:
- net GND: now also U_CHIP.AF11, U_CHIP.AG20; no longer U_CHIP.AF10, U_CHIP.AF12, U_CHIP.AF4, U_CHIP.AF8, U_CHIP.AG19, U_CHIP.AG21
- net VDD_CORE: no longer U_CHIP.AF11, U_CHIP.AF13, U_CHIP.AF3, U_CHIP.AF5, U_CHIP.AF7, U_CHIP.AF9, U_CHIP.AG18, U_CHIP.AG20
- new net PSRAM_CLK10: U_CHIP.AF7
- new net PSRAM_CLK11: U_CHIP.AF8
- new net PSRAM_CLK12: U_CHIP.AF9
- new net PSRAM_CLK13: U_CHIP.AF10
- new net PSRAM_CLK14: U_CHIP.AF12
- new net PSRAM_CLK15: U_CHIP.AF13
- new net PSRAM_CLK4: U_CHIP.AG18
- new net PSRAM_CLK5: U_CHIP.AG19
- new net PSRAM_CLK6: U_CHIP.AG21
- new net PSRAM_CLK7: U_CHIP.AF3
- new net PSRAM_CLK8: U_CHIP.AF4
- new net PSRAM_CLK9: U_CHIP.AF5
Changed lines of the file:
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@@
     (pin "A82")
     (pin "B82")
-    (instances (project "appliance" (path "/a44f63fc-7712-4594-9b92-4acfa967723a/c29c41d6-b0a9-4083-849c-c4aea6088c8b" (reference "J_EDGE") (unit 1))))
+    (instances (project "appliance" (path "/53a34ee7-8c3b-4e20-9ef1-ef0d8fcc1954/b343c77a-a6eb-41db-a475-c3a1e922dde8" (reference "J_EDGE") (unit 1))))
   )
   (global_label "+12V" (shape input) (at 87.46 197.87 180) (effects (font (size 0.8 0.8)) (justify right)) (property "Intersheetrefs" "${INTERSHEET_REFS}" (at 0 0 0) (effects (font (size 0.8 0.8)) hide)))
@@
     (pin "AH27")
     (pin "AH28")
-    (instances (project "appliance" (path "/a44f63fc-7712-4594-9b92-4acfa967723a/c29c41d6-b0a9-4083-849c-c4aea6088c8b" (reference "U_CHIP") (unit 1))))
+    (instances (project "appliance" (path "/53a34ee7-8c3b-4e20-9ef1-ef0d8fcc1954/b343c77a-a6eb-41db-a475-c3a1e922dde8" (reference "U_CHIP") (unit 1))))
   )
   (global_label "PSRAM_0_DQ0" (shape input) (at 261.6 591.57 180) (effects (font (size 0.8 0.8)) (justify right)) (property "Intersheetrefs" "${INTERSHEET_REFS}" (at 0 0 0) (effects (font (size 0.8 0.8)) hide)))
@@
   (global_label "VDD_CORE" (shape input) (at 554.89 600.38 270) (effects (font (size 0.8 0.8)) (justify left)) (property "Intersheetrefs" "${INTERSHEET_REFS}" (at 0 0 0) (effects (font (size 0.8 0.8)) hide)))
   (global_label "GND" (shape input) (at 557.43 600.38 270) (effects (font (size 0.8 0.8)) (justify left)) (property "Intersheetrefs" "${INTERSHEET_REFS}" (at 0 0 0) (effects (font (size 0.8 0.8)) hide)))
-  (global_label "VDD_CORE" (shape input) (at 559.97 600.38 270) (effects (font (size 0.8 0.8)) (justify left)) (property "Intersheetrefs" "${INTERSHEET_REFS}" (at 0 0 0) (effects (font (size 0.8 0.8)) hide)))
-  (global_label "GND" (shape input) (at 562.51 600.38 270) (effects (font (size 0.8 0.8)) (justify left)) (property "Intersheetrefs" "${INTERSHEET_REFS}" (at 0 0 0) (effects (font (size 0.8 0.8)) hide)))
-  (global_label "VDD_CORE" (shape input) (at 565.05 600.38 270) (effects (font (size 0.8 0.8)) (justify left)) (property "Intersheetrefs" "${INTERSHEET_REFS}" (at 0 0 0) (effects (font (size 0.8 0.8)) hide)))
+  (global_label "PSRAM_CLK7" (shape input) (at 559.97 600.38 270) (effects (font (size 0.8 0.8)) (justify left)) (property "Intersheetrefs" "${INTERSHEET_REFS}" (at 0 0 0) (effects (font (size 0.8 0.8)) hide)))
+  (global_label "PSRAM_CLK8" (shape input) (at 562.51 600.38 270) (effects (font (size 0.8 0.8)) (justify left)) (property "Intersheetrefs" "${INTERSHEET_REFS}" (at 0 0 0) (effects (font (size 0.8 0.8)) hide)))
+  (global_label "PSRAM_CLK9" (shape input) (at 565.05 600.38 270) (effects (font (size 0.8 0.8)) (justify left)) (property "Intersheetrefs" "${INTERSHEET_REFS}" (at 0 0 0) (effects (font (size 0.8 0.8)) hide)))
   (global_label "GND" (shape input) (at 567.59 600.38 270) (effects (font (size 0.8 0.8)) (justify left)) (property "Intersheetrefs" "${INTERSHEET_REFS}" (at 0 0 0) (effects (font (size 0.8 0.8)) hide)))
-  (global_label "VDD_CORE" (shape input) (at 570.13 600.38 270) (effects (font (size 0.8 0.8)) (justify left)) (property "Intersheetrefs" "${INTERSHEET_REFS}" (at 0 0 0) (effects (font (size 0.8 0.8)) hide)))
-  (global_label "GND" (shape input) (at 572.67 600.38 270) (effects (font (size 0.8 0.8)) (justify left)) (property "Intersheetrefs" "${INTERSHEET_REFS}" (at 0 0 0) (effects (font (size 0.8 0.8)) hide)))
-  (global_label "VDD_CORE" (shape input) (at 575.21 600.38 270) (effects (font (size 0.8 0.8)) (justify left)) (property "Intersheetrefs" "${INTERSHEET_REFS}" (at 0 0 0) (effects (font (size 0.8 0.8)) hide)))
-  (global_label "GND" (shape input) (at 577.75 600.38 270) (effects (font (size 0.8 0.8)) (justify left)) (property "Intersheetrefs" "${INTERSHEET_REFS}" (at 0 0 0) (effects (font (size 0.8 0.8)) hide)))
-  (global_label "VDD_CORE" (shape input) (at 580.29 600.38 270) (effects (font (size 0.8 0.8)) (justify left)) (property "Intersheetrefs" "${INTERSHEET_REFS}" (at 0 0 0) (effects (font (size 0.8 0.8)) hide)))
-  (global_label "GND" (shape input) (at 582.83 600.38 270) (effects (font (size 0.8 0.8)) (justify left)) (property "Intersheetrefs" "${INTERSHEET_REFS}" (at 0 0 0) (effects (font (size 0.8 0.8)) hide)))
-  (global_label "VDD_CORE" (shape input) (at 585.37 600.38 270) (effects (font (size 0.8 0.8)) (justify left)) (property "Intersheetrefs" "${INTERSHEET_REFS}" (at 0 0 0) (effects (font (size 0.8 0.8)) hide)))
+  (global_label "PSRAM_CLK10" (shape input) (at 570.13 600.38 270) (effects (font (size 0.8 0.8)) (justify left)) (property "Intersheetrefs" "${INTERSHEET_REFS}" (at 0 0 0) (effects (font (size 0.8 0.8)) hide)))
+  (global_label "PSRAM_CLK11" (shape input) (at 572.67 600.38 270) (effects (font (size 0.8 0.8)) (justify left)) (property "Intersheetrefs" "${INTERSHEET_REFS}" (at 0 0 0) (effects (font (size 0.8 0.8)) hide)))
+  (global_label "PSRAM_CLK12" (shape input) (at 575.21 600.38 270) (effects (font (size 0.8 0.8)) (justify left)) (property "Intersheetrefs" "${INTERSHEET_REFS}" (at 0 0 0) (effects (font (size 0.8 0.8)) hide)))
+  (global_label "PSRAM_CLK13" (shape input) (at 577.75 600.38 270) (effects (font (size 0.8 0.8)) (justify left)) (property "Intersheetrefs" "${INTERSHEET_REFS}" (at 0 0 0) (effects (font (size 0.8 0.8)) hide)))
+  (global_label "GND" (shape input) (at 580.29 600.38 270) (effects (font (size 0.8 0.8)) (justify left)) (property "Intersheetrefs" "${INTERSHEET_REFS}" (at 0 0 0) (effects (font (size 0.8 0.8)) hide)))
+  (global_label "PSRAM_CLK14" (shape input) (at 582.83 600.38 270) (effects (font (size 0.8 0.8)) (justify left)) (property "Intersheetrefs" "${INTERSHEET_REFS}" (at 0 0 0) (effects (font (size 0.8 0.8)) hide)))
+  (global_label "PSRAM_CLK15" (shape input) (at 585.37 600.38 270) (effects (font (size 0.8 0.8)) (justify left)) (property "Intersheetrefs" "${INTERSHEET_REFS}" (at 0 0 0) (effects (font (size 0.8 0.8)) hide)))
   (global_label "GND" (shape input) (at 587.91 600.38 270) (effects (font (size 0.8 0.8)) (justify left)) (property "Intersheetrefs" "${INTERSHEET_REFS}" (at 0 0 0) (effects (font (size 0.8 0.8)) hide)))
   (global_label "VDD_CORE" (shape input) (at 590.45 600.38 270) (effects (font (size 0.8 0.8)) (justify left)) (property "Intersheetrefs" "${INTERSHEET_REFS}" (at 0 0 0) (effects (font (size 0.8 0.8)) hide)))
@@
   (global_label "PSRAM_CLK2" (shape input) (at 664.11 600.38 270) (effects (font (size 0.8 0.8)) (justify left)) (property "Intersheetrefs" "${INTERSHEET_REFS}" (at 0 0 0) (effects (font (size 0.8 0.8)) hide)))
   (global_label "PSRAM_CLK3" (shape input) (at 666.65 600.38 270) (effects (font (size 0.8 0.8)) (justify left)) (property "Intersheetrefs" "${INTERSHEET_REFS}" (at 0 0 0) (effects (font (size 0.8 0.8)) hide)))
-  (global_label "VDD_CORE" (shape input) (at 669.19 600.38 270) (effects (font (size 0.8 0.8)) (justify left)) (property "Intersheetrefs" "${INTERSHEET_REFS}" (at 0 0 0) (effects (font (size 0.8 0.8)) hide)))
-  (global_label "GND" (shape input) (at 671.73 600.38 270) (effects (font (size 0.8 0.8)) (justify left)) (property "Intersheetrefs" "${INTERSHEET_REFS}" (at 0 0 0) (effects (font (size 0.8 0.8)) hide)))
-  (global_label "VDD_CORE" (shape input) (at 674.27 600.38 270) (effects (font (size 0.8 0.8)) (justify left)) (property "Intersheetrefs" "${INTERSHEET_REFS}" (at 0 0 0) (effects (font (size 0.8 0.8)) hide)))
-  (global_label "GND" (shape input) (at 676.81 600.38 270) (effects (font (size 0.8 0.8)) (justify left)) (property "Intersheetrefs" "${INTERSHEET_REFS}" (at 0 0 0) (effects (font (size 0.8 0.8)) hide)))
+  (global_label "PSRAM_CLK4" (shape input) (at 669.19 600.38 270) (effects (font (size 0.8 0.8)) (justify left)) (property "Intersheetrefs" "${INTERSHEET_REFS}" (at 0 0 0) (effects (font (size 0.8 0.8)) hide)))
+  (global_label "PSRAM_CLK5" (shape input) (at 671.73 600.38 270) (effects (font (size 0.8 0.8)) (justify left)) (property "Intersheetrefs" "${INTERSHEET_REFS}" (at 0 0 0) (effects (font (size 0.8 0.8)) hide)))
+  (global_label "GND" (shape input) (at 674.27 600.38 270) (effects (font (size 0.8 0.8)) (justify left)) (property "Intersheetrefs" "${INTERSHEET_REFS}" (at 0 0 0) (effects (font (size 0.8 0.8)) hide)))
+  (global_label "PSRAM_CLK6" (shape input) (at 676.81 600.38 270) (effects (font (size 0.8 0.8)) (justify left)) (property "Intersheetrefs" "${INTERSHEET_REFS}" (at 0 0 0) (effects (font (size 0.8 0.8)) hide)))
   (global_label "LINK_OUT_DATA1" (shape input) (at 679.35 600.38 270) (effects (font (size 0.8 0.8)) (justify left)) (property "Intersheetrefs" "${INTERSHEET_REFS}" (at 0 0 0) (effects (font (size 0.8 0.8)) hide)))
   (global_label "LINK_OUT_DATA3" (shape input) (at 681.89 600.38 270) (effects (font (size 0.8 0.8)) (justify left)) (property "Intersheetrefs" "${INTERSHEET_REFS}" (at 0 0 0) (effects (font (size 0.8 0.8)) hide)))

Commit message: Move the PSRAM clock balls to the north edge beside the memory
A small interface may now name its own package edge in
package_selection.edges; psram_clk: N puts the sixteen clocks in the row
just inside the north memory rows, sixteen of its eighteen positions
between the east and west strips, so each clock escapes with its memory
and runs 15 to 55 mm to its device instead of round the package.  The
report lists them and counts them among the balls that need a build-up
escape.  The clock study keeps the south placement as its second case
and sweeps the point-to-point trace over the north lengths.

Co-Authored-By: Claude Fable 5.1 <noreply@anthropic.com>
Claude-Session: https://claude.ai/code/session_01VmmvkZe8Ctg3RAykNGsQBn
Connections:
- net GND: now also U_CHIP.AF10, U_CHIP.AF12, U_CHIP.AF4, U_CHIP.AF8, U_CHIP.AG13, U_CHIP.AG17, U_CHIP.AG19, U_CHIP.AG21; no longer U_CHIP.AF11, U_CHIP.AG20, U_CHIP.F10, U_CHIP.F12, U_CHIP.F14, U_CHIP.F16, U_CHIP.F18, U_CHIP.F20, U_CHIP.F6, U_CHIP.F8
- net PSRAM_CLK0: now also U_CHIP.F6; no longer U_CHIP.AG13
- net PSRAM_CLK1: now also U_CHIP.F7; no longer U_CHIP.AG14
- net PSRAM_CLK10: now also U_CHIP.F16; no longer U_CHIP.AF7
- net PSRAM_CLK11: now also U_CHIP.F17; no longer U_CHIP.AF8
- net PSRAM_CLK12: now also U_CHIP.F18; no longer U_CHIP.AF9
- net PSRAM_CLK13: now also U_CHIP.F19; no longer U_CHIP.AF10
- net PSRAM_CLK14: now also U_CHIP.F20; no longer U_CHIP.AF12
- net PSRAM_CLK15: now also U_CHIP.F21; no longer U_CHIP.AF13
- net PSRAM_CLK2: now also U_CHIP.F8; no longer U_CHIP.AG16
- net PSRAM_CLK3: now also U_CHIP.F9; no longer U_CHIP.AG17
- net PSRAM_CLK4: now also U_CHIP.F10; no longer U_CHIP.AG18
- net PSRAM_CLK5: now also U_CHIP.F11; no longer U_CHIP.AG19
- net PSRAM_CLK6: now also U_CHIP.F12; no longer U_CHIP.AG21
- net PSRAM_CLK7: now also U_CHIP.F13; no longer U_CHIP.AF3
- net PSRAM_CLK8: now also U_CHIP.F14; no longer U_CHIP.AF4
- net PSRAM_CLK9: now also U_CHIP.F15; no longer U_CHIP.AF5
- net VDD_CORE: now also U_CHIP.AF11, U_CHIP.AF13, U_CHIP.AF3, U_CHIP.AF5, U_CHIP.AF7, U_CHIP.AF9, U_CHIP.AG14, U_CHIP.AG16, U_CHIP.AG18, U_CHIP.AG20; no longer U_CHIP.AA16, U_CHIP.AA6, U_CHIP.F13, U_CHIP.F15, U_CHIP.F17, U_CHIP.F19, U_CHIP.F7, U_CHIP.F9
- net VDD_IO_1V8: now also U_CHIP.W14, U_CHIP.Y15; no longer U_CHIP.F11, U_CHIP.F21
- net VDD_PLL_0V9: now also U_CHIP.AA16, U_CHIP.AA6; no longer U_CHIP.W14, U_CHIP.Y15
