File: hw/kicad_psram/module_memory.kicad_sch (KiCad schematic)
At the start: 16 parts

Commit message: Choose the PSRAM and write its HPI controller
The PSRAM board's device is the AP Memory APS512XXN-OB9-BG: 512 Mb, the
Xccela DDR interface in x16 (HPI) mode, 250 MHz, 1.8 V, a 24-ball 6 x 8
mm BGA.  fabric/hpi.py carries its geometry, the mode-register
encodings, the command frame and the striping of the die's memory port
over sixteen devices in page-sized stripes; fabric_hpi.sv is the
controller: a per-device channel with the power-up sequence, global
reset, mode registers and an identity check, the command phase on both
clock edges, fixed-latency writes with data mask, and reads captured by
the device's strobe through a gray-pointer ring so refresh push-out
costs nothing; and a stripe unit that splits a burst into concurrent
per-device chunks, returns read data in order and completes a write
only when every chunk is in the device.  A behavioural device model
checks the protocol (tCEM, tCPH, even addresses, x16 mode) and the
testbench runs random bursts over one, two, four and sixteen devices
against the striped image.

The memory port's burst count widens to 12 bits so a head's state is
one burst across all devices, and the map aligns regions to a page.
The board gains the real part, its DQS/DM naming, and the four shared
clocks as a small interface the pinout places with the management
signals and the card wires to its devices; the connector count is
unchanged.

Co-Authored-By: Claude Fable 5.1 <noreply@anthropic.com>
Claude-Session: https://claude.ai/code/session_01VmmvkZe8Ctg3RAykNGsQBn
Parts:
- U_M0_0, U_M0_1, U_M0_10, U_M0_11, U_M0_12, U_M0_13, U_M0_14, U_M0_15, U_M0_2, U_M0_3, U_M0_4, U_M0_5, U_M0_6, U_M0_7, U_M0_8, U_M0_9: footprint appliance:FBGA49_7x7_P1.0 -> appliance:BGA24_5x5_P1.0
Connections:
- net MEM0_CS is gone; now on net MEM0_DQ4: U_M0_0.E5
- net MEM0_RWDS0 is gone; now on net MEM0_DQ2: U_M0_0.E3
- net MEM0_RWDS1 is gone; now on net MEM0_DQ3: U_M0_0.E4
- net MEM10_CS is gone; now on net MEM10_DQ4: U_M0_10.E5
- net MEM10_RWDS0 is gone; now on net MEM10_DQ2: U_M0_10.E3
- net MEM10_RWDS1 is gone; now on net MEM10_DQ3: U_M0_10.E4
- net MEM11_CS is gone; now on net MEM11_DQ4: U_M0_11.E5
- net MEM11_RWDS0 is gone; now on net MEM11_DQ2: U_M0_11.E3
- net MEM11_RWDS1 is gone; now on net MEM11_DQ3: U_M0_11.E4
- net MEM12_CS is gone; now on net MEM12_DQ4: U_M0_12.E5
- net MEM12_RWDS0 is gone; now on net MEM12_DQ2: U_M0_12.E3
- net MEM12_RWDS1 is gone; now on net MEM12_DQ3: U_M0_12.E4
- net MEM13_CS is gone; now on net MEM13_DQ4: U_M0_13.E5
- net MEM13_RWDS0 is gone; now on net MEM13_DQ2: U_M0_13.E3
- net MEM13_RWDS1 is gone; now on net MEM13_DQ3: U_M0_13.E4
- net MEM14_CS is gone; now on net MEM14_DQ4: U_M0_14.E5
- net MEM14_RWDS0 is gone; now on net MEM14_DQ2: U_M0_14.E3
- net MEM14_RWDS1 is gone; now on net MEM14_DQ3: U_M0_14.E4
- net MEM15_CS is gone; now on net MEM15_DQ4: U_M0_15.E5
- net MEM15_RWDS0 is gone; now on net MEM15_DQ2: U_M0_15.E3
- net MEM15_RWDS1 is gone; now on net MEM15_DQ3: U_M0_15.E4
- net MEM1_CS is gone; now on net MEM1_DQ4: U_M0_1.E5
- net MEM1_RWDS0 is gone; now on net MEM1_DQ2: U_M0_1.E3
- net MEM1_RWDS1 is gone; now on net MEM1_DQ3: U_M0_1.E4
- net MEM2_CS is gone; now on net MEM2_DQ4: U_M0_2.E5
- net MEM2_RWDS0 is gone; now on net MEM2_DQ2: U_M0_2.E3
- net MEM2_RWDS1 is gone; now on net MEM2_DQ3: U_M0_2.E4
- net MEM3_CS is gone; now on net MEM3_DQ4: U_M0_3.E5
- net MEM3_RWDS0 is gone; now on net MEM3_DQ2: U_M0_3.E3
- net MEM3_RWDS1 is gone; now on net MEM3_DQ3: U_M0_3.E4
- net MEM4_CS is gone; now on net MEM4_DQ4: U_M0_4.E5
- net MEM4_RWDS0 is gone; now on net MEM4_DQ2: U_M0_4.E3
- net MEM4_RWDS1 is gone; now on net MEM4_DQ3: U_M0_4.E4
- net MEM5_CS is gone; now on net MEM5_DQ4: U_M0_5.E5
- net MEM5_RWDS0 is gone; now on net MEM5_DQ2: U_M0_5.E3
- net MEM5_RWDS1 is gone; now on net MEM5_DQ3: U_M0_5.E4
- net MEM6_CS is gone; now on net MEM6_DQ4: U_M0_6.E5
- net MEM6_RWDS0 is gone; now on net MEM6_DQ2: U_M0_6.E3
- net MEM6_RWDS1 is gone; now on net MEM6_DQ3: U_M0_6.E4
- net MEM7_CS is gone; now on net MEM7_DQ4: U_M0_7.E5
- net MEM7_RWDS0 is gone; now on net MEM7_DQ2: U_M0_7.E3
- net MEM7_RWDS1 is gone; now on net MEM7_DQ3: U_M0_7.E4
- net MEM8_CS is gone; now on net MEM8_DQ4: U_M0_8.E5
- net MEM8_RWDS0 is gone; now on net MEM8_DQ2: U_M0_8.E3
- net MEM8_RWDS1 is gone; now on net MEM8_DQ3: U_M0_8.E4
- net MEM9_CS is gone; now on net MEM9_DQ4: U_M0_9.E5
- net MEM9_RWDS0 is gone; now on net MEM9_DQ2: U_M0_9.E3
- net MEM9_RWDS1 is gone; now on net MEM9_DQ3: U_M0_9.E4
- net GND: no longer U_M0_0.A7, U_M0_0.B2, U_M0_0.B4, U_M0_0.B6, U_M0_0.C1, U_M0_0.C3, U_M0_0.C5, U_M0_0.C7, U_M0_0.D2, U_M0_0.D4, U_M0_0.D6, U_M0_0.E7, U_M0_1.A7, U_M0_1.B2, U_M0_1.B4, U_M0_1.B6, U_M0_1.C1, U_M0_1.C3, U_M0_1.C5, U_M0_1.C7, U_M0_1.D2, U_M0_1.D4, U_M0_1.D6, U_M0_1.E7, U_M0_10.A7, U_M0_10.B2, U_M0_10.B4, U_M0_10.B6, U_M0_10.C1, U_M0_10.C3, U_M0_10.C5, U_M0_10.C7, U_M0_10.D2, U_M0_10.D4, U_M0_10.D6, U_M0_10.E7, U_M0_11.A7, U_M0_11.B2, U_M0_11.B4, U_M0_11.B6, U_M0_11.C1, U_M0_11.C3, U_M0_11.C5, U_M0_11.C7, U_M0_11.D2, U_M0_11.D4, U_M0_11.D6, U_M0_11.E7, U_M0_12.A7, U_M0_12.B2, U_M0_12.B4, U_M0_12.B6, U_M0_12.C1, U_M0_12.C3, U_M0_12.C5, U_M0_12.C7, U_M0_12.D2, U_M0_12.D4, U_M0_12.D6, U_M0_12.E7, U_M0_13.A7, U_M0_13.B2, U_M0_13.B4, U_M0_13.B6, U_M0_13.C1, U_M0_13.C3, U_M0_13.C5, U_M0_13.C7, U_M0_13.D2, U_M0_13.D4, U_M0_13.D6, U_M0_13.E7, U_M0_14.A7, U_M0_14.B2, U_M0_14.B4, U_M0_14.B6, U_M0_14.C1, U_M0_14.C3, U_M0_14.C5, U_M0_14.C7, U_M0_14.D2, U_M0_14.D4, U_M0_14.D6, U_M0_14.E7, U_M0_15.A7, U_M0_15.B2, U_M0_15.B4, U_M0_15.B6, U_M0_15.C1, U_M0_15.C3, U_M0_15.C5, U_M0_15.C7, U_M0_15.D2, U_M0_15.D4, U_M0_15.D6, U_M0_15.E7, U_M0_2.A7, U_M0_2.B2, U_M0_2.B4, U_M0_2.B6, U_M0_2.C1, U_M0_2.C3, U_M0_2.C5, U_M0_2.C7, U_M0_2.D2, U_M0_2.D4, U_M0_2.D6, U_M0_2.E7, U_M0_3.A7, U_M0_3.B2, U_M0_3.B4, U_M0_3.B6, U_M0_3.C1, U_M0_3.C3, U_M0_3.C5, U_M0_3.C7, U_M0_3.D2, U_M0_3.D4, U_M0_3.D6, U_M0_3.E7, U_M0_4.A7, U_M0_4.B2, U_M0_4.B4, U_M0_4.B6, U_M0_4.C1, U_M0_4.C3, U_M0_4.C5, U_M0_4.C7, U_M0_4.D2, U_M0_4.D4, U_M0_4.D6, U_M0_4.E7, U_M0_5.A7, U_M0_5.B2, U_M0_5.B4, U_M0_5.B6, U_M0_5.C1, U_M0_5.C3, U_M0_5.C5, U_M0_5.C7, U_M0_5.D2, U_M0_5.D4, U_M0_5.D6, U_M0_5.E7, U_M0_6.A7, U_M0_6.B2, U_M0_6.B4, U_M0_6.B6, U_M0_6.C1, U_M0_6.C3, U_M0_6.C5, U_M0_6.C7, U_M0_6.D2, U_M0_6.D4, U_M0_6.D6, U_M0_6.E7, U_M0_7.A7, U_M0_7.B2, U_M0_7.B4, U_M0_7.B6, U_M0_7.C1, U_M0_7.C3, U_M0_7.C5, U_M0_7.C7, U_M0_7.D2, U_M0_7.D4, U_M0_7.D6, U_M0_7.E7, U_M0_8.A7, U_M0_8.B2, U_M0_8.B4, U_M0_8.B6, U_M0_8.C1, U_M0_8.C3, U_M0_8.C5, U_M0_8.C7, U_M0_8.D2, U_M0_8.D4, U_M0_8.D6, U_M0_8.E7, U_M0_9.A7, U_M0_9.B2, U_M0_9.B4, U_M0_9.B6, U_M0_9.C1, U_M0_9.C3, U_M0_9.C5, U_M0_9.C7, U_M0_9.D2, U_M0_9.D4, U_M0_9.D6, U_M0_9.E7
- net MEM0_DQ0: now also U_M0_0.E1; no longer U_M0_0.G1
- net MEM0_DQ1: now also U_M0_0.E2; no longer U_M0_0.G2
- net MEM0_DQ10: now also U_M0_0.C1; no longer U_M0_0.F4
- net MEM0_DQ11: now also U_M0_0.C2; no longer U_M0_0.F5
- net MEM0_DQ12: now also U_M0_0.C3; no longer U_M0_0.F6
- net MEM0_DQ13: now also U_M0_0.C4; no longer U_M0_0.F7
- net MEM0_DQ14: now also U_M0_0.C5; no longer U_M0_0.E1
- net MEM0_DQ15: now also U_M0_0.B1; no longer U_M0_0.E2
- net MEM0_DQ2: no longer U_M0_0.G3
- net MEM0_DQ3: no longer U_M0_0.G4
- net MEM0_DQ4: no longer U_M0_0.G5
- net MEM0_DQ5: now also U_M0_0.D1; no longer U_M0_0.G6
- net MEM0_DQ6: now also U_M0_0.D2; no longer U_M0_0.G7
- net MEM0_DQ7: now also U_M0_0.D3; no longer U_M0_0.F1
- net MEM0_DQ8: now also U_M0_0.D4; no longer U_M0_0.F2
- net MEM0_DQ9: now also U_M0_0.D5; no longer U_M0_0.F3
- net MEM10_DQ0: now also U_M0_10.E1; no longer U_M0_10.G1
- net MEM10_DQ1: now also U_M0_10.E2; no longer U_M0_10.G2
- net MEM10_DQ10: now also U_M0_10.C1; no longer U_M0_10.F4
- net MEM10_DQ11: now also U_M0_10.C2; no longer U_M0_10.F5
- net MEM10_DQ12: now also U_M0_10.C3; no longer U_M0_10.F6
- net MEM10_DQ13: now also U_M0_10.C4; no longer U_M0_10.F7
- net MEM10_DQ14: now also U_M0_10.C5; no longer U_M0_10.E1
- net MEM10_DQ15: now also U_M0_10.B1; no longer U_M0_10.E2
- net MEM10_DQ2: no longer U_M0_10.G3
- net MEM10_DQ3: no longer U_M0_10.G4
- net MEM10_DQ4: no longer U_M0_10.G5
- net MEM10_DQ5: now also U_M0_10.D1; no longer U_M0_10.G6
- net MEM10_DQ6: now also U_M0_10.D2; no longer U_M0_10.G7
- net MEM10_DQ7: now also U_M0_10.D3; no longer U_M0_10.F1
- net MEM10_DQ8: now also U_M0_10.D4; no longer U_M0_10.F2
- net MEM10_DQ9: now also U_M0_10.D5; no longer U_M0_10.F3
- net MEM11_DQ0: now also U_M0_11.E1; no longer U_M0_11.G1
- net MEM11_DQ1: now also U_M0_11.E2; no longer U_M0_11.G2
- net MEM11_DQ10: now also U_M0_11.C1; no longer U_M0_11.F4
- net MEM11_DQ11: now also U_M0_11.C2; no longer U_M0_11.F5
- net MEM11_DQ12: now also U_M0_11.C3; no longer U_M0_11.F6
- net MEM11_DQ13: now also U_M0_11.C4; no longer U_M0_11.F7
- net MEM11_DQ14: now also U_M0_11.C5; no longer U_M0_11.E1
- net MEM11_DQ15: now also U_M0_11.B1; no longer U_M0_11.E2
- net MEM11_DQ2: no longer U_M0_11.G3
- net MEM11_DQ3: no longer U_M0_11.G4
- net MEM11_DQ4: no longer U_M0_11.G5
- net MEM11_DQ5: now also U_M0_11.D1; no longer U_M0_11.G6
- net MEM11_DQ6: now also U_M0_11.D2; no longer U_M0_11.G7
- net MEM11_DQ7: now also U_M0_11.D3; no longer U_M0_11.F1
- net MEM11_DQ8: now also U_M0_11.D4; no longer U_M0_11.F2
- net MEM11_DQ9: now also U_M0_11.D5; no longer U_M0_11.F3
- net MEM12_DQ0: now also U_M0_12.E1; no longer U_M0_12.G1
- net MEM12_DQ1: now also U_M0_12.E2; no longer U_M0_12.G2
- net MEM12_DQ10: now also U_M0_12.C1; no longer U_M0_12.F4
- net MEM12_DQ11: now also U_M0_12.C2; no longer U_M0_12.F5
- net MEM12_DQ12: now also U_M0_12.C3; no longer U_M0_12.F6
- net MEM12_DQ13: now also U_M0_12.C4; no longer U_M0_12.F7
- net MEM12_DQ14: now also U_M0_12.C5; no longer U_M0_12.E1
- net MEM12_DQ15: now also U_M0_12.B1; no longer U_M0_12.E2
- net MEM12_DQ2: no longer U_M0_12.G3
- net MEM12_DQ3: no longer U_M0_12.G4
- net MEM12_DQ4: no longer U_M0_12.G5
- net MEM12_DQ5: now also U_M0_12.D1; no longer U_M0_12.G6
- net MEM12_DQ6: now also U_M0_12.D2; no longer U_M0_12.G7
- net MEM12_DQ7: now also U_M0_12.D3; no longer U_M0_12.F1
- net MEM12_DQ8: now also U_M0_12.D4; no longer U_M0_12.F2
- net MEM12_DQ9: now also U_M0_12.D5; no longer U_M0_12.F3
- net MEM13_DQ0: now also U_M0_13.E1; no longer U_M0_13.G1
- net MEM13_DQ1: now also U_M0_13.E2; no longer U_M0_13.G2
- net MEM13_DQ10: now also U_M0_13.C1; no longer U_M0_13.F4
- net MEM13_DQ11: now also U_M0_13.C2; no longer U_M0_13.F5
- net MEM13_DQ12: now also U_M0_13.C3; no longer U_M0_13.F6
- net MEM13_DQ13: now also U_M0_13.C4; no longer U_M0_13.F7
- net MEM13_DQ14: now also U_M0_13.C5; no longer U_M0_13.E1
- net MEM13_DQ15: now also U_M0_13.B1; no longer U_M0_13.E2
- net MEM13_DQ2: no longer U_M0_13.G3
- net MEM13_DQ3: no longer U_M0_13.G4
- net MEM13_DQ4: no longer U_M0_13.G5
- net MEM13_DQ5: now also U_M0_13.D1; no longer U_M0_13.G6
- net MEM13_DQ6: now also U_M0_13.D2; no longer U_M0_13.G7
- net MEM13_DQ7: now also U_M0_13.D3; no longer U_M0_13.F1
- net MEM13_DQ8: now also U_M0_13.D4; no longer U_M0_13.F2
- net MEM13_DQ9: now also U_M0_13.D5; no longer U_M0_13.F3
- net MEM14_DQ0: now also U_M0_14.E1; no longer U_M0_14.G1
- net MEM14_DQ1: now also U_M0_14.E2; no longer U_M0_14.G2
- net MEM14_DQ10: now also U_M0_14.C1; no longer U_M0_14.F4
- net MEM14_DQ11: now also U_M0_14.C2; no longer U_M0_14.F5
- net MEM14_DQ12: now also U_M0_14.C3; no longer U_M0_14.F6
- net MEM14_DQ13: now also U_M0_14.C4; no longer U_M0_14.F7
- net MEM14_DQ14: now also U_M0_14.C5; no longer U_M0_14.E1
- net MEM14_DQ15: now also U_M0_14.B1; no longer U_M0_14.E2
- net MEM14_DQ2: no longer U_M0_14.G3
- net MEM14_DQ3: no longer U_M0_14.G4
- net MEM14_DQ4: no longer U_M0_14.G5
- net MEM14_DQ5: now also U_M0_14.D1; no longer U_M0_14.G6
- net MEM14_DQ6: now also U_M0_14.D2; no longer U_M0_14.G7
- net MEM14_DQ7: now also U_M0_14.D3; no longer U_M0_14.F1
- net MEM14_DQ8: now also U_M0_14.D4; no longer U_M0_14.F2
- net MEM14_DQ9: now also U_M0_14.D5; no longer U_M0_14.F3
- net MEM15_DQ0: now also U_M0_15.E1; no longer U_M0_15.G1
- net MEM15_DQ1: now also U_M0_15.E2; no longer U_M0_15.G2
- net MEM15_DQ10: now also U_M0_15.C1; no longer U_M0_15.F4
- net MEM15_DQ11: now also U_M0_15.C2; no longer U_M0_15.F5
- net MEM15_DQ12: now also U_M0_15.C3; no longer U_M0_15.F6
- net MEM15_DQ13: now also U_M0_15.C4; no longer U_M0_15.F7
- net MEM15_DQ14: now also U_M0_15.C5; no longer U_M0_15.E1
- net MEM15_DQ15: now also U_M0_15.B1; no longer U_M0_15.E2
- net MEM15_DQ2: no longer U_M0_15.G3
- net MEM15_DQ3: no longer U_M0_15.G4
- net MEM15_DQ4: no longer U_M0_15.G5
- net MEM15_DQ5: now also U_M0_15.D1; no longer U_M0_15.G6
- net MEM15_DQ6: now also U_M0_15.D2; no longer U_M0_15.G7
- net MEM15_DQ7: now also U_M0_15.D3; no longer U_M0_15.F1
- net MEM15_DQ8: now also U_M0_15.D4; no longer U_M0_15.F2
- net MEM15_DQ9: now also U_M0_15.D5; no longer U_M0_15.F3
- net MEM1_DQ0: now also U_M0_1.E1; no longer U_M0_1.G1
- net MEM1_DQ1: now also U_M0_1.E2; no longer U_M0_1.G2
- net MEM1_DQ10: now also U_M0_1.C1; no longer U_M0_1.F4
- net MEM1_DQ11: now also U_M0_1.C2; no longer U_M0_1.F5
- net MEM1_DQ12: now also U_M0_1.C3; no longer U_M0_1.F6
- net MEM1_DQ13: now also U_M0_1.C4; no longer U_M0_1.F7
- net MEM1_DQ14: now also U_M0_1.C5; no longer U_M0_1.E1
- net MEM1_DQ15: now also U_M0_1.B1; no longer U_M0_1.E2
- net MEM1_DQ2: no longer U_M0_1.G3
- net MEM1_DQ3: no longer U_M0_1.G4
- net MEM1_DQ4: no longer U_M0_1.G5
- net MEM1_DQ5: now also U_M0_1.D1; no longer U_M0_1.G6
- net MEM1_DQ6: now also U_M0_1.D2; no longer U_M0_1.G7
- net MEM1_DQ7: now also U_M0_1.D3; no longer U_M0_1.F1
- net MEM1_DQ8: now also U_M0_1.D4; no longer U_M0_1.F2
- net MEM1_DQ9: now also U_M0_1.D5; no longer U_M0_1.F3
- net MEM2_DQ0: now also U_M0_2.E1; no longer U_M0_2.G1
- net MEM2_DQ1: now also U_M0_2.E2; no longer U_M0_2.G2
- net MEM2_DQ10: now also U_M0_2.C1; no longer U_M0_2.F4
- net MEM2_DQ11: now also U_M0_2.C2; no longer U_M0_2.F5
- net MEM2_DQ12: now also U_M0_2.C3; no longer U_M0_2.F6
- net MEM2_DQ13: now also U_M0_2.C4; no longer U_M0_2.F7
- net MEM2_DQ14: now also U_M0_2.C5; no longer U_M0_2.E1
- net MEM2_DQ15: now also U_M0_2.B1; no longer U_M0_2.E2
- net MEM2_DQ2: no longer U_M0_2.G3
- net MEM2_DQ3: no longer U_M0_2.G4
- net MEM2_DQ4: no longer U_M0_2.G5
- net MEM2_DQ5: now also U_M0_2.D1; no longer U_M0_2.G6
- net MEM2_DQ6: now also U_M0_2.D2; no longer U_M0_2.G7
- net MEM2_DQ7: now also U_M0_2.D3; no longer U_M0_2.F1
- net MEM2_DQ8: now also U_M0_2.D4; no longer U_M0_2.F2
- net MEM2_DQ9: now also U_M0_2.D5; no longer U_M0_2.F3
- net MEM3_DQ0: now also U_M0_3.E1; no longer U_M0_3.G1
- net MEM3_DQ1: now also U_M0_3.E2; no longer U_M0_3.G2
- net MEM3_DQ10: now also U_M0_3.C1; no longer U_M0_3.F4
- net MEM3_DQ11: now also U_M0_3.C2; no longer U_M0_3.F5
- net MEM3_DQ12: now also U_M0_3.C3; no longer U_M0_3.F6
- net MEM3_DQ13: now also U_M0_3.C4; no longer U_M0_3.F7
- net MEM3_DQ14: now also U_M0_3.C5; no longer U_M0_3.E1
- net MEM3_DQ15: now also U_M0_3.B1; no longer U_M0_3.E2
- net MEM3_DQ2: no longer U_M0_3.G3
- net MEM3_DQ3: no longer U_M0_3.G4
- net MEM3_DQ4: no longer U_M0_3.G5
- net MEM3_DQ5: now also U_M0_3.D1; no longer U_M0_3.G6
- net MEM3_DQ6: now also U_M0_3.D2; no longer U_M0_3.G7
- net MEM3_DQ7: now also U_M0_3.D3; no longer U_M0_3.F1
- net MEM3_DQ8: now also U_M0_3.D4; no longer U_M0_3.F2
- net MEM3_DQ9: now also U_M0_3.D5; no longer U_M0_3.F3
- net MEM4_DQ0: now also U_M0_4.E1; no longer U_M0_4.G1
- net MEM4_DQ1: now also U_M0_4.E2; no longer U_M0_4.G2
- net MEM4_DQ10: now also U_M0_4.C1; no longer U_M0_4.F4
- net MEM4_DQ11: now also U_M0_4.C2; no longer U_M0_4.F5
- net MEM4_DQ12: now also U_M0_4.C3; no longer U_M0_4.F6
- net MEM4_DQ13: now also U_M0_4.C4; no longer U_M0_4.F7
- net MEM4_DQ14: now also U_M0_4.C5; no longer U_M0_4.E1
- net MEM4_DQ15: now also U_M0_4.B1; no longer U_M0_4.E2
- net MEM4_DQ2: no longer U_M0_4.G3
- net MEM4_DQ3: no longer U_M0_4.G4
- net MEM4_DQ4: no longer U_M0_4.G5
- net MEM4_DQ5: now also U_M0_4.D1; no longer U_M0_4.G6
- net MEM4_DQ6: now also U_M0_4.D2; no longer U_M0_4.G7
- net MEM4_DQ7: now also U_M0_4.D3; no longer U_M0_4.F1
- net MEM4_DQ8: now also U_M0_4.D4; no longer U_M0_4.F2
- net MEM4_DQ9: now also U_M0_4.D5; no longer U_M0_4.F3
- net MEM5_DQ0: now also U_M0_5.E1; no longer U_M0_5.G1
- net MEM5_DQ1: now also U_M0_5.E2; no longer U_M0_5.G2
- net MEM5_DQ10: now also U_M0_5.C1; no longer U_M0_5.F4
- net MEM5_DQ11: now also U_M0_5.C2; no longer U_M0_5.F5
- net MEM5_DQ12: now also U_M0_5.C3; no longer U_M0_5.F6
- net MEM5_DQ13: now also U_M0_5.C4; no longer U_M0_5.F7
- net MEM5_DQ14: now also U_M0_5.C5; no longer U_M0_5.E1
- net MEM5_DQ15: now also U_M0_5.B1; no longer U_M0_5.E2
- net MEM5_DQ2: no longer U_M0_5.G3
- net MEM5_DQ3: no longer U_M0_5.G4
- net MEM5_DQ4: no longer U_M0_5.G5
- net MEM5_DQ5: now also U_M0_5.D1; no longer U_M0_5.G6
- net MEM5_DQ6: now also U_M0_5.D2; no longer U_M0_5.G7
- net MEM5_DQ7: now also U_M0_5.D3; no longer U_M0_5.F1
- net MEM5_DQ8: now also U_M0_5.D4; no longer U_M0_5.F2
- net MEM5_DQ9: now also U_M0_5.D5; no longer U_M0_5.F3
- net MEM6_DQ0: now also U_M0_6.E1; no longer U_M0_6.G1
- net MEM6_DQ1: now also U_M0_6.E2; no longer U_M0_6.G2
- net MEM6_DQ10: now also U_M0_6.C1; no longer U_M0_6.F4
- net MEM6_DQ11: now also U_M0_6.C2; no longer U_M0_6.F5
- net MEM6_DQ12: now also U_M0_6.C3; no longer U_M0_6.F6
- net MEM6_DQ13: now also U_M0_6.C4; no longer U_M0_6.F7
- net MEM6_DQ14: now also U_M0_6.C5; no longer U_M0_6.E1
- net MEM6_DQ15: now also U_M0_6.B1; no longer U_M0_6.E2
- net MEM6_DQ2: no longer U_M0_6.G3
- net MEM6_DQ3: no longer U_M0_6.G4
- net MEM6_DQ4: no longer U_M0_6.G5
- net MEM6_DQ5: now also U_M0_6.D1; no longer U_M0_6.G6
- net MEM6_DQ6: now also U_M0_6.D2; no longer U_M0_6.G7
- net MEM6_DQ7: now also U_M0_6.D3; no longer U_M0_6.F1
- net MEM6_DQ8: now also U_M0_6.D4; no longer U_M0_6.F2
- net MEM6_DQ9: now also U_M0_6.D5; no longer U_M0_6.F3
- net MEM7_DQ0: now also U_M0_7.E1; no longer U_M0_7.G1
- net MEM7_DQ1: now also U_M0_7.E2; no longer U_M0_7.G2
- net MEM7_DQ10: now also U_M0_7.C1; no longer U_M0_7.F4
- net MEM7_DQ11: now also U_M0_7.C2; no longer U_M0_7.F5
- net MEM7_DQ12: now also U_M0_7.C3; no longer U_M0_7.F6
- net MEM7_DQ13: now also U_M0_7.C4; no longer U_M0_7.F7
- net MEM7_DQ14: now also U_M0_7.C5; no longer U_M0_7.E1
- net MEM7_DQ15: now also U_M0_7.B1; no longer U_M0_7.E2
- net MEM7_DQ2: no longer U_M0_7.G3
- net MEM7_DQ3: no longer U_M0_7.G4
- net MEM7_DQ4: no longer U_M0_7.G5
- net MEM7_DQ5: now also U_M0_7.D1; no longer U_M0_7.G6
- net MEM7_DQ6: now also U_M0_7.D2; no longer U_M0_7.G7
- net MEM7_DQ7: now also U_M0_7.D3; no longer U_M0_7.F1
- net MEM7_DQ8: now also U_M0_7.D4; no longer U_M0_7.F2
- net MEM7_DQ9: now also U_M0_7.D5; no longer U_M0_7.F3
- net MEM8_DQ0: now also U_M0_8.E1; no longer U_M0_8.G1
- net MEM8_DQ1: now also U_M0_8.E2; no longer U_M0_8.G2
- net MEM8_DQ10: now also U_M0_8.C1; no longer U_M0_8.F4
- net MEM8_DQ11: now also U_M0_8.C2; no longer U_M0_8.F5
- net MEM8_DQ12: now also U_M0_8.C3; no longer U_M0_8.F6
- net MEM8_DQ13: now also U_M0_8.C4; no longer U_M0_8.F7
- net MEM8_DQ14: now also U_M0_8.C5; no longer U_M0_8.E1
- net MEM8_DQ15: now also U_M0_8.B1; no longer U_M0_8.E2
- net MEM8_DQ2: no longer U_M0_8.G3
- net MEM8_DQ3: no longer U_M0_8.G4
- net MEM8_DQ4: no longer U_M0_8.G5
- net MEM8_DQ5: now also U_M0_8.D1; no longer U_M0_8.G6
- net MEM8_DQ6: now also U_M0_8.D2; no longer U_M0_8.G7
- net MEM8_DQ7: now also U_M0_8.D3; no longer U_M0_8.F1
- net MEM8_DQ8: now also U_M0_8.D4; no longer U_M0_8.F2
- net MEM8_DQ9: now also U_M0_8.D5; no longer U_M0_8.F3
- net MEM9_DQ0: now also U_M0_9.E1; no longer U_M0_9.G1
- net MEM9_DQ1: now also U_M0_9.E2; no longer U_M0_9.G2
- net MEM9_DQ10: now also U_M0_9.C1; no longer U_M0_9.F4
- net MEM9_DQ11: now also U_M0_9.C2; no longer U_M0_9.F5
- net MEM9_DQ12: now also U_M0_9.C3; no longer U_M0_9.F6
- net MEM9_DQ13: now also U_M0_9.C4; no longer U_M0_9.F7
- net MEM9_DQ14: now also U_M0_9.C5; no longer U_M0_9.E1
- net MEM9_DQ15: now also U_M0_9.B1; no longer U_M0_9.E2
- net MEM9_DQ2: no longer U_M0_9.G3
- net MEM9_DQ3: no longer U_M0_9.G4
- net MEM9_DQ4: no longer U_M0_9.G5
- net MEM9_DQ5: now also U_M0_9.D1; no longer U_M0_9.G6
- net MEM9_DQ6: now also U_M0_9.D2; no longer U_M0_9.G7
- net MEM9_DQ7: now also U_M0_9.D3; no longer U_M0_9.F1
- net MEM9_DQ8: now also U_M0_9.D4; no longer U_M0_9.F2
- net MEM9_DQ9: now also U_M0_9.D5; no longer U_M0_9.F3
- net VDD_IO_1V8: no longer U_M0_0.A6, U_M0_0.B1, U_M0_0.B3, U_M0_0.B5, U_M0_0.B7, U_M0_0.C2, U_M0_0.C4, U_M0_0.C6, U_M0_0.D1, U_M0_0.D3, U_M0_0.D5, U_M0_0.D7, U_M0_0.E6, U_M0_1.A6, U_M0_1.B1, U_M0_1.B3, U_M0_1.B5, U_M0_1.B7, U_M0_1.C2, U_M0_1.C4, U_M0_1.C6, U_M0_1.D1, U_M0_1.D3, U_M0_1.D5, U_M0_1.D7, U_M0_1.E6, U_M0_10.A6, U_M0_10.B1, U_M0_10.B3, U_M0_10.B5, U_M0_10.B7, U_M0_10.C2, U_M0_10.C4, U_M0_10.C6, U_M0_10.D1, U_M0_10.D3, U_M0_10.D5, U_M0_10.D7, U_M0_10.E6, U_M0_11.A6, U_M0_11.B1, U_M0_11.B3, U_M0_11.B5, U_M0_11.B7, U_M0_11.C2, U_M0_11.C4, U_M0_11.C6, U_M0_11.D1, U_M0_11.D3, U_M0_11.D5, U_M0_11.D7, U_M0_11.E6, U_M0_12.A6, U_M0_12.B1, U_M0_12.B3, U_M0_12.B5, U_M0_12.B7, U_M0_12.C2, U_M0_12.C4, U_M0_12.C6, U_M0_12.D1, U_M0_12.D3, U_M0_12.D5, U_M0_12.D7, U_M0_12.E6, U_M0_13.A6, U_M0_13.B1, U_M0_13.B3, U_M0_13.B5, U_M0_13.B7, U_M0_13.C2, U_M0_13.C4, U_M0_13.C6, U_M0_13.D1, U_M0_13.D3, U_M0_13.D5, U_M0_13.D7, U_M0_13.E6, U_M0_14.A6, U_M0_14.B1, U_M0_14.B3, U_M0_14.B5, U_M0_14.B7, U_M0_14.C2, U_M0_14.C4, U_M0_14.C6, U_M0_14.D1, U_M0_14.D3, U_M0_14.D5, U_M0_14.D7, U_M0_14.E6, U_M0_15.A6, U_M0_15.B1, U_M0_15.B3, U_M0_15.B5, U_M0_15.B7, U_M0_15.C2, U_M0_15.C4, U_M0_15.C6, U_M0_15.D1, U_M0_15.D3, U_M0_15.D5, U_M0_15.D7, U_M0_15.E6, U_M0_2.A6, U_M0_2.B1, U_M0_2.B3, U_M0_2.B5, U_M0_2.B7, U_M0_2.C2, U_M0_2.C4, U_M0_2.C6, U_M0_2.D1, U_M0_2.D3, U_M0_2.D5, U_M0_2.D7, U_M0_2.E6, U_M0_3.A6, U_M0_3.B1, U_M0_3.B3, U_M0_3.B5, U_M0_3.B7, U_M0_3.C2, U_M0_3.C4, U_M0_3.C6, U_M0_3.D1, U_M0_3.D3, U_M0_3.D5, U_M0_3.D7, U_M0_3.E6, U_M0_4.A6, U_M0_4.B1, U_M0_4.B3, U_M0_4.B5, U_M0_4.B7, U_M0_4.C2, U_M0_4.C4, U_M0_4.C6, U_M0_4.D1, U_M0_4.D3, U_M0_4.D5, U_M0_4.D7, U_M0_4.E6, U_M0_5.A6, U_M0_5.B1, U_M0_5.B3, U_M0_5.B5, U_M0_5.B7, U_M0_5.C2, U_M0_5.C4, U_M0_5.C6, U_M0_5.D1, U_M0_5.D3, U_M0_5.D5, U_M0_5.D7, U_M0_5.E6, U_M0_6.A6, U_M0_6.B1, U_M0_6.B3, U_M0_6.B5, U_M0_6.B7, U_M0_6.C2, U_M0_6.C4, U_M0_6.C6, U_M0_6.D1, U_M0_6.D3, U_M0_6.D5, U_M0_6.D7, U_M0_6.E6, U_M0_7.A6, U_M0_7.B1, U_M0_7.B3, U_M0_7.B5, U_M0_7.B7, U_M0_7.C2, U_M0_7.C4, U_M0_7.C6, U_M0_7.D1, U_M0_7.D3, U_M0_7.D5, U_M0_7.D7, U_M0_7.E6, U_M0_8.A6, U_M0_8.B1, U_M0_8.B3, U_M0_8.B5, U_M0_8.B7, U_M0_8.C2, U_M0_8.C4, U_M0_8.C6, U_M0_8.D1, U_M0_8.D3, U_M0_8.D5, U_M0_8.D7, U_M0_8.E6, U_M0_9.A6, U_M0_9.B1, U_M0_9.B3, U_M0_9.B5, U_M0_9.B7, U_M0_9.C2, U_M0_9.C4, U_M0_9.C6, U_M0_9.D1, U_M0_9.D3, U_M0_9.D5, U_M0_9.D7, U_M0_9.E6
- new net MEM0_CE: U_M0_0.B4
- new net MEM0_DQS0: U_M0_0.B2
- new net MEM0_DQS1: U_M0_0.B3
- new net MEM10_CE: U_M0_10.B4
- new net MEM10_DQS0: U_M0_10.B2
- new net MEM10_DQS1: U_M0_10.B3
- new net MEM11_CE: U_M0_11.B4
- new net MEM11_DQS0: U_M0_11.B2
- new net MEM11_DQS1: U_M0_11.B3
- new net MEM12_CE: U_M0_12.B4
- new net MEM12_DQS0: U_M0_12.B2
- new net MEM12_DQS1: U_M0_12.B3
- new net MEM13_CE: U_M0_13.B4
- new net MEM13_DQS0: U_M0_13.B2
- new net MEM13_DQS1: U_M0_13.B3
- new net MEM14_CE: U_M0_14.B4
- new net MEM14_DQS0: U_M0_14.B2
- new net MEM14_DQS1: U_M0_14.B3
- new net MEM15_CE: U_M0_15.B4
- new net MEM15_DQS0: U_M0_15.B2
- new net MEM15_DQS1: U_M0_15.B3
- new net MEM1_CE: U_M0_1.B4
- new net MEM1_DQS0: U_M0_1.B2
- new net MEM1_DQS1: U_M0_1.B3
- new net MEM2_CE: U_M0_2.B4
- new net MEM2_DQS0: U_M0_2.B2
- new net MEM2_DQS1: U_M0_2.B3
- new net MEM3_CE: U_M0_3.B4
- new net MEM3_DQS0: U_M0_3.B2
- new net MEM3_DQS1: U_M0_3.B3
- new net MEM4_CE: U_M0_4.B4
- new net MEM4_DQS0: U_M0_4.B2
- new net MEM4_DQS1: U_M0_4.B3
- new net MEM5_CE: U_M0_5.B4
- new net MEM5_DQS0: U_M0_5.B2
- new net MEM5_DQS1: U_M0_5.B3
- new net MEM6_CE: U_M0_6.B4
- new net MEM6_DQS0: U_M0_6.B2
- new net MEM6_DQS1: U_M0_6.B3
- new net MEM7_CE: U_M0_7.B4
- new net MEM7_DQS0: U_M0_7.B2
- new net MEM7_DQS1: U_M0_7.B3
- new net MEM8_CE: U_M0_8.B4
- new net MEM8_DQS0: U_M0_8.B2
- new net MEM8_DQS1: U_M0_8.B3
- new net MEM9_CE: U_M0_9.B4
- new net MEM9_DQS0: U_M0_9.B2
- new net MEM9_DQS1: U_M0_9.B3
- new net PSRAM_CLK0: U_M0_0.B5, U_M0_1.B5, U_M0_2.B5, U_M0_3.B5
- new net PSRAM_CLK1: U_M0_4.B5, U_M0_5.B5, U_M0_6.B5, U_M0_7.B5
- new net PSRAM_CLK2: U_M0_10.B5, U_M0_11.B5, U_M0_8.B5, U_M0_9.B5
- new net PSRAM_CLK3: U_M0_12.B5, U_M0_13.B5, U_M0_14.B5, U_M0_15.B5

Commit message: Add the PHY delay lines with their DLL, and settle the PSRAM clock by simulation
fabric_phy.sv is the PHY: a behavioural 256-tap delay line and a master
DLL that measures the clock period in taps with a replica line and a
phase detector, walking the code through one period and then dithering
a tap either side of it; the quarter code drives the slave lines (the
device clock and the two DQS strobes per channel), which take a new
code only while every channel has CE# high.  A line that cannot span
the period is reported rather than searched forever.  The channel
waits for the lock before starting the device, and tb_hpi and
tb_mem_bridge run the whole controller through the delay lines at taps
of 25 to 90 ps in place of the ideal quarter-period delays.

hw/si.py is a small time-domain solver for lossless transmission-line
networks (LC ladder, 1 mm segments, 2 ps steps, Thevenin driver, the
datasheet's 5 pF package input per receiver) and hw/si_psram_clock.md
its answer to whether four devices can share one 250 MHz clock: the
star of four and the fly-by, terminated or not, cannot meet the
device's 0.6 ns edge without ringing past its absolute maximum, two per
clock passes only in a narrow band, and one clock per device passes
from 33 to 50 ohm at every length on the card.  The board takes a
clock per device: sixteen psram_clk balls, the small interfaces
allowed a third row on the south edge, the card's nets one per device,
the derived pinout and KiCad outputs regenerated.

Co-Authored-By: Claude Fable 5.1 <noreply@anthropic.com>
Claude-Session: https://claude.ai/code/session_01VmmvkZe8Ctg3RAykNGsQBn
Connections:
- net PSRAM_CLK0: no longer U_M0_1.B5, U_M0_2.B5, U_M0_3.B5
- net PSRAM_CLK1: now also U_M0_1.B5; no longer U_M0_4.B5, U_M0_5.B5, U_M0_6.B5, U_M0_7.B5
- net PSRAM_CLK2: now also U_M0_2.B5; no longer U_M0_10.B5, U_M0_11.B5, U_M0_8.B5, U_M0_9.B5
- net PSRAM_CLK3: now also U_M0_3.B5; no longer U_M0_12.B5, U_M0_13.B5, U_M0_14.B5, U_M0_15.B5
- new net PSRAM_CLK10: U_M0_10.B5
- new net PSRAM_CLK11: U_M0_11.B5
- new net PSRAM_CLK12: U_M0_12.B5
- new net PSRAM_CLK13: U_M0_13.B5
- new net PSRAM_CLK14: U_M0_14.B5
- new net PSRAM_CLK15: U_M0_15.B5
- new net PSRAM_CLK4: U_M0_4.B5
- new net PSRAM_CLK5: U_M0_5.B5
- new net PSRAM_CLK6: U_M0_6.B5
- new net PSRAM_CLK7: U_M0_7.B5
- new net PSRAM_CLK8: U_M0_8.B5
- new net PSRAM_CLK9: U_M0_9.B5
